File: 2000EATX-KiCAD/2000ATX.kicad_pcb (KiCad board)
At the start: 2 copper layers, 304.8 x 330.2 mm, 55 parts, among them CN600 Amiga-2000-CPU-Slot, CN601 Amiga-2000-Zorro-Slot, CN602 Amiga-2000-Zorro-Slot, CN603 Amiga-2000-Zorro-Slot, CN604 Amiga-2000-Zorro-Slot, CN605 Amiga-2000-Zorro-Slot, U1 74LS08, U100 68000D, U103 74LS245, U104 74LS373, U105 74LS245, U106 74LS373, U600 74LS245, U601 74LS245, U602 74LS245, U603 74LS245, U604 74LS245, U605 74LS245

Commit message: Add files via upload
Parts:
- removed RNX1, RNX2: 2.7k, Resistor_THT:R_Array_SIP10
- removed RNX1, RNX2: 2.7k, Resistor_THT:R_Array_SIP9
- added C400: 220uF, Capacitor_SMD:CP_Elec_8x10.5, F.Cu at (355.7, 151.6)
- added C401: 0.1uf, Capacitor_SMD:C_1206_3216Metric, F.Cu at (356.2, 128.2)
- added C402: 47uF, Capacitor_SMD:CP_Elec_8x10.5, F.Cu at (369.3, 118.5)
- added C403: 47uF, Capacitor_SMD:CP_Elec_8x10.5, F.Cu at (333.4, 131.5)
- added C404: 47uF, Capacitor_SMD:CP_Elec_8x10.5, F.Cu at (315.7, 143.9)
- added C405: 47uF, Capacitor_SMD:CP_Elec_8x10.5, F.Cu at (369.4, 130.8)
- added C406: 47uF, Capacitor_SMD:CP_Elec_8x10.5, F.Cu at (329.0, 143.9)
- added C407: 0.1uf, Capacitor_SMD:C_1206_3216Metric, F.Cu at (327.7, 153.8)
- added C408: 47uF, Capacitor_SMD:CP_Elec_8x10.5, F.Cu at (346.7, 131.5)
- added C409: 0.1uf, Capacitor_SMD:C_1206_3216Metric, F.Cu at (316.4, 155.3)
- added C412: 47uF, Capacitor_SMD:CP_Elec_8x10.5, F.Cu at (336.6, 215.9)
- added C413: 0.1uf, Capacitor_SMD:C_1206_3216Metric, F.Cu at (315.0, 96.4)
- added C416: 220uF, Capacitor_SMD:CP_Elec_8x10, F.Cu at (117.7, 145.5)
- added C417: 220uF, Capacitor_SMD:CP_Elec_8x10, F.Cu at (138.0, 150.6)
- added C418: 220uF, Capacitor_SMD:CP_Elec_8x10, F.Cu at (159.6, 139.2)
- added C419: 220uF, Capacitor_SMD:CP_Elec_8x10, F.Cu at (177.2, 144.5)
- added C420: 47uF, Capacitor_SMD:CP_Elec_8x10.5, F.Cu at (355.7, 141.6)
- added C421: 47uF, Capacitor_SMD:CP_Elec_8x10.5, F.Cu at (342.4, 151.6)
- added C422: 47uF, Capacitor_SMD:CP_Elec_8x10.5, F.Cu at (369.4, 143.5)
- added C606: 0.1uF, Capacitor_SMD:C_1206_3216Metric, F.Cu at (210.3, 192.3)
- added C617: 1000pF, Capacitor_SMD:C_1206_3216Metric, F.Cu at (179.1, 207.7)
- added C619: 1000pF, Capacitor_SMD:C_1206_3216Metric, F.Cu at (179.1, 213.4)
- added C620: 1000pF, Capacitor_SMD:C_1206_3216Metric, F.Cu at (179.1, 210.4)
- added C621: 1000pF, Capacitor_SMD:C_1206_3216Metric, F.Cu at (179.1, 216.3)
- added C622: 1000pF, Capacitor_SMD:C_1206_3216Metric, F.Cu at (138.3, 222.1)
- added C623: 1000pF, Capacitor_SMD:C_1206_3216Metric, F.Cu at (178.9, 219.2)
- added C624: 1000pF, Capacitor_SMD:C_1206_3216Metric, F.Cu at (138.2, 225.0)
- added C625: 1000pF, Capacitor_SMD:C_1206_3216Metric, F.Cu at (179.0, 222.2)
- added C626: 1000pF, Capacitor_SMD:C_1206_3216Metric, F.Cu at (138.2, 227.8)
- added C627: 1000pF, Capacitor_SMD:C_1206_3216Metric, F.Cu at (179.0, 225.0)
- added C628: 1000pF, Capacitor_SMD:C_1206_3216Metric, F.Cu at (178.9, 230.8)
- added C629: 1000pF, Capacitor_SMD:C_1206_3216Metric, F.Cu at (178.9, 227.9)
- added C630: 1000pF, Capacitor_SMD:C_1206_3216Metric, F.Cu at (138.2, 230.6)
- added C631: 1000pF, Capacitor_SMD:C_1206_3216Metric, F.Cu at (178.8, 233.7)
- added C632: 1000pF, Capacitor_SMD:C_1206_3216Metric, F.Cu at (138.2, 233.6)
- added C633: 1000pF, Capacitor_SMD:C_1206_3216Metric, F.Cu at (138.2, 236.3)
- added C635: 1000pF, Capacitor_SMD:C_1206_3216Metric, F.Cu at (138.2, 239.4)
- added C637: 1000pF, Capacitor_SMD:C_1206_3216Metric, F.Cu at (138.2, 242.2)
- added C639: 1000pF, Capacitor_SMD:C_1206_3216Metric, F.Cu at (138.2, 245.0)
- added C641: 1000pF, Capacitor_SMD:C_1206_3216Metric, F.Cu at (138.0, 247.9)
- added C645: 1000pF, Capacitor_SMD:C_1206_3216Metric, F.Cu at (178.7, 253.0)
- added C647: 1000pF, Capacitor_SMD:C_1206_3216Metric, F.Cu at (178.7, 255.8)
- added C649: 1000pF, Capacitor_SMD:C_1206_3216Metric, F.Cu at (178.7, 258.6)
- added C650: 1000pF, Capacitor_SMD:C_1206_3216Metric, F.Cu at (178.7, 264.3)
- added C651: 1000pF, Capacitor_SMD:C_1206_3216Metric, F.Cu at (178.7, 261.4)
- added C652: 1000pF, Capacitor_SMD:C_1206_3216Metric, F.Cu at (178.7, 267.0)
- added C654: 1000pF, Capacitor_SMD:C_1206_3216Metric, F.Cu at (178.7, 269.7)
- added C655: 1000pF, Capacitor_SMD:C_1206_3216Metric, F.Cu at (178.7, 272.5)
- added C657: 1000pF, Capacitor_SMD:C_1206_3216Metric, F.Cu at (178.7, 278.3)
- added C658: 1000pF, Capacitor_SMD:C_1206_3216Metric, F.Cu at (178.7, 275.3)
- added C659: 1000pF, Capacitor_SMD:C_1206_3216Metric, F.Cu at (138.7, 269.7)
- added C660: 1000pF, Capacitor_SMD:C_1206_3216Metric, F.Cu at (138.7, 272.8)
- added C661: 1000pF, Capacitor_SMD:C_1206_3216Metric, F.Cu at (138.7, 275.6)
- added C662: 1000pF, Capacitor_SMD:C_1206_3216Metric, F.Cu at (138.7, 278.4)
- added C663: 1000pF, Capacitor_SMD:C_1206_3216Metric, F.Cu at (138.7, 281.2)
- added C664: 1000pF, Capacitor_SMD:C_1206_3216Metric, F.Cu at (138.7, 284.0)
- added C665: 1000pF, Capacitor_SMD:C_1206_3216Metric, F.Cu at (138.7, 286.8)
- added C666: 1000pF, Capacitor_SMD:C_1206_3216Metric, F.Cu at (138.7, 289.6)
- added C667: 1000pF, Capacitor_SMD:C_1206_3216Metric, F.Cu at (138.7, 292.4)
- added C668: 1000pF, Capacitor_SMD:C_1206_3216Metric, F.Cu at (138.7, 295.1)
- added C669: 1000pF, Capacitor_SMD:C_1206_3216Metric, F.Cu at (179.1, 293.4)
- added C670: 1000pF, Capacitor_SMD:C_1206_3216Metric, F.Cu at (179.1, 296.2)
- added C671: 1000pF, Capacitor_SMD:C_1206_3216Metric, F.Cu at (179.1, 299.0)
- added C672: 1000pF, Capacitor_SMD:C_1206_3216Metric, F.Cu at (179.1, 301.8)
- added C673: 1000pF, Capacitor_SMD:C_1206_3216Metric, F.Cu at (179.1, 304.5)
- added C674: 1000pF, Capacitor_SMD:C_1206_3216Metric, F.Cu at (179.1, 307.3)
- added C675: 1000pF, Capacitor_SMD:C_1206_3216Metric, F.Cu at (179.1, 310.1)
- added C9000: 1uF, Capacitor_SMD:C_1206_3216Metric, F.Cu at (259.7, 193.8)
- added C9001: 0.33uF, Capacitor_SMD:C_1206_3216Metric, F.Cu at (243.6, 205.5)
- added C9002: 1uF, Capacitor_SMD:C_1206_3216Metric, F.Cu at (230.5, 150.7)
- added C9003: 10uF, Capacitor_SMD:C_1206_3216Metric, F.Cu at (249.3, 139.8)
- added C903: 0.1uf, Capacitor_SMD:C_1206_3216Metric, F.Cu at (379.2, 134.6)
- added C906: 0.1uf, Capacitor_SMD:C_1206_3216Metric, F.Cu at (322.1, 150.6)
- added C910: 0.1uf, Capacitor_SMD:C_1206_3216Metric, F.Cu at (384.4, 128.6)
- added CN400: ATX-24, Connector_Molex:Molex_Mini-Fit_Jr_5566-24A_2x12_P4.20mm_Vertical, F.Cu at (269.0, 178.4)
- added D9000: 1N4148, Diode_SMD:D_SOD-323, F.Cu at (222.5, 156.9)
- added D9001: 1N4148, Diode_SMD:D_SOD-323, F.Cu at (222.5, 153.9)
- added J9000: POWER_SWITCH, Connector_PinHeader_2.54mm:PinHeader_1x02_P2.54mm_Vertical, F.Cu at (234.8, 159.4)
- added R311: 1k, Resistor_SMD:R_1206_3216Metric, F.Cu at (138.6, 217.2)
- added R312: 1k, Resistor_SMD:R_1206_3216Metric, F.Cu at (138.6, 214.4)
- added R600A1: 10k, Resistor_SMD:R_1206_3216Metric, F.Cu at (150.8, 176.3)
- added R600B1: 10k, Resistor_SMD:R_1206_3216Metric, F.Cu at (143.4, 176.8)
- added R600C1: 10k, Resistor_SMD:R_1206_3216Metric, F.Cu at (159.6, 175.5)
- added R600D1: 10k, Resistor_SMD:R_1206_3216Metric, F.Cu at (166.1, 175.5)
- added R600E1: 10k, Resistor_SMD:R_1206_3216Metric, F.Cu at (190.6, 178.1)
- added R601: 1k, Resistor_SMD:R_1206_3216Metric, F.Cu at (182.1, 175.8)
- added R601A1: 1k, Resistor_SMD:R_1206_3216Metric, F.Cu at (159.4, 208.8)
- added R601B1: 1k, Resistor_SMD:R_1206_3216Metric, F.Cu at (159.4, 213.7)
- added R601C1: 1k, Resistor_SMD:R_1206_3216Metric, F.Cu at (159.3, 211.1)
- added R601D1: 1k, Resistor_SMD:R_1206_3216Metric, F.Cu at (159.4, 216.3)
- added R601E1: 1k, Resistor_SMD:R_1206_3216Metric, F.Cu at (118.4, 222.3)
- added R601F1: 1k, Resistor_SMD:R_1206_3216Metric, F.Cu at (159.3, 219.5)
- added R601G1: 1k, Resistor_SMD:R_1206_3216Metric, F.Cu at (118.6, 225.1)
- added R601H1: 1k, Resistor_SMD:R_1206_3216Metric, F.Cu at (159.4, 222.2)
- added R601I1: 1k, Resistor_SMD:R_1206_3216Metric, F.Cu at (118.7, 227.9)
- added R602A1: 1k, Resistor_SMD:R_1206_3216Metric, F.Cu at (159.4, 225.0)
- added R602B1: 1k, Resistor_SMD:R_1206_3216Metric, F.Cu at (159.8, 230.9)
- added R602C1: 1k, Resistor_SMD:R_1206_3216Metric, F.Cu at (159.6, 228.0)
- added R602D1: 1k, Resistor_SMD:R_1206_3216Metric, F.Cu at (118.2, 230.6)
- added R602E1: 1k, Resistor_SMD:R_1206_3216Metric, F.Cu at (159.8, 233.7)
- added R602F1: 1k, Resistor_SMD:R_1206_3216Metric, F.Cu at (118.4, 233.7)
- added R602G1: 1k, Resistor_SMD:R_1206_3216Metric, F.Cu at (118.9, 236.3)
- added R602H1: 1k, Resistor_SMD:R_1206_3216Metric, F.Cu at (118.7, 239.6)
- added R602I1: 1k, Resistor_SMD:R_1206_3216Metric, F.Cu at (118.2, 242.4)
- added R603: 1k, Resistor_SMD:R_1206_3216Metric, F.Cu at (169.9, 169.7)
- added R603A1: 1k, Resistor_SMD:R_1206_3216Metric, F.Cu at (118.4, 245.2)
- added R603B1: 1k, Resistor_SMD:R_1206_3216Metric, F.Cu at (118.2, 247.9)
- added R603C1: 1k, Resistor_SMD:R_1206_3216Metric, F.Cu at (159.4, 253.5)
- added R603D1: 1k, Resistor_SMD:R_1206_3216Metric, F.Cu at (159.4, 256.1)
- added R603E1: 1k, Resistor_SMD:R_1206_3216Metric, F.Cu at (159.1, 258.7)
- added R603F1: 1k, Resistor_SMD:R_1206_3216Metric, F.Cu at (159.3, 264.3)
- added R603G1: 1k, Resistor_SMD:R_1206_3216Metric, F.Cu at (159.1, 261.4)
- added R603H1: 1k, Resistor_SMD:R_1206_3216Metric, F.Cu at (159.3, 267.0)
- added R603I1: 1k, Resistor_SMD:R_1206_3216Metric, F.Cu at (159.3, 269.6)
- added R604: 1k, Resistor_SMD:R_1206_3216Metric, F.Cu at (118.4, 287.1)
- added R604A1: 1k, Resistor_SMD:R_1206_3216Metric, F.Cu at (159.6, 272.5)
- added R604B1: 1k, Resistor_SMD:R_1206_3216Metric, F.Cu at (159.8, 278.4)
- added R604C1: 1k, Resistor_SMD:R_1206_3216Metric, F.Cu at (159.7, 275.1)
- added R604D1: 1k, Resistor_SMD:R_1206_3216Metric, F.Cu at (118.2, 271.5)
- added R604E1: 1k, Resistor_SMD:R_1206_3216Metric, F.Cu at (118.2, 274.1)
- added R604F1: 1k, Resistor_SMD:R_1206_3216Metric, F.Cu at (118.3, 276.5)
- added R604G1: 1k, Resistor_SMD:R_1206_3216Metric, F.Cu at (118.2, 278.5)
- added R604H1: 1k, Resistor_SMD:R_1206_3216Metric, F.Cu at (118.2, 281.2)
- added R604I1: 1k, Resistor_SMD:R_1206_3216Metric, F.Cu at (118.3, 284.2)
- added R605: 1k, Resistor_SMD:R_1206_3216Metric, F.Cu at (118.7, 289.3)
- added R605A1: 1k, Resistor_SMD:R_1206_3216Metric, F.Cu at (118.4, 292.4)
- added R605B1: 1k, Resistor_SMD:R_1206_3216Metric, F.Cu at (118.4, 295.1)
- added R605C1: 1k, Resistor_SMD:R_1206_3216Metric, F.Cu at (158.8, 293.5)
- added R605D1: 1k, Resistor_SMD:R_1206_3216Metric, F.Cu at (158.8, 296.3)
- added R605E1: 1k, Resistor_SMD:R_1206_3216Metric, F.Cu at (158.5, 299.2)
- added R605F1: 1k, Resistor_SMD:R_1206_3216Metric, F.Cu at (158.6, 301.8)
- added R605G1: 1k, Resistor_SMD:R_1206_3216Metric, F.Cu at (158.8, 304.5)
- added R605H1: 1k, Resistor_SMD:R_1206_3216Metric, F.Cu at (158.6, 307.5)
- added R605I1: 1k, Resistor_SMD:R_1206_3216Metric, F.Cu at (158.8, 310.1)
- added R607A1: 1k, Resistor_SMD:R_1206_3216Metric, F.Cu at (175.5, 173.9)
- added R607B1: 1k, Resistor_SMD:R_1206_3216Metric, F.Cu at (118.5, 208.3)
- added R607C1: 1k, Resistor_SMD:R_1206_3216Metric, F.Cu at (118.5, 203.7)
- added R607D1: 1k, Resistor_SMD:R_1206_3216Metric, F.Cu at (138.8, 204.3)
- added R607E1: 1k, Resistor_SMD:R_1206_3216Metric, F.Cu at (159.4, 206.4)
- added R9000: 10k, Resistor_SMD:R_1206_3216Metric, F.Cu at (254.8, 149.0)
- added R9001: 10k, Resistor_SMD:R_1206_3216Metric, F.Cu at (249.2, 152.3)
- added R9002: 470, Resistor_SMD:R_1206_3216Metric, F.Cu at (243.6, 152.3)
- added RNX1A1: 2.7k, Resistor_SMD:R_1206_3216Metric, F.Cu at (288.4, 310.8)
- added RNX1A2: 2.7k, Resistor_SMD:R_1206_3216Metric, F.Cu at (244.7, 310.8)
- added RNX1A3: 2.7k, Resistor_SMD:R_1206_3216Metric, F.Cu at (244.7, 308.2)
- added RNX1A4: 2.7k, Resistor_SMD:R_1206_3216Metric, F.Cu at (244.7, 305.7)
- added RNX1A5: 2.7k, Resistor_SMD:R_1206_3216Metric, F.Cu at (288.4, 308.2)
- added RNX1A6: 2.7k, Resistor_SMD:R_1206_3216Metric, F.Cu at (288.4, 305.7)
- added RNX1A7: 2.7k, Resistor_SMD:R_1206_3216Metric, F.Cu at (288.4, 303.1)
- added RNX1A8: 2.7k, Resistor_SMD:R_1206_3216Metric, F.Cu at (288.3, 300.6)
- added RNX1A9: 2.7k, Resistor_SMD:R_1206_3216Metric, F.Cu at (244.7, 313.2)
- added RNX2A1: 2.7k, Resistor_SMD:R_1206_3216Metric, F.Cu at (244.7, 303.1)
- added RNX2B1: 2.7k, Resistor_SMD:R_1206_3216Metric, F.Cu at (244.7, 300.6)
- added RNX2C1: 2.7k, Resistor_SMD:R_1206_3216Metric, F.Cu at (244.7, 298.1)
- added RNX2D1: 2.7k, Resistor_SMD:R_1206_3216Metric, F.Cu at (244.7, 295.5)
- added RNX2E1: 2.7k, Resistor_SMD:R_1206_3216Metric, F.Cu at (244.7, 293.0)
- added RNX2F1: 2.7k, Resistor_SMD:R_1206_3216Metric, F.Cu at (244.7, 290.4)
- added RNX2G1: 2.7k, Resistor_SMD:R_1206_3216Metric, F.Cu at (244.7, 287.8)
- added RNX2H1: 2.7k, Resistor_SMD:R_1206_3216Metric, F.Cu at (244.7, 285.4)
- added U606: 74LS32, Package_SO:SOIC-14_3.9x8.7mm_P1.27mm, F.Cu at (209.3, 201.8)
- added U9000: MC7905, Package_TO_SOT_SMD:TO-263-2, F.Cu at (261.5, 205.7)
- added U9001: 74HC14, Package_SO:SOIC-14_3.9x8.7mm_P1.27mm, F.Cu at (237.1, 139.8)
- added U9002: 74HC74, Package_SO:SOIC-14_3.9x8.7mm_P1.27mm, F.Cu at (222.1, 139.6)
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Connections:
- net Net-(CN601-Pad64) renamed _EBG5
- net Net-(CN601-Pad9) renamed _SLAVE5
- net Net-(CN602-Pad64) renamed _EBG4
- net Net-(CN602-Pad9) renamed _SLAVE4
- net Net-(CN603-Pad64) renamed _EBG3
- net Net-(CN603-Pad9) renamed _SLAVE3
- net Net-(CN604-Pad64) renamed _EBG2
- net Net-(CN604-Pad9) renamed _SLAVE2
- net Net-(CN605-Pad64) renamed _EBG1
- net Net-(CN605-Pad9) renamed _SLAVE1
- CN601 pad 1: Net-(CN601-Pad1) -> GND
- CN601 pad 10: Net-(CN601-Pad10) -> +12V
- CN601 pad 100: Net-(CN601-Pad100) -> GND
- CN601 pad 12: Net-(CN601-Pad12) -> /Zorro_Expansion/_CFGOUT5
- CN601 pad 13: Net-(CN601-Pad13) -> GND
- CN601 pad 14: Net-(CN601-Pad14) -> EC3
- CN601 pad 15: Net-(CN601-Pad15) -> ECDAC
- CN601 pad 16: Net-(CN601-Pad16) -> _EC1
- CN601 pad 17: Net-(CN601-Pad17) -> _OVR
- CN601 pad 18: Net-(CN601-Pad18) -> XRDY
- CN601 pad 19: Net-(CN601-Pad19) -> _INT2
- CN601 pad 2: Net-(CN601-Pad2) -> GND
- CN601 pad 20: Net-(CN601-Pad20) -> -12V
- CN601 pad 21: Net-(CN601-Pad21) -> BA5
- CN601 pad 22: Net-(CN601-Pad22) -> _INT6
- CN601 pad 23: Net-(CN601-Pad23) -> BA6
- CN601 pad 24: Net-(CN601-Pad24) -> BA4
- CN601 pad 25: Net-(CN601-Pad25) -> GND
- CN601 pad 26: Net-(CN601-Pad26) -> BA3
- CN601 pad 27: Net-(CN601-Pad27) -> BA2
- CN601 pad 28: Net-(CN601-Pad28) -> BA7
- CN601 pad 29: Net-(CN601-Pad29) -> BA1
- CN601 pad 3: Net-(CN601-Pad3) -> GND
- CN601 pad 30: Net-(CN601-Pad30) -> BA8
- CN601 pad 31: Net-(CN601-Pad31) -> BFC0
- CN601 pad 32: Net-(CN601-Pad32) -> BA9
- CN601 pad 33: Net-(CN601-Pad33) -> BFC1
- CN601 pad 34: Net-(CN601-Pad34) -> BA10
- CN601 pad 35: Net-(CN601-Pad35) -> BFC2
- CN601 pad 36: Net-(CN601-Pad36) -> BA11
- CN601 pad 37: Net-(CN601-Pad37) -> GND
- CN601 pad 38: Net-(CN601-Pad38) -> BA12
- CN601 pad 39: Net-(CN601-Pad39) -> BA13
- CN601 pad 4: Net-(CN601-Pad4) -> GND
- CN601 pad 40: Net-(CN601-Pad40) -> _EINT7
- CN601 pad 41: Net-(CN601-Pad41) -> BA14
- CN601 pad 42: Net-(CN601-Pad42) -> _EINT5
- CN601 pad 43: Net-(CN601-Pad43) -> BA15
- CN601 pad 44: Net-(CN601-Pad44) -> _EINT4
- CN601 pad 45: Net-(CN601-Pad45) -> BA16
- CN601 pad 46: Net-(CN601-Pad46) -> _BEER
- CN601 pad 47: Net-(CN601-Pad47) -> BA17
- CN601 pad 48: Net-(CN601-Pad48) -> _VPA
- CN601 pad 49: Net-(CN601-Pad49) -> GND
- CN601 pad 5: Net-(CN601-Pad5) -> +5V
- CN601 pad 50: Net-(CN601-Pad50) -> E
- CN601 pad 51: Net-(CN601-Pad51) -> _VMA
- CN601 pad 52: Net-(CN601-Pad52) -> BA18
- CN601 pad 53: Net-(CN601-Pad53) -> _RST
- CN601 pad 54: Net-(CN601-Pad54) -> BA19
- CN601 pad 55: Net-(CN601-Pad55) -> _HLT
- CN601 pad 56: Net-(CN601-Pad56) -> BA20
- CN601 pad 57: Net-(CN601-Pad57) -> BA22
- CN601 pad 58: Net-(CN601-Pad58) -> BA21
- CN601 pad 59: Net-(CN601-Pad59) -> BA23
- CN601 pad 6: Net-(CN601-Pad6) -> +5V
- CN601 pad 60: Net-(CN601-Pad60) -> _EBR5
- CN601 pad 61: Net-(CN601-Pad61) -> GND
- CN601 pad 62: Net-(CN601-Pad62) -> _BGACK
- CN601 pad 63: Net-(CN601-Pad63) -> BD15
- CN601 pad 65: Net-(CN601-Pad65) -> BD14
- CN601 pad 66: Net-(CN601-Pad66) -> _DTACK
- CN601 pad 67: Net-(CN601-Pad67) -> BD13
- CN601 pad 68: Net-(CN601-Pad68) -> READ
- CN601 pad 69: Net-(CN601-Pad69) -> BD12
- CN601 pad 7: Net-(CN601-Pad7) -> _OWN
- CN601 pad 70: Net-(CN601-Pad70) -> _BLDS
- CN601 pad 71: Net-(CN601-Pad71) -> BD11
- CN601 pad 72: Net-(CN601-Pad72) -> _BUDS
- CN601 pad 73: Net-(CN601-Pad73) -> GND
- CN601 pad 74: Net-(CN601-Pad74) -> _BAS
- CN601 pad 75: Net-(CN601-Pad75) -> BD0
- CN601 pad 76: Net-(CN601-Pad76) -> BD10
- CN601 pad 77: Net-(CN601-Pad77) -> BD1
- CN601 pad 78: Net-(CN601-Pad78) -> BD9
- CN601 pad 79: Net-(CN601-Pad79) -> BD2
- CN601 pad 8: Net-(CN601-Pad8) -> -5V
- CN601 pad 80: Net-(CN601-Pad80) -> BD8
- CN601 pad 81: Net-(CN601-Pad81) -> BD3
- CN601 pad 82: Net-(CN601-Pad82) -> BD7
- CN601 pad 83: Net-(CN601-Pad83) -> BD4
- CN601 pad 84: Net-(CN601-Pad84) -> BD6
- CN601 pad 85: Net-(CN601-Pad85) -> GND
- CN601 pad 86: Net-(CN601-Pad86) -> BD5
- CN601 pad 87: Net-(CN601-Pad87) -> GND
- CN601 pad 88: Net-(CN601-Pad88) -> GND
- CN601 pad 89: Net-(CN601-Pad89) -> GND
- CN601 pad 90: Net-(CN601-Pad90) -> GND
- CN601 pad 91: Net-(CN601-Pad91) -> GND
- CN601 pad 92: Net-(CN601-Pad92) -> E7M
- CN601 pad 93: Net-(CN601-Pad93) -> DOE
- CN601 pad 94: Net-(CN601-Pad94) -> _BURST
- CN601 pad 95: Net-(CN601-Pad95) -> _GBG
- CN601 pad 96: Net-(CN601-Pad96) -> _EINT1
- CN601 pad 99: Net-(CN601-Pad99) -> GND
- CN602 pad 1: Net-(CN602-Pad1) -> GND
- CN602 pad 10: Net-(CN602-Pad10) -> +12V
- CN602 pad 100: Net-(CN602-Pad100) -> GND
- CN602 pad 11: Net-(CN602-Pad11) -> /Zorro_Expansion/_CFGIN4
- CN602 pad 12: Net-(CN602-Pad12) -> /Zorro_Expansion/_CFGOUT4
- CN602 pad 13: Net-(CN602-Pad13) -> GND
- CN602 pad 14: Net-(CN602-Pad14) -> EC3
- CN602 pad 15: Net-(CN602-Pad15) -> ECDAC
- CN602 pad 16: Net-(CN602-Pad16) -> _EC1
- CN602 pad 17: Net-(CN602-Pad17) -> _OVR
- CN602 pad 18: Net-(CN602-Pad18) -> XRDY
- CN602 pad 19: Net-(CN602-Pad19) -> _INT2
- CN602 pad 2: Net-(CN602-Pad2) -> GND
- CN602 pad 20: Net-(CN602-Pad20) -> -12V
- CN602 pad 21: Net-(CN602-Pad21) -> BA5
- CN602 pad 22: Net-(CN602-Pad22) -> _INT6
- CN602 pad 23: Net-(CN602-Pad23) -> BA6
- CN602 pad 24: Net-(CN602-Pad24) -> BA4
- CN602 pad 25: Net-(CN602-Pad25) -> GND
- CN602 pad 26: Net-(CN602-Pad26) -> BA3
- CN602 pad 27: Net-(CN602-Pad27) -> BA2
- CN602 pad 28: Net-(CN602-Pad28) -> BA7
- CN602 pad 29: Net-(CN602-Pad29) -> BA1
- CN602 pad 3: Net-(CN602-Pad3) -> GND
- CN602 pad 30: Net-(CN602-Pad30) -> BA8
- CN602 pad 31: Net-(CN602-Pad31) -> BFC0
- CN602 pad 32: Net-(CN602-Pad32) -> BA9
- CN602 pad 33: Net-(CN602-Pad33) -> BFC1
- CN602 pad 34: Net-(CN602-Pad34) -> BA10
- CN602 pad 35: Net-(CN602-Pad35) -> BFC2
- CN602 pad 36: Net-(CN602-Pad36) -> BA11
- CN602 pad 37: Net-(CN602-Pad37) -> GND
- CN602 pad 38: Net-(CN602-Pad38) -> BA12
- CN602 pad 39: Net-(CN602-Pad39) -> BA13
- CN602 pad 4: Net-(CN602-Pad4) -> GND
- CN602 pad 40: Net-(CN602-Pad40) -> _EINT7
- CN602 pad 41: Net-(CN602-Pad41) -> BA14
- CN602 pad 42: Net-(CN602-Pad42) -> _EINT5
- CN602 pad 43: Net-(CN602-Pad43) -> BA15
- CN602 pad 44: Net-(CN602-Pad44) -> _EINT4
- CN602 pad 45: Net-(CN602-Pad45) -> BA16
- CN602 pad 46: Net-(CN602-Pad46) -> _BEER
- CN602 pad 47: Net-(CN602-Pad47) -> BA17
- CN602 pad 48: Net-(CN602-Pad48) -> _VPA
- CN602 pad 49: Net-(CN602-Pad49) -> GND
- CN602 pad 5: Net-(CN602-Pad5) -> +5V
- CN602 pad 50: Net-(CN602-Pad50) -> E
- CN602 pad 51: Net-(CN602-Pad51) -> _VMA
- CN602 pad 52: Net-(CN602-Pad52) -> BA18
- CN602 pad 53: Net-(CN602-Pad53) -> _RST
- CN602 pad 54: Net-(CN602-Pad54) -> BA19
- CN602 pad 55: Net-(CN602-Pad55) -> _HLT
- CN602 pad 56: Net-(CN602-Pad56) -> BA20
- CN602 pad 57: Net-(CN602-Pad57) -> BA22
- CN602 pad 58: Net-(CN602-Pad58) -> BA21
- CN602 pad 59: Net-(CN602-Pad59) -> BA23
- CN602 pad 6: Net-(CN602-Pad6) -> +5V
- CN602 pad 60: Net-(CN602-Pad60) -> _EBR4
- CN602 pad 61: Net-(CN602-Pad61) -> GND
- CN602 pad 62: Net-(CN602-Pad62) -> _BGACK
- CN602 pad 63: Net-(CN602-Pad63) -> BD15
- CN602 pad 65: Net-(CN602-Pad65) -> BD14
- CN602 pad 66: Net-(CN602-Pad66) -> _DTACK
- CN602 pad 67: Net-(CN602-Pad67) -> BD13
- CN602 pad 68: Net-(CN602-Pad68) -> READ
- CN602 pad 69: Net-(CN602-Pad69) -> BD12
- CN602 pad 7: Net-(CN602-Pad7) -> _OWN
- CN602 pad 70: Net-(CN602-Pad70) -> _BLDS
- CN602 pad 71: Net-(CN602-Pad71) -> BD11
- CN602 pad 72: Net-(CN602-Pad72) -> _BUDS
- CN602 pad 73: Net-(CN602-Pad73) -> GND
- CN602 pad 74: Net-(CN602-Pad74) -> _BAS
- CN602 pad 75: Net-(CN602-Pad75) -> BD0
- CN602 pad 76: Net-(CN602-Pad76) -> BD10
- CN602 pad 77: Net-(CN602-Pad77) -> BD1
- CN602 pad 78: Net-(CN602-Pad78) -> BD9
- CN602 pad 79: Net-(CN602-Pad79) -> BD2
- CN602 pad 8: Net-(CN602-Pad8) -> -5V
- CN602 pad 80: Net-(CN602-Pad80) -> BD8
- CN602 pad 81: Net-(CN602-Pad81) -> BD3
- CN602 pad 82: Net-(CN602-Pad82) -> BD7
- CN602 pad 83: Net-(CN602-Pad83) -> BD4
- CN602 pad 84: Net-(CN602-Pad84) -> BD6
- CN602 pad 85: Net-(CN602-Pad85) -> GND
- CN602 pad 86: Net-(CN602-Pad86) -> BD5
- CN602 pad 87: Net-(CN602-Pad87) -> GND
- CN602 pad 88: Net-(CN602-Pad88) -> GND
- CN602 pad 89: Net-(CN602-Pad89) -> GND
- CN602 pad 90: Net-(CN602-Pad90) -> GND
- CN602 pad 91: Net-(CN602-Pad91) -> GND
- CN602 pad 92: Net-(CN602-Pad92) -> E7M
- CN602 pad 93: Net-(CN602-Pad93) -> DOE
- CN602 pad 94: Net-(CN602-Pad94) -> _BURST
- CN602 pad 95: Net-(CN602-Pad95) -> _GBG
- CN602 pad 96: Net-(CN602-Pad96) -> _EINT1
- CN602 pad 97: Net-(CN602-Pad97) -> Net-(CN601-Pad97)
- CN602 pad 98: Net-(CN602-Pad98) -> Net-(CN601-Pad98)
- CN602 pad 99: Net-(CN602-Pad99) -> GND
- CN603 pad 1: Net-(CN603-Pad1) -> GND
- CN603 pad 10: Net-(CN603-Pad10) -> +12V
- CN603 pad 100: Net-(CN603-Pad100) -> GND
- CN603 pad 11: Net-(CN603-Pad11) -> /Zorro_Expansion/_CFGIN3
- CN603 pad 12: Net-(CN603-Pad12) -> /Zorro_Expansion/_CFGOUT3
- CN603 pad 13: Net-(CN603-Pad13) -> GND
- CN603 pad 14: Net-(CN603-Pad14) -> EC3
- CN603 pad 15: Net-(CN603-Pad15) -> ECDAC
- CN603 pad 16: Net-(CN603-Pad16) -> _EC1
- CN603 pad 17: Net-(CN603-Pad17) -> _OVR
- CN603 pad 18: Net-(CN603-Pad18) -> XRDY
- CN603 pad 19: Net-(CN603-Pad19) -> _INT2
- CN603 pad 2: Net-(CN603-Pad2) -> GND
- CN603 pad 20: Net-(CN603-Pad20) -> -12V
- CN603 pad 21: Net-(CN603-Pad21) -> BA5
- CN603 pad 22: Net-(CN603-Pad22) -> _INT6
- CN603 pad 23: Net-(CN603-Pad23) -> BA6
- CN603 pad 24: Net-(CN603-Pad24) -> BA4
- CN603 pad 25: Net-(CN603-Pad25) -> GND
- CN603 pad 26: Net-(CN603-Pad26) -> BA3
- CN603 pad 27: Net-(CN603-Pad27) -> BA2
- CN603 pad 28: Net-(CN603-Pad28) -> BA7
- CN603 pad 29: Net-(CN603-Pad29) -> BA1
- CN603 pad 3: Net-(CN603-Pad3) -> GND
- CN603 pad 30: Net-(CN603-Pad30) -> BA8
- CN603 pad 31: Net-(CN603-Pad31) -> BFC0
- CN603 pad 32: Net-(CN603-Pad32) -> BA9
- CN603 pad 33: Net-(CN603-Pad33) -> BFC1
- CN603 pad 34: Net-(CN603-Pad34) -> BA10
- CN603 pad 35: Net-(CN603-Pad35) -> BFC2
- CN603 pad 36: Net-(CN603-Pad36) -> BA11
- CN603 pad 37: Net-(CN603-Pad37) -> GND
- CN603 pad 38: Net-(CN603-Pad38) -> BA12
- CN603 pad 39: Net-(CN603-Pad39) -> BA13
- CN603 pad 4: Net-(CN603-Pad4) -> GND
- CN603 pad 40: Net-(CN603-Pad40) -> _EINT7
- CN603 pad 41: Net-(CN603-Pad41) -> BA14
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Routing:
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- added copper zone on F.Cu, net +12V
- added copper zone on F.Cu, net +5V
- added copper zone on F.Cu, net -12V
- added copper zone on B.Cu, net GND
Other:
- net class GND1 added: clearance 0.2, trace_width 0.381, via_dia 0.8, via_drill 0.4
- net class PWR1 added: clearance 0.2, trace_width 0.4572, via_dia 0.8, via_drill 0.4

Commit message: Add files via upload
Parts:
- removed RN100: 4.7k, Resistor_THT:R_Array_SIP10
- removed RN101: 2.7k, Resistor_THT:R_Array_SIP10
- added R100A1: 4.7k, Resistor_SMD:R_1206_3216Metric, F.Cu at (288.2, 242.2)
- added R100B1: 4.7k, Resistor_SMD:R_1206_3216Metric, F.Cu at (288.2, 244.7)
- added R100C1: 4.7k, Resistor_SMD:R_1206_3216Metric, F.Cu at (288.2, 247.3)
- added R100D1: 4.7k, Resistor_SMD:R_1206_3216Metric, F.Cu at (288.2, 249.8)
- added R100E1: 4.7k, Resistor_SMD:R_1206_3216Metric, F.Cu at (288.2, 252.3)
- added R100F1: 4.7k, Resistor_SMD:R_1206_3216Metric, F.Cu at (288.2, 254.9)
- added R100G1: 4.7k, Resistor_SMD:R_1206_3216Metric, F.Cu at (288.2, 282.8)
- added R100H1: 4.7k, Resistor_SMD:R_1206_3216Metric, F.Cu at (337.9, 249.0)
- added R100I1: 4.7k, Resistor_SMD:R_1206_3216Metric, F.Cu at (288.2, 280.3)
- added R101A1: 2.7k, Resistor_SMD:R_1206_3216Metric, F.Cu at (288.2, 267.6)
- added R101B1: 2.7k, Resistor_SMD:R_1206_3216Metric, F.Cu at (288.2, 270.1)
- added R101C1: 2.7k, Resistor_SMD:R_1206_3216Metric, F.Cu at (288.2, 287.9)
- added R101D1: 2.7k, Resistor_SMD:R_1206_3216Metric, F.Cu at (288.2, 298.1)
- added R101E1: 2.7k, Resistor_SMD:R_1206_3216Metric, F.Cu at (288.2, 290.4)
- added R101F1: 2.7k, Resistor_SMD:R_1206_3216Metric, F.Cu at (288.2, 295.5)
- added R101G1: 2.7k, Resistor_SMD:R_1206_3216Metric, F.Cu at (288.2, 293.0)
- added R101H1: 2.7k, Resistor_SMD:R_1206_3216Metric, F.Cu at (288.2, 265.0)
- added R101I1: 2.7k, Resistor_SMD:R_1206_3216Metric, F.Cu at (288.2, 260.0)
- C400, C402, C403, C404, C405, C406, C408, C412, C420, C421, C422: footprint Capacitor_SMD:CP_Elec_8x10.5 -> Capacitor_SMD:CP_Elec_6.3x5.8
- C416, C417, C418, C419: footprint Capacitor_SMD:CP_Elec_8x10 -> Capacitor_SMD:CP_Elec_6.3x5.8
- moved C405 162.2 mm to (218.8, 190.9), turned to 270 degrees
- moved C402 120.1 mm to (257.9, 163.5), turned to 180 degrees
- moved C413 112.6 mm to (318.0, 208.9)
- moved C400 100.4 mm to (257.9, 174.0), turned to 180 degrees
- moved C416 94.3 mm to (200.2, 191.3), turned to 90 degrees
- moved C408 84.8 mm to (291.8, 196.2)
- moved U105 82.2 mm to (313.5, 324.0)
- moved U9002 78.5 mm to (298.8, 156.5)
- moved C403 78.5 mm to (257.9, 153.2), turned to 180 degrees
- moved C406 72.3 mm to (257.6, 132.3), turned to 180 degrees
- moved U9001 68.0 mm to (298.8, 168.5)
- moved C9002 63.8 mm to (291.1, 170.8), turned to 270 degrees
- moved D9000 63.5 mm to (285.8, 151.7), turned to 270 degrees
- moved D9001 63.4 mm to (285.8, 158.2), turned to 270 degrees
- moved C422 61.5 mm to (329.2, 190.1), turned to 180 degrees
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Routing:
- net GND: track 1184.7 -> 1865.0 mm, vias 5 -> 9
- net +5V: track 238.2 -> 355.8 mm
- net _DTACK: track 84.5 -> 186.0 mm, vias 0 -> 1
- net /Power/+5VSB: track 0.00 -> 69.5 mm
- net _UDS: track 0.00 -> 55.5 mm
- net _AS: track 0.00 -> 55.5 mm
- net R_W: track 0.00 -> 55.5 mm
- net _LDS: track 0.00 -> 55.5 mm
- net _HLT: track 144.7 -> 198.5 mm, vias 0 -> 1
- net _RST: track 143.6 -> 196.8 mm, vias 0 -> 1
- net _VMA: track 141.7 -> 194.2 mm, vias 0 -> 2
- net _VPA: track 137.7 -> 190.1 mm, vias 0 -> 2
- net _BEER: track 135.0 -> 181.0 mm, vias 0 -> 2
- net E: track 136.7 -> 182.8 mm, vias 0 -> 2
- net _BGACK: track 86.9 -> 132.9 mm, vias 0 -> 1
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- added copper zone on B.Cu, net +12V
- added copper zone on F.Cu, net GND
- removed copper zone on F.Cu, net +12V

Commit message: Add files via upload
Parts:
- removed the REF** at (196.8, 35.6)
- added C1V1: 100nF, Capacitor_SMD:C_1206_3216Metric, F.Cu at (258.5, 47.4)
- added C201: 0.22uF, Capacitor_SMD:C_0603_1608Metric, F.Cu at (443.4, 75.6)
- added C205: 0.1uF, Capacitor_SMD:C_0603_1608Metric, F.Cu at (463.1, 80.2)
- added C206: 0.1uF, Capacitor_SMD:C_0603_1608Metric, F.Cu at (455.7, 74.9)
- added C214: 470uF, Capacitor_SMD:CP_Elec_6.3x5.8, F.Cu at (459.8, 190.9)
- added C226: 470uF, Capacitor_SMD:CP_Elec_6.3x5.8, F.Cu at (447.2, 190.9)
- added C2V1: 100nF, Capacitor_SMD:C_1206_3216Metric, F.Cu at (267.5, 47.4)
- added C3V1: 100nF, Capacitor_SMD:C_1206_3216Metric, F.Cu at (276.7, 47.4)
- added C913: 47pF, Capacitor_SMD:C_1206_3216Metric, F.Cu at (443.9, 81.1)
- added C914: 100pF, Capacitor_SMD:C_0603_1608Metric, F.Cu at (449.9, 75.4)
- added C915: 0.1uF, Capacitor_SMD:C_1206_3216Metric, F.Cu at (450.5, 81.0)
- added CN201: Amiga-2000-Video-Slot, AmigaFootprints:2x18_P2.54mm_Horizontal, F.Cu at (209.5, 71.7)
- added CN202: DB15_Female_HighDensity, Connector_Dsub:DSUB-15-HD_Female_Horizontal_P2.29x1.98mm_EdgePinOffset3.03mm_Housed_MountingHolesOffset4.94mm, F.Cu at (262.5, 32.8)
- added CN203: Amiga-2000-Video-Slot, AmigaFootprints:2x18_P2.54mm_Horizontal, F.Cu at (209.4, 125.2)
- added CP1: 0.1uF, Capacitor_SMD:C_1206_3216Metric, F.Cu at (470.0, 139.3)
- added CP2: 0.1uf, Capacitor_SMD:C_1206_3216Metric, F.Cu at (490.2, 134.2)
- added CP3: 0.1uF, Capacitor_SMD:C_1206_3216Metric, F.Cu at (475.6, 139.3)
- added EMI200: 100pF, AmigaFootprints:C_1206_3216_Feedthrough, F.Cu at (354.7, 33.8)
- added EMI206: 100pF, AmigaFootprints:C_1206_3216_Feedthrough, F.Cu at (275.9, 38.3)
- added EMI207: 100pF, AmigaFootprints:C_1206_3216_Feedthrough, F.Cu at (281.4, 38.3)
- added EMI229: 100pF, AmigaFootprints:C_1206_3216_Feedthrough, F.Cu at (339.0, 33.9)
- added FB900: Ferrite_Bead, Capacitor_SMD:C_1206_3216Metric, F.Cu at (262.5, 38.4)
- added FB901: Ferrite_Bead, Capacitor_SMD:C_1206_3216Metric, F.Cu at (264.8, 38.4)
- added FB902: Ferrite_Bead, Capacitor_SMD:C_1206_3216Metric, F.Cu at (267.2, 38.4)
- added G***: LOGO, AmigaFootprints:RaspberryPiZerowithHoles, F.Cu at (146.2, 79.0)
- added JPP1: JP1, Connector_PinHeader_2.54mm:PinHeader_1x03_P2.54mm_Vertical, F.Cu at (481.6, 31.3)
- added JPP2: Push Button, Connector_PinHeader_2.54mm:PinHeader_1x02_P2.54mm_Vertical, F.Cu at (481.2, 54.4)
- added JPP3: Raspberry_Pi_0, Connector_PinSocket_2.54mm:PinSocket_2x20_P2.54mm_Vertical, F.Cu at (435.4, 16.8)
- added Q1V1: MMBT3904, Package_TO_SOT_SMD:SOT-23, F.Cu at (256.7, 55.1)
- added Q2V1: MMBT3904, Package_TO_SOT_SMD:SOT-23, F.Cu at (265.8, 55.1)
- added Q3V1: MMBT3904, Package_TO_SOT_SMD:SOT-23, F.Cu at (275.2, 55.1)
- added R10V1: 2k, Resistor_SMD:R_1206_3216Metric, F.Cu at (275.5, 62.8)
- added R11V1: 4k, Resistor_SMD:R_1206_3216Metric, F.Cu at (278.0, 62.8)
- added R12V1: 8k, Resistor_SMD:R_1206_3216Metric, F.Cu at (280.5, 62.8)
- added R13V1: 470, Resistor_SMD:R_1206_3216Metric, F.Cu at (252.7, 62.8)
- added R14V1: 390, Resistor_SMD:R_1206_3216Metric, F.Cu at (255.2, 62.8)
- added R15V1: 470, Resistor_SMD:R_1206_3216Metric, F.Cu at (267.8, 62.8)
- added R16V1: 390, Resistor_SMD:R_1206_3216Metric, F.Cu at (270.4, 62.8)
- added R17V1: 470, Resistor_SMD:R_1206_3216Metric, F.Cu at (283.1, 62.8)
- added R18V1: 390, Resistor_SMD:R_1206_3216Metric, F.Cu at (285.6, 62.8)
- added R19V1: 75, Resistor_SMD:R_1206_3216Metric, F.Cu at (253.3, 47.4)
- added R1V1: 1k, Resistor_SMD:R_1206_3216Metric, F.Cu at (242.8, 62.8)
- added R203: 10k, Resistor_SMD:R_1206_3216Metric, F.Cu at (421.6, 81.5)
- added R203A1: 47, Resistor_SMD:R_1206_3216Metric, F.Cu at (414.8, 74.0)
- added R203B1: 47, Resistor_SMD:R_1206_3216Metric, F.Cu at (414.7, 57.4)
- added R20V1: 75, Resistor_SMD:R_1206_3216Metric, F.Cu at (255.9, 47.4)
- added R211: 10k, Resistor_SMD:R_1206_3216Metric, F.Cu at (412.8, 95.9)
- added R212: 22, Resistor_SMD:R_1206_3216Metric, F.Cu at (414.4, 79.4)
- added R215: 1, Resistor_SMD:R_1206_3216Metric, F.Cu at (413.6, 112.5)
- added R216: 10k, Resistor_SMD:R_1206_3216Metric, F.Cu at (420.7, 87.4)
- added R21V1: 75, Resistor_SMD:R_1206_3216Metric, F.Cu at (262.3, 47.4)
- added R22V1: 75, Resistor_SMD:R_1206_3216Metric, F.Cu at (264.9, 47.4)
- added R23V1: 75, Resistor_SMD:R_1206_3216Metric, F.Cu at (271.4, 47.4)
- added R24V1: 75, Resistor_SMD:R_1206_3216Metric, F.Cu at (274.1, 47.4)
- added R2V1: 4k, Resistor_SMD:R_1206_3216Metric, F.Cu at (247.7, 62.8)
- added R3V1: 2k, Resistor_SMD:R_1206_3216Metric, F.Cu at (245.3, 62.8)
- added R4V1: 8k, Resistor_SMD:R_1206_3216Metric, F.Cu at (250.1, 62.8)
- added R5V1: 1k, Resistor_SMD:R_1206_3216Metric, F.Cu at (257.7, 62.8)
- added R6V1: 2k, Resistor_SMD:R_1206_3216Metric, F.Cu at (260.3, 62.8)
- added R7V1: 4k, Resistor_SMD:R_1206_3216Metric, F.Cu at (262.7, 62.8)
- added R8V1: 8k, Resistor_SMD:R_1206_3216Metric, F.Cu at (265.2, 62.8)
- added R9V1: 1k, Resistor_SMD:R_1206_3216Metric, F.Cu at (273.0, 62.8)
- added RN201A1: 47, Resistor_SMD:R_1206_3216Metric, F.Cu at (421.9, 74.2)
- added RN201B1: 47, Resistor_SMD:R_1206_3216Metric, F.Cu at (421.9, 69.2)
- added RN201C1: 47, Resistor_SMD:R_1206_3216Metric, F.Cu at (456.8, 81.0)
- added RN201D1: 47, Resistor_SMD:R_1206_3216Metric, F.Cu at (415.1, 69.0)
- added RN203E1: 47, Resistor_SMD:R_1206_3216Metric, F.Cu at (419.9, 99.1)
- added RN205A1: 1k, Resistor_SMD:R_1206_3216Metric, F.Cu at (415.1, 51.7)
- added RN205B1: 1k, Resistor_SMD:R_1206_3216Metric, F.Cu at (460.3, 181.3)
- added RN205C1: 1k, Resistor_SMD:R_1206_3216Metric, F.Cu at (413.1, 101.6)
- added RN205D1: 1k, Resistor_SMD:R_1206_3216Metric, F.Cu at (422.0, 110.1)
- added RN904A1: 4.7k, Resistor_SMD:R_1206_3216Metric, F.Cu at (423.2, 46.4)
- added RN904B1: 4.7k, Resistor_SMD:R_1206_3216Metric, F.Cu at (421.8, 63.1)
- added RN904C1: 4.7k, Resistor_SMD:R_1206_3216Metric, F.Cu at (462.5, 74.9)
- added RN904D1: 4.7k, Resistor_SMD:R_1206_3216Metric, F.Cu at (421.7, 57.7)
- added RN905A1: 4.7k, Resistor_SMD:R_1206_3216Metric, F.Cu at (413.3, 90.7)
- added RN905B1: 4.7k, Resistor_SMD:R_1206_3216Metric, F.Cu at (413.6, 85.3)
- added RN905C1: 4.7k, Resistor_SMD:R_1206_3216Metric, F.Cu at (421.2, 104.3)
- added RN905D1: 4.7k, Resistor_SMD:R_1206_3216Metric, F.Cu at (414.3, 63.3)
- added RN906A1: 4.7k, Resistor_SMD:R_1206_3216Metric, F.Cu at (420.7, 93.3)
- added RN906B1: 4.7k, Resistor_SMD:R_1206_3216Metric, F.Cu at (413.0, 106.9)
- added RN906C1: 4.7k, Resistor_SMD:R_1206_3216Metric, F.Cu at (415.0, 46.3)
- added RN906D1: 4.7k, Resistor_SMD:R_1206_3216Metric, F.Cu at (421.3, 51.7)
- added RP1: 3k3, Resistor_SMD:R_1206_3216Metric, F.Cu at (456.4, 66.4)
- added U201: Denise, Package_DIP:DIP-48_W15.24mm, F.Cu at (304.7, 103.0)
- added U205: 74HCT244, Package_SO:SOIC-20W_7.5x12.8mm_P1.27mm, F.Cu at (256.0, 88.2)
- added U206: 74HCT244, Package_SO:SOIC-20W_7.5x12.8mm_P1.27mm, F.Cu at (282.0, 88.1)
- added U303: 74LS08, Package_SO:SOIC-14_3.9x8.7mm_P1.27mm, F.Cu at (445.1, 215.5)
- added UP1: 74AHC86N, Package_SO:SOIC-14_3.9x8.7mm_P1.27mm, F.Cu at (496.4, 51.6)
- added UP2: 74LVC574A, Package_SO:SOIC-20W_7.5x12.8mm_P1.27mm, F.Cu at (433.3, 31.0)
- added UP3: 74LVC574A, Package_SO:SOIC-20W_7.5x12.8mm_P1.27mm, F.Cu at (467.6, 53.3)
- added VIDIOT: HY200, Connector_PinSocket_2.54mm:PinSocket_1x22_P2.54mm_Vertical, F.Cu at (243.5, 72.5)
- moved U106 80.1 mm to (325.9, 232.8)
Connections:
- net Net-(CN400-Pad1) renamed +3V3
Routing:
- net GND: track 1865.0 -> 2036.3 mm, vias 9 -> 11
- net +VID: track 0.00 -> 115.5 mm, vias 0 -> 4
- net /Video/BLUE: track 0.00 -> 50.7 mm, vias 0 -> 2
- net /Video/RED: track 0.00 -> 43.6 mm, vias 0 -> 2
- net /Video/GREEN: track 0.00 -> 42.9 mm, vias 0 -> 2
- net Net-(Q3V1-Pad2): track 0.00 -> 18.5 mm
- net Net-(Q2V1-Pad2): track 0.00 -> 18.3 mm
- net Net-(Q1V1-Pad2): track 0.00 -> 18.0 mm
- net Net-(CN202-Pad14): track 0.00 -> 17.7 mm, vias 0 -> 1
- net Net-(CN202-Pad13): track 0.00 -> 16.3 mm
- net R2: track 0.00 -> 11.7 mm
- net R3: track 0.00 -> 11.5 mm
- net R1: track 0.00 -> 11.3 mm
- net R0: track 0.00 -> 11.1 mm
- net G0: track 0.00 -> 9.85 mm
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Other:
- board text added: "VIDIOT CIRCUIT"

Commit message: Add files via upload
Parts:
- added C800: 0.1uF, Capacitor_SMD:C_1206_3216Metric, F.Cu at (157.8, 331.4)
- added C802: 0.1uF, Capacitor_SMD:C_1206_3216Metric, F.Cu at (211.5, 343.0)
- added C803: 0.1uF, Capacitor_SMD:C_1206_3216Metric, F.Cu at (227.0, 342.0)
- added C804: 0.1uF, Capacitor_SMD:C_1206_3216Metric, F.Cu at (242.6, 341.7)
- added C904: 100pF, Capacitor_SMD:C_1206_3216Metric, F.Cu at (168.5, 346.6)
- added C920: 100pF, Capacitor_SMD:C_1206_3216Metric, F.Cu at (175.8, 346.7)
- added R800: 1k, Resistor_SMD:R_1206_3216Metric, F.Cu at (107.2, 331.6)
- added R806: 4.7k, Resistor_SMD:R_1206_3216Metric, F.Cu at (181.0, 326.5)
- added R807: 4.7k, Resistor_SMD:R_1206_3216Metric, F.Cu at (181.0, 332.5)
- added R904: 47, Resistor_SMD:R_1206_3216Metric, F.Cu at (107.4, 324.8)
- added R905: 47, Resistor_SMD:R_1206_3216Metric, F.Cu at (161.2, 346.8)
- added RN800A1: 1k, Resistor_SMD:R_1206_3216Metric, F.Cu at (188.1, 346.6)
- added RN800B1: 1k, Resistor_SMD:R_1206_3216Metric, F.Cu at (183.0, 346.8)
- added RN800C1: 1k, Resistor_SMD:R_1206_3216Metric, F.Cu at (204.9, 347.2)
- added RN800D1: 1k, Resistor_SMD:R_1206_3216Metric, F.Cu at (199.6, 346.5)
- added RN800E1: 1k, Resistor_SMD:R_1206_3216Metric, F.Cu at (194.1, 347.0)
- added RN801A1: 4.7k, Resistor_SMD:R_1206_3216Metric, F.Cu at (234.0, 322.1)
- added RN801B1: 4.7k, Resistor_SMD:R_1206_3216Metric, F.Cu at (229.0, 321.8)
- added RN801C1: 4.7k, Resistor_SMD:R_1206_3216Metric, F.Cu at (224.2, 322.2)
- added RN801D1: 4.7k, Resistor_SMD:R_1206_3216Metric, F.Cu at (221.3, 322.2)
- added RN801E1: 4.7k, Resistor_SMD:R_1206_3216Metric, F.Cu at (212.9, 322.0)
- added RN801F1: 4.7k, Resistor_SMD:R_1206_3216Metric, F.Cu at (218.1, 322.2)
- added RN801G1: 4.7k, Resistor_SMD:R_1206_3216Metric, F.Cu at (207.3, 321.9)
- added U302: 74LS32, Package_SO:SOIC-14_3.9x8.7mm_P1.27mm, F.Cu at (281.8, 340.4)
- added U800: BUSTER, Package_DIP:DIP-48_W15.24mm, F.Cu at (114.6, 338.5)
- added U802: 74LS138, Package_SO:SOIC-16_3.9x9.9mm_P1.27mm, F.Cu at (211.4, 331.5)
- added U803: 74LS08, Package_SO:SOIC-14_3.9x8.7mm_P1.27mm, F.Cu at (227.1, 331.7)
- added U804: 74LS148, Package_SO:SOIC-16_3.9x9.9mm_P1.27mm, F.Cu at (242.5, 331.9)
- renumbered VIDIOT to VIDIOT1
Routing:
- added copper zone on F.Cu, net _CIPL0

Commit message: Add files via upload
Parts:
- removed the REF** at (118.1, 262.9)
- removed the REF** at (118.1, 190.5)
- removed the REF** at (242.6, 262.9)
- removed the REF** at (242.6, 190.5)
- added BT800: Battery_Cell, Battery:BatteryHolder_ComfortableElectronic_CH273-2450_1x2450, F.Cu at (432.9, 327.1)
- added C811: 2.2uF, Capacitor_SMD:C_1206_3216Metric, F.Cu at (464.3, 331.4)
- added C812: 0.1uF, Capacitor_SMD:C_1206_3216Metric, F.Cu at (477.2, 314.5)
- added CN700: Bus_ISA_8bit, AmigaFootprints:ISA_2x31_P2.54mm_Horizontal, F.Cu at (110.3, 40.6)
- added CN701: Bus_ISA_8bit, AmigaFootprints:ISA_2x31_P2.54mm_Horizontal, F.Cu at (130.7, 40.6)
- added CN702: Bus_ISA_8bit, AmigaFootprints:ISA_2x31_P2.54mm_Horizontal, F.Cu at (151.0, 40.5)
- added CN704: Bus_ISA_16bit, Connector_Samtec_HLE_THT:Samtec_HLE-118-02-xx-DV-TE_2x18_P2.54mm_Horizontal, F.Cu at (108.0, 126.9)
- added CN705: Bus_ISA_16bit, Connector_Samtec_HLE_THT:Samtec_HLE-118-02-xx-DV-TE_2x18_P2.54mm_Horizontal, F.Cu at (127.4, 127.0)
- added CN706: Bus_ISA_16bit, Connector_Samtec_HLE_THT:Samtec_HLE-118-02-xx-DV-TE_2x18_P2.54mm_Horizontal, F.Cu at (148.5, 127.0)
- added D800: BAT54CT, Package_TO_SOT_SMD:SOT-23, F.Cu at (463.7, 338.6)
- added R801: 220, Resistor_SMD:R_1206_3216Metric, F.Cu at (464.3, 334.7)
- added R803: 220, Resistor_SMD:R_1206_3216Metric, F.Cu at (477.2, 317.7)
- added R804: 10k, Resistor_SMD:R_1206_3216Metric, F.Cu at (469.9, 331.4)
- added R804A1: 10k, Resistor_SMD:R_1206_3216Metric, F.Cu at (477.2, 321.0)
- added REF**: MountingHole_4.3mm_M4_Pad, MountingHole:MountingHole_4.3mm_M4_Pad, F.Cu at (118.2, 262.9)
- added REF**: MountingHole_4.3mm_M4_Pad, MountingHole:MountingHole_4.3mm_M4_Pad, F.Cu at (118.2, 190.5)
- added REF**: MountingHole_4.3mm_M4_Pad, MountingHole:MountingHole_4.3mm_M4_Pad, F.Cu at (242.6, 262.9)
- added REF**: MountingHole_4.3mm_M4_Pad, MountingHole:MountingHole_4.3mm_M4_Pad, F.Cu at (242.6, 190.5)
- added U801: RTC62423, Package_SO:SOIC-24W_7.5x15.4mm_P1.27mm, F.Cu at (467.9, 321.3)
- UP1: footprint Package_SO:SOIC-14_3.9x8.7mm_P1.27mm -> Package_SO:SOIC-20W_7.5x12.8mm_P1.27mm
- moved G*** 382.2 mm to (528.4, 77.8), turned to 90 degrees
- moved C920 282.8 mm to (196.5, 64.7), turned to 180 degrees
- moved R905 280.3 mm to (195.4, 68.6), turned to 180 degrees
- moved U800 257.4 mm to (178.7, 89.2), turned to 0 degrees
- moved R601I1 256.8 mm to (369.4, 282.6)
- moved R602D1 256.4 mm to (368.3, 288.2)
- moved C800 250.8 mm to (186.0, 82.1)
- moved R904 249.4 mm to (199.8, 93.1)
- moved C630 243.3 mm to (374.6, 288.2)
- moved C626 242.5 mm to (374.4, 282.5)
- moved RN800A1 230.4 mm to (186.1, 116.1), turned to 180 degrees
- moved RN800B1 228.2 mm to (186.1, 118.7), turned to 180 degrees
- moved RN800C1 226.8 mm to (186.1, 121.2), turned to 180 degrees
- moved RN800D1 223.1 mm to (186.1, 123.7), turned to 180 degrees
- moved RN800E1 220.8 mm to (186.0, 126.3), turned to 180 degrees
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Routing:
- net GND: track 2036.3 -> 1576.5 mm, vias 11 -> 9
- net DOE: track 84.5 -> 387.2 mm
- net _GBG: track 84.5 -> 371.6 mm, vias 0 -> 2
- net _EBG3: track 0.00 -> 273.1 mm
- net _EBG2: track 0.00 -> 260.6 mm
- net _EBG1: track 0.00 -> 244.7 mm
- net _EBR5: track 0.00 -> 242.9 mm, vias 0 -> 2
- net _EBR1: track 0.00 -> 229.8 mm, vias 0 -> 1
- net _EBR2: track 0.00 -> 207.4 mm, vias 0 -> 1
- net _EBR3: track 0.00 -> 204.2 mm, vias 0 -> 1
- net _EBR4: track 0.00 -> 185.2 mm, vias 0 -> 1
- net _EBG4: track 0.00 -> 182.7 mm, vias 0 -> 2
- net _EBG5: track 0.00 -> 182.1 mm, vias 0 -> 2
- net BA23: track 115.4 -> 281.3 mm, vias 0 -> 2
- net BA22: track 118.4 -> 278.5 mm, vias 0 -> 2
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Other:
- board text added: "ISA SUBSYSTEM"
