File: 2000EATX-KiCAD/2000ATX.kicad_pcb (KiCad board)
At the start: 2 copper layers, 304.8 x 330.2 mm, 364 parts, among them CN201 Amiga-2000-Video-Slot, CN202 DB15_Female_HighDensity, CN203 Amiga-2000-Video-Slot, CN400 ATX-24, CN600 Amiga-2000-CPU-Slot, CN601 Amiga-2000-Zorro-Slot, CN602 Amiga-2000-Zorro-Slot, CN603 Amiga-2000-Zorro-Slot, CN604 Amiga-2000-Zorro-Slot, CN605 Amiga-2000-Zorro-Slot, CN700 Bus_ISA_8bit, CN701 Bus_ISA_8bit, CN702 Bus_ISA_8bit, CN704 Bus_ISA_16bit, CN705 Bus_ISA_16bit, CN706 Bus_ISA_16bit, J9000 POWER_SWITCH, Q1V1 MMBT3904, Q2V1 MMBT3904, Q3V1 MMBT3904, U1 74LS08, U100 68000D, U103 74LS245, U104 74LS373, U105 74LS245, U106 74LS373, U201 Denise, U205 74HCT244, U206 74HCT244, U302 74LS32, U303 74LS08, U600 74LS245, U601 74LS245, U602 74LS245, U603 74LS245, U604 74LS245, U605 74LS245, U606 74LS32, U800 BUSTER, U801 RTC62423, U802 74LS138, U803 74LS08, U804 74LS148, U9000 MC7905, U9001 74HC14, U9002 74HC74

Commit message: Add files via upload
Parts:
- added C101: 0.1uF, Capacitor_SMD:C_1206_3216Metric, F.Cu at (329.9, 174.1)
- added C102: 0.1uF, Capacitor_SMD:C_1206_3216Metric, F.Cu at (381.7, 116.6)
- added C107: 0.1uF, Capacitor_SMD:C_1206_3216Metric, F.Cu at (381.2, 201.3)
- added C110: 0.1uF, Capacitor_SMD:C_1206_3216Metric, F.Cu at (287.7, 185.4)
- added C415: 4.7uF, Capacitor_SMD:CP_Elec_6.3x5.8, F.Cu at (266.8, 185.7)
- added C905: 100pF, Capacitor_SMD:C_1206_3216Metric, F.Cu at (388.3, 219.0)
- added C907: 100pF, Capacitor_SMD:C_1206_3216Metric, F.Cu at (386.8, 198.0)
- added C908: 47pF, Capacitor_SMD:C_1206_3216Metric, F.Cu at (388.3, 215.7)
- added C918: 0.1uF, Capacitor_SMD:C_1206_3216Metric, F.Cu at (393.9, 212.4)
- added FB101: Ferrite_Bead, Capacitor_SMD:C_1206_3216Metric, F.Cu at (297.4, 189.6)
- added FB102: Ferrite_Bead, Capacitor_SMD:C_1206_3216Metric, F.Cu at (381.2, 198.0)
- added J102: Short for NTSC/Open for PAL, Jumper:SolderJumper-2_P1.3mm_Bridged_RoundedPad1.0x1.5mm, F.Cu at (272.8, 190.8)
- added J900: Enable Chip RAM slowdown during DMA, Jumper:SolderJumper-2_P1.3mm_Bridged_RoundedPad1.0x1.5mm, F.Cu at (397.5, 236.8)
- added Q1V1: MMBT3904, Package_TO_SOT_SMD:SOT-23, F.Cu at (280.9, 1.11)
- added R101: 4.7k, Resistor_SMD:R_1206_3216Metric, F.Cu at (399.7, 201.1)
- added R105: 22, Resistor_SMD:R_1206_3216Metric, F.Cu at (370.7, 216.4)
- added R106: 22, Resistor_SMD:R_1206_3216Metric, F.Cu at (351.3, 267.9)
- added R109: 4.7k, Resistor_SMD:R_1206_3216Metric, F.Cu at (296.8, 182.1)
- added R110: 330, Resistor_SMD:R_1206_3216Metric, F.Cu at (296.8, 185.0)
- added R114: 330, Resistor_SMD:R_1206_3216Metric, F.Cu at (399.8, 207.7)
- added R115: 330, Resistor_SMD:R_1206_3216Metric, F.Cu at (370.7, 219.6)
- added R916: 4.7k, Resistor_SMD:R_1206_3216Metric, F.Cu at (379.2, 206.1)
- added RN102A1: 47, Resistor_SMD:R_1206_3216Metric, F.Cu at (376.3, 216.4)
- added RN102B1: 47, Resistor_SMD:R_1206_3216Metric, F.Cu at (393.9, 219.0)
- added RN102C1: 47, Resistor_SMD:R_1206_3216Metric, F.Cu at (184.2, 58.6)
- added RN102D1: 47, Resistor_SMD:R_1206_3216Metric, F.Cu at (391.1, 222.2)
- added RN902A1: 47, Resistor_SMD:R_1206_3216Metric, F.Cu at (381.2, 225.0)
- added RN902B1: 47, Resistor_SMD:R_1206_3216Metric, F.Cu at (399.8, 204.4)
- added RN902C1: 47, Resistor_SMD:R_1206_3216Metric, F.Cu at (398.1, 233.4)
- added RN907A1: 47, Resistor_SMD:R_1206_3216Metric, F.Cu at (393.9, 215.7)
- added RN907B1: 47, Resistor_SMD:R_1206_3216Metric, F.Cu at (386.8, 201.3)
- added RN907C1: 47, Resistor_SMD:R_1206_3216Metric, F.Cu at (379.2, 209.4)
- added U101: FATTERAGNUS, Package_LCC:PLCC-84_THT-Socket, F.Cu at (335.2, 196.6)
- added U102: Gary, Package_DIP:DIP-48_W15.24mm, F.Cu at (420.0, 180.6)
- added U107: 74LS04, Package_SO:SOIC-14_3.9x8.7mm_P1.27mm, F.Cu at (372.1, 209.6)
- added U900: 7400, Package_SO:SOIC-14_3.9x8.7mm_P1.27mm, F.Cu at (392.2, 165.6)
- added X1: 28.63636MHz, Oscillator:Oscillator_DIP-14, F.Cu at (295.2, 198.7)
- moved C214 267.9 mm to (232.6, 48.9)
- moved C226 251.4 mm to (232.7, 59.7)
- moved RN201C1 232.1 mm to (224.8, 74.0)
- moved RN201A1 197.1 mm to (224.8, 70.4)
- moved RN201B1 196.4 mm to (225.6, 72.2)
- moved RN201D1 190.2 mm to (225.0, 76.1), turned to 180 degrees
- moved R203A1 131.0 mm to (288.3, 39.8)
- moved RN906D1 129.1 mm to (314.4, 124.0)
- moved RN906C1 128.2 mm to (314.4, 125.7)
- moved R203B1 127.0 mm to (288.4, 44.2)
- moved RN904C1 126.7 mm to (344.2, 120.2)
- moved R215 115.3 mm to (302.9, 80.0)
- moved RN905D1 114.5 mm to (314.1, 118.7)
- moved RN906A1 109.5 mm to (313.6, 116.4)
- moved RN905C1 107.1 mm to (314.1, 107.4)
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Connections:
- R20V1 pad 1: Net-(Q1V1-Pad1) -> Net-(R20V1-Pad1)
- U302 pad 10: (no net) -> GND
- U302 pad 8: (no net) -> Net-(RN907B1-Pad2)
- U302 pad 9: (no net) -> Net-(RN907A1-Pad2)
Routing:
- net _OVR: track 124.2 -> 234.4 mm
- net A18: track 39.6 -> 147.5 mm, vias 0 -> 1
- net _BUDS: track 198.7 -> 305.5 mm, vias 0 -> 1
- net _BLDS: track 197.0 -> 303.5 mm, vias 0 -> 1
- net A16: track 37.0 -> 139.1 mm
- net _BAS: track 200.5 -> 302.3 mm, vias 0 -> 1
- net A19: track 42.6 -> 144.1 mm, vias 0 -> 2
- net READ: track 195.1 -> 296.3 mm, vias 0 -> 1
- net A17: track 37.7 -> 137.2 mm, vias 0 -> 1
- net A14: track 44.4 -> 139.2 mm
- net A15: track 46.0 -> 140.1 mm
- net A12: track 40.9 -> 131.0 mm
- net A13: track 43.4 -> 133.0 mm
- net _BG: track 92.1 -> 2.94 mm
- net A10: track 38.5 -> 124.0 mm
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- removed copper zone on F.Cu, net _CIPL0
Other:
- board text added: "ISA/BRIDGEBOARD SUBSYSTEM"
- board text removed: "ISA SUBSYSTEM"

Commit message: Add files via upload
Parts:
- added C200: 0.1uF, Capacitor_SMD:C_1206_3216Metric, F.Cu at (272.2, -75.0)
- added C202: 0.1uF, Capacitor_SMD:C_1206_3216Metric, F.Cu at (207.7, -12.2)
- added C204: 0.1uF, Capacitor_SMD:C_1206_3216Metric, F.Cu at (196.5, -12.5)
- added C210: 0.047uF, Capacitor_SMD:C_1206_3216Metric, F.Cu at (252.5, -63.6)
- added C211: 0.047uF, Capacitor_SMD:C_1206_3216Metric, F.Cu at (209.3, -22.1)
- added C212: 0.047uF, Capacitor_SMD:C_1206_3216Metric, F.Cu at (242.3, -46.8)
- added C213: 0.047uF, Capacitor_SMD:C_1206_3216Metric, F.Cu at (214.9, -22.1)
- added C218: 0.1uF, Capacitor_SMD:C_1206_3216Metric, F.Cu at (190.9, -12.5)
- added C219: 0.22uF, Capacitor_SMD:C_1206_3216Metric, F.Cu at (258.1, -63.6)
- added C220: 0.22uF, Capacitor_SMD:C_1206_3216Metric, F.Cu at (209.3, -15.5)
- added C221: 0.22uF, Capacitor_SMD:C_1206_3216Metric, F.Cu at (261.0, -75.0)
- added C222: 47uF, Capacitor_SMD:CP_Elec_6.3x5.8, F.Cu at (211.7, -44.1)
- added C223: 47uF, Capacitor_SMD:CP_Elec_6.3x5.8, F.Cu at (222.2, -44.1)
- added C224: 4.7uF, Capacitor_SMD:CP_Elec_6.3x5.8, F.Cu at (211.7, -36.0)
- added C225: 470uF, Capacitor_SMD:CP_Elec_6.3x5.8, F.Cu at (244.7, -52.6)
- added C230: 0.1uF, Capacitor_SMD:C_1206_3216Metric, F.Cu at (209.3, -18.8)
- added C231: 6800pF, Capacitor_SMD:C_1206_3216Metric, F.Cu at (261.0, -71.7)
- added C232: 3900pF, Capacitor_SMD:C_1206_3216Metric, F.Cu at (266.6, -75.0)
- added C233: 22uF, Capacitor_SMD:CP_Elec_6.3x5.8, F.Cu at (211.7, -27.8)
- added C234: 0.1uF, Capacitor_SMD:C_1206_3216Metric, F.Cu at (202.1, -12.5)
- added C240: 0.1uF, Capacitor_SMD:C_1206_3216Metric, F.Cu at (263.7, -63.8)
- added C241: 6800pF, Capacitor_SMD:C_1206_3216Metric, F.Cu at (252.5, -60.3)
- added C242: 3900pF, Capacitor_SMD:C_1206_3216Metric, F.Cu at (261.0, -68.5)
- added C243: 22uF, Capacitor_SMD:CP_Elec_6.3x5.8, F.Cu at (222.2, -36.0)
- added C244: 0.1uF, Capacitor_SMD:C_1206_3216Metric, F.Cu at (219.8, -30.3)
- added C900: 0.1uF, Capacitor_SMD:C_1206_3216Metric, F.Cu at (219.8, -27.0)
- added C901: 0.1uF, Capacitor_SMD:C_1206_3216Metric, F.Cu at (252.7, -57.0)
- added CN200: DB9_Male_Stack, AmigaFootprints:DSUB-9_Male_Stack, F.Cu at (312.7, 25.6)
- added CN205: AudioJack, Connector_Audio:Jack_3.5mm_CUI_SJ1-3533NG_Horizontal_CircularHoles, F.Cu at (289.9, 27.4)
- added EMI230: 100pF, AmigaFootprints:C_1206_3216_Feedthrough, F.Cu at (225.4, -29.9)
- added EMI231: 100pF, AmigaFootprints:C_1206_3216_Feedthrough, F.Cu at (266.6, -71.4)
- added EMI232: 100pF, AmigaFootprints:C_1206_3216_Feedthrough, F.Cu at (231.0, -32.0)
- added EMI233: 100pF, AmigaFootprints:C_1206_3216_Feedthrough, F.Cu at (214.9, -18.5)
- added EMI234: 100pF, AmigaFootprints:C_1206_3216_Feedthrough, F.Cu at (238.7, -43.2)
- added EMI235: 100pF, AmigaFootprints:C_1206_3216_Feedthrough, F.Cu at (230.2, -36.0)
- added EMI236: 100pF, AmigaFootprints:C_1206_3216_Feedthrough, F.Cu at (220.5, -23.3)
- added EMI237: 100pF, AmigaFootprints:C_1206_3216_Feedthrough, F.Cu at (247.9, -46.5)
- added EMI238: 100pF, AmigaFootprints:C_1206_3216_Feedthrough, F.Cu at (220.5, -19.4)
- added EMI239: 100pF, AmigaFootprints:C_1206_3216_Feedthrough, F.Cu at (238.7, -39.2)
- added EMI240: 100pF, AmigaFootprints:C_1206_3216_Feedthrough, F.Cu at (214.9, -14.5)
- added EMI241: 100pF, AmigaFootprints:C_1206_3216_Feedthrough, F.Cu at (272.2, -71.4)
- added EMI242: 100pF, AmigaFootprints:C_1206_3216_Feedthrough, F.Cu at (266.6, -67.4)
- added EMI243: 100pF, AmigaFootprints:C_1206_3216_Feedthrough, F.Cu at (231.8, -24.8)
- added F1: 4A, Fuse:Fuse_1206_3216Metric, F.Cu at (258.3, -53.7)
- added FB401: Ferrite_Bead, Capacitor_SMD:C_1206_3216Metric, F.Cu at (258.3, -57.0)
- added Q200: MMBFJ211, Package_TO_SOT_SMD:SOT-23, F.Cu at (247.2, -35.7)
- added Q201: MMBFJ211, Package_TO_SOT_SMD:SOT-23, F.Cu at (231.2, -20.5)
- added Q202: MMBT3906, Package_TO_SOT_SMD:SOT-23, F.Cu at (274.4, -63.9)
- added R202: 10k, Resistor_SMD:R_1206_3216Metric, F.Cu at (277.8, -75.0)
- added R204: 470k, Resistor_SMD:R_1206_3216Metric, F.Cu at (252.7, -50.4)
- added R205: 470k, Resistor_SMD:R_1206_3216Metric, F.Cu at (231.0, -28.4)
- added R206: 10k, Resistor_SMD:R_1206_3216Metric, F.Cu at (226.1, -25.1)
- added R207: 10, Resistor_SMD:R_1206_3216Metric, F.Cu at (277.8, -71.7)
- added R208: 10, Resistor_SMD:R_1206_3216Metric, F.Cu at (226.1, -21.8)
- added R209: 1.2k, Resistor_SMD:R_1206_3216Metric, F.Cu at (258.1, -60.3)
- added R210: 1.2k, Resistor_SMD:R_1206_3216Metric, F.Cu at (263.7, -60.5)
- added R213: 2.7k, Resistor_SMD:R_1206_3216Metric, F.Cu at (236.6, -35.6)
- added R214: 10k, Resistor_SMD:R_1206_3216Metric, F.Cu at (236.6, -32.3)
- added R230: 360, Resistor_SMD:R_1206_3216Metric, F.Cu at (272.2, -67.8)
- added R231: 10k, Resistor_SMD:R_1206_3216Metric, F.Cu at (244.3, -39.6)
- added R232: 10k, Resistor_SMD:R_1206_3216Metric, F.Cu at (220.5, -15.7)
- added R233: 1k, Resistor_SMD:R_1206_3216Metric, F.Cu at (253.5, -47.1)
- added R234: 390, Resistor_SMD:R_1206_3216Metric, F.Cu at (242.2, -35.6)
- added R240: 360, Resistor_SMD:R_1206_3216Metric, F.Cu at (244.3, -42.9)
- added R241: 10k, Resistor_SMD:R_1206_3216Metric, F.Cu at (269.3, -63.8)
- added R242: 10k, Resistor_SMD:R_1206_3216Metric, F.Cu at (263.9, -57.2)
- added R243: 1k, Resistor_SMD:R_1206_3216Metric, F.Cu at (283.4, -75.0)
- added R244: 390, Resistor_SMD:R_1206_3216Metric, F.Cu at (220.5, -12.5)
- added R900: 1k, Resistor_SMD:R_1206_3216Metric, F.Cu at (236.6, -29.0)
- added RN200A1: 4.7k, Resistor_SMD:R_1206_3216Metric, F.Cu at (258.3, -50.4)
- added RN200B1: 4.7k, Resistor_SMD:R_1206_3216Metric, F.Cu at (226.1, -18.5)
- added RN200C1: 4.7k, Resistor_SMD:R_1206_3216Metric, F.Cu at (249.9, -42.9)
- added RN200D1: 4.7k, Resistor_SMD:R_1206_3216Metric, F.Cu at (269.3, -60.5)
- added RN200E1: 4.7k, Resistor_SMD:R_1206_3216Metric, F.Cu at (252.7, -53.7)
- added RN200F1: 4.7k, Resistor_SMD:R_1206_3216Metric, F.Cu at (242.2, -32.3)
- added RN200G1: 4.7k, Resistor_SMD:R_1206_3216Metric, F.Cu at (263.9, -53.9)
- added RN200G2: 4.7k, Resistor_SMD:R_1206_3216Metric, F.Cu at (249.9, -39.6)
- added RN204A1: 68, Resistor_SMD:R_1206_3216Metric, F.Cu at (259.1, -47.1)
- added RN204B1: 68, Resistor_SMD:R_1206_3216Metric, F.Cu at (226.1, -15.3)
- added RN204C1: 68, Resistor_SMD:R_1206_3216Metric, F.Cu at (283.4, -71.7)
- added RN204D1: 68, Resistor_SMD:R_1206_3216Metric, F.Cu at (277.8, -68.5)
- added U200: PAULA, Package_DIP:DIP-48_W15.24mm, F.Cu at (371.1, 119.3)
- added U202: 74LS157, Package_SO:SOIC-16_3.9x9.9mm_P1.27mm, F.Cu at (253.9, -71.0)
- added U204: LF347, Package_SO:SOIC-14_3.9x8.7mm_P1.27mm, F.Cu at (231.6, -43.1)
- U102: value Gary -> GARY
- U201: value Denise -> DENISE
- moved R101 155.8 mm to (539.6, 269.5)
- moved C905 155.8 mm to (528.3, 287.4)
- moved C907 155.8 mm to (526.7, 266.5)
- moved FB102 155.8 mm to (521.1, 266.5)
- moved RN102B1 155.8 mm to (533.9, 287.4)
- moved RN907C1 155.8 mm to (519.1, 277.9)
- moved C107 155.8 mm to (521.1, 269.8)
- moved C908 155.8 mm to (528.3, 284.1)
- moved C918 155.8 mm to (533.9, 280.9)
- moved R105 155.8 mm to (510.7, 284.8)
- moved R115 155.8 mm to (510.7, 288.1)
- moved R916 155.8 mm to (519.1, 274.6)
- moved RN902A1 155.8 mm to (521.1, 293.5)
- moved RN907A1 155.8 mm to (533.9, 284.1)
- moved RN907B1 155.8 mm to (526.7, 269.8)
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- renumbered CN700 to CN1, CN704 to CN2, CN701 to CN3, CN705 to CN4, CN706 to CN5, CN702 to CN6
Connections:
- net _LPEN renamed _FIR1
- C1V1 pad 1: +VID -> Net-(C1V1-Pad1)
- C2V1 pad 1: +VID -> Net-(C2V1-Pad1)
- C3V1 pad 1: +VID -> Net-(C3V1-Pad1)
- C600 pad 1: +5V -> Net-(C600-Pad1)
- C601 pad 1: +5V -> Net-(C601-Pad1)
- C602 pad 1: +5V -> Net-(C602-Pad1)
- C603 pad 1: +5V -> Net-(C603-Pad1)
- C604 pad 1: +5V -> Net-(C604-Pad1)
- C9002 pad 2: GND -> Net-(C9002-Pad2)
- C9003 pad 2: GND -> Net-(C9002-Pad2)
- J9000 pad 2: GND -> Net-(C9002-Pad2)
- Q1V1 pad 3: +VID -> Net-(C1V1-Pad1)
- Q2V1 pad 3: +VID -> Net-(C2V1-Pad1)
- Q3V1 pad 3: +VID -> Net-(C3V1-Pad1)
- R13V1 pad 2: +VID -> Net-(C1V1-Pad1)
- R15V1 pad 2: +VID -> Net-(C2V1-Pad1)
- R17V1 pad 2: +VID -> Net-(C3V1-Pad1)
- U600 pad 20: +5V -> Net-(C600-Pad1)
- U601 pad 20: +5V -> Net-(C601-Pad1)
- U602 pad 20: +5V -> Net-(C602-Pad1)
- U603 pad 20: +5V -> Net-(C603-Pad1)
- U604 pad 20: +5V -> Net-(C604-Pad1)
- U9001 pad 7: GND -> Net-(C9002-Pad2)
- U9002 pad 7: GND -> Net-(C9002-Pad2)

Commit message: Add files via upload
Parts:
- removed JPP1: JP1, Connector_PinHeader_2.54mm:PinHeader_1x03_P2.54mm_Vertical
- removed JPP2: Push Button, Connector_PinHeader_2.54mm:PinHeader_1x02_P2.54mm_Vertical
- removed JPP3: Raspberry_Pi_0, Connector_PinSocket_2.54mm:PinSocket_2x20_P2.54mm_Vertical
- removed RP1: 3k3, Resistor_SMD:R_1206_3216Metric
- removed UP1: 74AHC86N, Package_SO:SOIC-20W_7.5x12.8mm_P1.27mm
- removed UP2, UP3: 74LVC574A, Package_SO:SOIC-20W_7.5x12.8mm_P1.27mm
- added ATX-RESET1: ATX RESET, Connector_PinHeader_2.54mm:PinHeader_1x02_P2.54mm_Vertical, F.Cu at (408.1, -38.7)
- added C301: 0.1uF, Capacitor_SMD:C_1206_3216Metric, F.Cu at (471.8, -76.6)
- added C304: 100pF, Capacitor_SMD:C_1206_3216Metric, F.Cu at (290.7, 61.7)
- added C305: 0.1uF, Capacitor_SMD:C_1206_3216Metric, F.Cu at (401.6, -62.8)
- added C306: 100pF, Capacitor_SMD:C_1206_3216Metric, F.Cu at (355.0, 66.4)
- added C310: 1000pF, Capacitor_SMD:C_1206_3216Metric, F.Cu at (311.1, 69.3)
- added C311: 1000pF, Capacitor_SMD:C_1206_3216Metric, F.Cu at (311.1, 66.9)
- added C312: 1000pF, Capacitor_SMD:C_1206_3216Metric, F.Cu at (296.1, 83.1)
- added C313: 1000pF, Capacitor_SMD:C_1206_3216Metric, F.Cu at (296.1, 80.7)
- added C314: 1000pF, Capacitor_SMD:C_1206_3216Metric, F.Cu at (355.0, 68.8)
- added C315: 1000pF, Capacitor_SMD:C_1206_3216Metric, F.Cu at (355.0, 71.2)
- added C316: 1000pF, Capacitor_SMD:C_1206_3216Metric, F.Cu at (348.2, 83.0)
- added C317: 22uF, Capacitor_SMD:CP_Elec_6.3x5.8, F.Cu at (349.1, 50.6)
- added C318: 22uF, Capacitor_SMD:CP_Elec_6.3x5.8, F.Cu at (301.0, 50.7)
- added C805: 0.1uF, Capacitor_SMD:C_1206_3216Metric, F.Cu at (424.0, -75.1)
- added C813: 22uF, Capacitor_SMD:CP_Elec_6.3x5.8, F.Cu at (509.3, -98.9)
- added C814: 22uF, Capacitor_SMD:CP_Elec_6.3x5.8, F.Cu at (498.6, -94.4)
- added C815: 0.1uF, Capacitor_SMD:C_1206_3216Metric, F.Cu at (500.4, -104.7)
- added C919: 0.1uF, Capacitor_SMD:C_1206_3216Metric, F.Cu at (429.7, -75.1)
- added CN305: DB25_Stack_FemaleAndMale, AmigaFootprints:DSUB-25_Stack_Female_Bottom_Male_Top, F.Cu at (326.0, 25.5)
- added CN306: POWER LED, Connector_PinHeader_2.54mm:PinHeader_1x03_P2.54mm_Vertical, F.Cu at (354.7, -36.2)
- added D300: 1N4148, Diode_SMD:D_SOD-323, F.Cu at (484.4, -94.6)
- added D802: 1N4148, Diode_SMD:D_SOD-323, F.Cu at (501.5, -111.3)
- added EMI300: C_Feedthrough, AmigaFootprints:C_1206_3216_Feedthrough, F.Cu at (313.3, 59.9)
- added EMI301: C_Feedthrough, AmigaFootprints:C_1206_3216_Feedthrough, F.Cu at (303.2, 60.0)
- added EMI302: C_Feedthrough, AmigaFootprints:C_1206_3216_Feedthrough, F.Cu at (309.9, 59.9)
- added EMI303: C_Feedthrough, AmigaFootprints:C_1206_3216_Feedthrough, F.Cu at (316.7, 59.9)
- added EMI304: C_Feedthrough, AmigaFootprints:C_1206_3216_Feedthrough, F.Cu at (320.1, 59.9)
- added EMI305: C_Feedthrough, AmigaFootprints:C_1206_3216_Feedthrough, F.Cu at (323.5, 59.9)
- added EMI306: C_Feedthrough, AmigaFootprints:C_1206_3216_Feedthrough, F.Cu at (326.9, 59.9)
- added EMI307: C_Feedthrough, AmigaFootprints:C_1206_3216_Feedthrough, F.Cu at (330.4, 60.0)
- added EMI308: C_Feedthrough, AmigaFootprints:C_1206_3216_Feedthrough, F.Cu at (333.8, 60.0)
- added EMI309: C_Feedthrough, AmigaFootprints:C_1206_3216_Feedthrough, F.Cu at (337.1, 60.0)
- added EMI310: C_Feedthrough, AmigaFootprints:C_1206_3216_Feedthrough, F.Cu at (306.5, 59.9)
- added EMI325: 100pF, AmigaFootprints:C_1206_3216_Feedthrough, F.Cu at (319.7, 49.3)
- added EMI326: 100pF, AmigaFootprints:C_1206_3216_Feedthrough, F.Cu at (340.2, 49.3)
- added EMI327: 100pF, AmigaFootprints:C_1206_3216_Feedthrough, F.Cu at (333.3, 49.4)
- added EMI328: 100pF, AmigaFootprints:C_1206_3216_Feedthrough, F.Cu at (336.8, 49.3)
- added EMI329: 100pF, AmigaFootprints:C_1206_3216_Feedthrough, F.Cu at (329.9, 49.4)
- added EMI330: 100pF, AmigaFootprints:C_1206_3216_Feedthrough, F.Cu at (326.5, 49.4)
- added EMI331: 100pF, AmigaFootprints:C_1206_3216_Feedthrough, F.Cu at (323.1, 49.4)
- added EMI332: 100pF, AmigaFootprints:C_1206_3216_Feedthrough, F.Cu at (316.3, 49.4)
- added EMI333: 100pF, AmigaFootprints:C_1206_3216_Feedthrough, F.Cu at (309.5, 49.4)
- added EMI334: 100pF, AmigaFootprints:C_1206_3216_Feedthrough, F.Cu at (312.9, 49.4)
- added EMI335: C_Feedthrough, AmigaFootprints:C_1206_3216_Feedthrough, F.Cu at (340.5, 60.0)
- added EMI336: C_Feedthrough, AmigaFootprints:C_1206_3216_Feedthrough, F.Cu at (344.0, 60.0)
- added EMI337: C_Feedthrough, AmigaFootprints:C_1206_3216_Feedthrough, F.Cu at (347.4, 60.0)
- added EMI338: C_Feedthrough, AmigaFootprints:C_1206_3216_Feedthrough, F.Cu at (350.8, 60.0)
- added F2: 4A, Fuse:Fuse_1206_3216Metric, F.Cu at (334.6, 67.0)
- added Q300: MMBT3904, Package_TO_SOT_SMD:SOT-23, F.Cu at (445.7, -81.3)
- added Q302: MMBT3906, Package_TO_SOT_SMD:SOT-23, F.Cu at (445.7, -85.9)
- added R302: 1k, Resistor_SMD:R_1206_3216Metric, F.Cu at (289.5, 56.2)
- added R305: 10k, Resistor_SMD:R_1206_3216Metric, F.Cu at (457.9, -101.4)
- added R306: 10k, Resistor_SMD:R_1206_3216Metric, F.Cu at (418.4, -64.6)
- added R307: 68, Resistor_SMD:R_1206_3216Metric, F.Cu at (435.3, -72.3)
- added R308: 200, Resistor_SMD:R_1206_3216Metric, F.Cu at (452.4, -70.0)
- added R802: 1k, Resistor_SMD:R_1206_3216Metric, F.Cu at (475.2, -107.2)
- added R802A1: 1k, Resistor_SMD:R_1206_3216Metric, F.Cu at (429.7, -64.5)
- added R802B1: 1k, Resistor_SMD:R_1206_3216Metric, F.Cu at (435.3, -69.0)
- added R802C1: 1k, Resistor_SMD:R_1206_3216Metric, F.Cu at (469.6, -103.2)
- added R802D1: 1k, Resistor_SMD:R_1206_3216Metric, F.Cu at (453.4, -107.6)
- added R802E1: 1k, Resistor_SMD:R_1206_3216Metric, F.Cu at (443.4, -64.4)
- added R805: 1k, Resistor_SMD:R_1206_3216Metric, F.Cu at (424.0, -60.5)
- added R902: 4.7k, Resistor_SMD:R_1206_3216Metric, F.Cu at (440.9, -76.3)
- added RRESET1: 1k, Resistor_SMD:R_1206_3216Metric, F.Cu at (417.0, -35.5)
- added U301: U8520, Package_DIP:DIP-40_W15.24mm, F.Cu at (463.0, -85.0)
- added U304: SN75188DR, Package_SO:SOIC-14_3.9x8.7mm_P1.27mm, F.Cu at (343.0, 69.4)
- added U305: SN75189DR, Package_SO:SOIC-14_3.9x8.7mm_P1.27mm, F.Cu at (323.0, 69.3)
- added U805: LM339, Package_SO:SOIC-14_3.9x8.7mm_P1.27mm, F.Cu at (491.0, -104.9)
- U200: value PAULA -> Paula
- U201: value DENISE -> Denise
- moved R202 164.0 mm to (360.9, 66.3), turned to 270 degrees
- moved R230 68.5 mm to (329.2, -105.7), turned to 180 degrees
- moved CN205 67.8 mm to (357.6, 28.6)
- moved CN200 65.9 mm to (378.6, 25.5)
- moved EMI229 43.2 mm to (378.7, 50.9)
Connections:
- U302 pad 4: (no net) -> _VMA
- U302 pad 5: (no net) -> A13
- U302 pad 6: (no net) -> Net-(U301-Pad23)
- U303 pad 4: (no net) -> +5V
- U303 pad 5: (no net) -> _LED
- U303 pad 6: (no net) -> Net-(R902-Pad2)
Routing:
- net GND: track 1625.1 -> 1754.6 mm
- net Net-(C313-Pad1): track 0.00 -> 40.1 mm, vias 0 -> 2
- net /Serial/CTS: track 0.00 -> 34.5 mm, vias 0 -> 2
- net Net-(C311-Pad1): track 0.00 -> 32.2 mm, vias 0 -> 2
- net /Serial/AO: track 0.00 -> 31.7 mm
- net Net-(EMI332-Pad2): track 0.00 -> 30.0 mm, vias 0 -> 2
- net Net-(C312-Pad1): track 0.00 -> 29.2 mm, vias 0 -> 2
- net Net-(CN305-Pad16): track 0.00 -> 27.5 mm, vias 0 -> 1
- net Net-(C310-Pad1): track 0.00 -> 27.0 mm, vias 0 -> 2
- net /Serial/DSR: track 0.00 -> 27.0 mm, vias 0 -> 2
- net Net-(CN305-Pad14): track 0.00 -> 26.7 mm, vias 0 -> 1
- net /Serial/CD: track 0.00 -> 26.1 mm, vias 0 -> 2
- net Net-(CN305-Pad13): track 0.00 -> 25.5 mm, vias 0 -> 1
- net Net-(CN305-Pad12): track 0.00 -> 25.3 mm, vias 0 -> 1
- net Net-(CN305-Pad11): track 0.00 -> 25.0 mm, vias 0 -> 1
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