File: 2000EATX-KiCAD/power.sch (KiCad schematic (older format))
At the start: 32 parts, among them CN400 ATX-24, J9000 POWER_SWITCH, U9000 MC7905, U9001 74HC14, U9002 74HC74

Commit message: Add files via upload
Connections:
- wire segments 129 -> 128
Changed lines of the file:
@@
 $Descr A4 11693 8268
 encoding utf-8
-Sheet 5 9
+Sheet 5 10
 Title ""
 Date ""
@@
 $EndComp
 $Comp
-L Amiga~3000~library:GND #PWR0165
+L power:GND #PWR0165
 U 1 1 60A5B857
 P 4150 3900
@@
 $EndComp
 $Comp
-L Amiga~3000~library:GND #PWR0166
+L power:GND #PWR0166
 U 1 1 60A630E8
 P 1600 2200
@@
 	2450 2000 2450 2100
 $Comp
-L Amiga~3000~library:-12V #PWR0167
+L power:-12V #PWR0167
 U 1 1 60A6467A
 P 8550 950
@@
 $EndComp
 $Comp
-L Amiga~3000~library:-5V #PWR0168
+L power:-5V #PWR0168
 U 1 1 60A64F47
 P 8800 950
@@
 $EndComp
 $Comp
-L Amiga~3000~library:GND #PWR0169
+L power:GND #PWR0169
 U 1 1 60A6AF77
 P 2150 6800
@@
 	6650 6300 6650 6800
 Connection ~ 3250 6800
-Wire Wire Line
-	2150 6800 2300 6800
 Connection ~ 2300 6800
 Wire Wire Line
 	2300 6800 3250 6800
 Wire Wire Line
-	2150 6800 1100 6800
-Wire Wire Line
 	1100 6800 1100 6250
-Connection ~ 2150 6800
 Connection ~ 3250 5100
 Wire Wire Line
@@
 	3400 1400 3750 1400
 $Comp
-L Amiga~3000~library:GND #PWR0170
+L power:GND #PWR0170
 U 1 1 60B02E26
 P 8050 1400
@@
 Connection ~ 3850 1400
 $Comp
-L Amiga~3000~library:+12V #PWR0171
+L power:+12V #PWR0171
 U 1 1 60B0BBA9
 P 8050 950
@@
 	3850 1800 4300 1800
 $Comp
-L Amiga~3000~library:+5V #PWR0172
+L power:+5V #PWR0172
 U 1 1 60B329EC
 P 8300 950
@@
 Wire Wire Line
 	2100 1850 2250 1850
+Wire Wire Line
+	1100 6800 2300 6800
 $EndSCHEMATC

Commit message: Add files via upload
Parts:
- added H1, H10, H11, H12, H2, H3, H4, H5, H6, H7, H8, H9: MountingHole_Pad, MountingHole:MountingHole_4.3mm_M4_Pad, symbol Mechanical:MountingHole_Pad
Connections:
- net GND: now also H1.1, H10.1, H11.1, H12.1, H2.1, H3.1, H4.1, H5.1, H6.1, H7.1, H8.1, H9.1
Other:
- note added: "MOUNTING\nHOLES"
Changed lines of the file:
@@
 Wire Wire Line
 	1100 6800 2300 6800
+$Comp
+L Mechanical:MountingHole_Pad H1
+U 1 1 6079CD83
+P 9100 3500
+F 0 "H1" V 9100 3650 50  0000 L CNN
+F 1 "MountingHole_Pad" V 9145 3650 50  0001 L CNN
+F 2 "MountingHole:MountingHole_4.3mm_M4_Pad" H 9100 3500 50  0001 C CNN
+F 3 "~" H 9100 3500 50  0001 C CNN
+	1    9100 3500
+	0    1    1    0
+$EndComp
+$Comp
+L Mechanical:MountingHole_Pad H4
+U 1 1 607A300A
+P 9100 3700
+F 0 "H4" V 9100 3850 50  0000 L CNN
+F 1 "MountingHole_Pad" V 9145 3850 50  0001 L CNN
+F 2 "MountingHole:MountingHole_4.3mm_M4_Pad" H 9100 3700 50  0001 C CNN
+F 3 "~" H 9100 3700 50  0001 C CNN
+	1    9100 3700
+	0    1    1    0
+$EndComp
+$Comp
+L Mechanical:MountingHole_Pad H7
+U 1 1 607A343C
+P 9100 3900
+F 0 "H7" V 9100 4050 50  0000 L CNN
+F 1 "MountingHole_Pad" V 9145 4050 50  0001 L CNN
+F 2 "MountingHole:MountingHole_4.3mm_M4_Pad" H 9100 3900 50  0001 C CNN
+F 3 "~" H 9100 3900 50  0001 C CNN
+	1    9100 3900
+	0    1    1    0
+$EndComp
+$Comp
+L Mechanical:MountingHole_Pad H10
+U 1 1 607A38D0
+P 9100 4100
+F 0 "H10" V 9100 4250 50  0000 L CNN
+F 1 "MountingHole_Pad" V 9145 4250 50  0001 L CNN
+F 2 "MountingHole:MountingHole_4.3mm_M4_Pad" H 9100 4100 50  0001 C CNN
+F 3 "~" H 9100 4100 50  0001 C CNN
+	1    9100 4100
+	0    1    1    0
+$EndComp
+$Comp
+L Mechanical:MountingHole_Pad H2
+U 1 1 607A449F
+P 9500 3500
+F 0 "H2" V 9500 3650 50  0000 L CNN
+F 1 "MountingHole_Pad" V 9545 3650 50  0001 L CNN
+F 2 "MountingHole:MountingHole_4.3mm_M4_Pad" H 9500 3500 50  0001 C CNN
+F 3 "~" H 9500 3500 50  0001 C CNN
+	1    9500 3500
+	0    1    1    0
+$EndComp
+$Comp
+L Mechanical:MountingHole_Pad H5
+U 1 1 607A48FE
+P 9500 3700
+F 0 "H5" V 9500 3850 50  0000 L CNN
+F 1 "MountingHole_Pad" V 9545 3850 50  0001 L CNN
+F 2 "MountingHole:MountingHole_4.3mm_M4_Pad" H 9500 3700 50  0001 C CNN
+F 3 "~" H 9500 3700 50  0001 C CNN
+	1    9500 3700
+	0    1    1    0
+$EndComp
+$Comp
+L Mechanical:MountingHole_Pad H8
+U 1 1 607A4E77
+P 9500 3900
+F 0 "H8" V 9500 4050 50  0000 L CNN
+F 1 "MountingHole_Pad" V 9545 4050 50  0001 L CNN
+F 2 "MountingHole:MountingHole_4.3mm_M4_Pad" H 9500 3900 50  0001 C CNN
+F 3 "~" H 9500 3900 50  0001 C CNN
+	1    9500 3900
+	0    1    1    0
+$EndComp
+$Comp
+L Mechanical:MountingHole_Pad H11
+U 1 1 607A52EF
+P 9500 4100
+F 0 "H11" V 9500 4250 50  0000 L CNN
+F 1 "MountingHole_Pad" V 9545 4250 50  0001 L CNN
+F 2 "MountingHole:MountingHole_4.3mm_M4_Pad" H 9500 4100 50  0001 C CNN
+F 3 "~" H 9500 4100 50  0001 C CNN
+	1    9500 4100
+	0    1    1    0
+$EndComp
+$Comp
+L Mechanical:MountingHole_Pad H3
+U 1 1 607B44AE
+P 9900 3500
+F 0 "H3" V 9900 3650 50  0000 L CNN
+F 1 "MountingHole_Pad" V 9945 3650 50  0001 L CNN
+F 2 "MountingHole:MountingHole_4.3mm_M4_Pad" H 9900 3500 50  0001 C CNN
+F 3 "~" H 9900 3500 50  0001 C CNN
+	1    9900 3500
+	0    1    1    0
+$EndComp
+$Comp
+L Mechanical:MountingHole_Pad H9
+U 1 1 607B4AE3
+P 9900 3900
+F 0 "H9" V 9900 4050 50  0000 L CNN
+F 1 "MountingHole_Pad" V 9945 4050 50  0001 L CNN
+F 2 "MountingHole:MountingHole_4.3mm_M4_Pad" H 9900 3900 50  0001 C CNN
+F 3 "~" H 9900 3900 50  0001 C CNN
+	1    9900 3900
+	0    1    1    0
+$EndComp
+$Comp
+L Mechanical:MountingHole_Pad H6
+U 1 1 607B5071
+P 9900 3700
+F 0 "H6" V 9900 3850 50  0000 L CNN
+F 1 "MountingHole_Pad" V 9945 3850 50  0001 L CNN
+F 2 "MountingHole:MountingHole_4.3mm_M4_Pad" H 9900 3700 50  0001 C CNN
+F 3 "~" H 9900 3700 50  0001 C CNN
+	1    9900 3700
+	0    1    1    0
+$EndComp
+$Comp
+L Mechanical:MountingHole_Pad H12
+U 1 1 607BA784
+P 9900 4100
+F 0 "H12" V 9900 4250 50  0000 L CNN
+F 1 "MountingHole_Pad" V 9945 4250 50  0001 L CNN
+F 2 "MountingHole:MountingHole_4.3mm_M4_Pad" H 9900 4100 50  0001 C CNN
+F 3 "~" H 9900 4100 50  0001 C CNN
+	1    9900 4100
+	0    1    1    0
+$EndComp
+Wire Wire Line
+	9400 3500 9400 3700
+Wire Wire Line
+	9400 4400 9000 4400
+Wire Wire Line
+	9000 4400 9000 4100
+Connection ~ 9400 3700
+Wire Wire Line
+	9400 3700 9400 3900
+Connection ~ 9400 3900
+Wire Wire Line
+	9400 3900 9400 4100
+Connection ~ 9400 4100
+Wire Wire Line
+	9400 4100 9400 4400
+Connection ~ 9000 3700
+Wire Wire Line
+	9000 3700 9000 3500
+Connection ~ 9000 3900
+Wire Wire Line
+	9000 3900 9000 3700
+Connection ~ 9000 4100
+Wire Wire Line
+	9000 4100 9000 3900
+Wire Wire Line
+	9800 3500 9800 3700
+Wire Wire Line
+	9800 4400 9400 4400
+Connection ~ 9800 3700
+Wire Wire Line
+	9800 3700 9800 3900
+Connection ~ 9800 3900
+Wire Wire Line
+	9800 3900 9800 4100
+Connection ~ 9800 4100
+Wire Wire Line
+	9800 4100 9800 4400
+Connection ~ 9400 4400
+$Comp
+L power:GND #PWR0357
+U 1 1 607C700A
+P 9400 4400
+F 0 "#PWR0357" H 9400 4150 50  0001 C CNN
+F 1 "GND" H 9405 4227 50  0000 C CNN
+F 2 "" H 9400 4400 50  0001 C CNN
+F 3 "" H 9400 4400 50  0001 C CNN
+	1    9400 4400
+	1    0    0    -1
+$EndComp
+Wire Notes Line
+	8800 2800 8800 4700
+Wire Notes Line
+	8800 4700 10250 4700
+Wire Notes Line
+	10250 4700 10250 2800
+Wire Notes Line
+	10250 2800 8800 2800
+Text Notes 9050 3250 0    118  ~ 0
+MOUNTING\nHOLES
 $EndSCHEMATC

Commit message: Add files via upload
Connections:
- net GND: now also C9002.2, C9003.2, J9000.2 (Pin_2), U9001.7 (GND), U9002.7 (GND)
Changed lines of the file:
@@
 L power:GND #PWR0169
 U 1 1 60A6AF77
-P 2150 6800
-F 0 "#PWR0169" H 2150 6550 50  0001 C CNN
-F 1 "GND" H 2155 6627 50  0000 C CNN
-F 2 "" H 2150 6800 50  0001 C CNN
-F 3 "" H 2150 6800 50  0001 C CNN
-	1    2150 6800
+P 2300 6800
+F 0 "#PWR0169" H 2300 6550 50  0001 C CNN
+F 1 "GND" H 2305 6627 50  0000 C CNN
+F 2 "" H 2300 6800 50  0001 C CNN
+F 3 "" H 2300 6800 50  0001 C CNN
+	1    2300 6800
 	1    0    0    -1
 $EndComp
@@
 Wire Wire Line
 	2100 1850 2250 1850
-Wire Wire Line
-	1100 6800 2300 6800
 $Comp
 L Mechanical:MountingHole_Pad H1
@@
 Text Notes 9050 3250 0    118  ~ 0
 MOUNTING\nHOLES
+$Comp
+L power:GND #PWR0177
+U 1 1 608A0106
+P 1100 6800
+F 0 "#PWR0177" H 1100 6550 50  0001 C CNN
+F 1 "GND" H 1105 6627 50  0000 C CNN
+F 2 "" H 1100 6800 50  0001 C CNN
+F 3 "" H 1100 6800 50  0001 C CNN
+	1    1100 6800
+	1    0    0    -1
+$EndComp
 $EndSCHEMATC
