File: 2000EATX-KiCAD/floppyparallel.sch (KiCad schematic (older format))
At the start: 16 parts, among them CN305 DB25_Stack_FemaleAndMale

Commit message: Add files via upload
Parts:
- added J1: DIN-5_180degree, AmigaFootprints:DIN5, symbol Connector:DIN-5_180degree
- added U2: 8520, Package_DIP:DIP-40_W15.24mm, symbol Amiga-Library:8520
Changed lines of the file:
@@
 $Descr B 17000 11000
 encoding utf-8
-Sheet 12 12
+Sheet 12 13
 Title ""
 Date ""
@@
 Wire Wire Line
 	9350 5350 9350 5550
+$Comp
+L Amiga-Library:8520 U2
+U 1 1 605D485E
+P 2150 3650
+F 0 "U2" H 2125 5875 50  0000 C CNN
+F 1 "8520" H 2125 5784 50  0000 C CNN
+F 2 "Package_DIP:DIP-40_W15.24mm" H 2150 5000 50  0001 C CNN
+F 3 "" H 2150 5000 50  0001 C CNN
+	1    2150 3650
+	1    0    0    -1
+$EndComp
+$Comp
+L Connector:DIN-5_180degree J1
+U 1 1 605D6665
+P 6800 1500
+F 0 "J1" H 6800 1225 50  0000 C CNN
+F 1 "DIN-5_180degree" H 6800 1134 50  0000 C CNN
+F 2 "AmigaFootprints:DIN5" H 6800 1500 50  0001 C CNN
+F 3 "http://www.mouser.com/ds/2/18/40_c091_abd_e-75918.pdf" H 6800 1500 50  0001 C CNN
+F 4 "SDS-50J" H 6800 1500 50  0001 C CNN "Part"
+	1    6800 1500
+	1    0    0    -1
+$EndComp
 $EndSCHEMATC

Commit message: Add files via upload
Parts:
- added C203, C300, C302, C607, C909, C916: 0.1uF, Capacitor_SMD:C_1206_3216Metric, symbol Device:C
- added C259, C260, C261: 100pF, Capacitor_SMD:C_1206_3216Metric, symbol Device:C
- added C912: 470uF, Capacitor_SMD:CP_Elec_6.3x5.8, symbol Device:CP
- added CN303: FLOPPY, Connector_PinHeader_2.54mm:PinHeader_2x17_P2.54mm_Vertical, symbol Connector_Generic:Conn_02x17_Odd_Even
- added FB301, FB302, FB303: Ferrite_Bead, Capacitor_SMD:C_1206_3216Metric, symbol Device:Ferrite_Bead
- added J301: CLOSE FOR DF1, Connector_PinHeader_2.54mm:PinHeader_1x02_P2.54mm_Vertical, symbol Connector:Conn_01x02_Male
- added Q301: MMBT3906, Package_TO_SOT_SMD:SOT-23, symbol Transistor_BJT:2N3904
- added R201, R300, R309: 4.7k, Resistor_SMD:R_1206_3216Metric, symbol Device:R
- added R301, R602: 1k, Resistor_SMD:R_1206_3216Metric, symbol Device:R
- added R310: 47 0.5W, Resistor_SMD:R_1206_3216Metric, symbol Device:R
- added R914: 1 0.5W, Resistor_SMD:R_1206_3216Metric, symbol Device:R
- added RN300: 10k, Resistor_THT:R_Array_SIP10, symbol Device:R_Network09
- added RN301: 1k, Resistor_THT:R_Array_SIP6, symbol Device:R_Network05
- added U102: GARY, Package_DIP:DIP-48_W15.24mm_Socket, symbol Amiga-Library:Gary
- added U108: 74LS74, Package_SO:SOIC-14_3.9x8.7mm_P1.27mm, symbol 74xx:74LS74
- added U203: 74LS38, Package_SO:SOIC-14_3.9x8.7mm_P1.27mm, symbol 74xx:74LS38
- added unit 2 of U300
- added U302: 74LS32, symbol 74xx:74LS32
- added U607: 74LS08, Package_SO:SOIC-14_3.9x8.7mm_P1.27mm, symbol 74xx:74LS08
- added U900: 74LS00, Package_SO:SOIC-14_3.9x8.7mm_P1.27mm, symbol 74xx:74LS00
- CN300: renamed from J1; value DIN-5_180degree -> KEYBOARD
- renumbered U2 to U300
Connections:
- net GND: now also CN300.5, C203.1, C259.2, C260.2, C261.2, C300.1, C302.1, C607.1, C909.2, C912.2, C916.2, CN303.1 (Pin_1), CN303.11 (Pin_11), CN303.13 (Pin_13), CN303.15 (Pin_15), CN303.17 (Pin_17), CN303.19 (Pin_19), CN303.21 (Pin_21), CN303.23 (Pin_23), CN303.25 (Pin_25), CN303.27 (Pin_27), CN303.29 (Pin_29), CN303.31 (Pin_31), CN303.33 (Pin_33), CN303.5 (Pin_5), CN303.7 (Pin_7), CN303.9 (Pin_9), Q301.1 (E), U203.7 (GND), U300.1 (GND1), U302.7 (GND), U607.7 (GND)
- net PPD0: now reaches U300.10 (PB0)
- net PPD0: now also EMI302.1
- net PPD1: now reaches U300.11 (PB1)
- net PPD1: now also EMI303.1
- net PPD2: now reaches U300.12 (PB2)
- net PPD2: now also EMI304.1
- net PPD3: now reaches U300.13 (PB3)
- net PPD3: now also EMI305.1
- net PPD4: now reaches U300.14 (PB4)
- net PPD4: now also EMI306.1
- net PPD5: now reaches U300.15 (PB5)
- net PPD5: now also EMI307.1
- net PPD6: now reaches U300.16 (PB6)
- net PPD6: now also EMI308.1
- net PPD7: now reaches U300.17 (PB7)
- net PPD7: now also EMI309.1
- net PSTROBE: now reaches U300.18 (_PC)
- net PSTROBE: now also EMI301.1, RN300.2 (R1)
- net TBASE: now reaches U300.19 (TICK)
- net OVL: now reaches U300.2 (PA0)
- net _INT2: now reaches U300.21 (_INT)
- net R_W: now reaches U300.22 (_W)
- net at U300.23 (_CS): now also U302.3
- net _PACK: now reaches U300.24 (_F)
- net _PACK: now also EMI335.1, RN300.5 (R4)
- net E: now reaches U300.25 (E)
- net D7: now reaches U300.26 (D7)
- net D7: now also CN305.9, EMI309.2
- net D6: now reaches U300.27 (D6)
- net D6: now also CN305.8, EMI308.2
- net D5: now reaches U300.28 (D5)
- net D5: now also CN305.7, EMI307.2
- net D4: now reaches U300.29 (D4)
- net D4: now also CN305.6, EMI306.2
- net _LED: now reaches U300.3 (PA1)
- net D3: now reaches U300.30 (D3)
- net D3: now also CN305.5, EMI305.2
- net D2: now reaches U300.31 (D2)
- net D2: now also CN305.4, EMI304.2
- net D1: now reaches U300.32 (D1)
- net D1: now also CN305.3, EMI303.2
- net D0: now reaches U300.33 (D0)
- net D0: now also CN305.2, EMI302.2
- net _BRST: now reaches U300.34 (_RESET)
- net _BRST: now also C909.1, R602.2, U108.10 (~S), U607.10, U607.12, U607.3, U607.5
- net A11: now reaches U300.35 (RS3)
- net A10: now reaches U300.36 (RS2)
- net A9: now reaches U300.37 (RS1)
- net A8: now reaches U300.38 (RS0)
- net at U300.39 (S): now also FB303.2, RN300.10 (R9)
- net CHNG: now reaches U300.4 (PA2)
- net CHNG: now also CN303.2 (Pin_2), RN301.2 (R1)
- net _KBCLK: now reaches U300.40 (C)
- net _KBCLK: now also FB302.2, RN300.9 (R8)
- net WPROT: now reaches U300.5 (PA3)
- net WPROT: now also CN303.28 (Pin_28), RN301.4 (R3)
- net TRK0: now reaches U300.6 (PA4)
- net TRK0: now also CN303.26 (Pin_26), RN301.3 (R2)
- net RDY: now reaches U300.7 (PA5)
- net RDY: now also CN303.34 (Pin_34), J301.2 (Pin_2), RN301.5 (R4)
- net _FIR0: now reaches U300.8 (PA6)
- net _FIR1: now reaches U300.9 (PA7)
- net KBDATA: now reaches CN300.2
- net KBDATA: now also C261.1, FB303.1
- net KBCLK: now reaches CN300.3
- net KBCLK: now also C260.1, FB302.1
- net at CN300.4: now also C259.1, C912.1, FB301.1
- net PBUSY: now reaches EMI336.1
- net PBUSY: now also RN300.6 (R5)
- net PPOUT: now reaches EMI337.1
- net PPOUT: now also RN300.7 (R6)
- net POUT: now reaches CN305.12, EMI337.2
- net PSEL: now reaches EMI338.1
- net PSEL: now also RN300.8 (R7)
- net SEL: now reaches CN305.13, EMI338.2
- net _IORST: now reaches EMI300.2
- net _IORST: now also C916.1, U607.8
- net at EMI310.2: now also R310.1
- new net: FB301.2, R914.2
- new net: U102.44 (DKWEB), U203.13
- new net: U102.45 (DKWDB), U203.10
- new net: R309.2, U102.46 (MTRON), U900.2
- new net: U102.47 (MTRX), U203.2
- new net: U108.11 (C), U203.5, U900.6
- new net: J301.1 (Pin_1), U203.6
- new net: Q301.2 (B), R300.1, R309.1
- new net: R300.2, U108.8 (~Q)
- new net +5V: C203.2, C300.2, C302.2, C607.2, R201.1, R301.1, R310.2, R602.1, R914.1, RN300.1 (common), RN301.1 (common), U108.13 (~R), U203.1, U203.12, U203.14 (VCC), U203.9, U300.20 (VCC), U302.14 (VCC), U607.1, U607.13, U607.14 (VCC), U607.4, U607.9, U900.1, U900.4
- new net A12: U302.1
- new net DIR: CN303.18 (Pin_18)
- new net DKWDB: CN303.22 (Pin_22), U203.8
- new net DKWE: U102.8 (DKWE)
- new net DKWEB: CN303.24 (Pin_24), U203.11
- new net INUSE1: CN303.14 (Pin_14), CN303.4 (Pin_4), U108.9 (Q), U203.4
- new net MTROD: CN303.16 (Pin_16), Q301.3 (C)
- new net _BUSRST: U607.11
- new net _DKRD: CN303.30 (Pin_30), R301.2
- new net _DKRST: U607.6
- new net _DKWD: U102.9 (_DKWD)
- new net _INDEX: CN303.8 (Pin_8), RN301.6 (R5)
- new net _INUSE0: CN303.6 (Pin_6), U900.3
- new net _KBRST: R201.2, U102.5 (_KBRST)
- new net _MTR: U102.7 (_MTR), U108.12 (D)
- new net _MTRX: U203.3
- new net _RST: U607.2
- new net _SEL0: CN303.10 (Pin_10), U102.16 (_SEL)
- new net _SEL1: CN303.12 (Pin_12), U900.5
- new net _SIDE: CN303.32 (Pin_32)
- new net _STEP: CN303.20 (Pin_20)
- new net _VMA: U302.2
- no-connect marks 1 -> 7
Other:
- note added: "KEY"
- note added: "NOTE: J300 IS OMITTED IN FAVOR OF\nUSING THE _VSYNC SIGNAL IN PLACE OF TICK."
- moved on the sheet: CN300, CN305A, EMI300, EMI301, EMI302, EMI303, EMI304, EMI305, EMI306, EMI307, EMI308, EMI309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

Commit message: Add files via upload
Parts:
- added C108: 0.1uF, Capacitor_SMD:C_1206_3216Metric, symbol Device:C
- added unit 3 of U108
Connections:
- net +5V: now also C108.2, U108.14 (VCC)
- net GND: now also C108.1, U108.7 (GND)
Changed lines of the file:
@@
 L power:GND #PWR0378
 U 1 1 615EAC3E
-P 9600 10250
-F 0 "#PWR0378" H 9600 10000 50  0001 C CNN
-F 1 "GND" H 9605 10077 50  0000 C CNN
-F 2 "" H 9600 10250 50  0001 C CNN
-F 3 "" H 9600 10250 50  0001 C CNN
-	1    9600 10250
+P 10650 10300
+F 0 "#PWR0378" H 10650 10050 50  0001 C CNN
+F 1 "GND" H 10655 10127 50  0000 C CNN
+F 2 "" H 10650 10300 50  0001 C CNN
+F 3 "" H 10650 10300 50  0001 C CNN
+	1    10650 10300
 	1    0    0    -1
 $EndComp
@@
 Connection ~ 8950 9400
 Wire Wire Line
-	9600 10050 9600 10150
-Wire Wire Line
 	8950 10400 9300 10400
 Wire Wire Line
-	9300 10400 9300 10150
-Wire Wire Line
-	9300 10150 9600 10150
+	9300 10400 9300 10300
 Connection ~ 8950 10400
-Connection ~ 9600 10150
-Wire Wire Line
-	9600 10150 9600 10250
 Wire Wire Line
 	8300 9750 8300 9400
@@
 Wire Wire Line
 	5750 9400 5050 9400
+$Comp
+L 74xx:74LS74 U108
+U 3 1 612EFF3A
+P 10250 9900
+F 0 "U108" H 10250 9850 50  0000 C CNN
+F 1 "74LS74" H 10250 9950 50  0000 C CNN
+F 2 "Package_SO:SOIC-14_3.9x8.7mm_P1.27mm" H 10250 9900 50  0001 C CNN
+F 3 "74xx/74hc_hct74.pdf" H 10250 9900 50  0001 C CNN
+	3    10250 9900
+	1    0    0    -1
+$EndComp
+Wire Wire Line
+	9600 9400 10250 9400
+Wire Wire Line
+	10250 9400 10250 9500
+Connection ~ 9600 9400
+Wire Wire Line
+	10250 10300 9600 10300
+Connection ~ 10250 10300
+Connection ~ 9600 10300
+Wire Wire Line
+	9600 10300 9300 10300
+Wire Wire Line
+	9600 10050 9600 10300
+$Comp
+L Device:C C108
+U 1 1 613B4947
+P 10650 9900
+F 0 "C108" H 10535 9854 50  0000 R CNN
+F 1 "0.1uF" H 10535 9945 50  0000 R CNN
+F 2 "Capacitor_SMD:C_1206_3216Metric" H 10688 9750 50  0001 C CNN
+F 3 "~" H 10650 9900 50  0001 C CNN
+	1    10650 9900
+	-1   0    0    1
+$EndComp
+Wire Wire Line
+	10250 10300 10650 10300
+Wire Wire Line
+	10650 10300 10650 10050
+Connection ~ 10650 10300
+Wire Wire Line
+	10650 9750 10650 9400
+Wire Wire Line
+	10650 9400 10250 9400
+Connection ~ 10250 9400
 $EndSCHEMATC

Commit message: Add files via upload
Other:
- note added: "PARALLEL"
Changed lines of the file:
@@
 	10650 9400 10250 9400
 Connection ~ 10250 9400
+Text Notes 8650 6050 0    79   ~ 0
+PARALLEL
 $EndSCHEMATC

Commit message: Add files via upload
Parts:
- J301: value CLOSE FOR DF1 -> SHORT FOR DF1
Changed lines of the file:
@@
 P 15550 5850
 F 0 "J301" H 15522 5732 50  0000 R CNN
-F 1 "CLOSE FOR DF1" H 15522 5823 50  0000 R CNN
+F 1 "SHORT FOR DF1" H 15522 5823 50  0000 R CNN
 F 2 "Connector_PinHeader_2.54mm:PinHeader_1x02_P2.54mm_Vertical" H 15550 5850 50  0001 C CNN
 F 3 "~" H 15550 5850 50  0001 C CNN

Commit message: Add files via upload
Connections:
- net PSTROBE: now also RN300.9 (R8); no longer RN300.2 (R1)
- net _KBCLK: now also RN300.3 (R2); no longer RN300.9 (R8)
- net at FB303.2, U300.39 (S): now also RN300.4 (R3); no longer RN300.10 (R9)
Changed lines of the file:
@@
 Wire Wire Line
 	3850 5400 3150 5400
-Wire Wire Line
-	4400 1800 4400 2000
 Connection ~ 4400 3100
 Wire Wire Line
-	4400 3100 6450 3100
+	4400 3100 5100 3100
 Text GLabel 1400 1700 0    50   Input ~ 0
 PSTROBE
@@
 Wire Wire Line
 	4300 2000 4400 2000
-Connection ~ 4400 2000
 Wire Wire Line
 	4400 2000 4400 3100
@@
 	6250 1750 6250 2000
 Wire Wire Line
-	3150 2500 5200 2500
-Wire Wire Line
-	6050 2250 5100 2250
+	3150 2500 4600 2500
 Wire Wire Line
 	3450 2250 3450 2050
@@
 	1    0    0    -1
 $EndComp
-NoConn ~ 4500 1800
-NoConn ~ 4600 1800
-Wire Wire Line
-	5100 1800 5100 2250
-Connection ~ 5100 2250
-Wire Wire Line
-	5100 2250 3450 2250
-Wire Wire Line
-	5200 1800 5200 2500
-Connection ~ 5200 2500
-Wire Wire Line
-	5200 2500 6350 2500
 Wire Wire Line
 	2650 9500 2650 10050
@@
 Text Notes 8650 6050 0    79   ~ 0
 PARALLEL
+Wire Wire Line
+	4500 1800 4500 2250
+Connection ~ 4500 2250
+Wire Wire Line
+	4500 2250 3450 2250
+Wire Wire Line
+	4500 2250 6050 2250
+NoConn ~ 5200 1800
+Wire Wire Line
+	4600 1800 4600 2500
+Connection ~ 4600 2500
+Wire Wire Line
+	4600 2500 6350 2500
+NoConn ~ 4400 1800
+Wire Wire Line
+	5100 1800 5100 3100
+Connection ~ 5100 3100
+Wire Wire Line
+	5100 3100 6450 3100
 $EndSCHEMATC

Commit message: Add files via upload
Connections:
- net TBASE renamed _VSYNC
Changed lines of the file:
@@
 Wire Wire Line
 	1850 6000 2300 6000
-Connection ~ 1850 6000
 Wire Wire Line
 	1850 6250 1850 6000
 Wire Wire Line
 	1550 6250 1850 6250
-Wire Wire Line
-	1550 6000 1850 6000
 Text GLabel 1550 6250 0    50   Input ~ 0
 _VSYNC
@@
 Text GLabel 1550 7100 0    50   Output ~ 0
 OVL
-Text GLabel 1550 6000 0    50   Output ~ 0
-TBASE
 $Comp
 L power:+5V #PWR0363
