File: 2000EATX-KiCAD/memory.sch (KiCad schematic (older format))
At the start: 3 parts, among them U500 27C400, U500A1 AT27C4096

Commit message: Add files via upload
Parts:
- removed U500A1: AT27C4096, Package_DIP:DIP-40_W15.24mm, symbol Amiga-Library:AT27C4096
- added C500, C501: 0.1uF, Capacitor_SMD:C_1206_3216Metric, symbol Device:C
- added J500: Conn_01x02_Male, Connector_PinHeader_2.54mm:PinHeader_1x02_P2.54mm_Vertical, symbol Connector:Conn_01x02_Male
- added R500: 4.7k, Resistor_SMD:R_1206_3216Metric, symbol Device:R
- added R5001D, R500A, R500B, R500C, R500D, R500E (x2), R501A, R501B, R501C: 47, Resistor_SMD:R_1206_3216Metric, symbol Device:R
- added R502A, R502B, R502C, R502D: 22, Resistor_SMD:R_1206_3216Metric, symbol Device:R
- added R503A, R503B, R503C, R503D, R503E, R503F, R503G, R503H, R503I: 470, Resistor_SMD:R_1206_3216Metric, symbol Device:R
- added U500: CY62157, Package_SO:TSOP-II-44_10.16x18.41mm_P0.8mm, symbol Amiga-Library:CY62157
- added U501: 74LS00, Package_SO:SOIC-14_3.9x8.7mm_P1.27mm, symbol 74xx:74LS00
- added U502, U503: 74LS574, Package_SO:SOIC-20W_7.5x12.8mm_P1.27mm, symbol 74xx:74LS574
- added U504: 74LS00, Package_SO:TSOP-II-44_10.16x18.41mm_P0.8mm, symbol Amiga-Library:CY62157
- added U540, U541: 74LS244, Package_SO:SOIC-20W_7.5x12.8mm_P1.27mm, symbol 74xx:74LS244
- U500: value 27C400 -> CY62157; footprint Package_DIP:DIP-40_W15.24mm -> Package_SO:TSOP-II-44_10.16x18.41mm_P0.8mm
Connections:
- net +5V: now also C500.1, C501.1, R500.1, R503A.2, R503B.2, R503C.2, R503D.2, R503E.2, R503F.2, R503G.2, R503H.2, R503I.2, U500.11 (Vcc), U501.14 (VCC)
- net GND: now also C500.2, C501.2, J500.1 (Pin_1), U500.12 (Vss), U500.34 (Vss), U501.12, U501.13, U501.7 (GND), U502.1 (OE), U502.10 (GND), U503.1 (OE), U503.10 (GND), U503.3 (D1), U503.4 (D2), U503.5 (D3), U503.6 (D4), U503.7 (D5), U503.8 (D6), U503.9 (D7), U540.10 (GND), U541.10 (GND)
- new net: R500D.2, U540.12 (O3a)
- new net: R500C.2, U540.14 (O2a)
- new net: R500B.2, U540.16 (O1a)
- new net: R500A.2, U540.18 (O0a)
- new net: R501C.2, U540.3 (O3b)
- new net: R501B.2, U540.5 (O2b)
- new net: R501A.2, U540.7 (O1b)
- new net: R500E.2, U540.9 (O0b)
- new net: R502B.2, U541.12 (O3a)
- new net: R502A.2, U541.14 (O2a)
- new net: R500E.2, U541.16 (O1a)
- new net: R5001D.2, U541.18 (O0a)
- new net: R502D.2, U541.3 (O3b)
- new net: R502C.2, U541.7 (O1b)
- new net DRA0: R500A.1, R503A.1, U502.2 (D0), U540.2 (I0a)
- new net DRA1: R500B.1, R503B.1, U502.3 (D1), U540.4 (I1a)
- new net DRA2: R500C.1, R503C.1, U502.4 (D2), U540.6 (I2a)
- new net DRA3: R500D.1, R503D.1, U502.5 (D3), U540.8 (I3a)
- new net DRA4: R500E.1, R503E.1, U502.6 (D4), U540.17 (I3b)
- new net DRA5: R501A.1, R503F.1, U502.7 (D5), U540.15 (I2b)
- new net DRA6: R501B.1, R503G.1, U502.8 (D6), U540.13 (I1b)
- new net DRA7: R501C.1, R503H.1, U502.9 (D7), U540.11 (I0b)
- new net DRA8: R5001D.1, R503I.1, U503.2 (D0), U541.2 (I0a)
- new net MA0: U502.19 (Q0)
- new net MA1: U502.18 (Q1)
- new net MA2: U502.17 (Q2)
- new net MA3: U502.16 (Q3)
- new net MA4: U502.15 (Q4)
- new net MA5: U502.14 (Q5)
- new net MA6: U502.13 (Q6)
- new net MA7: U502.12 (Q7)
- new net MA8: U503.19 (Q0)
- new net _CAS: U501.10, U501.6
- new net _CASL: R500E.1, U501.4, U541.4 (I1a)
- new net _CASU: R502A.1, U501.5, U541.6 (I2a)
- new net _EXRAM: J500.2 (Pin_2), R500.2
- new net _MEMCLK: U501.3, U501.9, U502.11 (Cp), U503.11 (Cp)
- new net _RAS0: R502B.1, U501.1, U541.8 (I3a)
- new net _RAS1: R502C.1, U501.2, U541.13 (I1b)
- new net _SRAMCE: U501.8
- new net _WE: R502D.1, U541.17 (I3b)
- no-connect marks 0 -> 10
Other:
- note added: "KICKSTART"
- note added: "OPEN FOR 1M CHIP RAM\nCLOSED FOR 512k"

Commit message: Add files via upload
Parts:
- removed R503A, R503B, R503C, R503D, R503E, R503F, R503G, R503H, R503I: 470, Resistor_SMD:R_1206_3216Metric, symbol Device:R
- removed U502, U503: 74LS574, Package_SO:SOIC-20W_7.5x12.8mm_P1.27mm, symbol 74xx:74LS574
- added C502, C540, C541: 0.1uF, Capacitor_SMD:C_1206_3216Metric, symbol Device:C
- added RN503: 470, Resistor_THT:R_Array_SIP10, symbol Device:R_Network09
- added U502: CY74FCT821T, Package_SO:SOIC-24W_7.5x15.4mm_P1.27mm, symbol Amiga-Library:CY74FCT821T
- U500: value CY62157 -> 27C400; footprint Package_SO:TSOP-II-44_10.16x18.41mm_P0.8mm -> Package_DIP:DIP-40_W15.24mm
- U503: renamed from U504; value 74LS00 -> CY62157
- renumbered C500 to C503, R500A to R500A1, R500B to R500B1, R500C to R500C1, R500D to R500D1, R500E to R500E1, R500E to R500E2, R501A to R501A1, R501B to R501B1, R501C to R501C1, R5001D to R501D1, R502A to R502A1, R502B to R502B1, R502C to R502C1, R502D to R502D1, U500 to U503
Connections:
- net +5V: now also U540.20 (VCC), U541.20 (VCC), C502.1, C540.1, C541.1, RN503.1 (common), U502.24 (Vcc)
- net DRA0: no longer R500A1.1
- net DRA1: no longer R500B1.1
- net DRA2: no longer R500C1.1
- net DRA3: no longer R500D1.1
- net DRA4: no longer R500E2.1
- net DRA5: no longer R501A1.1
- net DRA6: no longer R501B1.1
- net DRA7: no longer R501C1.1
- net DRA8: no longer R501D1.1
- net GND: now also U503.41 (_OE), C502.2, C540.2, C541.2, U502.1 (_OE), U502.11 (D9), U502.12 (GND)
- net _CASL: no longer R500E1.1, U501.4
- net _CASU: no longer R502A1.1, U501.5
- net _MEMCLK: now also U502.13 (CP)
- net _RAS0: no longer R502B1.1, U501.1
- net _RAS1: no longer R502C1.1, U501.2
- net _SRAMCE: now also U503.6 (_CE)
- net _WE: no longer R502D1.1
- net DRAC4: now reaches U503.1 (A4)
- net DRAC4: now also U502.19 (Y4)
- net DRD3: now reaches U503.10 (O3)
- net DRD4: now reaches U503.13 (O4)
- net DRD5: now reaches U503.14 (O5)
- net DRD6: now reaches U503.15 (O6)
- net DRD7: now reaches U503.16 (O7)
- net _MWE: now reaches U503.17 (_WE)
- net _MWE: now also R502D1.1
- net _MRAS0: now reaches U503.18 (A18)
- net _MRAS0: now also R502B1.1, U501.1
- net DRAB8: now reaches U503.19 (A17)
- net DRAB8: now also R501D1.1, RN503.10 (R9), U502.10 (D8)
- net DRAC3: now reaches U503.2 (A3)
- net DRAC3: now also U502.20 (Y3)
- net DRAB7: now reaches U503.20 (A16)
- net DRAB7: now also R501C1.1, RN503.2 (R1), U502.9 (D7)
- net DRAB6: now reaches U503.21 (A15)
- net DRAB6: now also R501B1.1, RN503.4 (R3), U502.8 (D6)
- net DRAB5: now reaches U503.22 (A14)
- net DRAB5: now also R501A1.1, RN503.7 (R6), U502.7 (D5)
- net DRAB4: now reaches U503.23 (A13)
- net DRAB4: now also R500E2.1, RN503.9 (R8), U502.6 (D4)
- net DRAB3: now reaches U503.24 (A12)
- net DRAB3: now also R500D1.1, RN503.8 (R7), U502.5 (D3)
- net DRAB2: now reaches U503.25 (A11)
- net DRAB2: now also R500C1.1, RN503.6 (R5), U502.4 (D2)
- net DRAB1: now reaches U503.26 (A10)
- net DRAB1: now also R500B1.1, RN503.5 (R4), U502.3 (D1)
- net DRAB0: now reaches U503.27 (A9)
- net DRAB0: now also R500A1.1, RN503.3 (R2), U502.2 (D0)
- net DRAC8: now reaches U503.28 (A8)
- net DRAC8: now also U502.15 (Y8)
- net DRD8: now reaches U503.29 (O8)
- net DRAC2: now reaches U503.3 (A2)
- net DRAC2: now also U502.21 (Y2)
- net DRD9: now reaches U503.30 (O9)
- net DRD10: now reaches U503.31 (O10)
- net DRD11: now reaches U503.32 (O11)
- net DRD12: now reaches U503.35 (O12)
- net DRD13: now reaches U503.36 (O13)
- net DRD14: now reaches U503.37 (014)
- net DRD15: now reaches U503.38 (O15)
- net _MLCAS: now reaches U503.39 (_BLE)
- net DRAC1: now reaches U503.4 (A1)
- net DRAC1: now also U502.22 (Y1)
- net _MUCAS: now reaches U503.40 (_BHE)
- net DRAC7: now reaches U503.42 (A7)
- net DRAC7: now also U502.16 (Y7)
- net DRAC6: now reaches U503.43 (A6)
- net DRAC6: now also U502.17 (Y6)
- net DRAC5: now reaches U503.44 (A5)
- net DRAC5: now also U502.18 (Y5)
- net DRAC0: now reaches U503.5 (A0)
- net DRAC0: now also U502.23 (Y0)
- net DRD0: now reaches U503.7 (O0)
- net DRD1: now reaches U503.8 (O1)
- net DRD2: now reaches U503.9 (O2)
- new net _MCASL: R500E1.1, U501.4
- new net _MCASU: R502A1.1, U501.5
- new net _MRAS1: R502C1.1, U501.2
- no-connect marks 10 -> 4
Other:
- note added: "512K x 16 SRAM"
- note added: "OPTIONAL 27C4096 EPROM"
- moved on the sheet: U503A

Commit message: Add files via upload
Parts:
- U500: value 27C400 -> KICKSTART
Changed lines of the file:
@@
 AR Path="/6089B263/605DC51E" Ref="U500"  Part="1"
 F 0 "U500" H 3550 7445 50  0000 C CNN
-F 1 "27C400" H 3550 7354 50  0000 C CNN
+F 1 "KICKSTART" H 3550 7354 50  0000 C CNN
 F 2 "Package_DIP:DIP-40_W15.24mm" H 3450 6880 50  0001 C CNN
 F 3 "" H 3450 6880 50  0001 C CNN
@@
 AR Path="/6089B263/60752CFC" Ref="U500"  Part="2"
 F 0 "U500" H 8878 10196 50  0000 L CNN
-F 1 "27C400" H 8878 10105 50  0000 L CNN
+F 1 "KICKSTART" H 8878 10105 50  0000 L CNN
 F 2 "Package_DIP:DIP-40_W15.24mm" H 8550 10580 50  0001 C CNN
 F 3 "" H 8550 10580 50  0001 C CNN

Commit message: Add files via upload
Parts:
- removed J500: Conn_01x02_Male, Connector_PinHeader_2.54mm:PinHeader_1x02_P2.54mm_Vertical, symbol Connector:Conn_01x02_Male
Other:
- note added: "SETTING IS PERMANENTLY \nSET TO 1M CHIP RAM"
- note removed: "OPEN FOR 1M CHIP RAM\nCLOSED FOR 512k"
Changed lines of the file:
@@
 NoConn ~ 8000 4550
-$Comp
-L Connector:Conn_01x02_Male J500
-U 1 1 607C1B72
-P 3150 3050
-F 0 "J500" V 3258 3094 50  0000 L CNN
-F 1 "Conn_01x02_Male" V 3303 3094 50  0001 L CNN
-F 2 "Connector_PinHeader_2.54mm:PinHeader_1x02_P2.54mm_Vertical" H 3150 3050 50  0001 C CNN
-F 3 "~" H 3150 3050 50  0001 C CNN
-	1    3150 3050
-	0    1    1    0
-$EndComp
 $Comp
 L Device:R R500
@@
 Wire Wire Line
 	2750 3250 2600 3250
-Wire Wire Line
-	2750 3250 3050 3250
-Connection ~ 2750 3250
-Wire Wire Line
-	3150 3250 3400 3250
-$Comp
-L power:GND #PWR0349
-U 1 1 608059F6
-P 3400 3250
-F 0 "#PWR0349" H 3400 3000 50  0001 C CNN
-F 1 "GND" H 3405 3077 50  0000 C CNN
-F 2 "" H 3400 3250 50  0001 C CNN
-F 3 "" H 3400 3250 50  0001 C CNN
-	1    3400 3250
-	1    0    0    -1
-$EndComp
 $Comp
 L power:+5V #PWR0350
@@
 	3650 2600 2050 2600
 Text Notes 2250 3550 0    50   ~ 0
-OPEN FOR 1M CHIP RAM\nCLOSED FOR 512k
+SETTING IS PERMANENTLY \nSET TO 1M CHIP RAM
 $Comp
 L power:GND #PWR0351

Commit message: Add files via upload
Connections:
- net _MLCAS is gone; now on net _MCASL: U503.39 (_BLE)
- net _MUCAS is gone; now on net _MCASU: U503.40 (_BHE)
- net DRA4: now also U540.11 (I0b); no longer U540.17 (I3b)
- net DRA5: now also U540.13 (I1b); no longer U540.15 (I2b)
- net DRA6: now also U540.15 (I2b); no longer U540.13 (I1b)
- net DRA7: now also U540.17 (I3b); no longer U540.11 (I0b)
- net GND: now also U540.1 (OEa), U540.19 (OEb), U541.1 (OEa), U541.19 (OEb)
Other:
- note added: "J500 IS OMITTED\nPERMANENTLY SET \nTO 1M CHIP RAM"
- note added: "OPTIONAL 27C4096 EPROM\nFUTURE"
- note removed: "OPTIONAL 27C4096 EPROM"
- note removed: "SETTING IS PERMANENTLY \nSET TO 1M CHIP RAM"
Changed lines of the file:
@@
 	4150 9700 6100 9700
-Wire Wire Line
-	6100 9700 6100 7500
-Wire Wire Line
-	6100 7500 2900 7500
-Wire Wire Line
-	2900 7500 2900 7100
 Wire Wire Line
 	2900 7100 3050 7100
@@
 DRA3
 Text GLabel 5800 2750 0    50   Input ~ 0
+DRA7
+Text GLabel 5800 2600 0    50   Input ~ 0
+DRA6
+Text GLabel 5800 2450 0    50   Input ~ 0
+DRA5
+Text GLabel 5800 2300 0    50   Input ~ 0
 DRA4
-Text GLabel 5800 2600 0    50   Input ~ 0
-DRA5
-Text GLabel 5800 2450 0    50   Input ~ 0
-DRA6
-Text GLabel 5800 2300 0    50   Input ~ 0
-DRA7
 Text GLabel 5800 2900 0    50   Input ~ 0
 DRA8
@@
 Wire Notes Line
 	3650 2600 2050 2600
-Text Notes 2250 3550 0    50   ~ 0
-SETTING IS PERMANENTLY \nSET TO 1M CHIP RAM
+Text Notes 2750 3550 0    50   ~ 0
+J500 IS OMITTED\nPERMANENTLY SET \nTO 1M CHIP RAM
 $Comp
 L power:GND #PWR0351
@@
 _MRAS0
 Text Label 15300 3600 0    50   ~ 0
-_MUCAS
+_MCASU
 Text Label 15300 3700 0    50   ~ 0
-_MLCAS
+_MCASL
 Wire Wire Line
 	14500 4000 14500 3650
@@
 Text Label 13100 2250 0    50   ~ 0
 DRAC6
-Text Notes 2600 10350 0    118  ~ 0
-OPTIONAL 27C4096 EPROM
+Text Notes 3150 10450 0    118  ~ 0
+OPTIONAL 27C4096 EPROM\nFUTURE
 Wire Wire Line
 	16150 5600 16150 3350
@@
 Wire Wire Line
 	11500 2150 12400 2150
+$Comp
+L power:GND #PWR?
+U 1 1 609B0376
+P 8000 3000
+F 0 "#PWR?" H 8000 2750 50  0001 C CNN
+F 1 "GND" H 8005 2827 50  0000 C CNN
+F 2 "" H 8000 3000 50  0001 C CNN
+F 3 "" H 8000 3000 50  0001 C CNN
+	1    8000 3000
+	1    0    0    -1
+$EndComp
+$Comp
+L power:GND #PWR?
+U 1 1 609B0A18
+P 8000 5150
+F 0 "#PWR?" H 8000 4900 50  0001 C CNN
+F 1 "GND" H 8005 4977 50  0000 C CNN
+F 2 "" H 8000 5150 50  0001 C CNN
+F 3 "" H 8000 5150 50  0001 C CNN
+	1    8000 5150
+	1    0    0    -1
+$EndComp
+Wire Wire Line
+	8000 2750 8000 2850
+Connection ~ 8000 2850
+Wire Wire Line
+	8000 2850 8000 3000
+Wire Wire Line
+	8000 4850 8000 4950
+Connection ~ 8000 4950
+Wire Wire Line
+	8000 4950 8000 5150
+Wire Wire Line
+	2900 7600 6100 7600
+Wire Wire Line
+	6100 7500 6100 7600
+Connection ~ 6100 7600
+Wire Wire Line
+	6100 7600 6100 9700
+Wire Wire Line
+	2900 7100 2900 7600
 $EndSCHEMATC

Commit message: Add files via upload
Other:
- note added: "Memory and Kickstart\nAmiga 2000 EATX"
Changed lines of the file:
@@
 	11500 2150 12400 2150
 $Comp
-L power:GND #PWR?
+L power:GND #PWR0208
 U 1 1 609B0376
 P 8000 3000
-F 0 "#PWR?" H 8000 2750 50  0001 C CNN
+F 0 "#PWR0208" H 8000 2750 50  0001 C CNN
 F 1 "GND" H 8005 2827 50  0000 C CNN
 F 2 "" H 8000 3000 50  0001 C CNN
@@
 $EndComp
 $Comp
-L power:GND #PWR?
+L power:GND #PWR0209
 U 1 1 609B0A18
 P 8000 5150
-F 0 "#PWR?" H 8000 4900 50  0001 C CNN
+F 0 "#PWR0209" H 8000 4900 50  0001 C CNN
 F 1 "GND" H 8005 4977 50  0000 C CNN
 F 2 "" H 8000 5150 50  0001 C CNN
@@
 Wire Wire Line
 	2900 7100 2900 7600
+Text Notes 12300 9850 0    197  ~ 0
+Memory and Kickstart\nAmiga 2000 EATX
 $EndSCHEMATC
