File: 2000EATX-KiCAD/video.sch (KiCad schematic (older format))
At the start: 39 parts, among them CN201 Amiga-2000-Video-Slot, CN202 DB15_Female_HighDensity, CN203 Amiga-2000-Video-Slot, U201 DENISE, U205 74HCT244, U206 74HCT244, U303 74LS08

Commit message: Add files via upload
Connections:
- net COMPVID is gone; now on net COMP: CN203.13
- no-connect marks 39 -> 35
Other:
- moved on the sheet: C214, C226
Changed lines of the file:
@@
 Wire Wire Line
 	8900 1750 8900 2050
-NoConn ~ 8900 2050
 Text Label 8900 2050 3    50   ~ 0
 COMPSYNC
@@
 	2850 1850 2850 1200
 Text Label 2850 1200 1    50   ~ 0
-COMPVID
-NoConn ~ 2850 1200
+COMP
 $Comp
 L Amiga-Library:Denise U201
@@
 Wire Wire Line
 	4500 6000 4500 5900
-Text Notes 12550 1240 0    118  ~ 0
+Text Notes 11950 1790 0    118  ~ 0
 VIDIOT
 Wire Wire Line
@@
 Wire Notes Line
 	11300 5450 11300 6550
-Text Label 12800 1600 2    47   ~ 0
+Text Label 12200 2150 2    47   ~ 0
 COMP
-Text Label 12800 1500 2    47   ~ 0
+Text Label 12200 2050 2    47   ~ 0
 COMPSYNC
-NoConn ~ 12800 1500
-NoConn ~ 12800 1600
-Wire Wire Line
-	13250 1500 12800 1500
-Wire Wire Line
-	13250 1600 12800 1600
-Text Label 13250 1800 2    47   ~ 0
+Wire Wire Line
+	12650 2050 12200 2050
+Wire Wire Line
+	12650 2150 12200 2150
+Text Label 12650 2350 2    47   ~ 0
 BLUE
-Text Label 13250 2300 2    47   ~ 0
+Text Label 12650 2850 2    47   ~ 0
 GREEN
-Text Label 13250 2800 2    47   ~ 0
+Text Label 12650 3350 2    47   ~ 0
 RED
 Wire Wire Line
-	12850 1300 13250 1300
-Wire Wire Line
-	12850 3400 12850 1300
-Wire Wire Line
-	13250 3400 12850 3400
+	12250 1850 12650 1850
+Wire Wire Line
+	12250 3950 12250 1850
+Wire Wire Line
+	12650 3950 12250 3950
 $Comp
 L power:GND #PWR0206
 U 1 1 60CF6FB1
-P 13250 3400
-F 0 "#PWR0206" H 13250 3150 50  0001 C CNN
-F 1 "GND" H 13255 3227 50  0000 C CNN
-F 2 "" H 13250 3400 50  0001 C CNN
-F 3 "" H 13250 3400 50  0001 C CNN
-	1    13250 3400
-	1    0    0    -1
-$EndComp
-Connection ~ 12950 3300
-Wire Wire Line
-	12950 1400 13250 1400
-Wire Wire Line
-	12950 3300 12950 1400
-Wire Wire Line
-	12950 3300 12950 3750
-Wire Wire Line
-	13250 3300 12950 3300
-Wire Wire Line
-	12700 3600 12700 3750
+P 12650 3950
+F 0 "#PWR0206" H 12650 3700 50  0001 C CNN
+F 1 "GND" H 12655 3777 50  0000 C CNN
+F 2 "" H 12650 3950 50  0001 C CNN
+F 3 "" H 12650 3950 50  0001 C CNN
+	1    12650 3950
+	1    0    0    -1
+$EndComp
+Connection ~ 12350 3850
+Wire Wire Line
+	12350 1950 12650 1950
+Wire Wire Line
+	12350 3850 12350 1950
+Wire Wire Line
+	12350 3850 12350 4300
+Wire Wire Line
+	12650 3850 12350 3850
+Wire Wire Line
+	12100 4150 12100 4300
 $Comp
 L Amiga-Library:+VID #PWR0205
 U 1 1 60C92D13
-P 12700 3600
-F 0 "#PWR0205" H 12700 3750 50  0001 C CNN
-F 1 "+VID" H 12700 3750 50  0000 C CNN
-F 2 "" H 12700 3600 50  0001 C CNN
-F 3 "" H 12700 3600 50  0001 C CNN
-	1    12700 3600
+P 12100 4150
+F 0 "#PWR0205" H 12100 4300 50  0001 C CNN
+F 1 "+VID" H 12100 4300 50  0000 C CNN
+F 2 "" H 12100 4150 50  0001 C CNN
+F 3 "" H 12100 4150 50  0001 C CNN
+	1    12100 4150
 	1    0    0    -1
 $EndComp
@@
 L power:GND #PWR0204
 U 1 1 60C92513
-P 13300 4050
-F 0 "#PWR0204" H 13300 3800 50  0001 C CNN
-F 1 "GND" H 13305 3877 50  0000 C CNN
-F 2 "" H 13300 4050 50  0001 C CNN
-F 3 "" H 13300 4050 50  0001 C CNN
-	1    13300 4050
-	1    0    0    -1
-$EndComp
-Connection ~ 13300 3950
-Wire Wire Line
-	13300 3950 13300 4050
-Wire Wire Line
-	12950 3950 13300 3950
-Connection ~ 12950 3750
-Wire Wire Line
-	12950 3750 12700 3750
-Wire Wire Line
-	12950 3750 13300 3750
-Text Label 13250 1700 2    47   ~ 0
+P 12700 4600
+F 0 "#PWR0204" H 12700 4350 50  0001 C CNN
+F 1 "GND" H 12705 4427 50  0000 C CNN
+F 2 "" H 12700 4600 50  0001 C CNN
+F 3 "" H 12700 4600 50  0001 C CNN
+	1    12700 4600
+	1    0    0    -1
+$EndComp
+Connection ~ 12700 4500
+Wire Wire Line
+	12700 4500 12700 4600
+Wire Wire Line
+	12350 4500 12700 4500
+Connection ~ 12350 4300
+Wire Wire Line
+	12350 4300 12100 4300
+Wire Wire Line
+	12350 4300 12700 4300
+Text Label 12650 2250 2    47   ~ 0
 _CSYNC
-Text Label 13250 1900 2    47   ~ 0
+Text Label 12650 2450 2    47   ~ 0
 B0
-Text Label 13250 2000 2    47   ~ 0
+Text Label 12650 2550 2    47   ~ 0
 B1
-Text Label 13250 2100 2    47   ~ 0
+Text Label 12650 2650 2    47   ~ 0
 B2
-Text Label 13250 2200 2    47   ~ 0
+Text Label 12650 2750 2    47   ~ 0
 B3
-Text Label 13250 2400 2    47   ~ 0
+Text Label 12650 2950 2    47   ~ 0
 G0
-Text Label 13250 2500 2    47   ~ 0
+Text Label 12650 3050 2    47   ~ 0
 G1
-Text Label 13250 2600 2    47   ~ 0
+Text Label 12650 3150 2    47   ~ 0
 G2
-Text Label 13250 2700 2    47   ~ 0
+Text Label 12650 3250 2    47   ~ 0
 G3
-Text Label 13250 2900 2    47   ~ 0
+Text Label 12650 3450 2    47   ~ 0
 R0
-Text Label 13250 3000 2    47   ~ 0
+Text Label 12650 3550 2    47   ~ 0
 R1
-Text Label 13250 3100 2    47   ~ 0
+Text Label 12650 3650 2    47   ~ 0
 R2
-Text Label 13250 3200 2    47   ~ 0
+Text Label 12650 3750 2    47   ~ 0
 R3
 $Comp
 L Connector:Conn_01x22_Male VIDIOT1
 U 1 1 60820DFB
-P 13450 2400
-F 0 "VIDIOT1" H 13300 2400 50  0001 C CNN
-F 1 "HY200" H 13422 2328 50  0000 R CNN
-F 2 "Connector_PinSocket_2.54mm:PinSocket_1x22_P2.54mm_Vertical" H 13450 2400 50  0001 C CNN
-F 3 "~" H 13450 2400 50  0001 C CNN
-	1    13450 2400
+P 12850 2950
+F 0 "VIDIOT1" H 12700 2950 50  0001 C CNN
+F 1 "HY200" H 12822 2878 50  0000 R CNN
+F 2 "Connector_PinSocket_2.54mm:PinSocket_1x22_P2.54mm_Vertical" H 12850 2950 50  0001 C CNN
+F 3 "~" H 12850 2950 50  0001 C CNN
+	1    12850 2950
 	-1   0    0    1
 $EndComp
@@
 L Device:CP_Small C214
 U 1 1 61608713
-P 12950 3850
-F 0 "C214" V 13175 3850 50  0000 C CNN
-F 1 "470uF" V 13084 3850 50  0000 C CNN
-F 2 "Capacitor_SMD:CP_Elec_6.3x5.8" H 12950 3850 50  0001 C CNN
-F 3 "~" H 12950 3850 50  0001 C CNN
-	1    12950 3850
+P 12350 4400
+F 0 "C214" V 12575 4400 50  0000 C CNN
+F 1 "470uF" V 12484 4400 50  0000 C CNN
+F 2 "Capacitor_SMD:CP_Elec_6.3x5.8" H 12350 4400 50  0001 C CNN
+F 3 "~" H 12350 4400 50  0001 C CNN
+	1    12350 4400
 	1    0    0    -1
 $EndComp
@@
 L Device:CP_Small C226
 U 1 1 61607EA7
-P 13300 3850
-F 0 "C226" V 13525 3850 50  0000 C CNN
-F 1 "470uF" V 13434 3850 50  0000 C CNN
-F 2 "Capacitor_SMD:CP_Elec_6.3x5.8" H 13300 3850 50  0001 C CNN
-F 3 "~" H 13300 3850 50  0001 C CNN
-	1    13300 3850
-	1    0    0    -1
-$EndComp
-Connection ~ 13250 3400
+P 12700 4400
+F 0 "C226" V 12925 4400 50  0000 C CNN
+F 1 "470uF" V 12834 4400 50  0000 C CNN
+F 2 "Capacitor_SMD:CP_Elec_6.3x5.8" H 12700 4400 50  0001 C CNN
+F 3 "~" H 12700 4400 50  0001 C CNN
+	1    12700 4400
+	1    0    0    -1
+$EndComp
+Connection ~ 12650 3950
 Wire Wire Line
 	2350 3300 2800 3300

Commit message: Add files via upload
Connections:
- net at U201.29 (G1), U206.6 (1A2): now also RN906.6 (R5); no longer RN906.4 (R3)
Changed lines of the file:
@@
 	2350 5900 2950 5900
-Wire Wire Line
-	2350 5800 2850 5800
 Wire Wire Line
 	2350 5700 2750 5700
@@
 	2650 5150 2450 5150
 Connection ~ 2450 5150
-NoConn ~ 3050 5550
+NoConn ~ 2850 5550
 Wire Wire Line
 	2650 5550 2650 5600
@@
 Wire Wire Line
 	2750 5700 4100 5700
-Wire Wire Line
-	2850 5550 2850 5800
-Connection ~ 2850 5800
-Wire Wire Line
-	2850 5800 4200 5800
 Wire Wire Line
 	2950 5550 2950 5900
@@
 Wire Wire Line
 	2600 3100 3200 3100
+Wire Wire Line
+	3050 5800 3050 5550
+Connection ~ 3050 5800
+Wire Wire Line
+	3050 5800 4200 5800
+Wire Wire Line
+	2350 5800 3050 5800
 $EndSCHEMATC

Commit message: Add files via upload
Parts:
- CN202: footprint Connector_Dsub:DSUB-15-HD_Female_Horizontal_P2.29x1.98mm_EdgePinOffset3.03mm_Housed_MountingHolesOffset4.94mm -> Connector_Dsub:DSUB-15-HD_Female_Horizontal_P2.29x1.98mm_EdgePinOffset8.35mm_Housed_MountingHolesOffset10.89mm
Changed lines of the file:
@@
 F 0 "CN202" H 10000 6017 50  0000 C CNN
 F 1 "DB15_Female_HighDensity" H 10000 5926 50  0000 C CNN
-F 2 "Connector_Dsub:DSUB-15-HD_Female_Horizontal_P2.29x1.98mm_EdgePinOffset3.03mm_Housed_MountingHolesOffset4.94mm" H 9050 5550 50  0001 C CNN
+F 2 "Connector_Dsub:DSUB-15-HD_Female_Horizontal_P2.29x1.98mm_EdgePinOffset8.35mm_Housed_MountingHolesOffset10.89mm" H 9050 5550 50  0001 C CNN
 F 3 " ~" H 9050 5550 50  0001 C CNN
 	1    10000 5150

Commit message: Add files via upload
Parts:
- CN202: footprint Connector_Dsub:DSUB-15-HD_Female_Horizontal_P2.29x1.98mm_EdgePinOffset8.35mm_Housed_MountingHolesOffset10.89mm -> AmigaFootprints:DSUB-15-HD_Female_Horizontal_P2.29x1.98mm_EdgePinOffset8.35mm_Housed_MountingHolesOffset10.89mm
Changed lines of the file:
@@
 F 0 "CN202" H 10000 6017 50  0000 C CNN
 F 1 "DB15_Female_HighDensity" H 10000 5926 50  0000 C CNN
-F 2 "Connector_Dsub:DSUB-15-HD_Female_Horizontal_P2.29x1.98mm_EdgePinOffset8.35mm_Housed_MountingHolesOffset10.89mm" H 9050 5550 50  0001 C CNN
+F 2 "AmigaFootprints:DSUB-15-HD_Female_Horizontal_P2.29x1.98mm_EdgePinOffset8.35mm_Housed_MountingHolesOffset10.89mm" H 9050 5550 50  0001 C CNN
 F 3 " ~" H 9050 5550 50  0001 C CNN
 	1    10000 5150

Commit message: Add files via upload
Connections:
- net TBASE is gone; now on net _VSYNC: C915.1, CN203.14
- net HSYNC: no longer names the net of EMI206.1, R203B1.1
- net VSYNC: no longer names the net of EMI207.1, R203A1.1
- no-connect marks 35 -> 13
Other:
- note removed: "Optional. Allows use of Raspberry Pi Zero to output HDMI. See Github for details."
- note removed: "Raspberry Pi HDMI Video Out"
- note removed: "https://github.com/jasonsbeer/Amiga-HDMI-Through-Hole"

Commit message: Add files via upload
Connections:
- net _VSYNC: no longer C915.1, CN203.14
- new net TBASE: C915.1, CN203.14
Other:
- note added: "Video\nAmiga 2000 EATX"
- note removed: "VIDEO"
Changed lines of the file:
@@
 Comment4 ""
 $EndDescr
-Text Notes 12330 9600 0    197  ~ 0
-VIDEO
+Text Notes 12350 9850 0    197  ~ 0
+Video\nAmiga 2000 EATX
 $Comp
 L Connector:DB15_Female_HighDensity CN202
@@
 R0
 Text GLabel 950  1450 0    50   Input ~ 0
-_VSYNC
+TBASE
 $Comp
 L Amiga-Library:C_Small C915

Commit message: Add files via upload
Parts:
- removed RN904, RN905, RN906: 4.7k, Resistor_THT:R_Array_SIP6, symbol Device:R_Network05
Connections:
- no-connect marks 13 -> 10
Changed lines of the file:
@@
-	1    0    0    -1
-$EndComp
-$Comp
-L Amiga-Library:Denise U201
-U 2 1 61235FB8
-P 2050 7250
-F 0 "U201" H 2328 7321 50  0000 L CNN
-F 1 "DENISE" H 2328 7230 50  0000 L CNN
-F 2 "Package_DIP:DIP-48_W15.24mm" H 2050 7250 50  0001 C CNN
-F 3 "" H 2050 7250 50  0001 C CNN
-	2    2050 7250
 	1    0    0    -1
 $EndComp
@@
 $EndComp
 Wire Wire Line
-	2050 6900 2450 6900
-Wire Wire Line
 	1300 7000 1550 7000
 Wire Wire Line
 	1550 7000 1550 6900
-Wire Wire Line
-	1550 6900 2050 6900
-Connection ~ 2050 6900
 $Comp
 L Amiga-Library:C_Feedthrough EMI200
@@
 	9400 5250 9400 5450
 Connection ~ 4300 2550
-$Comp
-L Device:R_Network05 RN904
-U 1 1 607131D9
-P 2800 4550
-F 0 "RN904" H 3088 4596 50  0000 L CNN
-F 1 "4.7k" H 3088 4505 50  0000 L CNN
-F 2 "Resistor_THT:R_Array_SIP6" V 3175 4550 50  0001 C CNN
-F 3 "http://www.vishay.com/docs/31509/csc.pdf" H 2800 4550 50  0001 C CNN
-	1    2800 4550
-	1    0    0    -1
-$EndComp
-Wire Wire Line
-	2350 4800 2600 4800
-Wire Wire Line
-	2350 4900 2700 4900
-Wire Wire Line
-	2350 5000 2800 5000
-Wire Wire Line
-	2350 5100 2900 5100
-Wire Wire Line
-	2450 4350 2600 4350
 Wire Wire Line
 	2350 4400 2350 4250
 Wire Wire Line
 	2350 4250 3500 4250
-Wire Wire Line
-	2600 4750 2600 4800
-Connection ~ 2600 4800
-Wire Wire Line
-	2600 4800 3600 4800
-Wire Wire Line
-	2700 4750 2700 4900
-Connection ~ 2700 4900
-Wire Wire Line
-	2700 4900 3700 4900
-Wire Wire Line
-	2800 4750 2800 5000
-Connection ~ 2800 5000
-Wire Wire Line
-	2800 5000 3800 5000
-Wire Wire Line
-	2900 4750 2900 5100
-Connection ~ 2900 5100
-Wire Wire Line
-	2900 5100 3900 5100
-NoConn ~ 3000 4750
-Wire Wire Line
-	2450 4350 2450 5150
-$Comp
-L Device:R_Network05 RN906
-U 1 1 609E4AA5
-P 2850 5350
-F 0 "RN906" H 3138 5396 50  0000 L CNN
-F 1 "4.7k" H 3138 5305 50  0000 L CNN
-F 2 "Resistor_THT:R_Array_SIP6" V 3225 5350 50  0001 C CNN
-F 3 "http://www.vishay.com/docs/31509/csc.pdf" H 2850 5350 50  0001 C CNN
-	1    2850 5350
-	1    0    0    -1
-$EndComp
-Wire Wire Line
-	2350 5900 2950 5900
-Wire Wire Line
-	2350 5700 2750 5700
-Wire Wire Line
-	2350 5600 2650 5600
-Wire Wire Line
-	2650 5150 2450 5150
-Connection ~ 2450 5150
-NoConn ~ 2850 5550
-Wire Wire Line
-	2650 5550 2650 5600
-Connection ~ 2650 5600
-Wire Wire Line
-	2650 5600 4000 5600
-Wire Wire Line
-	2750 5550 2750 5700
-Connection ~ 2750 5700
-Wire Wire Line
-	2750 5700 4100 5700
-Wire Wire Line
-	2950 5550 2950 5900
-Connection ~ 2950 5900
-Wire Wire Line
-	2950 5900 4300 5900
-Wire Wire Line
-	2350 6400 2650 6400
-Wire Wire Line
-	2350 6500 2750 6500
-Wire Wire Line
-	2350 6600 2850 6600
-Wire Wire Line
-	2350 6700 2950 6700
-Wire Wire Line
-	2450 5150 2450 5950
-$Comp
-L Device:R_Network05 RN905
-U 1 1 60C1E4EE
-P 2850 6150
-F 0 "RN905" H 3138 6196 50  0000 L CNN
-F 1 "4.7k" H 3138 6105 50  0000 L CNN
-F 2 "Resistor_THT:R_Array_SIP6" V 3225 6150 50  0001 C CNN
-F 3 "http://www.vishay.com/docs/31509/csc.pdf" H 2850 6150 50  0001 C CNN
-	1    2850 6150
-	1    0    0    -1
-$EndComp
-NoConn ~ 3050 6350
-Wire Wire Line
-	2650 5950 2450 5950
-Connection ~ 2450 5950
-Wire Wire Line
-	2450 5950 2450 6900
-Wire Wire Line
-	2650 6350 2650 6400
-Connection ~ 2650 6400
-Wire Wire Line
-	2650 6400 4400 6400
-Wire Wire Line
-	2750 6350 2750 6500
-Connection ~ 2750 6500
-Wire Wire Line
-	2750 6500 3550 6500
-Wire Wire Line
-	2850 6350 2850 6600
-Connection ~ 2850 6600
-Wire Wire Line
-	2850 6600 4050 6600
-Wire Wire Line
-	2950 6350 2950 6700
-Connection ~ 2950 6700
-Wire Wire Line
-	2950 6700 4250 6700
 $Comp
 L Device:R_Network05 RN205
@@
 	2600 3100 3200 3100
 Wire Wire Line
-	3050 5800 3050 5550
-Connection ~ 3050 5800
-Wire Wire Line
-	3050 5800 4200 5800
-Wire Wire Line
-	2350 5800 3050 5800
+	1550 6900 2050 6900
+$Comp
+L Amiga-Library:Denise U201
+U 2 1 61235FB8
+P 2050 7250
+F 0 "U201" H 2328 7321 50  0000 L CNN
+F 1 "DENISE" H 2328 7230 50  0000 L CNN
+F 2 "Package_DIP:DIP-48_W15.24mm" H 2050 7250 50  0001 C CNN
+F 3 "" H 2050 7250 50  0001 C CNN
+	2    2050 7250
+	1    0    0    -1
+$EndComp
+Wire Wire Line
+	2350 6400 4400 6400
+Wire Wire Line
+	2350 6500 3550 6500
+Wire Wire Line
+	2350 6600 4050 6600
+Wire Wire Line
+	2350 6700 4250 6700
+Wire Wire Line
+	2350 5600 4000 5600
+Wire Wire Line
+	2350 5700 4100 5700
+Wire Wire Line
+	2350 5900 4300 5900
+Wire Wire Line
+	2350 5800 4200 5800
+Wire Wire Line
+	2350 4800 3600 4800
+Wire Wire Line
+	2350 4900 3700 4900
+Wire Wire Line
+	2350 5000 3800 5000
+Wire Wire Line
+	2350 5100 3900 5100
 $EndSCHEMATC

Commit message: Add files via upload
Parts:
- C214, C226: footprint Capacitor_SMD:CP_Elec_6.3x5.8 -> Capacitor_SMD:CP_Elec_8x10
Changed lines of the file:
@@
 F 0 "C214" V 12575 4400 50  0000 C CNN
 F 1 "470uF" V 12484 4400 50  0000 C CNN
-F 2 "Capacitor_SMD:CP_Elec_6.3x5.8" H 12350 4400 50  0001 C CNN
+F 2 "Capacitor_SMD:CP_Elec_8x10" H 12350 4400 50  0001 C CNN
 F 3 "~" H 12350 4400 50  0001 C CNN
 	1    12350 4400
@@
 F 0 "C226" V 12925 4400 50  0000 C CNN
 F 1 "470uF" V 12834 4400 50  0000 C CNN
-F 2 "Capacitor_SMD:CP_Elec_6.3x5.8" H 12700 4400 50  0001 C CNN
+F 2 "Capacitor_SMD:CP_Elec_8x10" H 12700 4400 50  0001 C CNN
 F 3 "~" H 12700 4400 50  0001 C CNN
 	1    12700 4400
