File: 2000EATX-KiCAD/Processor.sch (KiCad schematic (older format))
At the start: 19 parts, among them U100 68000D, U103 74LS245, U104 74LS373, U105 74LS245, U106 74LS373, U303 74LS08

Commit message: Add files via upload
Parts:
- U100: value 68000D -> MC68000
Changed lines of the file:
@@
 P 4750 4050
 F 0 "U100" H 4750 6631 50  0000 C CNN
-F 1 "68000D" H 4750 6540 50  0000 C CNN
+F 1 "MC68000" H 4750 6540 50  0000 C CNN
 F 2 "Package_DIP:DIP-64_W25.4mm" H 4750 4050 50  0001 C CNN
 F 3 "https://www.nxp.com/docs/en/reference-manual/MC68000UM.pdf" H 4750 4050 50  0001 C CNN

Commit message: Add files via upload
Parts:
- R1000, R917: value 407 -> 470
- RN101: value 4.7k -> 2.7k
Changed lines of the file:
@@
 P 3700 4300
 F 0 "R917" H 3759 4346 50  0000 L CNN
-F 1 "407" H 3759 4255 50  0000 L CNN
+F 1 "470" H 3759 4255 50  0000 L CNN
 F 2 "Capacitor_SMD:C_1206_3216Metric" H 3700 4300 50  0001 C CNN
 F 3 "~" H 3700 4300 50  0001 C CNN
@@
 P 3200 4450
 F 0 "R1000" H 3259 4496 50  0000 L CNN
-F 1 "407" H 3259 4405 50  0000 L CNN
+F 1 "470" H 3259 4405 50  0000 L CNN
 F 2 "Capacitor_SMD:C_1206_3216Metric" H 3200 4450 50  0001 C CNN
 F 3 "~" H 3200 4450 50  0001 C CNN
@@
 P 1550 3750
 F 0 "RN101" H 2038 3796 50  0000 L CNN
-F 1 "4.7k" H 2038 3705 50  0000 L CNN
+F 1 "2.7k" H 2038 3705 50  0000 L CNN
 F 2 "Resistor_THT:R_Array_SIP10" V 2125 3750 50  0001 C CNN
 F 3 "http://www.vishay.com/docs/31509/csc.pdf" H 1550 3750 50  0001 C CNN

Commit message: Add files via upload
Other:
- note added: "Processor\nAmiga 2000 EATX"
- note removed: "PROCESSOR"
Changed lines of the file:
@@
 Wire Wire Line
 	3700 4850 2850 4850
-Text Notes 7100 6700 0    50   ~ 0
-PROCESSOR
+Text Notes 7050 7100 0    197  ~ 0
+Processor\nAmiga 2000 EATX
 Text GLabel 5750 1850 2    50   BiDi ~ 0
 A1

Commit message: Add files via upload
Parts:
- R1000, R104, R917, XR1: footprint Capacitor_SMD:C_1206_3216Metric -> Resistor_SMD:R_1206_3216Metric
- R111: value 407 -> 470; footprint Capacitor_SMD:C_1206_3216Metric -> Resistor_SMD:R_1206_3216Metric
Changed lines of the file:
@@
 F 0 "R917" H 3759 4346 50  0000 L CNN
 F 1 "470" H 3759 4255 50  0000 L CNN
-F 2 "Capacitor_SMD:C_1206_3216Metric" H 3700 4300 50  0001 C CNN
+F 2 "Resistor_SMD:R_1206_3216Metric" H 3700 4300 50  0001 C CNN
 F 3 "~" H 3700 4300 50  0001 C CNN
 	1    3700 4300
@@
 F 0 "R1000" H 3259 4496 50  0000 L CNN
 F 1 "470" H 3259 4405 50  0000 L CNN
-F 2 "Capacitor_SMD:C_1206_3216Metric" H 3200 4450 50  0001 C CNN
+F 2 "Resistor_SMD:R_1206_3216Metric" H 3200 4450 50  0001 C CNN
 F 3 "~" H 3200 4450 50  0001 C CNN
 	1    3200 4450
@@
 P 1950 4950
 F 0 "R111" H 2009 4996 50  0000 L CNN
-F 1 "407" H 2009 4905 50  0000 L CNN
-F 2 "Capacitor_SMD:C_1206_3216Metric" H 1950 4950 50  0001 C CNN
+F 1 "470" H 2009 4905 50  0000 L CNN
+F 2 "Resistor_SMD:R_1206_3216Metric" H 1950 4950 50  0001 C CNN
 F 3 "~" H 1950 4950 50  0001 C CNN
 	1    1950 4950
@@
 F 0 "R104" H 2059 2396 50  0000 L CNN
 F 1 "4.7k" H 2059 2305 50  0000 L CNN
-F 2 "Capacitor_SMD:C_1206_3216Metric" H 2000 2350 50  0001 C CNN
+F 2 "Resistor_SMD:R_1206_3216Metric" H 2000 2350 50  0001 C CNN
 F 3 "~" H 2000 2350 50  0001 C CNN
 	1    2000 2350
@@
 F 0 "XR1" H 2859 3996 50  0000 L CNN
 F 1 "68" H 2859 3905 50  0000 L CNN
-F 2 "Capacitor_SMD:C_1206_3216Metric" H 2800 3950 50  0001 C CNN
+F 2 "Resistor_SMD:R_1206_3216Metric" H 2800 3950 50  0001 C CNN
 F 3 "~" H 2800 3950 50  0001 C CNN
 	1    2800 3950

Commit message: Add files via upload
Parts:
- U103, U105: value 74LS245 -> 74HCT245
- U104, U106: value 74LS373 -> 74HCT373
- U303: value 74LS08 -> 74HCT08
Changed lines of the file:
@@
 P 7900 3100
 F 0 "U103" H 7900 4081 50  0000 C CNN
-F 1 "74LS245" H 7900 3990 50  0000 C CNN
+F 1 "74HCT245" H 7900 3990 50  0000 C CNN
 F 2 "Package_SO:SOIC-20W_7.5x12.8mm_P1.27mm" H 7900 3100 50  0001 C CNN
 F 3 "http://www.ti.com/lit/gpn/sn74LS245" H 7900 3100 50  0001 C CNN
@@
 P 7900 5250
 F 0 "U105" H 7900 6231 50  0000 C CNN
-F 1 "74LS245" H 7900 6140 50  0000 C CNN
+F 1 "74HCT245" H 7900 6140 50  0000 C CNN
 F 2 "Package_SO:SOIC-20W_7.5x12.8mm_P1.27mm" H 7900 5250 50  0001 C CNN
 F 3 "http://www.ti.com/lit/gpn/sn74LS245" H 7900 5250 50  0001 C CNN
@@
 P 9850 2550
 F 0 "U104" H 9850 3531 50  0000 C CNN
-F 1 "74LS373" H 9850 3440 50  0000 C CNN
+F 1 "74HCT373" H 9850 3440 50  0000 C CNN
 F 2 "Package_SO:SOIC-20W_7.5x12.8mm_P1.27mm" H 9850 2550 50  0001 C CNN
 F 3 "http://www.ti.com/lit/gpn/sn74LS373" H 9850 2550 50  0001 C CNN
@@
 P 9850 4700
 F 0 "U106" H 9850 5681 50  0000 C CNN
-F 1 "74LS373" H 9850 5590 50  0000 C CNN
+F 1 "74HCT373" H 9850 5590 50  0000 C CNN
 F 2 "Package_SO:SOIC-20W_7.5x12.8mm_P1.27mm" H 9850 4700 50  0001 C CNN
 F 3 "http://www.ti.com/lit/gpn/sn74LS373" H 9850 4700 50  0001 C CNN
@@
 P 2600 2550
 F 0 "U303" H 2600 2875 50  0000 C CNN
-F 1 "74LS08" H 2600 2784 50  0000 C CNN
+F 1 "74HCT08" H 2600 2784 50  0000 C CNN
 F 2 "Package_SO:SOIC-14_3.9x8.7mm_P1.27mm" H 2600 2550 50  0001 C CNN
 F 3 "http://www.ti.com/lit/gpn/sn74LS08" H 2600 2550 50  0001 C CNN
