File: 2000EATX-KiCAD/agnus.sch (KiCad schematic (older format))
At the start: 33 parts, among them J102 Short for NTSC/Open for PAL, J900 Enable Chip RAM slowdown duri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, U101 FATTERAGNUS, U102 GARY, U107 74LS04, U302 74LS32, U900 74LS00, X1 28.63636MHz

Commit message: Add files via upload
Parts:
- J102: value Short for NTSC/Open for PAL -> Short for NTSC
- U101: value FATTERAGNUS -> FATTER_AGNUS
Changed lines of the file:
@@
 P 8850 7150
 F 0 "U101" H 8850 4327 50  0000 C CNN
-F 1 "FATTERAGNUS" H 8850 4236 50  0000 C CNN
+F 1 "FATTER_AGNUS" H 8850 4236 50  0000 C CNN
 F 2 "Package_LCC:PLCC-84_THT-Socket" H 8750 8700 50  0001 C CNN
 F 3 "http://www.ti.com/lit/gpn/sn7400" H 8750 8700 50  0001 C CNN
@@
 P 10450 10000
 F 0 "J102" V 10350 9950 50  0000 C CNN
-F 1 "Short for NTSC/Open for PAL" V 10250 10000 50  0000 C CNN
+F 1 "Short for NTSC" V 10250 10000 50  0000 C CNN
 F 2 "Connector_PinHeader_2.54mm:PinHeader_1x02_P2.54mm_Vertical" H 10450 10000 50  0001 C CNN
 F 3 "~" H 10450 10000 50  0001 C CNN
@@
 P 11150 1550
 F 0 "U101" H 10550 1550 50  0000 L CNN
-F 1 "FATTERAGNUS" H 10300 1450 50  0000 L CNN
+F 1 "FATTER_AGNUS" H 10300 1450 50  0000 L CNN
 F 2 "Package_LCC:PLCC-84_THT-Socket" H 11150 1550 50  0001 C CNN
 F 3 "http://www.ti.com/lit/gpn/sn7400" H 11050 3100 50  0001 C CNN

Commit message: Add files via upload
Parts:
- J102: value Short for NTSC -> SHORT FOR NTSC
Connections:
- net +5V: now also U900.14 (VCC); no longer U900.7 (GND)
- net GND: now also U900.7 (GND); no longer U900.14 (VCC)
Changed lines of the file:
@@
 P 10450 10000
 F 0 "J102" V 10350 9950 50  0000 C CNN
-F 1 "Short for NTSC" V 10250 10000 50  0000 C CNN
+F 1 "SHORT FOR NTSC" V 10250 10000 50  0000 C CNN
 F 2 "Connector_PinHeader_2.54mm:PinHeader_1x02_P2.54mm_Vertical" H 10450 10000 50  0001 C CNN
 F 3 "~" H 10450 10000 50  0001 C CNN
@@
 U 5 1 60DDC760
 P 15200 1600
-F 0 "U900" H 14970 1554 50  0000 R CNN
-F 1 "74LS00" H 14970 1645 50  0000 R CNN
+F 0 "U900" H 15250 1550 50  0000 R CNN
+F 1 "74LS00" H 15300 1650 50  0000 R CNN
 F 2 "Package_SO:SOIC-14_3.9x8.7mm_P1.27mm" H 15200 1600 50  0001 C CNN
 F 3 "http://www.ti.com/lit/gpn/sn7400" H 15200 1600 50  0001 C CNN
 	5    15200 1600
-	-1   0    0    1
+	1    0    0    -1
 $EndComp
 Wire Wire Line
@@
 Wire Wire Line
 	13250 1200 13250 1100
-Wire Wire Line
-	15300 1100 15300 1050
 Connection ~ 12500 1200
 Wire Wire Line
@@
 	12700 1200 13200 1200
 Wire Wire Line
-	15200 2100 14500 2100
-Wire Wire Line
 	13000 2100 13000 1950
 Wire Wire Line
@@
 L power:GND #PWR0251
 U 1 1 60E2C45F
-P 15200 2100
-F 0 "#PWR0251" H 15200 1850 50  0001 C CNN
-F 1 "GND" H 15205 1927 50  0000 C CNN
-F 2 "" H 15200 2100 50  0001 C CNN
-F 3 "" H 15200 2100 50  0001 C CNN
-	1    15200 2100
-	1    0    0    -1
-$EndComp
-Connection ~ 15200 2100
+P 15800 2100
+F 0 "#PWR0251" H 15800 1850 50  0001 C CNN
+F 1 "GND" H 15805 1927 50  0000 C CNN
+F 2 "" H 15800 2100 50  0001 C CNN
+F 3 "" H 15800 2100 50  0001 C CNN
+	1    15800 2100
+	1    0    0    -1
+$EndComp
 $Comp
 L Device:C C101
@@
 	1    0    0    -1
 $EndComp
-Connection ~ 15200 1100
-Wire Wire Line
-	15200 1100 15300 1100
 Wire Wire Line
 	13850 1100 14500 1100
@@
 Connection ~ 14500 1100
 Wire Wire Line
-	14500 1100 15200 1100
-Wire Wire Line
 	13200 1350 13200 1200
 Connection ~ 13200 1200
@@
 L power:+5V #PWR0252
 U 1 1 60E766EA
-P 15300 1050
-F 0 "#PWR0252" H 15300 900 50  0001 C CNN
-F 1 "+5V" H 15315 1223 50  0000 C CNN
-F 2 "" H 15300 1050 50  0001 C CNN
-F 3 "" H 15300 1050 50  0001 C CNN
-	1    15300 1050
+P 15800 1100
+F 0 "#PWR0252" H 15800 950 50  0001 C CNN
+F 1 "+5V" H 15815 1273 50  0000 C CNN
+F 2 "" H 15800 1100 50  0001 C CNN
+F 3 "" H 15800 1100 50  0001 C CNN
+	1    15800 1100
 	1    0    0    -1
 $EndComp
@@
 	15800 1650 15800 2100
 Wire Wire Line
-	15800 2100 15200 2100
-Wire Wire Line
-	15300 1100 15800 1100
-Wire Wire Line
 	15800 1100 15800 1350
-Connection ~ 15300 1100
 $Comp
 L Device:Ferrite_Bead FB101
@@
 Text Notes 1800 10300 0    79   ~ 0
 28.37516MHz for PAL
+Connection ~ 15800 1100
+Connection ~ 15800 2100
+Wire Wire Line
+	14500 2100 15200 2100
+Wire Wire Line
+	14500 1100 15200 1100
+Connection ~ 15200 1100
+Wire Wire Line
+	15200 1100 15800 1100
+Connection ~ 15200 2100
+Wire Wire Line
+	15200 2100 15800 2100
 $EndSCHEMATC

Commit message: Add files via upload
Parts:
- U101: value FATTER_AGNUS -> 8372A_FATTER_AGNUS
Changed lines of the file:
@@
 P 8850 7150
 F 0 "U101" H 8850 4327 50  0000 C CNN
-F 1 "FATTER_AGNUS" H 8850 4236 50  0000 C CNN
+F 1 "8372A_FATTER_AGNUS" H 8850 4236 50  0000 C CNN
 F 2 "Package_LCC:PLCC-84_THT-Socket" H 8750 8700 50  0001 C CNN
 F 3 "http://www.ti.com/lit/gpn/sn7400" H 8750 8700 50  0001 C CNN
@@
 P 11150 1550
 F 0 "U101" H 10550 1550 50  0000 L CNN
-F 1 "FATTER_AGNUS" H 10300 1450 50  0000 L CNN
+F 1 "8372A_FATTER_AGNUS" H 10300 1450 50  0000 L CNN
 F 2 "Package_LCC:PLCC-84_THT-Socket" H 11150 1550 50  0001 C CNN
 F 3 "http://www.ti.com/lit/gpn/sn7400" H 11050 3100 50  0001 C CNN

Commit message: Add files via upload
Parts:
- added CX2: 0.1uF, Capacitor_SMD:C_1206_3216Metric, symbol Device:C
- added X2: 7C-28.63636MBB-T, Oscillator:Oscillator_SMD_SeikoEpson_SG8002LB-4Pin_5.0x3.2mm, symbol Oscillator:SG-5032CAN
Connections:
- net GND: now also CX2.2, X2.2 (GND)
- net at FB101.1, X1.8 (OUT): now also X2.3 (OUT)
- new net +3V3: CX2.1, X2.1 (~ST), X2.4 (VCC)
Other:
- note added: "OPTIONAL SMD CMOS XTAL. \nIF USED, DO NOT POPULATE \nX1 OR C110!"
- moved on the sheet: C110, FB101, X1
Changed lines of the file:
@@
 L Device:Ferrite_Bead FB101
 U 1 1 608A6DB7
-P 2900 9800
-F 0 "FB101" V 3082 9800 50  0000 C CNN
-F 1 "Ferrite_Bead" V 3083 9800 50  0001 C CNN
-F 2 "Capacitor_SMD:C_1206_3216Metric" V 2830 9800 50  0001 C CNN
-F 3 "~" H 2900 9800 50  0001 C CNN
-	1    2900 9800
-	0    -1   -1   0
+P 2750 9650
+F 0 "FB101" V 2932 9650 50  0000 C CNN
+F 1 "Ferrite_Bead" V 2933 9650 50  0001 C CNN
+F 2 "Capacitor_SMD:C_1206_3216Metric" V 2680 9650 50  0001 C CNN
+F 3 "~" H 2750 9650 50  0001 C CNN
+	1    2750 9650
+	1    0    0    -1
 $EndComp
 $Comp
 L Oscillator:ACO-xxxMHz X1
 U 1 1 608A92B4
-P 2450 9800
-F 0 "X1" H 2107 9846 50  0000 R CNN
-F 1 "28.63636MHz" H 2107 9755 50  0000 R CNN
-F 2 "Oscillator:Oscillator_DIP-14" H 2900 9450 50  0001 C CNN
-F 3 "" H 2350 9800 50  0001 C CNN
-	1    2450 9800
+P 2150 7350
+F 0 "X1" H 1807 7396 50  0000 R CNN
+F 1 "28.63636MHz" H 1807 7305 50  0000 R CNN
+F 2 "Oscillator:Oscillator_DIP-14" H 2600 7000 50  0001 C CNN
+F 3 "" H 2050 7350 50  0001 C CNN
+	1    2150 7350
 	1    0    0    -1
 $EndComp
@@
 L Device:C C110
 U 1 1 608AD688
-P 1200 9800
-F 0 "C110" H 1315 9846 50  0000 L CNN
-F 1 "0.1uF" H 1315 9755 50  0000 L CNN
-F 2 "Capacitor_SMD:C_1206_3216Metric" H 1238 9650 50  0001 C CNN
-F 3 "~" H 1200 9800 50  0001 C CNN
-	1    1200 9800
-	1    0    0    -1
-$EndComp
-Wire Wire Line
-	8150 9800 3050 9800
-Wire Wire Line
-	3050 9800 3050 9250
-Connection ~ 3050 9800
-Wire Wire Line
-	3050 9250 1950 9250
-Wire Wire Line
-	1200 9650 1200 9500
-Wire Wire Line
-	1200 9500 2450 9500
-Wire Wire Line
-	2450 10100 1200 10100
-Wire Wire Line
-	1200 10100 1200 9950
+P 900 7350
+F 0 "C110" H 1015 7396 50  0000 L CNN
+F 1 "0.1uF" H 1015 7305 50  0000 L CNN
+F 2 "Capacitor_SMD:C_1206_3216Metric" H 938 7200 50  0001 C CNN
+F 3 "~" H 900 7350 50  0001 C CNN
+	1    900  7350
+	1    0    0    -1
+$EndComp
+Wire Wire Line
+	900  7200 900  7050
+Wire Wire Line
+	900  7050 2150 7050
+Wire Wire Line
+	2150 7650 900  7650
+Wire Wire Line
+	900  7650 900  7500
 $Comp
 L power:GND #PWR0253
 U 1 1 608ED7B0
-P 1200 10100
-F 0 "#PWR0253" H 1200 9850 50  0001 C CNN
-F 1 "GND" H 1205 9927 50  0000 C CNN
-F 2 "" H 1200 10100 50  0001 C CNN
-F 3 "" H 1200 10100 50  0001 C CNN
-	1    1200 10100
-	1    0    0    -1
-$EndComp
-Connection ~ 1200 10100
-Text GLabel 1950 9250 0    50   Output ~ 0
+P 900 7650
+F 0 "#PWR0253" H 900 7400 50  0001 C CNN
+F 1 "GND" H 905 7477 50  0000 C CNN
+F 2 "" H 900 7650 50  0001 C CNN
+F 3 "" H 900 7650 50  0001 C CNN
+	1    900  7650
+	1    0    0    -1
+$EndComp
+Connection ~ 900  7650
+Text GLabel 1050 9800 0    50   Output ~ 0
 28M
 $Comp
 L power:+5V #PWR0254
 U 1 1 608FAF04
-P 1200 9500
-F 0 "#PWR0254" H 1200 9350 50  0001 C CNN
-F 1 "+5V" H 1215 9673 50  0000 C CNN
-F 2 "" H 1200 9500 50  0001 C CNN
-F 3 "" H 1200 9500 50  0001 C CNN
-	1    1200 9500
-	1    0    0    -1
-$EndComp
-Connection ~ 1200 9500
+P 900 7050
+F 0 "#PWR0254" H 900 6900 50  0001 C CNN
+F 1 "+5V" H 915 7223 50  0000 C CNN
+F 2 "" H 900 7050 50  0001 C CNN
+F 3 "" H 900 7050 50  0001 C CNN
+	1    900  7050
+	1    0    0    -1
+$EndComp
+Connection ~ 900  7050
 Wire Wire Line
 	8150 9700 6550 9700
@@
 Wire Wire Line
 	13700 6200 14000 6200
-Text Notes 1800 10300 0    79   ~ 0
+Text Notes 1200 6900 0    79   ~ 0
 28.37516MHz for PAL
 Connection ~ 15800 1100
@@
 Wire Wire Line
 	15200 2100 15800 2100
+$Comp
+L Oscillator:SG-5032CAN X2
+U 1 1 607A3CCE
+P 1650 8500
+F 0 "X2" H 1600 8100 50  0000 L CNN
+F 1 "7C-28.63636MBB-T" H 1300 8000 50  0000 L CNN
+F 2 "Oscillator:Oscillator_SMD_SeikoEpson_SG8002LB-4Pin_5.0x3.2mm" H 2350 8150 50  0001 C CNN
+F 3 "https://support.epson.biz/td/api/doc_check.php?dl=brief_SG5032CAN&lang=en" H 1550 8500 50  0001 C CNN
+	1    1650 8500
+	1    0    0    -1
+$EndComp
+Wire Wire Line
+	1050 9800 2750 9800
+Wire Wire Line
+	2750 9800 8150 9800
+Wire Wire Line
+	1350 8500 1350 8200
+Wire Wire Line
+	1350 8200 1650 8200
+Wire Wire Line
+	1950 8500 2750 8500
+Wire Wire Line
+	2750 8500 2750 9500
+Connection ~ 2750 8500
+$Comp
+L power:+3.3V #PWR0178
+U 1 1 60810017
+P 900 8200
+F 0 "#PWR0178" H 900 8050 50  0001 C CNN
+F 1 "+3.3V" H 915 8373 50  0000 C CNN
+F 2 "" H 900 8200 50  0001 C CNN
+F 3 "" H 900 8200 50  0001 C CNN
+	1    900  8200
+	1    0    0    -1
+$EndComp
+$Comp
+L Device:C CX2
+U 1 1 60810704
+P 900 8500
+F 0 "CX2" H 1015 8546 50  0000 L CNN
+F 1 "0.1uF" H 1015 8455 50  0000 L CNN
+F 2 "Capacitor_SMD:C_1206_3216Metric" H 938 8350 50  0001 C CNN
+F 3 "~" H 900 8500 50  0001 C CNN
+	1    900  8500
+	1    0    0    -1
+$EndComp
+Wire Wire Line
+	1650 8800 900  8800
+Wire Wire Line
+	900  8800 900  8650
+Wire Wire Line
+	900  8200 900  8350
+Wire Wire Line
+	1350 8200 900  8200
+Connection ~ 1350 8200
+Connection ~ 900  8200
+$Comp
+L power:GND #PWR0179
+U 1 1 6082C839
+P 900 8800
+F 0 "#PWR0179" H 900 8550 50  0001 C CNN
+F 1 "GND" H 905 8627 50  0000 C CNN
+F 2 "" H 900 8800 50  0001 C CNN
+F 3 "" H 900 8800 50  0001 C CNN
+	1    900  8800
+	1    0    0    -1
+$EndComp
+Connection ~ 900  8800
+Wire Notes Line
+	700  7950 700  9400
+Wire Notes Line
+	700  9400 2250 9400
+Wire Notes Line
+	2250 9400 2250 7950
+Wire Notes Line
+	2250 7950 700  7950
+Text Notes 800  9350 0    50   ~ 0
+OPTIONAL SMD CMOS XTAL. \nIF USED, DO NOT POPULATE \nX1 OR C110!
+Wire Wire Line
+	2450 7350 2750 7350
+Wire Wire Line
+	2750 7350 2750 8500
+Connection ~ 2750 9800
 $EndSCHEMATC

Commit message: Add files via upload
Changed lines of the file:
@@
 Wire Wire Line
 	8150 9600 5950 9600
-Text GLabel 5250 9600 0    50   Output ~ 0
+Text GLabel 5250 9600 0    50   Input ~ 0
 _XCLKEN
-Text GLabel 5250 9700 0    50   Output ~ 0
+Text GLabel 5250 9700 0    50   Input ~ 0
 XCLK
 $Comp

Commit message: Add files via upload
Other:
- note added: "Agnus\nAmiga 2000 EATX"
Changed lines of the file:
@@
 	2750 7350 2750 8500
 Connection ~ 2750 9800
+Text Notes 12300 9850 0    197  ~ 0
+Agnus\nAmiga 2000 EATX
 $EndSCHEMATC

Commit message: Add files via upload
Parts:
- C415: footprint Capacitor_SMD:CP_Elec_6.3x5.8 -> Capacitor_SMD:CP_Elec_4x5.8
Changed lines of the file:
@@
 F 0 "C415" H 12168 1596 50  0000 L CNN
 F 1 "4.7uF" H 12168 1505 50  0000 L CNN
-F 2 "Capacitor_SMD:CP_Elec_6.3x5.8" H 12088 1400 50  0001 C CNN
+F 2 "Capacitor_SMD:CP_Elec_4x5.8" H 12088 1400 50  0001 C CNN
 F 3 "~" H 12050 1550 50  0001 C CNN
 	1    12050 1550

Commit message: Add files via upload
Parts:
- U107: value 74LS04 -> 74HCT04
- U302: value 74LS32 -> 74HCT32
- U900: value 74LS00 -> 74HCT00
Changed lines of the file:
@@
 P 12500 3350
 F 0 "U107" H 12500 3667 50  0000 C CNN
-F 1 "74LS04" H 12500 3576 50  0000 C CNN
+F 1 "74HCT04" H 12500 3576 50  0000 C CNN
 F 2 "Package_SO:SOIC-14_3.9x8.7mm_P1.27mm" H 12500 3350 50  0001 C CNN
 F 3 "http://www.ti.com/lit/gpn/sn7400" H 12500 3350 50  0001 C CNN
@@
 P 12100 3800
 F 0 "U107" H 12100 4117 50  0000 C CNN
-F 1 "74LS04" H 12100 4026 50  0000 C CNN
+F 1 "74HCT04" H 12100 4026 50  0000 C CNN
 F 2 "Package_SO:SOIC-14_3.9x8.7mm_P1.27mm" H 12100 3800 50  0001 C CNN
 F 3 "http://www.ti.com/lit/gpn/sn7400" H 12100 3800 50  0001 C CNN
@@
 P 12550 4600
 F 0 "U107" H 12550 4917 50  0000 C CNN
-F 1 "74LS04" H 12550 4826 50  0000 C CNN
+F 1 "74HCT04" H 12550 4826 50  0000 C CNN
 F 2 "Package_SO:SOIC-14_3.9x8.7mm_P1.27mm" H 12550 4600 50  0001 C CNN
 F 3 "http://www.ti.com/lit/gpn/sn7400" H 12550 4600 50  0001 C CNN
@@
 P 12150 5050
 F 0 "U107" H 12150 5367 50  0000 C CNN
-F 1 "74LS04" H 12150 5276 50  0000 C CNN
+F 1 "74HCT04" H 12150 5276 50  0000 C CNN
 F 2 "Package_SO:SOIC-14_3.9x8.7mm_P1.27mm" H 12150 5050 50  0001 C CNN
 F 3 "http://www.ti.com/lit/gpn/sn7400" H 12150 5050 50  0001 C CNN
@@
 P 12550 5650
 F 0 "U107" H 12550 5967 50  0000 C CNN
-F 1 "74LS04" H 12550 5876 50  0000 C CNN
+F 1 "74HCT04" H 12550 5876 50  0000 C CNN
 F 2 "Package_SO:SOIC-14_3.9x8.7mm_P1.27mm" H 12550 5650 50  0001 C CNN
 F 3 "http://www.ti.com/lit/gpn/sn7400" H 12550 5650 50  0001 C CNN
@@
 P 12150 6200
 F 0 "U107" H 12150 6517 50  0000 C CNN
-F 1 "74LS04" H 12150 6426 50  0000 C CNN
+F 1 "74HCT04" H 12150 6426 50  0000 C CNN
 F 2 "Package_SO:SOIC-14_3.9x8.7mm_P1.27mm" H 12150 6200 50  0001 C CNN
 F 3 "http://www.ti.com/lit/gpn/sn7400" H 12150 6200 50  0001 C CNN
@@
 P 10850 8850
 F 0 "U302" H 10850 9175 50  0000 C CNN
-F 1 "74LS32" H 10850 9084 50  0000 C CNN
+F 1 "74HCT32" H 10850 9084 50  0000 C CNN
 F 2 "Package_SO:SOIC-14_3.9x8.7mm_P1.27mm" H 10850 8850 50  0001 C CNN
 F 3 "http://www.ti.com/lit/gpn/sn74LS32" H 10850 8850 50  0001 C CNN
@@
 P 6850 3900
 F 0 "U900" H 6850 3583 50  0000 C CNN
-F 1 "74LS00" H 6850 3674 50  0000 C CNN
+F 1 "74HCT00" H 6850 3674 50  0000 C CNN
 F 2 "Package_SO:SOIC-14_3.9x8.7mm_P1.27mm" H 6850 3900 50  0001 C CNN
 F 3 "http://www.ti.com/lit/gpn/sn7400" H 6850 3900 50  0001 C CNN
@@
 P 7700 3800
 F 0 "U900" H 7700 3483 50  0000 C CNN
-F 1 "74LS00" H 7700 3574 50  0000 C CNN
+F 1 "74HCT00" H 7700 3574 50  0000 C CNN
 F 2 "Package_SO:SOIC-14_3.9x8.7mm_P1.27mm" H 7700 3800 50  0001 C CNN
 F 3 "http://www.ti.com/lit/gpn/sn7400" H 7700 3800 50  0001 C CNN
@@
 P 13850 1600
 F 0 "U107" H 14080 1646 50  0000 L CNN
-F 1 "74LS04" H 14080 1555 50  0000 L CNN
+F 1 "74HCT04" H 14080 1555 50  0000 L CNN
 F 2 "Package_SO:SOIC-14_3.9x8.7mm_P1.27mm" H 13850 1600 50  0001 C CNN
 F 3 "http://www.ti.com/lit/gpn/sn7400" H 13850 1600 50  0001 C CNN
@@
 P 15200 1600
 F 0 "U900" H 15250 1550 50  0000 R CNN
-F 1 "74LS00" H 15300 1650 50  0000 R CNN
+F 1 "74HCT00" H 15300 1650 50  0000 R CNN
 F 2 "Package_SO:SOIC-14_3.9x8.7mm_P1.27mm" H 15200 1600 50  0001 C CNN
 F 3 "http://www.ti.com/lit/gpn/sn7400" H 15200 1600 50  0001 C CNN
