File: 2000EATX-KiCAD/paula.sch (KiCad schematic (older format))
At the start: 77 parts, among them CN200 DB9_Male_Stack, CN205 AudioJack, Q200 MMBFJ211, Q201 MMBFJ211, Q202 MMBT3906, U200 PAULA, U202 74LS157, U204 LF347

Commit message: Add files via upload
Parts:
- added FB215: Ferrite_Bead, Capacitor_SMD:C_1206_3216Metric, symbol Device:Ferrite_Bead
- added R200: 1, Resistor_SMD:R_1206_3216Metric, symbol Device:R
- C204: value 0.1uF -> 0.01uF
- renumbered EMI236 to EMI235, EMI235 to EMI236
Connections:
- net +5V: now also FB215.1, R200.1; no longer C200.1, C225.1, F1.1, R209.1, U200.27 (VCC)
- net at C243.1, U204.1: now also C241.1, U204.2 (-)
- new net: F1.1, FB215.2
- new net +AUD: C200.1, C225.1, R200.2, R209.1, U200.27 (VCC)
Other:
- note added: "JOY"
- note added: "MOUSE"
- moved on the sheet: F1
Changed lines of the file:
@@
 $EndComp
 $Comp
-L Amiga-Library:C_Feedthrough EMI236
+L Amiga-Library:C_Feedthrough EMI235
 U 1 1 605DFACF
 P 4600 8000
-F 0 "EMI236" H 4600 8305 50  0000 C CNN
+F 0 "EMI235" H 4600 8305 50  0000 C CNN
 F 1 "100pF" H 4600 8214 50  0000 C CNN
 F 2 "AmigaFootprints:C_1206_3216_Feedthrough" V 4600 8000 50  0001 C CNN
@@
 $EndComp
 $Comp
-L Amiga-Library:C_Feedthrough EMI235
+L Amiga-Library:C_Feedthrough EMI236
 U 1 1 605E12EA
 P 4600 8500
-F 0 "EMI235" H 4600 8805 50  0000 C CNN
+F 0 "EMI236" H 4600 8805 50  0000 C CNN
 F 1 "100pF" H 4600 8714 50  0000 C CNN
 F 2 "AmigaFootprints:C_1206_3216_Feedthrough" V 4600 8500 50  0001 C CNN
@@
 L Device:Fuse F1
 U 1 1 60BA328F
-P 9250 8100
-F 0 "F1" V 9053 8100 50  0000 C CNN
-F 1 "4A" V 9144 8100 50  0000 C CNN
-F 2 "Fuse:Fuse_1206_3216Metric" V 9180 8100 50  0001 C CNN
-F 3 "~" H 9250 8100 50  0001 C CNN
-	1    9250 8100
+P 9100 8100
+F 0 "F1" V 8903 8100 50  0000 C CNN
+F 1 "4A" V 8994 8100 50  0000 C CNN
+F 2 "Fuse:Fuse_1206_3216Metric" V 9030 8100 50  0001 C CNN
+F 3 "~" H 9100 8100 50  0001 C CNN
+	1    9100 8100
 	0    1    1    0
 $EndComp
@@
 	1    0    0    -1
 $EndComp
-Wire Wire Line
-	9400 8100 9700 8100
 Connection ~ 9700 8100
-Wire Wire Line
-	9100 8100 8950 8100
 Text Label 8950 8100 2    50   ~ 0
 +5VMOUSE
 Wire Notes Line
-	8650 8650 10150 8650
+	8500 8650 10150 8650
 Wire Notes Line
 	10150 8650 10150 7500
 Wire Notes Line
-	10150 7500 8650 7500
+	10150 7500 8500 7500
 Wire Notes Line
-	8650 7500 8650 8650
+	8500 7500 8500 8650
 Text Notes 8850 7750 0    50   ~ 0
 MOUSE/JOY POWER
@@
 L power:+5V #PWR0276
 U 1 1 60C0532B
-P 2250 900
-F 0 "#PWR0276" H 2250 750 50  0001 C CNN
-F 1 "+5V" H 2265 1073 50  0000 C CNN
-F 2 "" H 2250 900 50  0001 C CNN
-F 3 "" H 2250 900 50  0001 C CNN
-	1    2250 900
+P 1850 900
+F 0 "#PWR0276" H 1850 750 50  0001 C CNN
+F 1 "+5V" H 1865 1073 50  0000 C CNN
+F 2 "" H 1850 900 50  0001 C CNN
+F 3 "" H 1850 900 50  0001 C CNN
+	1    1850 900
 	1    0    0    -1
 $EndComp
@@
 Text GLabel 3100 1900 2    50   Input ~ 0
 _DKRD
-Text GLabel 3100 2100 2    50   Input ~ 0
+Text GLabel 3100 2100 2    50   Output ~ 0
 _DKWD
 Text GLabel 3100 2300 2    50   Output ~ 0
@@
 	9650 1850 10500 1850
 Wire Wire Line
-	10500 1850 10500 950
+	10500 1850 10500 1550
 Wire Wire Line
 	10500 950  8350 950
@@
 Connection ~ 10700 8600
 Wire Wire Line
-	10250 1550 10600 1550
+	10250 1550 10500 1550
 $Comp
 L Device:CP C243
@@
 P 8700 6100
 F 0 "C204" H 8815 6146 50  0000 L CNN
-F 1 "0.1uF" H 8815 6055 50  0000 L CNN
+F 1 "0.01uF" H 8815 6055 50  0000 L CNN
 F 2 "Capacitor_SMD:C_1206_3216Metric" H 8738 5950 50  0001 C CNN
 F 3 "~" H 8700 6100 50  0001 C CNN
@@
 Wire Wire Line
 	3000 8550 4200 8550
+Text Notes 6800 8350 0    50   ~ 0
+MOUSE
+Text Notes 6800 10050 0    50   ~ 0
+JOY
+$Comp
+L Device:Ferrite_Bead FB215
+U 1 1 609130CC
+P 9400 8100
+F 0 "FB215" V 9126 8100 50  0000 C CNN
+F 1 "Ferrite_Bead" V 9217 8100 50  0000 C CNN
+F 2 "Capacitor_SMD:C_1206_3216Metric" V 9330 8100 50  0001 C CNN
+F 3 "~" H 9400 8100 50  0001 C CNN
+	1    9400 8100
+	0    1    1    0
+$EndComp
+Wire Wire Line
+	9550 8100 9700 8100
+$Comp
+L Device:R R200
+U 1 1 60985958
+P 2100 900
+F 0 "R200" H 2170 946 50  0000 L CNN
+F 1 "1" H 2170 855 50  0000 L CNN
+F 2 "Resistor_SMD:R_1206_3216Metric" V 2030 900 50  0001 C CNN
+F 3 "~" H 2100 900 50  0001 C CNN
+	1    2100 900
+	0    -1   -1   0
+$EndComp
+Wire Wire Line
+	1850 900  1950 900
+Connection ~ 10500 1550
+Wire Wire Line
+	10500 1550 10500 950
+Wire Wire Line
+	10500 1550 10600 1550
 $EndSCHEMATC

Commit message: Add files via upload
Parts:
- added D200: S1MWF-7, Diode_SMD:D_SOD-123F, symbol Diode:1N4001
Connections:
- net +5VMOUSE: now also D200.1 (K); no longer F1.2
- new net: D200.2 (A), F1.2
Other:
- note added: "Paula\nAmiga 2000 EATX"
- note removed: "PAULA"
- moved on the sheet: C218, C219, C224, F1, FB215, R209, R210
Changed lines of the file:
@@
 L power:GND #PWR0272
 U 1 1 60BA1AC2
-P 9700 8400
-F 0 "#PWR0272" H 9700 8150 50  0001 C CNN
-F 1 "GND" H 9705 8227 50  0000 C CNN
-F 2 "" H 9700 8400 50  0001 C CNN
-F 3 "" H 9700 8400 50  0001 C CNN
-	1    9700 8400
+P 10300 8050
+F 0 "#PWR0272" H 10300 7800 50  0001 C CNN
+F 1 "GND" H 10305 7877 50  0000 C CNN
+F 2 "" H 10300 8050 50  0001 C CNN
+F 3 "" H 10300 8050 50  0001 C CNN
+	1    10300 8050
 	1    0    0    -1
 $EndComp
@@
 L Device:Fuse F1
 U 1 1 60BA328F
-P 9100 8100
-F 0 "F1" V 8903 8100 50  0000 C CNN
-F 1 "4A" V 8994 8100 50  0000 C CNN
-F 2 "Fuse:Fuse_1206_3216Metric" V 9030 8100 50  0001 C CNN
-F 3 "~" H 9100 8100 50  0001 C CNN
-	1    9100 8100
+P 9700 7750
+F 0 "F1" V 9503 7750 50  0000 C CNN
+F 1 "4A" V 9594 7750 50  0000 C CNN
+F 2 "Fuse:Fuse_1206_3216Metric" V 9630 7750 50  0001 C CNN
+F 3 "~" H 9700 7750 50  0001 C CNN
+	1    9700 7750
 	0    1    1    0
 $EndComp
@@
 L power:+5V #PWR0273
 U 1 1 60BA4681
-P 9700 7950
-F 0 "#PWR0273" H 9700 7800 50  0001 C CNN
-F 1 "+5V" H 9715 8123 50  0000 C CNN
-F 2 "" H 9700 7950 50  0001 C CNN
-F 3 "" H 9700 7950 50  0001 C CNN
-	1    9700 7950
+P 10300 7600
+F 0 "#PWR0273" H 10300 7450 50  0001 C CNN
+F 1 "+5V" H 10315 7773 50  0000 C CNN
+F 2 "" H 10300 7600 50  0001 C CNN
+F 3 "" H 10300 7600 50  0001 C CNN
+	1    10300 7600
 	1    0    0    -1
 $EndComp
@@
 L Device:C C218
 U 1 1 60BA6BF5
-P 9700 8250
-F 0 "C218" H 9815 8296 50  0000 L CNN
-F 1 "0.1uF" H 9815 8205 50  0000 L CNN
-F 2 "Capacitor_SMD:C_1206_3216Metric" H 9738 8100 50  0001 C CNN
-F 3 "~" H 9700 8250 50  0001 C CNN
-	1    9700 8250
-	1    0    0    -1
-$EndComp
-Connection ~ 9700 8100
-Text Label 8950 8100 2    50   ~ 0
+P 10300 7900
+F 0 "C218" H 10415 7946 50  0000 L CNN
+F 1 "0.1uF" H 10415 7855 50  0000 L CNN
+F 2 "Capacitor_SMD:C_1206_3216Metric" H 10338 7750 50  0001 C CNN
+F 3 "~" H 10300 7900 50  0001 C CNN
+	1    10300 7900
+	1    0    0    -1
+$EndComp
+Connection ~ 10300 7750
+Text Label 9250 7750 2    50   ~ 0
 +5VMOUSE
 Wire Notes Line
-	8500 8650 10150 8650
+	8700 8300 10750 8300
 Wire Notes Line
-	10150 8650 10150 7500
+	10750 8300 10750 7150
 Wire Notes Line
-	10150 7500 8500 7500
+	10750 7150 8700 7150
 Wire Notes Line
-	8500 7500 8500 8650
-Text Notes 8850 7750 0    50   ~ 0
+	8700 7150 8700 8300
+Text Notes 9450 7400 0    50   ~ 0
 MOUSE/JOY POWER
 Wire Wire Line
-	9700 8100 9700 7950
+	10300 7750 10300 7600
 Wire Wire Line
 	2500 8250 2700 8250
@@
 Text GLabel 3100 3700 2    50   Input ~ 0
 _INT2
-Text Notes 13300 9550 2    197  ~ 0
-PAULA
+Text Notes 12300 9850 0    197  ~ 0
+Paula\nAmiga 2000 EATX
 $Comp
 L Amiga-Library:+AUD #PWR0279
 U 1 1 60C49AD6
-P 10700 7700
-F 0 "#PWR0279" H 10700 7550 50  0001 C CNN
-F 1 "+AUD" H 10715 7873 50  0000 C CNN
-F 2 "" H 10700 7700 50  0001 C CNN
-F 3 "" H 10700 7700 50  0001 C CNN
-	1    10700 7700
+P 13800 5800
+F 0 "#PWR0279" H 13800 5650 50  0001 C CNN
+F 1 "+AUD" H 13815 5973 50  0000 C CNN
+F 2 "" H 13800 5800 50  0001 C CNN
+F 3 "" H 13800 5800 50  0001 C CNN
+	1    13800 5800
 	1    0    0    -1
 $EndComp
@@
 L Device:R R209
 U 1 1 60C4A170
-P 10700 7850
-F 0 "R209" H 10770 7896 50  0000 L CNN
-F 1 "1.2k" H 10770 7805 50  0000 L CNN
-F 2 "Resistor_SMD:R_1206_3216Metric" V 10630 7850 50  0001 C CNN
-F 3 "~" H 10700 7850 50  0001 C CNN
-	1    10700 7850
+P 13800 5950
+F 0 "R209" H 13870 5996 50  0000 L CNN
+F 1 "1.2k" H 13870 5905 50  0000 L CNN
+F 2 "Resistor_SMD:R_1206_3216Metric" V 13730 5950 50  0001 C CNN
+F 3 "~" H 13800 5950 50  0001 C CNN
+	1    13800 5950
 	1    0    0    -1
 $EndComp
@@
 L Device:R R210
 U 1 1 60C4A471
-P 10700 8300
-F 0 "R210" H 10770 8346 50  0000 L CNN
-F 1 "1.2k" H 10770 8255 50  0000 L CNN
-F 2 "Resistor_SMD:R_1206_3216Metric" V 10630 8300 50  0001 C CNN
-F 3 "~" H 10700 8300 50  0001 C CNN
-	1    10700 8300
+P 13800 6400
+F 0 "R210" H 13870 6446 50  0000 L CNN
+F 1 "1.2k" H 13870 6355 50  0000 L CNN
+F 2 "Resistor_SMD:R_1206_3216Metric" V 13730 6400 50  0001 C CNN
+F 3 "~" H 13800 6400 50  0001 C CNN
+	1    13800 6400
 	1    0    0    -1
 $EndComp
@@
 L Amiga-Library:AUDIO #PWR0280
 U 1 1 60C4ACCC
-P 10700 8600
-F 0 "#PWR0280" H 10700 8350 50  0001 C CNN
-F 1 "AUDIO" H 10705 8427 50  0000 C CNN
-F 2 "" H 10700 8600 50  0001 C CNN
-F 3 "" H 10700 8600 50  0001 C CNN
-	1    10700 8600
+P 13800 6700
+F 0 "#PWR0280" H 13800 6450 50  0001 C CNN
+F 1 "AUDIO" H 13805 6527 50  0000 C CNN
+F 2 "" H 13800 6700 50  0001 C CNN
+F 3 "" H 13800 6700 50  0001 C CNN
+	1    13800 6700
 	1    0    0    -1
 $EndComp
@@
 L Device:C C219
 U 1 1 60C4B08C
-P 11050 8300
-F 0 "C219" H 11165 8346 50  0000 L CNN
-F 1 "0.22uF" H 11165 8255 50  0000 L CNN
-F 2 "Capacitor_SMD:C_1206_3216Metric" H 11088 8150 50  0001 C CNN
-F 3 "~" H 11050 8300 50  0001 C CNN
-	1    11050 8300
+P 14150 6400
+F 0 "C219" H 14265 6446 50  0000 L CNN
+F 1 "0.22uF" H 14265 6355 50  0000 L CNN
+F 2 "Capacitor_SMD:C_1206_3216Metric" H 14188 6250 50  0001 C CNN
+F 3 "~" H 14150 6400 50  0001 C CNN
+	1    14150 6400
 	1    0    0    -1
 $EndComp
@@
 L Device:CP C224
 U 1 1 60C4C156
-P 11600 8300
-F 0 "C224" H 11718 8346 50  0000 L CNN
-F 1 "4.7uF" H 11718 8255 50  0000 L CNN
-F 2 "Capacitor_SMD:CP_Elec_6.3x5.8" H 11638 8150 50  0001 C CNN
-F 3 "~" H 11600 8300 50  0001 C CNN
-	1    11600 8300
-	1    0    0    -1
-$EndComp
-Wire Wire Line
-	10700 8000 11050 8000
-Connection ~ 10700 8000
-Wire Wire Line
-	10700 8600 11050 8600
-Wire Wire Line
-	11600 8600 11600 8450
-Wire Wire Line
-	11600 8150 11600 8000
-Connection ~ 11600 8000
-Wire Wire Line
-	11600 8000 12100 8000
-Wire Wire Line
-	11050 8150 11050 8000
-Connection ~ 11050 8000
-Wire Wire Line
-	11050 8000 11600 8000
-Wire Wire Line
-	11050 8450 11050 8600
-Connection ~ 11050 8600
-Wire Wire Line
-	11050 8600 11600 8600
+P 14700 6400
+F 0 "C224" H 14818 6446 50  0000 L CNN
+F 1 "4.7uF" H 14818 6355 50  0000 L CNN
+F 2 "Capacitor_SMD:CP_Elec_6.3x5.8" H 14738 6250 50  0001 C CNN
+F 3 "~" H 14700 6400 50  0001 C CNN
+	1    14700 6400
+	1    0    0    -1
+$EndComp
+Wire Wire Line
+	13800 6100 14150 6100
+Connection ~ 13800 6100
+Wire Wire Line
+	13800 6700 14150 6700
+Wire Wire Line
+	14700 6700 14700 6550
+Wire Wire Line
+	14700 6250 14700 6100
+Connection ~ 14700 6100
+Wire Wire Line
+	14700 6100 15200 6100
+Wire Wire Line
+	14150 6250 14150 6100
+Connection ~ 14150 6100
+Wire Wire Line
+	14150 6100 14700 6100
+Wire Wire Line
+	14150 6550 14150 6700
+Connection ~ 14150 6700
+Wire Wire Line
+	14150 6700 14700 6700
 Wire Notes Line
-	12750 8900 12750 7400
+	15850 7000 15850 5500
 Wire Notes Line
-	12750 7400 10400 7400
+	15850 5500 13500 5500
 Wire Notes Line
-	10400 7400 10400 8900
+	13500 5500 13500 7000
 Wire Notes Line
-	10400 8900 12750 8900
-Text Notes 11700 7750 2    50   ~ 0
+	13500 7000 15850 7000
+Text Notes 14800 5850 2    50   ~ 0
 Audio Vref
 $Comp
@@
 $EndComp
 Wire Wire Line
-	10700 8000 10700 8150
-Wire Wire Line
-	10700 8450 10700 8600
-Connection ~ 10700 8600
+	13800 6100 13800 6250
+Wire Wire Line
+	13800 6550 13800 6700
+Connection ~ 13800 6700
 Wire Wire Line
 	10250 1550 10500 1550
@@
 L Amiga-Library:VREF #VREF0103
 U 1 1 609668FD
-P 12100 8000
-F 0 "#VREF0103" H 12100 7850 50  0001 C CNN
-F 1 "VREF" H 12115 8173 50  0000 C CNN
-F 2 "" H 12100 8000 50  0001 C CNN
-F 3 "" H 12100 8000 50  0001 C CNN
-	1    12100 8000
+P 15200 6100
+F 0 "#VREF0103" H 15200 5950 50  0001 C CNN
+F 1 "VREF" H 15215 6273 50  0000 C CNN
+F 2 "" H 15200 6100 50  0001 C CNN
+F 3 "" H 15200 6100 50  0001 C CNN
+	1    15200 6100
 	1    0    0    -1
 $EndComp
@@
 L Device:Ferrite_Bead FB215
 U 1 1 609130CC
-P 9400 8100
-F 0 "FB215" V 9126 8100 50  0000 C CNN
-F 1 "Ferrite_Bead" V 9217 8100 50  0000 C CNN
-F 2 "Capacitor_SMD:C_1206_3216Metric" V 9330 8100 50  0001 C CNN
-F 3 "~" H 9400 8100 50  0001 C CNN
-	1    9400 8100
+P 10000 7750
+F 0 "FB215" V 9726 7750 50  0000 C CNN
+F 1 "Ferrite_Bead" V 9817 7750 50  0000 C CNN
+F 2 "Capacitor_SMD:C_1206_3216Metric" V 9930 7750 50  0001 C CNN
+F 3 "~" H 10000 7750 50  0001 C CNN
+	1    10000 7750
 	0    1    1    0
 $EndComp
 Wire Wire Line
-	9550 8100 9700 8100
+	10150 7750 10300 7750
 $Comp
 L Device:R R200
@@
 Wire Wire Line
 	10500 1550 10600 1550
+$Comp
+L Diode:1N4001 D200
+U 1 1 60B1681A
+P 9400 7750
+F 0 "D200" H 9400 7967 50  0000 C CNN
+F 1 "S1MWF-7" H 9400 7876 50  0000 C CNN
+F 2 "Diode_SMD:D_SOD-123F" H 9400 7575 50  0001 C CNN
+F 3 "" H 9400 7750 50  0001 C CNN
+	1    9400 7750
+	1    0    0    -1
+$EndComp
 $EndSCHEMATC

Commit message: Add files via upload
Connections:
- net +5VMOUSE: now also F1.2; no longer D200.1 (K)
- net at FB215.2: now also D200.2 (A); no longer F1.1
- new net: D200.1 (K), F1.1
Other:
- moved on the sheet: D200, F1
Changed lines of the file:
@@
 L Device:Fuse F1
 U 1 1 60BA328F
-P 9700 7750
-F 0 "F1" V 9503 7750 50  0000 C CNN
-F 1 "4A" V 9594 7750 50  0000 C CNN
-F 2 "Fuse:Fuse_1206_3216Metric" V 9630 7750 50  0001 C CNN
-F 3 "~" H 9700 7750 50  0001 C CNN
-	1    9700 7750
+P 9400 7750
+F 0 "F1" V 9203 7750 50  0000 C CNN
+F 1 "4A" V 9294 7750 50  0000 C CNN
+F 2 "Fuse:Fuse_1206_3216Metric" V 9330 7750 50  0001 C CNN
+F 3 "~" H 9400 7750 50  0001 C CNN
+	1    9400 7750
 	0    1    1    0
 $EndComp
@@
 L Diode:1N4001 D200
 U 1 1 60B1681A
-P 9400 7750
-F 0 "D200" H 9400 7967 50  0000 C CNN
-F 1 "S1MWF-7" H 9400 7876 50  0000 C CNN
-F 2 "Diode_SMD:D_SOD-123F" H 9400 7575 50  0001 C CNN
-F 3 "" H 9400 7750 50  0001 C CNN
-	1    9400 7750
-	1    0    0    -1
-$EndComp
+P 9700 7750
+F 0 "D200" H 9700 7967 50  0000 C CNN
+F 1 "S1MWF-7" H 9700 7876 50  0000 C CNN
+F 2 "Diode_SMD:D_SOD-123F" H 9700 7575 50  0001 C CNN
+F 3 "" H 9700 7750 50  0001 C CNN
+	1    9700 7750
+	1    0    0    -1
+$EndComp

Commit message: Add files via upload
Parts:
- removed C230, C240: 0.1uF, Capacitor_SMD:C_1206_3216Metric, symbol Device:C
Changed lines of the file:
@@
 Audio Vref
-$Comp
-L Device:C C240
-U 1 1 60C8AE4C
-P 7000 1200
-F 0 "C240" H 7115 1246 50  0000 L CNN
-F 1 "0.1uF" H 7115 1155 50  0000 L CNN
-F 2 "Capacitor_SMD:C_1206_3216Metric" H 7038 1050 50  0001 C CNN
-F 3 "~" H 7000 1200 50  0001 C CNN
-	1    7000 1200
-	1    0    0    -1
-$EndComp
 $Comp
 L Device:R R240
@@
 	1    0    0    -1
 $EndComp
-Wire Wire Line
-	7450 1350 7000 1350
-Connection ~ 7000 1350
-Wire Wire Line
-	7000 1350 6550 1350
-Wire Wire Line
-	6550 1050 7000 1050
-Connection ~ 7000 1050
-Wire Wire Line
-	7000 1050 8050 1050
 Wire Wire Line
 	7450 1550 7350 1550
@@
 	1    0    0    -1
 $EndComp
-$Comp
-L Device:C C230
-U 1 1 60604EE4
-P 7800 4250
-F 0 "C230" H 7915 4296 50  0000 L CNN
-F 1 "0.1uF" H 7915 4205 50  0000 L CNN
-F 2 "Capacitor_SMD:C_1206_3216Metric" H 7838 4100 50  0001 C CNN
-F 3 "~" H 7800 4250 50  0001 C CNN
-	1    7800 4250
-	1    0    0    -1
-$EndComp
-Wire Wire Line
-	8350 4400 7800 4400
 Connection ~ 7400 4400
-Connection ~ 7800 4400
-Wire Wire Line
-	7800 4400 7400 4400
-Wire Wire Line
-	7400 4100 7800 4100
 Wire Wire Line
 	8950 4100 8950 4500
-Connection ~ 7800 4100
-Wire Wire Line
-	7800 4100 8950 4100
 Wire Wire Line
 	8350 4600 8150 4600
@@
 	1    0    0    -1
 $EndComp
+Wire Wire Line
+	7400 4100 8950 4100
+Wire Wire Line
+	7400 4400 8350 4400
+Wire Wire Line
+	6550 1050 8050 1050
+Wire Wire Line
+	6550 1350 7450 1350
 $EndSCHEMATC

Commit message: Add files via upload
Parts:
- C224: footprint Capacitor_SMD:CP_Elec_6.3x5.8 -> Capacitor_SMD:CP_Elec_4x5.8
- C225: footprint Capacitor_SMD:CP_Elec_6.3x5.8 -> Capacitor_SMD:CP_Elec_8x10
Changed lines of the file:
@@
 F 0 "C225" H 3068 1096 50  0000 L CNN
 F 1 "470uF" H 3068 1005 50  0000 L CNN
-F 2 "Capacitor_SMD:CP_Elec_6.3x5.8" H 2988 900 50  0001 C CNN
+F 2 "Capacitor_SMD:CP_Elec_8x10" H 2988 900 50  0001 C CNN
 F 3 "~" H 2950 1050 50  0001 C CNN
 	1    2950 1050
@@
 F 0 "C224" H 14818 6446 50  0000 L CNN
 F 1 "4.7uF" H 14818 6355 50  0000 L CNN
-F 2 "Capacitor_SMD:CP_Elec_6.3x5.8" H 14738 6250 50  0001 C CNN
+F 2 "Capacitor_SMD:CP_Elec_4x5.8" H 14738 6250 50  0001 C CNN
 F 3 "~" H 14700 6400 50  0001 C CNN
 	1    14700 6400

Commit message: Add files via upload
Parts:
- U202: value 74LS157 -> 74HCT157
Changed lines of the file:
@@
 P 2000 8850
 F 0 "U202" H 2000 7669 50  0000 C CNN
-F 1 "74LS157" H 2000 7760 50  0000 C CNN
+F 1 "74HCT157" H 2000 7760 50  0000 C CNN
 F 2 "Package_SO:SOIC-16_3.9x9.9mm_P1.27mm" H 2000 8850 50  0001 C CNN
 F 3 "http://www.ti.com/lit/gpn/sn74LS157" H 2000 8850 50  0001 C CNN
