File: 2000EATX-KiCAD/serial.sch (KiCad schematic (older format))
At the start: 52 parts, among them CN305 DB25_Stack_FemaleAndMale, CN306 POWER LED, Q300 MMBT3904, Q302 MMBT3906, U301 8520, U302 74LS32, U303 74LS08, U304 SN75188DR, U305 SN75189DR, U805 LM339

Commit message: Add files via upload
Parts:
- added C303: 0.1uF, Capacitor_SMD:C_1206_3216Metric, symbol Device:C
- added U?: 74LS08, symbol 74xx:74LS08
Connections:
- net +5V: now also C303.1, U?.14 (VCC)
- net GND: now also C303.2, U?.7 (GND)
Other:
- moved on the sheet: U304B
Changed lines of the file:
@@
 L Amiga-Library:SN75188DR U304
 U 2 1 6066C22E
-P 8100 9900
-F 0 "U304" H 8378 9921 50  0000 L CNN
-F 1 "SN75188DR" H 8378 9830 50  0000 L CNN
-F 2 "Package_SO:SOIC-14_3.9x8.7mm_P1.27mm" H 8050 9050 50  0001 C CNN
-F 3 "https://www.ti.com/lit/ds/symlink/mc1488.pdf?HQS=dis-dk-null-digikeymode-dsf-pf-null-wwe&ts=1616552868480" H 8100 9100 50  0001 C CNN
-	2    8100 9900
+P 6350 9750
+F 0 "U304" H 6628 9771 50  0000 L CNN
+F 1 "SN75188DR" H 6628 9680 50  0000 L CNN
+F 2 "Package_SO:SOIC-14_3.9x8.7mm_P1.27mm" H 6300 8900 50  0001 C CNN
+F 3 "https://www.ti.com/lit/ds/symlink/mc1488.pdf?HQS=dis-dk-null-digikeymode-dsf-pf-null-wwe&ts=1616552868480" H 6350 8950 50  0001 C CNN
+	2    6350 9750
 	1    0    0    -1
 $EndComp
@@
 L power:+12V #PWR0297
 U 1 1 60673697
-P 8100 9600
-F 0 "#PWR0297" H 8100 9450 50  0001 C CNN
-F 1 "+12V" H 8115 9773 50  0000 C CNN
-F 2 "" H 8100 9600 50  0001 C CNN
-F 3 "" H 8100 9600 50  0001 C CNN
-	1    8100 9600
+P 6350 9450
+F 0 "#PWR0297" H 6350 9300 50  0001 C CNN
+F 1 "+12V" H 6365 9623 50  0000 C CNN
+F 2 "" H 6350 9450 50  0001 C CNN
+F 3 "" H 6350 9450 50  0001 C CNN
+	1    6350 9450
 	1    0    0    -1
 $EndComp
@@
 L power:GND #PWR0298
 U 1 1 6067399F
-P 8100 10250
-F 0 "#PWR0298" H 8100 10000 50  0001 C CNN
-F 1 "GND" H 8105 10077 50  0000 C CNN
-F 2 "" H 8100 10250 50  0001 C CNN
-F 3 "" H 8100 10250 50  0001 C CNN
-	1    8100 10250
+P 6350 10100
+F 0 "#PWR0298" H 6350 9850 50  0001 C CNN
+F 1 "GND" H 6355 9927 50  0000 C CNN
+F 2 "" H 6350 10100 50  0001 C CNN
+F 3 "" H 6350 10100 50  0001 C CNN
+	1    6350 10100
 	1    0    0    -1
 $EndComp
@@
 	-1   0    0    1
 $EndComp
+$Comp
+L 74xx:74LS08 U?
+U 5 1 60A7C756
+P 8200 9750
+F 0 "U?" H 8200 10075 50  0000 C CNN
+F 1 "74LS08" H 8200 9984 50  0000 C CNN
+F 2 "" H 8200 9750 50  0001 C CNN
+F 3 "http://www.ti.com/lit/gpn/sn74LS08" H 8200 9750 50  0001 C CNN
+	5    8200 9750
+	1    0    0    -1
+$EndComp
+$Comp
+L Device:C C303
+U 1 1 60A965B1
+P 8650 9750
+F 0 "C303" H 8765 9796 50  0000 L CNN
+F 1 "0.1uF" H 8765 9705 50  0000 L CNN
+F 2 "Capacitor_SMD:C_1206_3216Metric" H 8688 9600 50  0001 C CNN
+F 3 "~" H 8650 9750 50  0001 C CNN
+	1    8650 9750
+	1    0    0    -1
+$EndComp
+Wire Wire Line
+	9400 9600 8650 9600
+Connection ~ 9400 9600
+Wire Wire Line
+	8200 9250 8650 9250
+Wire Wire Line
+	8650 9250 8650 9600
+Connection ~ 8650 9600
+Wire Wire Line
+	9400 10250 8650 10250
+Connection ~ 9400 10250
+Wire Wire Line
+	8650 9900 8650 10250
+Connection ~ 8650 10250
+Wire Wire Line
+	8650 10250 8200 10250
 $EndSCHEMATC

Commit message: Add files via upload
Parts:
- removed D802: 1N4148, Diode_SMD:D_SOD-323, symbol Diode:1N4148
- removed RRESET1: 1k, Resistor_SMD:R_1206_3216Metric, symbol Device:R
- added XU1: DS1813, Package_TO_SOT_SMD:SOT-23, symbol Amiga-Library:DS1813
- gave numbers to parts that had none: 1
- renumbered ATX-RESET1 to J9001
Connections:
- net +5V: now also XU1.2 (Vcc)
- net GND: now also J9001.2 (Pin_2), XU1.3 (GND)
- net _KBRST: no longer J9001.1 (Pin_1)
- net RESET: now reaches C814.1, R805.2, U805.10 (-), U805.2
- net RESET: now also J9001.1 (Pin_1), XU1.1 (/RST)
Other:
- note removed: "DELETE XU1. NO MODERN EQUIVALENT?\nTHIS IS THE ORIGINAL B2000 RESET CIRCUIT."
- moved on the sheet: C814, J9001, R805
Changed lines of the file:
@@
 Wire Wire Line
 	12000 2150 12150 2150
-$Comp
-L Diode:1N4148 D802
-U 1 1 609295DA
-P 12350 1900
-F 0 "D802" V 12304 1980 50  0000 L CNN
-F 1 "1N4148" V 12395 1980 50  0000 L CNN
-F 2 "Diode_SMD:D_SOD-323" H 12350 1725 50  0001 C CNN
-F 3 "https://assets.nexperia.com/documents/data-sheet/1N4148_1N4448.pdf" H 12350 1900 50  0001 C CNN
-F 4 "1N4148WSTR" V 12350 1900 50  0001 C CNN "pART"
-	1    12350 1900
-	0    1    1    0
-$EndComp
-Wire Wire Line
-	12350 2050 12350 2150
-Connection ~ 12350 2150
-Wire Wire Line
-	12350 2150 12600 2150
-Wire Wire Line
-	12150 2050 12150 2150
-Connection ~ 12150 2150
-Wire Wire Line
-	12150 2150 12350 2150
+Wire Wire Line
+	12250 2050 12250 2150
+Connection ~ 12250 2150
 $Comp
 L Device:R R805
 U 1 1 609496BA
-P 12150 1900
-F 0 "R805" V 11943 1900 50  0000 C CNN
-F 1 "1k" V 12034 1900 50  0000 C CNN
-F 2 "Resistor_SMD:R_1206_3216Metric" V 12080 1900 50  0001 C CNN
-F 3 "~" H 12150 1900 50  0001 C CNN
-	1    12150 1900
+P 12250 1900
+F 0 "R805" V 12350 1900 50  0000 C CNN
+F 1 "1k" V 12250 1900 50  0000 C CNN
+F 2 "Resistor_SMD:R_1206_3216Metric" V 12180 1900 50  0001 C CNN
+F 3 "~" H 12250 1900 50  0001 C CNN
+	1    12250 1900
 	1    0    0    -1
 $EndComp
@@
 L Device:CP C814
 U 1 1 60949F6D
-P 12150 2300
-F 0 "C814" H 12268 2346 50  0000 L CNN
-F 1 "22uF" H 12268 2255 50  0000 L CNN
-F 2 "Capacitor_SMD:CP_Elec_6.3x5.8" H 12188 2150 50  0001 C CNN
-F 3 "~" H 12150 2300 50  0001 C CNN
-	1    12150 2300
-	1    0    0    -1
-$EndComp
-Wire Wire Line
-	12350 1750 12150 1750
+P 12250 2300
+F 0 "C814" H 12368 2346 50  0000 L CNN
+F 1 "22uF" H 12368 2255 50  0000 L CNN
+F 2 "Capacitor_SMD:CP_Elec_6.3x5.8" H 12288 2150 50  0001 C CNN
+F 3 "~" H 12250 2300 50  0001 C CNN
+	1    12250 2300
+	1    0    0    -1
+$EndComp
 $Comp
 L power:+5V #PWR0324
 U 1 1 60957A19
-P 12150 1750
-F 0 "#PWR0324" H 12150 1600 50  0001 C CNN
-F 1 "+5V" H 12165 1923 50  0000 C CNN
-F 2 "" H 12150 1750 50  0001 C CNN
-F 3 "" H 12150 1750 50  0001 C CNN
-	1    12150 1750
-	1    0    0    -1
-$EndComp
-Connection ~ 12150 1750
-Text Notes 11250 1300 0    50   ~ 0
-DELETE XU1. NO MODERN EQUIVALENT?\nTHIS IS THE ORIGINAL B2000 RESET CIRCUIT.
+P 12250 1500
+F 0 "#PWR0324" H 12250 1350 50  0001 C CNN
+F 1 "+5V" H 12265 1673 50  0000 C CNN
+F 2 "" H 12250 1500 50  0001 C CNN
+F 3 "" H 12250 1500 50  0001 C CNN
+	1    12250 1500
+	1    0    0    -1
+$EndComp
 Wire Wire Line
 	12600 2350 12600 2650
@@
 POWER FAIL/RESET
 $Comp
-L Connector:Conn_01x02_Male ATX-RESET1
+L Connector:Conn_01x02_Male J9001
 U 1 1 60A28FC2
-P 15250 1450
-F 0 "ATX-RESET1" V 15312 1494 50  0000 L CNN
-F 1 "RESET" V 15403 1494 50  0000 L CNN
-F 2 "Connector_PinHeader_2.54mm:PinHeader_1x02_P2.54mm_Vertical" H 15250 1450 50  0001 C CNN
-F 3 "~" H 15250 1450 50  0001 C CNN
-	1    15250 1450
+P 12150 1000
+F 0 "J9001" V 12000 850 50  0000 L CNN
+F 1 "RESET" V 12100 850 50  0000 L CNN
+F 2 "Connector_PinHeader_2.54mm:PinHeader_1x02_P2.54mm_Vertical" H 12150 1000 50  0001 C CNN
+F 3 "~" H 12150 1000 50  0001 C CNN
+	1    12150 1000
 	0    1    1    0
-$EndComp
-Wire Wire Line
-	15150 1650 14950 1650
-$Comp
-L Device:R RRESET1
-U 1 1 60A56EBC
-P 14950 1800
-F 0 "RRESET1" V 14743 1800 50  0000 C CNN
-F 1 "1k" V 14834 1800 50  0000 C CNN
-F 2 "Resistor_SMD:R_1206_3216Metric" V 14880 1800 50  0001 C CNN
-F 3 "~" H 14950 1800 50  0001 C CNN
-	1    14950 1800
-	1    0    0    -1
 $EndComp
 $Comp
 L power:GND #PWR0326
 U 1 1 60A59CE8
-P 14950 1950
-F 0 "#PWR0326" H 14950 1700 50  0001 C CNN
-F 1 "GND" H 14955 1777 50  0000 C CNN
-F 2 "" H 14950 1950 50  0001 C CNN
-F 3 "" H 14950 1950 50  0001 C CNN
-	1    14950 1950
-	1    0    0    -1
-$EndComp
-Wire Wire Line
-	14650 2500 15250 2500
-Wire Wire Line
-	15250 1650 15250 2500
-Connection ~ 15250 2500
-Wire Wire Line
-	15250 2500 15650 2500
+P 13900 1400
+F 0 "#PWR0326" H 13900 1150 50  0001 C CNN
+F 1 "GND" H 13905 1227 50  0000 C CNN
+F 2 "" H 13900 1400 50  0001 C CNN
+F 3 "" H 13900 1400 50  0001 C CNN
+	1    13900 1400
+	1    0    0    -1
+$EndComp
 $Comp
 L power:GND #PWR0327
 U 1 1 60A7BF0B
-P 12150 2450
-F 0 "#PWR0327" H 12150 2200 50  0001 C CNN
-F 1 "GND" H 12155 2277 50  0000 C CNN
-F 2 "" H 12150 2450 50  0001 C CNN
-F 3 "" H 12150 2450 50  0001 C CNN
-	1    12150 2450
+P 12250 2450
+F 0 "#PWR0327" H 12250 2200 50  0001 C CNN
+F 1 "GND" H 12255 2277 50  0000 C CNN
+F 2 "" H 12250 2450 50  0001 C CNN
+F 3 "" H 12250 2450 50  0001 C CNN
+	1    12250 2450
 	1    0    0    -1
 $EndComp
@@
 $EndComp
 $Comp
-L 74xx:74LS08 U?
+L 74xx:74LS08 U303
 U 5 1 60A7C756
 P 8200 9750
-F 0 "U?" H 8200 10075 50  0000 C CNN
+F 0 "U303" H 8200 10075 50  0000 C CNN
 F 1 "74LS08" H 8200 9984 50  0000 C CNN
 F 2 "" H 8200 9750 50  0001 C CNN
@@
 Wire Wire Line
 	8650 10250 8200 10250
+$Comp
+L Amiga-Library:DS1813 XU1
+U 1 1 607B0B2C
+P 13000 1400
+F 0 "XU1" V 12635 1300 50  0000 C CNN
+F 1 "DS1813" V 12726 1300 50  0000 C CNN
+F 2 "Package_TO_SOT_SMD:SOT-23" H 13000 1400 50  0001 C CNN
+F 3 "" H 13000 1400 50  0001 C CNN
+	1    13000 1400
+	0    1    1    0
+$EndComp
+Wire Wire Line
+	14650 2500 15650 2500
+Wire Wire Line
+	12250 2150 12600 2150
+Wire Wire Line
+	12550 1500 12250 1500
+Wire Wire Line
+	12250 1500 12250 1750
+Connection ~ 12250 1500
+Wire Wire Line
+	13250 1400 13900 1400
+Wire Wire Line
+	12550 1300 12550 1200
+Wire Wire Line
+	12550 1200 12150 1200
+Wire Wire Line
+	12150 1200 12150 2150
+Connection ~ 12150 2150
+Wire Wire Line
+	12150 2150 12250 2150
+Connection ~ 12150 1200
+$Comp
+L power:GND #PWR0176
+U 1 1 6083E71B
+P 12050 1200
+F 0 "#PWR0176" H 12050 950 50  0001 C CNN
+F 1 "GND" H 12055 1027 50  0000 C CNN
+F 2 "" H 12050 1200 50  0001 C CNN
+F 3 "" H 12050 1200 50  0001 C CNN
+	1    12050 1200
+	1    0    0    -1
+$EndComp
+Text Label 12150 1200 0    50   ~ 0
+RESET
 $EndSCHEMATC

Commit message: Add files via upload
Parts:
- removed Q300: MMBT3904, Package_TO_SOT_SMD:SOT-23, symbol Transistor_BJT:MMBT3904
- added Q300: MMBT3904, Package_TO_SOT_SMD:SOT-23, symbol Transistor_BJT:2SC1815
- R802: value 1k -> 10k
- R805: value 1k -> 47k
- renumbered CN306 to J9002
Connections:
- net GND: now also C813.2, Q300.1 (E)
- net PSEL: now also Q300.2 (C)
- net at D300.1 (K), R305.1, R306.2: now also Q300.3 (B)
- net at C815.1, RN802.1 (R1.1), RN802.4 (R2.2)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: no longer C813.2
- net D0 renamed D8
- net D1 renamed D9
- net D2 renamed D10
- net D3 renamed D11
- net D4 renamed D12
- net D5 renamed D13
- net D6 renamed D14
- net D7 renamed D15
Changed lines of the file:
@@
 	1050 5300 1950 5300
 Text GLabel 1050 3900 0    50   BiDi ~ 0
-D7
+D15
 Text GLabel 1050 4000 0    50   BiDi ~ 0
-D6
+D14
 Text GLabel 1050 4100 0    50   BiDi ~ 0
-D5
+D13
 Text GLabel 1050 4200 0    50   BiDi ~ 0
-D4
+D12
 Text GLabel 1050 4300 0    50   BiDi ~ 0
-D3
+D11
 Text GLabel 1050 4400 0    50   BiDi ~ 0
-D2
+D10
 Text GLabel 1050 4500 0    50   BiDi ~ 0
-D1
+D9
 Text GLabel 1050 4600 0    50   BiDi ~ 0
-D0
+D8
 Text GLabel 1050 5000 0    50   Input ~ 0
 A11
@@
 Wire Wire Line
 	4050 9400 1100 9400
-Text GLabel 1100 8150 0    50   Input ~ 0
+Text GLabel 1100 8150 0    50   Output ~ 0
 _STEP
-Text GLabel 1100 8300 0    50   Input ~ 0
+Text GLabel 1100 8300 0    50   Output ~ 0
 DIR
-Text GLabel 1100 8450 0    50   Input ~ 0
+Text GLabel 1100 8450 0    50   Output ~ 0
 _SIDE
-Text GLabel 1100 8600 0    50   Input ~ 0
+Text GLabel 1100 8600 0    50   Output ~ 0
 _SEL0
-Text GLabel 1100 8800 0    50   Input ~ 0
+Text GLabel 1100 8800 0    50   Output ~ 0
 _SEL1
-Text GLabel 1100 9000 0    50   Input ~ 0
+Text GLabel 1100 9000 0    50   Output ~ 0
 _SEL2
-Text GLabel 1100 9200 0    50   Input ~ 0
+Text GLabel 1100 9200 0    50   Output ~ 0
 _SEL3
-Text GLabel 1100 9400 0    50   Input ~ 0
+Text GLabel 1100 9400 0    50   Output ~ 0
 _MTR
 Wire Wire Line
@@
 	7600 1800 8000 1800
 $Comp
-L Connector:Conn_01x02_Male CN306
+L Connector:Conn_01x02_Male J9002
 U 1 1 60649299
 P 8200 1800
-F 0 "CN306" H 8172 1732 50  0000 R CNN
+F 0 "J9002" H 8172 1732 50  0000 R CNN
 F 1 "POWER LED" H 8172 1823 50  0000 R CNN
 F 2 "Connector_PinHeader_2.54mm:PinHeader_1x02_P2.54mm_Vertical" H 8200 1800 50  0001 C CNN
@@
 	1    10400 8800
 	1    0    0    -1
-$EndComp
-$Comp
-L Transistor_BJT:MMBT3904 Q300
-U 1 1 6073DFBC
-P 9850 8950
-F 0 "Q300" H 10041 8996 50  0000 L CNN
-F 1 "MMBT3904" H 10041 8905 50  0000 L CNN
-F 2 "Package_TO_SOT_SMD:SOT-23" H 10050 8875 50  0001 L CIN
-F 3 "https://www.fairchildsemi.com/datasheets/2N/2N3904.pdf" H 9850 8950 50  0001 L CNN
-	1    9850 8950
-	-1   0    0    -1
 $EndComp
 $Comp
@@
 	1    0    0    -1
 $EndComp
-Connection ~ 10050 8950
 Wire Wire Line
 	10050 8950 10400 8950
@@
 P 11000 1900
 F 0 "R802" V 10793 1900 50  0000 C CNN
-F 1 "1k" V 10884 1900 50  0000 C CNN
+F 1 "10k" V 10884 1900 50  0000 C CNN
 F 2 "Resistor_SMD:R_1206_3216Metric" V 10930 1900 50  0001 C CNN
 F 3 "~" H 11000 1900 50  0001 C CNN
@@
 Wire Wire Line
 	11000 2050 11400 2050
-Wire Wire Line
-	11000 3050 10600 3050
 Connection ~ 10050 3050
 Wire Wire Line
@@
 $EndComp
 Wire Wire Line
-	11400 3050 11000 3050
-Connection ~ 11000 3050
-Wire Wire Line
 	12000 2150 12150 2150
 Wire Wire Line
@@
 P 12250 1900
 F 0 "R805" V 12350 1900 50  0000 C CNN
-F 1 "1k" V 12250 1900 50  0000 C CNN
+F 1 "47k" V 12250 1900 50  0000 C CNN
 F 2 "Resistor_SMD:R_1206_3216Metric" V 12180 1900 50  0001 C CNN
 F 3 "~" H 12250 1900 50  0001 C CNN
@@
 	11400 2250 11400 3050
 Wire Wire Line
-	11000 2350 11000 3050
-Wire Wire Line
 	10050 2150 10050 3050
 Connection ~ 10050 2150
@@
 Wire Wire Line
 	13500 2650 13500 2250
-Text GLabel 15650 2500 2    50   Output ~ 0
+Text GLabel 15150 2500 2    50   Output ~ 0
 _KBRST
 Wire Notes Line
@@
 $EndComp
 Wire Wire Line
-	14650 2500 15650 2500
-Wire Wire Line
 	12250 2150 12600 2150
 Wire Wire Line
@@
 Text Label 12150 1200 0    50   ~ 0
 RESET
+$Comp
+L Transistor_BJT:2SC1815 Q300
+U 1 1 609BBF63
+P 9850 8950
+F 0 "Q300" H 10041 8996 50  0000 L CNN
+F 1 "MMBT3904" H 10041 8905 50  0000 L CNN
+F 2 "Package_TO_SOT_SMD:SOT-23" H 10050 8875 50  0001 L CIN
+F 3 "https://media.digikey.com/pdf/Data%20Sheets/Toshiba%20PDFs/2SC1815.pdf" H 9850 8950 50  0001 L CNN
+	1    9850 8950
+	-1   0    0    -1
+$EndComp
+Connection ~ 10050 8950
+Wire Wire Line
+	10600 3050 11400 3050
+$Comp
+L power:GND #PWR0180
+U 1 1 609F7B0F
+P 11000 2350
+F 0 "#PWR0180" H 11000 2100 50  0001 C CNN
+F 1 "GND" H 11005 2177 50  0000 C CNN
+F 2 "" H 11000 2350 50  0001 C CNN
+F 3 "" H 11000 2350 50  0001 C CNN
+	1    11000 2350
+	1    0    0    -1
+$EndComp
+Wire Wire Line
+	14650 2500 15150 2500
 $EndSCHEMATC

Commit message: Add files via upload
Other:
- note added: "Serial\nAmiga 2000 EATX"
Changed lines of the file:
@@
 Wire Wire Line
 	14650 2500 15150 2500
+Text Notes 12300 9850 0    197  ~ 0
+Serial\nAmiga 2000 EATX
 $EndSCHEMATC

Commit message: Add files via upload
Parts:
- added D400, D401: S1MWF-7, Diode_SMD:D_SOD-123F, symbol Diode:1N4001
Connections:
- net +12V: now also D400.2 (A); no longer F2.1
- net -12V: now also D401.1 (K); no longer EMI334.2
- new net: D401.2 (A), EMI334.2
- new net: D400.1 (K), F2.1
Changed lines of the file:
@@
 Wire Wire Line
 	14450 6650 14750 6650
-Wire Wire Line
-	15050 6650 15600 6650
 $Comp
 L power:+12V #PWR0312
@@
 Wire Wire Line
 	14050 7150 14650 7150
-Wire Wire Line
-	14450 7650 15650 7650
 $Comp
 L power:-12V #PWR0313
@@
 Text Notes 12300 9850 0    197  ~ 0
 Serial\nAmiga 2000 EATX
+$Comp
+L Diode:1N4001 D400
+U 1 1 607FC6A1
+P 15200 6650
+F 0 "D400" H 15200 6867 50  0000 C CNN
+F 1 "S1MWF-7" H 15200 6776 50  0000 C CNN
+F 2 "Diode_SMD:D_SOD-123F" H 15200 6475 50  0001 C CNN
+F 3 "" H 15200 6650 50  0001 C CNN
+	1    15200 6650
+	1    0    0    -1
+$EndComp
+$Comp
+L Diode:1N4001 D401
+U 1 1 607FD0E8
+P 15150 7650
+F 0 "D401" H 15150 7433 50  0000 C CNN
+F 1 "S1MWF-7" H 15150 7524 50  0000 C CNN
+F 2 "Diode_SMD:D_SOD-123F" H 15150 7475 50  0001 C CNN
+F 3 "" H 15150 7650 50  0001 C CNN
+	1    15150 7650
+	-1   0    0    1
+$EndComp
+Wire Wire Line
+	15650 7650 15300 7650
+Wire Wire Line
+	15000 7650 14450 7650
+Wire Wire Line
+	15350 6650 15600 6650
 $EndSCHEMATC

Commit message: Add files via upload
Parts:
- U302: value 74LS32 -> 74HCT32
- U303: value 74LS08 -> 74HCT08
Changed lines of the file:
@@
 P 1350 5800
 F 0 "U302" H 1350 5483 50  0000 C CNN
-F 1 "74LS32" H 1350 5574 50  0000 C CNN
+F 1 "74HCT32" H 1350 5574 50  0000 C CNN
 F 2 "" H 1350 5800 50  0001 C CNN
 F 3 "http://www.ti.com/lit/gpn/sn74LS32" H 1350 5800 50  0001 C CNN
@@
 P 4750 2850
 F 0 "U303" H 4750 3175 50  0000 C CNN
-F 1 "74LS08" H 4750 3084 50  0000 C CNN
+F 1 "74HCT08" H 4750 3084 50  0000 C CNN
 F 2 "" H 4750 2850 50  0001 C CNN
 F 3 "http://www.ti.com/lit/gpn/sn74LS08" H 4750 2850 50  0001 C CNN
@@
 U 5 1 60A7C756
 P 8200 9750
-F 0 "U303" H 8200 10075 50  0000 C CNN
-F 1 "74LS08" H 8200 9984 50  0000 C CNN
+F 0 "U303" H 8200 9800 50  0000 C CNN
+F 1 "74HCT08" H 8200 9700 50  0000 C CNN
 F 2 "" H 8200 9750 50  0001 C CNN
 F 3 "http://www.ti.com/lit/gpn/sn74LS08" H 8200 9750 50  0001 C CNN
