File: 2000EATX-KiCAD-R1/power.sch (KiCad schematic (older format))
At the start: 44 parts, among them CN400 ATX-24, J9000 POWER_SWITCH, U9000 MC7905, U9001 74HCT14, U9002 74HCT74

Commit message: Add files via upload
Parts:
- added C9101, C9102: 0.1uF, Capacitor_SMD:C_1206_3216Metric, symbol Device:C
- renumbered C9003 to C9103, C9002 to C9104, D9000 to D9100, D9001 to D9101, J9000 to J9100, R9000 to R9100, R9001 to R9101, R9002 to R9102, U9001 to U9101, U9002 to U9102
Connections:
- net +5VSB: now also C9101.1, C9102.1
- net GND: now also C9101.2, C9102.2
Other:
- moved on the sheet: U9101G
Changed lines of the file:
@@
 	3450 3900 3450 3800
 $Comp
-L Connector:Conn_01x02_Male J9000
+L Connector:Conn_01x02_Male J9100
 U 1 1 60A6A8CF
 P 900 6150
-F 0 "J9000" H 1008 6331 50  0000 C CNN
+F 0 "J9100" H 1008 6331 50  0000 C CNN
 F 1 "POWER_SWITCH" H 1008 6240 50  0000 C CNN
 F 2 "Connector_PinHeader_2.54mm:PinHeader_1x02_P2.54mm_Vertical" H 900 6150 50  0001 C CNN
@@
 	2450 1600 2450 1750
 $Comp
-L 74xx:74HC14 U9001
+L 74xx:74HC14 U9101
 U 1 1 60A74CD0
 P 3650 5750
-F 0 "U9001" H 3650 6067 50  0000 C CNN
+F 0 "U9101" H 3650 6067 50  0000 C CNN
 F 1 "74HCT14" H 3650 5976 50  0000 C CNN
 F 2 "Package_SO:SOIC-14_3.9x8.7mm_P1.27mm" H 3650 5750 50  0001 C CNN
@@
 $EndComp
 $Comp
-L 74xx:74HC14 U9001
+L 74xx:74HC14 U9101
 U 2 1 60A761E9
 P 3650 6300
-F 0 "U9001" H 3650 6617 50  0000 C CNN
+F 0 "U9101" H 3650 6617 50  0000 C CNN
 F 1 "74HCT14" H 3650 6526 50  0000 C CNN
 F 2 "Package_SO:SOIC-14_3.9x8.7mm_P1.27mm" H 3650 6300 50  0001 C CNN
@@
 $EndComp
 $Comp
-L 74xx:74HC14 U9001
+L 74xx:74HC14 U9101
 U 3 1 60A77188
 P 4250 6300
-F 0 "U9001" H 4250 6617 50  0000 C CNN
+F 0 "U9101" H 4250 6617 50  0000 C CNN
 F 1 "74HCT14" H 4250 6526 50  0000 C CNN
 F 2 "Package_SO:SOIC-14_3.9x8.7mm_P1.27mm" H 4250 6300 50  0001 C CNN
@@
 $EndComp
 $Comp
-L 74xx:74HC74 U9002
+L 74xx:74HC74 U9102
 U 2 1 60A7B12E
 P 5250 5950
-F 0 "U9002" H 5250 6431 50  0000 C CNN
+F 0 "U9102" H 5250 6431 50  0000 C CNN
 F 1 "74HCT74" H 5250 6340 50  0000 C CNN
 F 2 "Package_SO:SOIC-14_3.9x8.7mm_P1.27mm" H 5250 5950 50  0001 C CNN
@@
 PS_ON
 $Comp
-L Device:R R9000
+L Device:R R9100
 U 1 1 60A7EE32
 P 1800 5400
-F 0 "R9000" H 1870 5446 50  0000 L CNN
+F 0 "R9100" H 1870 5446 50  0000 L CNN
 F 1 "10k" H 1870 5355 50  0000 L CNN
 F 2 "Resistor_SMD:R_1206_3216Metric" V 1730 5400 50  0001 C CNN
@@
 $EndComp
 $Comp
-L Device:R R9001
+L Device:R R9101
 U 1 1 60A7F446
 P 2750 5250
-F 0 "R9001" H 2820 5296 50  0000 L CNN
+F 0 "R9101" H 2820 5296 50  0000 L CNN
 F 1 "10k" H 2820 5205 50  0000 L CNN
 F 2 "Resistor_SMD:R_1206_3216Metric" V 2680 5250 50  0001 C CNN
@@
 $EndComp
 $Comp
-L Device:R R9002
+L Device:R R9102
 U 1 1 60A7F8B4
 P 2050 5750
-F 0 "R9002" V 1843 5750 50  0000 C CNN
+F 0 "R9102" V 1843 5750 50  0000 C CNN
 F 1 "470" V 1934 5750 50  0000 C CNN
 F 2 "Resistor_SMD:R_1206_3216Metric" V 1980 5750 50  0001 C CNN
@@
 $EndComp
 $Comp
-L Device:D D9000
+L Device:D D9100
 U 1 1 60A8886E
 P 3250 5250
-F 0 "D9000" V 3204 5330 50  0000 L CNN
+F 0 "D9100" V 3204 5330 50  0000 L CNN
 F 1 "1N4148" V 3295 5330 50  0000 L CNN
 F 2 "Diode_SMD:D_SOD-323" H 3250 5250 50  0001 C CNN
@@
 $EndComp
 $Comp
-L Device:D D9001
+L Device:D D9101
 U 1 1 60A911F3
 P 2300 5250
-F 0 "D9001" V 2254 5330 50  0000 L CNN
+F 0 "D9101" V 2254 5330 50  0000 L CNN
 F 1 "1N4148" V 2345 5330 50  0000 L CNN
 F 2 "Diode_SMD:D_SOD-323" H 2300 5250 50  0001 C CNN
@@
 Connection ~ 6650 6300
 $Comp
-L Device:C_Small C9002
+L Device:C_Small C9104
 U 1 1 60AE28F0
 P 2300 6100
-F 0 "C9002" H 2392 6146 50  0000 L CNN
+F 0 "C9104" H 2392 6146 50  0000 L CNN
 F 1 "1uF" H 2392 6055 50  0000 L CNN
 F 2 "Capacitor_SMD:C_1206_3216Metric" H 2300 6100 50  0001 C CNN
@@
 $EndComp
 $Comp
-L Device:C_Small C9003
+L Device:C_Small C9103
 U 1 1 60AE3393
 P 3250 6550
-F 0 "C9003" H 3342 6596 50  0000 L CNN
+F 0 "C9103" H 3342 6596 50  0000 L CNN
 F 1 "10uF" H 3342 6505 50  0000 L CNN
 F 2 "Capacitor_SMD:C_1206_3216Metric" H 3250 6550 50  0001 C CNN
@@
 	4150 1400 4150 2200
 $Comp
-L 74xx:74HC14 U9001
+L 74xx:74HC14 U9101
 U 7 1 60B8C9CF
-P 7450 5700
-F 0 "U9001" H 7680 5746 50  0000 L CNN
-F 1 "74HCT14" H 7680 5655 50  0000 L CNN
-F 2 "Package_SO:SOIC-14_3.9x8.7mm_P1.27mm" H 7450 5700 50  0001 C CNN
-F 3 "74xx/74hc_hct74.pdf" H 7450 5700 50  0001 C CNN
-	7    7450 5700
-	1    0    0    -1
-$EndComp
-Wire Wire Line
-	7450 5200 7450 5100
-Wire Wire Line
-	7450 6200 7450 6300
-$Comp
-L 74xx:74HC74 U9002
+P 8150 5700
+F 0 "U9101" H 8380 5746 50  0000 L CNN
+F 1 "74HCT14" H 8380 5655 50  0000 L CNN
+F 2 "Package_SO:SOIC-14_3.9x8.7mm_P1.27mm" H 8150 5700 50  0001 C CNN
+F 3 "74xx/74hc_hct74.pdf" H 8150 5700 50  0001 C CNN
+	7    8150 5700
+	1    0    0    -1
+$EndComp
+$Comp
+L 74xx:74HC74 U9102
 U 3 1 60BA6B66
 P 6650 5700
-F 0 "U9002" H 6880 5746 50  0000 L CNN
+F 0 "U9102" H 6880 5746 50  0000 L CNN
 F 1 "74HCT74" H 6880 5655 50  0000 L CNN
 F 2 "Package_SO:SOIC-14_3.9x8.7mm_P1.27mm" H 6650 5700 50  0001 C CNN
@@
 Wire Wire Line
 	6750 2400 8800 2400
+$Comp
+L Device:C C9102
+U 1 1 609B825E
+P 7450 5650
+F 0 "C9102" H 7565 5696 50  0000 L CNN
+F 1 "0.1uF" H 7565 5605 50  0000 L CNN
+F 2 "Capacitor_SMD:C_1206_3216Metric" H 7488 5500 50  0001 C CNN
+F 3 "~" H 7450 5650 50  0001 C CNN
+	1    7450 5650
+	1    0    0    -1
+$EndComp
+$Comp
+L Device:C C9101
+U 1 1 609C9C6F
+P 8900 5650
+F 0 "C9101" H 9015 5696 50  0000 L CNN
+F 1 "0.1uF" H 9015 5605 50  0000 L CNN
+F 2 "Capacitor_SMD:C_1206_3216Metric" H 8938 5500 50  0001 C CNN
+F 3 "~" H 8900 5650 50  0001 C CNN
+	1    8900 5650
+	1    0    0    -1
+$EndComp
+Wire Wire Line
+	7450 5100 8150 5100
+Wire Wire Line
+	8900 5100 8900 5500
+Connection ~ 7450 5100
+Wire Wire Line
+	7450 6300 8150 6300
+Wire Wire Line
+	8900 6300 8900 5800
+Connection ~ 7450 6300
+Wire Wire Line
+	8150 6200 8150 6300
+Connection ~ 8150 6300
+Wire Wire Line
+	8150 6300 8900 6300
+Wire Wire Line
+	8150 5200 8150 5100
+Connection ~ 8150 5100
+Wire Wire Line
+	8150 5100 8900 5100
+Wire Wire Line
+	7450 5100 7450 5500
+Wire Wire Line
+	7450 5800 7450 6300
 $EndSCHEMATC

Commit message: Add files via upload
Parts:
- removed H8: MountingHole_Pad, MountingHole:MountingHole_4.3mm_M4_Pad, symbol Mechanical:MountingHole_Pad
- H1, H10, H11, H12, H2, H3, H4, H5, H6, H7, H9: footprint MountingHole:MountingHole_4.3mm_M4_Pad -> AmigaFootprints:MountingHole_Pad
Changed lines of the file:
@@
 F 0 "H1" V 9100 3650 50  0000 L CNN
 F 1 "MountingHole_Pad" V 9145 3650 50  0001 L CNN
-F 2 "MountingHole:MountingHole_4.3mm_M4_Pad" H 9100 3500 50  0001 C CNN
+F 2 "AmigaFootprints:MountingHole_Pad" H 9100 3500 50  0001 C CNN
 F 3 "~" H 9100 3500 50  0001 C CNN
 	1    9100 3500
@@
 F 0 "H4" V 9100 3850 50  0000 L CNN
 F 1 "MountingHole_Pad" V 9145 3850 50  0001 L CNN
-F 2 "MountingHole:MountingHole_4.3mm_M4_Pad" H 9100 3700 50  0001 C CNN
+F 2 "AmigaFootprints:MountingHole_Pad" H 9100 3700 50  0001 C CNN
 F 3 "~" H 9100 3700 50  0001 C CNN
 	1    9100 3700
@@
 F 0 "H7" V 9100 4050 50  0000 L CNN
 F 1 "MountingHole_Pad" V 9145 4050 50  0001 L CNN
-F 2 "MountingHole:MountingHole_4.3mm_M4_Pad" H 9100 3900 50  0001 C CNN
+F 2 "AmigaFootprints:MountingHole_Pad" H 9100 3900 50  0001 C CNN
 F 3 "~" H 9100 3900 50  0001 C CNN
 	1    9100 3900
@@
 F 0 "H10" V 9100 4250 50  0000 L CNN
 F 1 "MountingHole_Pad" V 9145 4250 50  0001 L CNN
-F 2 "MountingHole:MountingHole_4.3mm_M4_Pad" H 9100 4100 50  0001 C CNN
+F 2 "AmigaFootprints:MountingHole_Pad" H 9100 4100 50  0001 C CNN
 F 3 "~" H 9100 4100 50  0001 C CNN
 	1    9100 4100
@@
 F 0 "H2" V 9500 3650 50  0000 L CNN
 F 1 "MountingHole_Pad" V 9545 3650 50  0001 L CNN
-F 2 "MountingHole:MountingHole_4.3mm_M4_Pad" H 9500 3500 50  0001 C CNN
+F 2 "AmigaFootprints:MountingHole_Pad" H 9500 3500 50  0001 C CNN
 F 3 "~" H 9500 3500 50  0001 C CNN
 	1    9500 3500
@@
 F 0 "H5" V 9500 3850 50  0000 L CNN
 F 1 "MountingHole_Pad" V 9545 3850 50  0001 L CNN
-F 2 "MountingHole:MountingHole_4.3mm_M4_Pad" H 9500 3700 50  0001 C CNN
+F 2 "AmigaFootprints:MountingHole_Pad" H 9500 3700 50  0001 C CNN
 F 3 "~" H 9500 3700 50  0001 C CNN
 	1    9500 3700
-	0    1    1    0
-$EndComp
-$Comp
-L Mechanical:MountingHole_Pad H8
-U 1 1 607A4E77
-P 9500 3900
-F 0 "H8" V 9500 4050 50  0000 L CNN
-F 1 "MountingHole_Pad" V 9545 4050 50  0001 L CNN
-F 2 "MountingHole:MountingHole_4.3mm_M4_Pad" H 9500 3900 50  0001 C CNN
-F 3 "~" H 9500 3900 50  0001 C CNN
-	1    9500 3900
 	0    1    1    0
 $EndComp
@@
 F 0 "H11" V 9500 4250 50  0000 L CNN
 F 1 "MountingHole_Pad" V 9545 4250 50  0001 L CNN
-F 2 "MountingHole:MountingHole_4.3mm_M4_Pad" H 9500 4100 50  0001 C CNN
+F 2 "AmigaFootprints:MountingHole_Pad" H 9500 4100 50  0001 C CNN
 F 3 "~" H 9500 4100 50  0001 C CNN
 	1    9500 4100
-	0    1    1    0
-$EndComp
-$Comp
-L Mechanical:MountingHole_Pad H3
-U 1 1 607B44AE
-P 9900 3500
-F 0 "H3" V 9900 3650 50  0000 L CNN
-F 1 "MountingHole_Pad" V 9945 3650 50  0001 L CNN
-F 2 "MountingHole:MountingHole_4.3mm_M4_Pad" H 9900 3500 50  0001 C CNN
-F 3 "~" H 9900 3500 50  0001 C CNN
-	1    9900 3500
 	0    1    1    0
 $EndComp
@@
 F 0 "H9" V 9900 4050 50  0000 L CNN
 F 1 "MountingHole_Pad" V 9945 4050 50  0001 L CNN
-F 2 "MountingHole:MountingHole_4.3mm_M4_Pad" H 9900 3900 50  0001 C CNN
+F 2 "AmigaFootprints:MountingHole_Pad" H 9900 3900 50  0001 C CNN
 F 3 "~" H 9900 3900 50  0001 C CNN
 	1    9900 3900
@@
 F 0 "H6" V 9900 3850 50  0000 L CNN
 F 1 "MountingHole_Pad" V 9945 3850 50  0001 L CNN
-F 2 "MountingHole:MountingHole_4.3mm_M4_Pad" H 9900 3700 50  0001 C CNN
+F 2 "AmigaFootprints:MountingHole_Pad" H 9900 3700 50  0001 C CNN
 F 3 "~" H 9900 3700 50  0001 C CNN
 	1    9900 3700
@@
 F 0 "H12" V 9900 4250 50  0000 L CNN
 F 1 "MountingHole_Pad" V 9945 4250 50  0001 L CNN
-F 2 "MountingHole:MountingHole_4.3mm_M4_Pad" H 9900 4100 50  0001 C CNN
+F 2 "AmigaFootprints:MountingHole_Pad" H 9900 4100 50  0001 C CNN
 F 3 "~" H 9900 4100 50  0001 C CNN
 	1    9900 4100
@@
 	9000 4400 9000 4100
 Connection ~ 9400 3700
-Wire Wire Line
-	9400 3700 9400 3900
-Connection ~ 9400 3900
-Wire Wire Line
-	9400 3900 9400 4100
 Connection ~ 9400 4100
 Wire Wire Line
@@
 Wire Wire Line
 	7450 5800 7450 6300
+Wire Wire Line
+	9400 3700 9400 4100
+$Comp
+L Mechanical:MountingHole_Pad H3
+U 1 1 607B44AE
+P 9900 3500
+F 0 "H3" V 9900 3650 50  0000 L CNN
+F 1 "MountingHole_Pad" V 9945 3650 50  0001 L CNN
+F 2 "AmigaFootprints:MountingHole_Pad" H 9900 3500 50  0001 C CNN
+F 3 "~" H 9900 3500 50  0001 C CNN
+	1    9900 3500
+	0    1    1    0
+$EndComp
 $EndSCHEMATC
