File: 2000EATX-KiCAD-R11/Zorro_Expansion.sch (KiCad schematic (older format))
At the start: 111 parts, among them CN601 Amiga-2000-Zorro-Slot, CN602 Amiga-2000-Zorro-Slot, CN603 Amiga-2000-Zorro-Slot, CN604 Amiga-2000-Zorro-Slot, CN605 Amiga-2000-Zorro-Slot, U606 74HCT32

Commit message: Add files via upload
Parts:
- C416, C417, C418, C419: footprint Capacitor_SMD:CP_Elec_6.3x5.8 -> Capacitor_SMD:CP_Elec_8x10
Changed lines of the file:
@@
 F 0 "C416" V 3578 1550 50  0000 C CNN
 F 1 "220uF" V 3487 1550 50  0000 C CNN
-F 2 "Capacitor_SMD:CP_Elec_6.3x5.8" H 3350 1550 50  0001 C CNN
+F 2 "Capacitor_SMD:CP_Elec_8x10" H 3350 1550 50  0001 C CNN
 F 3 "~" H 3350 1550 50  0001 C CNN
 	1    3350 1550
@@
 F 0 "C417" V 4528 1550 50  0000 C CNN
 F 1 "220uF" V 4437 1550 50  0000 C CNN
-F 2 "Capacitor_SMD:CP_Elec_6.3x5.8" H 4300 1550 50  0001 C CNN
+F 2 "Capacitor_SMD:CP_Elec_8x10" H 4300 1550 50  0001 C CNN
 F 3 "~" H 4300 1550 50  0001 C CNN
 	1    4300 1550
@@
 F 0 "C418" V 5528 1550 50  0000 C CNN
 F 1 "220uF" V 5437 1550 50  0000 C CNN
-F 2 "Capacitor_SMD:CP_Elec_6.3x5.8" H 5300 1550 50  0001 C CNN
+F 2 "Capacitor_SMD:CP_Elec_8x10" H 5300 1550 50  0001 C CNN
 F 3 "~" H 5300 1550 50  0001 C CNN
 	1    5300 1550
@@
 F 0 "C419" V 6478 1550 50  0000 C CNN
 F 1 "220uF" V 6387 1550 50  0000 C CNN
-F 2 "Capacitor_SMD:CP_Elec_6.3x5.8" H 6250 1550 50  0001 C CNN
+F 2 "Capacitor_SMD:CP_Elec_8x10" H 6250 1550 50  0001 C CNN
 F 3 "~" H 6250 1550 50  0001 C CNN
 	1    6250 1550
