File: 2000EATX-KiCAD-R11/Processor.sch (KiCad schematic (older format))
At the start: 19 parts, among them U100 MC68000, U103 74HCT245, U104 74HCT373, U105 74HCT245, U106 74HCT373, U303 74HCT08

Commit message: Add files via upload
Parts:
- U100: footprint Package_DIP:DIP-64_W25.4mm -> Package_DIP:DIP-64_W22.86mm_Socket
Changed lines of the file:
@@
 F 0 "U100" H 4750 6631 50  0000 C CNN
 F 1 "MC68000" H 4750 6540 50  0000 C CNN
-F 2 "Package_DIP:DIP-64_W25.4mm" H 4750 4050 50  0001 C CNN
+F 2 "Package_DIP:DIP-64_W22.86mm_Socket" H 4750 4050 50  0001 C CNN
 F 3 "https://www.nxp.com/docs/en/reference-manual/MC68000UM.pdf" H 4750 4050 50  0001 C CNN
 	1    4750 4050
