File: 2000EATX-KiCAD-R11/bus.sch (KiCad schematic (older format))
At the start: 26 parts, among them U302 74HCT32, U800 BUSTER, U801 RTC62423, U802 74HCT138, U803 74HCT08, U804 74LS148

Commit message: Add files via upload
Parts:
- U801: footprint Package_SO:SOP-24_7.5x15.4mm_P1.27mm -> Package_SO:SOIC-24W_7.5x15.4mm_P1.27mm
Changed lines of the file:
@@
 F 0 "U801" H 8325 9065 50  0000 C CNN
 F 1 "RTC62423" H 8325 8974 50  0000 C CNN
-F 2 "Package_SO:SOP-24_7.5x15.4mm_P1.27mm" H 8150 8600 50  0001 C CNN
+F 2 "Package_SO:SOIC-24W_7.5x15.4mm_P1.27mm" H 8150 8600 50  0001 C CNN
 F 3 "" H 8150 8600 50  0001 C CNN
 	1    8350 8350
