File: 2000EATX-KiCAD-R11/coprocessor.sch (KiCad schematic (older format))
At the start: 17 parts, among them CN600 Amiga-2000-CPU-Slot, U600 74HCT245, U601 74HCT245, U602 74HCT245, U603 74HCT245, U604 74HCT245, U605 74HCT245

Commit message: Add files via upload
Connections:
- net +5V: now also C600.1, C601.1, C602.1, C603.1, C604.1, U600.20 (VCC), U601.20 (VCC), U602.20 (VCC), U603.20 (VCC), U604.20 (VCC)
Changed lines of the file:
@@
 L power:+5V #PWR0143
 U 1 1 60E89AA3
-P 6150 4150
-F 0 "#PWR0143" H 6150 4000 50  0001 C CNN
-F 1 "+5V" H 6167 4373 50  0000 C CNN
-F 2 "" H 6150 4150 50  0001 C CNN
-F 3 "" H 6150 4150 50  0001 C CNN
-	1    6150 4150
+P 6200 4150
+F 0 "#PWR0143" H 6200 4000 50  0001 C CNN
+F 1 "+5V" H 6217 4373 50  0000 C CNN
+F 2 "" H 6200 4150 50  0001 C CNN
+F 3 "" H 6200 4150 50  0001 C CNN
+	1    6200 4150
 	1    0    0    -1
 $EndComp
@@
 	3100 1700 3100 2550
 Wire Wire Line
-	6850 2400 7300 2400
-Wire Wire Line
-	10250 3450 10700 3450
-Wire Wire Line
-	10250 1200 10600 1200
-Wire Wire Line
-	5800 800  6150 800
-Wire Wire Line
-	6000 4150 6500 4150
+	6850 2400 7150 2400
+Wire Wire Line
+	10250 3450 10500 3450
+Wire Wire Line
+	10250 1200 10500 1200
+Wire Wire Line
+	5800 800  6050 800
+Wire Wire Line
+	6000 4150 6200 4150
 $Comp
 L Device:R_Network09 RNX1
@@
 Text Notes 7050 7100 0    197  ~ 0
 Coprocessor\nAmiga 2000 EATX
+Connection ~ 7150 2400
+Wire Wire Line
+	7150 2400 7300 2400
+Connection ~ 6050 800
+Wire Wire Line
+	6050 800  6150 800
+Connection ~ 6200 4150
+Wire Wire Line
+	6200 4150 6500 4150
+Connection ~ 3450 5800
+Connection ~ 10500 3450
+Wire Wire Line
+	10500 3450 10700 3450
+Connection ~ 10500 1200
+Wire Wire Line
+	10500 1200 10600 1200
 $EndSCHEMATC
