File: 2000EATX-KiCAD-R11/floppyparallel.sch (KiCad schematic (older format))
At the start: 50 parts, among them CN300 KEYBOARD, CN303 FLOPPY, CN305 DB25_Stack_FemaleAndMale, J301 SHORT FOR DF1, Q301 MMBT3906, U102 GARY, U108 74HCT74, U203 74LS38, U300 8520, U302 74HCT32, U607 74HCT08, U900 74HCT00

Commit message: Add files via upload
Parts:
- removed Q301: MMBT3906, Package_TO_SOT_SMD:SOT-23, symbol Transistor_BJT:2N3904
- added Q301: MMBT3906, Package_TO_SOT_SMD:SOT-23, symbol Transistor_BJT:MMBT3906
Connections:
- net GND: now also Q301.2 (E)
- net MTROD: now also Q301.3 (C)
- net at R300.1, R309.1: now also Q301.1 (B)
Changed lines of the file:
@@
 	12500 5500 12850 5500
-$Comp
-L Transistor_BJT:2N3904 Q301
-U 1 1 60D03916
-P 13650 5500
-F 0 "Q301" H 13841 5546 50  0000 L CNN
-F 1 "MMBT3906" H 13841 5455 50  0000 L CNN
-F 2 "Package_TO_SOT_SMD:SOT-23" H 13850 5425 50  0001 L CIN
-F 3 "https://www.fairchildsemi.com/datasheets/2N/2N3904.pdf" H 13650 5500 50  0001 L CNN
-	1    13650 5500
-	1    0    0    -1
-$EndComp
 $Comp
 L power:GND #PWR0371
@@
 Wire Wire Line
 	850  6400 2300 6400
+$Comp
+L Transistor_BJT:MMBT3906 Q301
+U 1 1 60EC67CE
+P 13650 5500
+F 0 "Q301" H 13841 5546 50  0000 L CNN
+F 1 "MMBT3906" H 13841 5455 50  0000 L CNN
+F 2 "Package_TO_SOT_SMD:SOT-23" H 13850 5425 50  0001 L CIN
+F 3 "https://www.fairchildsemi.com/datasheets/2N/2N3906.pdf" H 13650 5500 50  0001 L CNN
+	1    13650 5500
+	1    0    0    -1
+$EndComp
 $EndSCHEMATC
