File: 2000EATX-KiCAD-R11/paula.sch (KiCad schematic (older format))
At the start: 78 parts, among them CN200 DB9_Male_Stack, CN205 AudioJack, Q200 MMBFJ211, Q201 MMBFJ211, Q202 MMBT3906, U200 PAULA, U202 74HCT157, U204 LF347

Commit message: Add files via upload
Parts:
- C222, C223: footprint Capacitor_SMD:CP_Elec_6.3x5.8 -> Capacitor_SMD:CP_Elec_8x10
Changed lines of the file:
@@
 F 0 "C222" V 14405 8000 50  0000 C CNN
 F 1 "47uF" V 14314 8000 50  0000 C CNN
-F 2 "Capacitor_SMD:CP_Elec_6.3x5.8" H 14188 7850 50  0001 C CNN
+F 2 "Capacitor_SMD:CP_Elec_8x10" H 14188 7850 50  0001 C CNN
 F 3 "~" H 14150 8000 50  0001 C CNN
 	1    14150 8000
@@
 F 0 "C223" V 14405 8300 50  0000 C CNN
 F 1 "47uF" V 14314 8300 50  0000 C CNN
-F 2 "Capacitor_SMD:CP_Elec_6.3x5.8" H 14188 8150 50  0001 C CNN
+F 2 "Capacitor_SMD:CP_Elec_8x10" H 14188 8150 50  0001 C CNN
 F 3 "~" H 14150 8300 50  0001 C CNN
 	1    14150 8300

Commit message: Add files via upload
Parts:
- removed Q202: MMBT3906, Package_TO_SOT_SMD:SOT-23, symbol Transistor_BJT:2N3906
- added Q202: MMBT3906, Package_TO_SOT_SMD:SOT-23, symbol Transistor_BJT:MMBT3906
Connections:
- net +AV: now also Q202.2 (E)
- net at C204.1, R204.1, R205.1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: now also Q202.3 (C)
- net at R213.2, R214.2: now also Q202.1 (B)
Changed lines of the file:
@@
 	1    0    0    -1
-$EndComp
-$Comp
-L Transistor_BJT:2N3906 Q202
-U 1 1 606A3F54
-P 10650 5750
-F 0 "Q202" H 10841 5704 50  0000 L CNN
-F 1 "MMBT3906" H 10841 5795 50  0000 L CNN
-F 2 "Package_TO_SOT_SMD:SOT-23" H 10850 5675 50  0001 L CIN
-F 3 "https://www.fairchildsemi.com/datasheets/2N/2N3906.pdf" H 10650 5750 50  0001 L CNN
-F 4 "MMBT3906-7-F" H 10650 5750 50  0001 C CNN "Part"
-	1    10650 5750
-	-1   0    0    1
 $EndComp
 Wire Wire Line
@@
 Wire Wire Line
 	6550 1350 7450 1350
+$Comp
+L Transistor_BJT:MMBT3906 Q202
+U 1 1 60E68FB6
+P 10650 5750
+F 0 "Q202" H 10841 5704 50  0000 L CNN
+F 1 "MMBT3906" H 10841 5795 50  0000 L CNN
+F 2 "Package_TO_SOT_SMD:SOT-23" H 10850 5675 50  0001 L CIN
+F 3 "https://www.fairchildsemi.com/datasheets/2N/2N3906.pdf" H 10650 5750 50  0001 L CNN
+	1    10650 5750
+	-1   0    0    1
+$EndComp
 $EndSCHEMATC
