File: 2000EATX-KiCAD-R11/serial.sch (KiCad schematic (older format))
At the start: 54 parts, among them CN305 DB25_Stack_FemaleAndMale, J9001 RESET, J9002 POWER LED, Q300 MMBT3904, Q302 MMBT3906, U301 8520, U302 74HCT32, U303 74HCT08, U304 SN75188DR, U305 SN75189DR, U805 LM339

Commit message: Add files via upload
Parts:
- removed Q300: MMBT3904, Package_TO_SOT_SMD:SOT-23, symbol Transistor_BJT:2SC1815
- removed Q302: MMBT3906, Package_TO_SOT_SMD:SOT-23, symbol Transistor_BJT:2N3906
- added Q300: MMBT3904, Package_TO_SOT_SMD:SOT-23, symbol Transistor_BJT:MMBT3904
- added Q302: MMBT3906, Package_TO_SOT_SMD:SOT-23, symbol Transistor_BJT:MMBT3906
Connections:
- net +5V: now also Q302.2 (E)
- net GND: now also Q300.2 (E)
- net PSEL: now also Q300.3 (C)
- net at R902.1: now also Q302.1 (B)
- net at R307.2: now also Q302.3 (C)
- net at D300.1 (K), R305.1, R306.2: now also Q300.1 (B)
Changed lines of the file:
@@
 	5850 1600 6200 1600
-$Comp
-L Transistor_BJT:2N3906 Q302
-U 1 1 605D6763
-P 6400 1600
-F 0 "Q302" H 6591 1554 50  0000 L CNN
-F 1 "MMBT3906" H 6591 1645 50  0000 L CNN
-F 2 "Package_TO_SOT_SMD:SOT-23" H 6600 1525 50  0001 L CIN
-F 3 "" H 6400 1600 50  0001 L CNN
-	1    6400 1600
-	1    0    0    1
-$EndComp
 $Comp
 L power:+5V #PWR0293
@@
 Text Label 12150 1200 0    50   ~ 0
 RESET
-$Comp
-L Transistor_BJT:2SC1815 Q300
-U 1 1 609BBF63
-P 9850 8950
-F 0 "Q300" H 10041 8996 50  0000 L CNN
-F 1 "MMBT3904" H 10041 8905 50  0000 L CNN
-F 2 "Package_TO_SOT_SMD:SOT-23" H 10050 8875 50  0001 L CIN
-F 3 "https://media.digikey.com/pdf/Data%20Sheets/Toshiba%20PDFs/2SC1815.pdf" H 9850 8950 50  0001 L CNN
-	1    9850 8950
-	-1   0    0    -1
-$EndComp
-Connection ~ 10050 8950
 Wire Wire Line
 	10600 3050 11400 3050
@@
 Wire Wire Line
 	15350 6650 15600 6650
+$Comp
+L Transistor_BJT:MMBT3904 Q300
+U 1 1 60E33EB1
+P 9850 8950
+F 0 "Q300" H 10041 8996 50  0000 L CNN
+F 1 "MMBT3904" H 10041 8905 50  0000 L CNN
+F 2 "Package_TO_SOT_SMD:SOT-23" H 10050 8875 50  0001 L CIN
+F 3 "https://www.fairchildsemi.com/datasheets/2N/2N3904.pdf" H 9850 8950 50  0001 L CNN
+	1    9850 8950
+	-1   0    0    -1
+$EndComp
+Connection ~ 10050 8950
+$Comp
+L Transistor_BJT:MMBT3906 Q302
+U 1 1 60E53945
+P 6400 1600
+F 0 "Q302" H 6591 1554 50  0000 L CNN
+F 1 "MMBT3906" H 6591 1645 50  0000 L CNN
+F 2 "Package_TO_SOT_SMD:SOT-23" H 6600 1525 50  0001 L CIN
+F 3 "https://www.fairchildsemi.com/datasheets/2N/2N3906.pdf" H 6400 1600 50  0001 L CNN
+	1    6400 1600
+	1    0    0    1
+$EndComp
 $EndSCHEMATC
