File: 2000EATX-KiCAD-R11/video.sch (KiCad schematic (older format))
At the start: 36 parts, among them CN201 Amiga-2000-Video-Slot, CN202 DB15_Female_HighDensity, CN203 Amiga-2000-Video-Slot, U201 DENISE, U205 74HCT244, U206 74HCT244, U303 74HCT08

Commit message: Add files via upload
Parts:
- U205, U206: value 74HCT244 -> 74AHCT244
Changed lines of the file:
@@
 P 5000 3350
 F 0 "U205" H 5000 4331 50  0000 C CNN
-F 1 "74HCT244" H 5000 4240 50  0000 C CNN
+F 1 "74AHCT244" H 5000 4240 50  0000 C CNN
 F 2 "Package_SO:SOIC-20W_7.5x12.8mm_P1.27mm" H 5000 3350 50  0001 C CNN
 F 3 "https://assets.nexperia.com/documents/data-sheet/74HC_HCT244.pdf" H 5000 3350 50  0001 C CNN
@@
 P 5000 5500
 F 0 "U206" H 5000 6481 50  0000 C CNN
-F 1 "74HCT244" H 5000 6390 50  0000 C CNN
+F 1 "74AHCT244" H 5000 6390 50  0000 C CNN
 F 2 "Package_SO:SOIC-20W_7.5x12.8mm_P1.27mm" H 5000 5500 50  0001 C CNN
 F 3 "https://assets.nexperia.com/documents/data-sheet/74HC_HCT244.pdf" H 5000 5500 50  0001 C CNN

Commit message: Add files via upload
Parts:
- HY200: renamed from VIDIOT1; value HY200 -> VIDIOT
Changed lines of the file:
@@
 R3
 $Comp
-L Connector:Conn_01x22_Male VIDIOT1
+L Connector:Conn_01x22_Male HY200
 U 1 1 60820DFB
 P 12850 2950
-F 0 "VIDIOT1" H 12700 2950 50  0001 C CNN
-F 1 "HY200" H 12822 2878 50  0000 R CNN
+F 0 "HY200" H 12700 2950 50  0001 C CNN
+F 1 "VIDIOT" H 12822 2878 50  0000 R CNN
 F 2 "Connector_PinSocket_2.54mm:PinSocket_1x22_P2.54mm_Vertical" H 12850 2950 50  0001 C CNN
 F 3 "~" H 12850 2950 50  0001 C CNN
