File: 2000EATX-KiCAD-R12/coprocessor.sch (KiCad schematic (older format))
At the start: 17 parts, among them CN600 Amiga-2000-CPU-Slot, U600 74HCT245, U601 74HCT245, U602 74HCT245, U603 74HCT245, U604 74HCT245, U605 74HCT245

Commit message: Add files via upload
Connections:
- net _COPCGF renamed _COPCFG
Changed lines of the file:
@@
 _VC1
 Text GLabel 850  1800 0    47   Output ~ 0
-_COPCGF
+_COPCFG
 Text GLabel 850  2300 0    47   Output ~ 0
 _OVR
