File: 2000EATX-KiCAD-R12/serial.sch (KiCad schematic (older format))
At the start: 54 parts, among them CN305 DB25_Stack_FemaleAndMale, J9001 RESET, J9002 POWER LED, Q300 MMBT3904, Q302 MMBT3906, U301 8520, U302 74HCT32, U303 74HCT08, U304 SN75188DR, U305 SN75189DR, U805 LM339

Commit message: Add files via upload
Connections:
- net _SEL2: no longer names the net of U301.15 (PB5)
- net _SEL3: no longer names the net of U301.16 (PB6)
- no-connect marks 16 -> 18
Changed lines of the file:
@@
 	3500 8800 1100 8800
-Wire Wire Line
-	2800 6900 3650 6900
-Wire Wire Line
-	3650 6900 3650 9000
-Wire Wire Line
-	3650 9000 1100 9000
-Wire Wire Line
-	2800 6700 3850 6700
-Wire Wire Line
-	3850 6700 3850 9200
-Wire Wire Line
-	3850 9200 1100 9200
 Wire Wire Line
 	2800 6500 4050 6500
@@
 Text GLabel 1100 8800 0    50   Output ~ 0
 _SEL1
-Text GLabel 1100 9000 0    50   Output ~ 0
-_SEL2
-Text GLabel 1100 9200 0    50   Output ~ 0
-_SEL3
 Text GLabel 1100 9400 0    50   Output ~ 0
 _MTR
@@
 Wire Wire Line
 	12100 2450 12250 2450
+NoConn ~ 2800 6900
+NoConn ~ 2800 6700
 $EndSCHEMATC
