File: 2000EATX-KiCAD-R12/agnus.sch (KiCad schematic (older format))
At the start: 35 parts, among them J102 SHORT FOR NTSC, J900 Enable Chip RAM slowdown duri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, U101 8372A_FATTER_AGNUS, U102 GARY, U107 74HCT04, U302 74HCT32, U900 74HCT00, X1 28.63636MHz, X2 7C-28.63636MBB-T

Commit message: Add files via upload
Changed lines of the file:
@@
 Wire Wire Line
 	6850 1450 8850 1450
-Wire Wire Line
-	6850 1000 7550 1000
 $Comp
 L power:+5V #PWR0248
@@
 	1    0    0    -1
 $EndComp
-Connection ~ 7550 1000
 $Comp
 L 74xx:7400 U900
@@
 Text Notes 12300 9850 0    197  ~ 0
 Agnus\nAmiga 2000 EATX
+$Comp
+L power:+5V #PWR?
+U 1 1 60EBF4D7
+P 6850 1000
+F 0 "#PWR?" H 6850 850 50  0001 C CNN
+F 1 "+5V" H 6865 1173 50  0000 C CNN
+F 2 "" H 6850 1000 50  0001 C CNN
+F 3 "" H 6850 1000 50  0001 C CNN
+	1    6850 1000
+	1    0    0    -1
+$EndComp
 $EndSCHEMATC

Commit message: Add files via upload
Changed lines of the file:
@@
 U 3 1 60CF8B16
 P 6850 3900
-F 0 "U900" H 6850 3583 50  0000 C CNN
-F 1 "74HCT00" H 6850 3674 50  0000 C CNN
+F 0 "U900" H 6850 4250 50  0000 C CNN
+F 1 "74HCT00" H 6850 4150 50  0000 C CNN
 F 2 "Package_SO:SOIC-14_3.9x8.7mm_P1.27mm" H 6850 3900 50  0001 C CNN
 F 3 "http://www.ti.com/lit/gpn/sn7400" H 6850 3900 50  0001 C CNN
 	3    6850 3900
-	-1   0    0    1
+	-1   0    0    -1
 $EndComp
 $Comp
@@
 	-1   0    0    1
 $EndComp
-Wire Wire Line
-	7150 3800 7400 3800
-Wire Wire Line
-	6250 1850 7250 1850
-Wire Wire Line
-	7150 4000 7250 4000
-Wire Wire Line
-	7250 4000 7250 1850
-Connection ~ 7250 1850
-Wire Wire Line
-	7250 1850 8850 1850
 Wire Wire Line
 	5750 3700 5750 3900
@@
 	1    0    0    -1
 $EndComp
+Wire Wire Line
+	6250 1850 7150 1850
+Wire Wire Line
+	7150 4000 7400 4000
+Wire Wire Line
+	7400 4000 7400 3800
+Wire Wire Line
+	7150 3800 7150 1850
+Connection ~ 7150 1850
+Wire Wire Line
+	7150 1850 8850 1850
 $EndSCHEMATC
