File: 2000EATX-KiCAD-R12/paula.sch (KiCad schematic (older format))
At the start: 78 parts, among them CN200 DB9_Male_Stack, CN205 AudioJack, Q200 MMBFJ211, Q201 MMBFJ211, Q202 MMBT3906, U200 PAULA, U202 74HCT157, U204 LF347

Commit message: Add files via upload
Other:
- note added: "JUMPER 200 OMITTED AND FIXED \nTO "STANDARD" ("A500") CONFIGURATION"
- note removed: "JUMPER 200 OMITTED AND FIXED \nTO "STANDARD" OR "A500" CONFIGURATION"
Changed lines of the file:
@@
 	10150 9950 10150 9750
 Text Notes 10250 10200 0    50   ~ 0
-JUMPER 200 OMITTED AND FIXED \nTO "STANDARD" OR "A500" CONFIGURATION
+JUMPER 200 OMITTED AND FIXED \nTO "STANDARD" ("A500") CONFIGURATION
 Text GLabel 10400 9150 2    50   Output ~ 0
 _FIR0

Commit message: Add files via upload
Connections:
- net AUDIO: now also C210.2, C211.2, C212.2, C213.2, U200.34 (A_GND)
- net GND: no longer C210.2, C211.2, C212.2, C213.2, U200.34 (A_GND)
Changed lines of the file:
@@
 Text GLabel 1850 6450 0    50   Input ~ 0
 _RST
-Wire Wire Line
-	4300 6450 4300 6550
-$Comp
-L power:GND #PWR0257
-U 1 1 605A38FC
-P 4300 6550
-F 0 "#PWR0257" H 4300 6300 50  0001 C CNN
-F 1 "GND" H 4305 6377 50  0000 C CNN
-F 2 "" H 4300 6550 50  0001 C CNN
-F 3 "" H 4300 6550 50  0001 C CNN
-	1    4300 6550
-	1    0    0    -1
-$EndComp
 $Comp
 L Device:C C210
@@
 Connection ~ 4100 6450
 Wire Wire Line
-	4100 6450 4300 6450
-Wire Wire Line
 	3600 6350 3600 6450
 Connection ~ 3600 6450
@@
 Connection ~ 3150 5300
 Wire Wire Line
-	4300 6450 4600 6450
-Wire Wire Line
 	4600 6450 4600 6400
-Connection ~ 4300 6450
 $Comp
 L 74xx:74LS157 U202
@@
 Wire Wire Line
 	10150 9950 10150 9750
-Text Notes 10250 10200 0    50   ~ 0
+Text Notes 9750 10300 0    79   ~ 0
 JUMPER 200 OMITTED AND FIXED \nTO "STANDARD" ("A500") CONFIGURATION
 Text GLabel 10400 9150 2    50   Output ~ 0
@@
 	-1   0    0    1
 $EndComp
+$Comp
+L Amiga-Library:AUDIO #PWR?
+U 1 1 60EEDA6C
+P 4600 6450
+F 0 "#PWR?" H 4600 6200 50  0001 C CNN
+F 1 "AUDIO" H 4605 6277 50  0000 C CNN
+F 2 "" H 4600 6450 50  0001 C CNN
+F 3 "" H 4600 6450 50  0001 C CNN
+	1    4600 6450
+	1    0    0    -1
+$EndComp
+Connection ~ 4600 6450
+Wire Wire Line
+	4100 6450 4600 6450
 $EndSCHEMATC

Commit message: Add files via upload
Connections:
- net AUDIO: now also CN205.S
- net GND: no longer CN205.S
Changed lines of the file:
@@
 	14950 2950 15250 2950
-$Comp
-L power:GND #PWR0282
-U 1 1 60E0B223
-P 15250 2950
-F 0 "#PWR0282" H 15250 2700 50  0001 C CNN
-F 1 "GND" H 15255 2777 50  0000 C CNN
-F 2 "" H 15250 2950 50  0001 C CNN
-F 3 "" H 15250 2950 50  0001 C CNN
-	1    15250 2950
-	1    0    0    -1
-$EndComp
 $Comp
 L Amiga-Library:DB9_Male_Stack CN200
@@
 $EndComp
 $Comp
-L Amiga-Library:AUDIO #PWR?
+L Amiga-Library:AUDIO #PWR0218
 U 1 1 60EEDA6C
 P 4600 6450
-F 0 "#PWR?" H 4600 6200 50  0001 C CNN
+F 0 "#PWR0218" H 4600 6200 50  0001 C CNN
 F 1 "AUDIO" H 4605 6277 50  0000 C CNN
 F 2 "" H 4600 6450 50  0001 C CNN
@@
 Wire Wire Line
 	4100 6450 4600 6450
+$Comp
+L Amiga-Library:AUDIO #PWR0219
+U 1 1 60EC6665
+P 15250 2950
+F 0 "#PWR0219" H 15250 2700 50  0001 C CNN
+F 1 "AUDIO" H 15255 2777 50  0000 C CNN
+F 2 "" H 15250 2950 50  0001 C CNN
+F 3 "" H 15250 2950 50  0001 C CNN
+	1    15250 2950
+	1    0    0    -1
+$EndComp
 $EndSCHEMATC

Commit message: Add files via upload
Connections:
- net FIR0: now also CN200.6; no longer CN200.15
- net at CN200.1: now also EMI234.2; no longer EMI230.2
- net at CN200.2: now also EMI235.2; no longer EMI231.2
- net at CN200.3: now also EMI236.2; no longer EMI232.2
- net at CN200.4: now also EMI237.2; no longer EMI233.2
- net at CN200.5: now also EMI243.2; no longer EMI240.1
- net at EMI238.1: now also CN200.15; no longer CN200.6
- net at CN200.9: now also EMI242.2; no longer EMI239.1
- net at CN200.10: now also EMI230.2; no longer EMI234.2
- net at CN200.11: now also EMI231.2; no longer EMI235.2
- net at CN200.12: now also EMI232.2; no longer EMI236.2
- net at CN200.13: now also EMI233.2; no longer EMI237.2
- net at CN200.14: now also EMI240.1; no longer EMI243.2
- net at CN200.18: now also EMI239.1; no longer EMI242.2
Other:
- moved on the sheet: CN200A, CN200B
Changed lines of the file:
@@
 _FIR1
-Wire Wire Line
-	6300 10450 9100 10450
 Wire Wire Line
 	10150 9750 10400 9750
@@
 L Amiga-Library:DB9_Male_Stack CN200
 U 1 1 605BDCC9
-P 6600 9900
-F 0 "CN200" H 6780 9946 50  0000 L CNN
-F 1 "DB9_Male_Stack" H 6780 9855 50  0000 L CNN
-F 2 "AmigaFootprints:DSUB-9_Male_Stack" H 6600 9900 50  0001 C CNN
-F 3 " ~" H 6600 9900 50  0001 C CNN
-	1    6600 9900
-	1    0    0    -1
-$EndComp
-Wire Wire Line
-	6300 10200 6300 10450
-$Comp
-L Amiga-Library:DB9_Male_Stack CN200
-U 2 1 605DF9E0
 P 6600 8150
 F 0 "CN200" H 6780 8196 50  0000 L CNN
@@
 F 2 "AmigaFootprints:DSUB-9_Male_Stack" H 6600 8150 50  0001 C CNN
 F 3 " ~" H 6600 8150 50  0001 C CNN
-	2    6600 8150
+	1    6600 8150
 	1    0    0    -1
 $EndComp
@@
 	1    0    0    -1
 $EndComp
+$Comp
+L Amiga-Library:DB9_Male_Stack CN200
+U 2 1 605DF9E0
+P 6600 9900
+F 0 "CN200" H 6780 9946 50  0000 L CNN
+F 1 "DB9_Male_Stack" H 6780 9855 50  0000 L CNN
+F 2 "AmigaFootprints:DSUB-9_Male_Stack" H 6600 9900 50  0001 C CNN
+F 3 " ~" H 6600 9900 50  0001 C CNN
+	2    6600 9900
+	1    0    0    -1
+$EndComp
+Wire Wire Line
+	6100 10450 6100 10200
+Wire Wire Line
+	6100 10200 6300 10200
+Wire Wire Line
+	6100 10450 9100 10450
 $EndSCHEMATC
