File: 2000EATX-KiCAD-R12/bus.sch (KiCad schematic (older format))
At the start: 26 parts, among them U302 74HCT32, U800 BUSTER, U801 RTC62423, U802 74HCT138, U803 74HCT08, U804 74LS148

Commit message: Add files via upload
Parts:
- U801: footprint Package_SO:SOIC-24W_7.5x15.4mm_P1.27mm -> AmigaFootprints:SOIC-24W_RTC62423
Changed lines of the file:
@@
 F 3 "http://www.ti.com/lit/gpn/sn74LS32" H 1300 5550 50  0001 C CNN
 	4    1300 5550
-	-1   0    0    1
+	-1   0    0    -1
 $EndComp
 Text GLabel 1000 5550 0    50   Output ~ 0
@@
 	1    0    0    -1
 $EndComp
-Wire Wire Line
-	1600 5650 1750 5650
 $Comp
 L power:+5V #PWR0226
@@
 Connection ~ 2600 7950
 Wire Wire Line
-	1750 4950 1750 5650
-Wire Wire Line
-	1600 5450 1650 5450
-Wire Wire Line
-	1650 5450 1650 5750
+	1750 4950 1750 5450
 Wire Wire Line
 	9500 2900 9500 3000
@@
 L power:GND #PWR0229
 U 1 1 605C2481
-P 4050 8150
-F 0 "#PWR0229" H 4050 7900 50  0001 C CNN
-F 1 "GND" H 4055 7977 50  0000 C CNN
-F 2 "" H 4050 8150 50  0001 C CNN
-F 3 "" H 4050 8150 50  0001 C CNN
-	1    4050 8150
+P 4050 8250
+F 0 "#PWR0229" H 4050 8000 50  0001 C CNN
+F 1 "GND" H 4055 8077 50  0000 C CNN
+F 2 "" H 4050 8250 50  0001 C CNN
+F 3 "" H 4050 8250 50  0001 C CNN
+	1    4050 8250
 	1    0    0    -1
 $EndComp
@@
 L power:GND #PWR0234
 U 1 1 605C2FFC
-P 1650 5750
-F 0 "#PWR0234" H 1650 5500 50  0001 C CNN
-F 1 "GND" H 1655 5577 50  0000 C CNN
-F 2 "" H 1650 5750 50  0001 C CNN
-F 3 "" H 1650 5750 50  0001 C CNN
-	1    1650 5750
+P 1600 5950
+F 0 "#PWR0234" H 1600 5700 50  0001 C CNN
+F 1 "GND" H 1605 5777 50  0000 C CNN
+F 2 "" H 1600 5950 50  0001 C CNN
+F 3 "" H 1600 5950 50  0001 C CNN
+	1    1600 5950
 	1    0    0    -1
 $EndComp
@@
 F 0 "U801" H 8325 9065 50  0000 C CNN
 F 1 "RTC62423" H 8325 8974 50  0000 C CNN
-F 2 "Package_SO:SOIC-24W_7.5x15.4mm_P1.27mm" H 8150 8600 50  0001 C CNN
+F 2 "AmigaFootprints:SOIC-24W_RTC62423" H 8150 8600 50  0001 C CNN
 F 3 "" H 8150 8600 50  0001 C CNN
 	1    8350 8350
@@
 Wire Wire Line
 	8850 4250 11300 4250
+Wire Wire Line
+	1600 5650 1600 5950
+Wire Wire Line
+	1600 5450 1750 5450
+Wire Wire Line
+	4050 8250 4050 8150
 $EndSCHEMATC
