File: 2000EATX-KiCAD-INSANE-JUMPER-EDITION/memory.sch (KiCad schematic (older format))
At the start: 44 parts, among them U500 KICKSTART, U501 74HCT00, U502 CY74FCT821T, U503 CY62167ELL-45ZXI SRAM, U504 CY74FCT821T, U540 74AHCT244, U541 74AHCT244

Commit message: Add files via upload
Parts:
- removed JA23, JA24, JA25, JA26, JA27, JA28, JA29, JA30, JA31, JA32, JA33: 8375/8372A, Jumper:SolderJumper-3_P1.3mm_Bridged12_RoundedPad1.0x1.5mm, symbol Jumper:SolderJumper_3_Bridged12
- added U505: CY62157, Package_SO:TSOP-II-44_10.16x18.41mm_P0.8mm, symbol Amiga-Library:CY62157
- R500-1, R500-10, R500-11, R500-12, R500-13, R500-14, R500-15, R500-2, R500-3, R500-4, R500-5, R500-6, R500-7, R500-8, R500-9: renamed from R?; footprint (none) -> Resistor_SMD:R_1206_3216Metric
- U503: value CY62167ELL-45ZXI SRAM -> CY62167ELL-45ZXI 1MX16 SRAM; footprint Package_SO:TSOP-II-44_10.16x18.41mm_P0.8mm -> Package_SO:TSOP-I-48_18.4x12mm_P0.5mm
- U503: value CY62167ELL-45ZXI SRAM -> CY62167ELL-45ZXI 1MX16 SRAM; footprint (none) -> Package_SO:TSOP-I-48_18.4x12mm_P0.5mm
- U540, U541: footprint (none) -> Package_SO:SOIC-20W_7.5x12.8mm_P1.27mm
Connections:
- net CAS: now also U501.6; no longer U501.3
- net DRAB9: now also JA22.1 (A)
- net GND: now also U505.41 (_OE)
- net RAS: now also U501.3; no longer U501.6
- net _MCASL: now also U501.4, U505.39 (_BLE); no longer U501.1
- net _MCASU: now also U501.5, U505.40 (_BHE); no longer U501.2
- net _MRAS1: now also JA22.3 (B); no longer R500-15.1, U501.5
- net _MWE: now also U505.17 (_WE)
- net _SRAMCE: now reaches U501.8, U503.26 (_CE1)
- net _SRAMCE: now also U505.6 (_CE)
- net DRAC5: now reaches U503.1 (A15)
- net DRAC5: now also U502.19 (Y4), U505.22 (A14)
- net DRAC8: now reaches U503.16 (A18)
- net DRAC8: now also U502.22 (Y1), U505.19 (A17)
- net DRAC7: now reaches U503.17 (A17)
- net DRAC7: now also U502.21 (Y2), U505.20 (A16)
- net DRAD7: now reaches U503.18 (A7), U504.21 (Y2)
- net DRAD7: now also U505.42 (A7)
- net DRAD6: now reaches U503.19 (A6), U504.20 (Y3)
- net DRAD6: now also U505.43 (A6)
- net DRAC4: now reaches U503.2 (A14)
- net DRAC4: now also U502.18 (Y5), U505.23 (A13)
- net DRAD5: now reaches U503.20 (A5), U504.19 (Y4)
- net DRAD5: now also U505.44 (A5)
- net DRAD4: now reaches U503.21 (A4), U504.18 (Y5)
- net DRAD4: now also U505.1 (A4)
- net DRAD3: now reaches U503.22 (A3), U504.17 (Y6)
- net DRAD3: now also U505.2 (A3)
- net DRAD2: now reaches U503.23 (A2), U504.16 (Y7)
- net DRAD2: now also U505.3 (A2)
- net DRAD1: now reaches U503.24 (A1), U504.15 (Y8)
- net DRAD1: now also U505.4 (A1)
- net DRAD0: now reaches U503.25 (A0), U504.14 (Y9)
- net DRAD0: now also U505.5 (A0)
- net DRAC3: now reaches U503.3 (A13)
- net DRAC3: now also U502.17 (Y6), U505.24 (A12)
- net DRAC2: now reaches U503.4 (A12)
- net DRAC2: now also U502.16 (Y7), U505.25 (A11)
- net DRAC6: now reaches U503.48 (A16)
- net DRAC6: now also U502.20 (Y3), U505.21 (A15)
- net DRAC1: now reaches U503.5 (A11)
- net DRAC1: now also U502.15 (Y8), U505.26 (A10)
- net DRAC0: now reaches U503.6 (A10)
- net DRAC0: now also U502.14 (Y9), U505.27 (A9)
- net at JA22.2 (C): now also U502.2 (D0); no longer U503.7 (A9)
- net DRAD8: now reaches U503.8 (A8), U504.22 (Y1)
- net DRAD8: now also U505.28 (A8)
- net DRAC9: now reaches U503.9 (A19)
- net DRAC9: now also U502.23 (Y0), U505.18 (A18)
- net DRAD9: now reaches U504.23 (Y0)
- net DRAD9: now also U503.7 (A9); no longer JA22.1 (A)
- net _MRAS0: no longer names the net of R500-14.1
- net _MRAS0: now also U501.1; no longer U501.4
- new net: R500-15.1, U501.2
Other:
- note added: "2.0"
- moved on the sheet: C540, C541, R500, R500-1, R500-10, R500-11, R500-12, R500-13, R500-14, R500-15, R500-2, R500-3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

Commit message: Add files via upload
Connections:
- net +5V: now also C540.2, C541.2, U540.20 (VCC), U541.20 (VCC); no longer C540.1, C541.1
- net DRA0: now also U540.2 (I0a); no longer U541.4 (I1a)
- net DRA1: now also U540.4 (I1a); no longer U541.2 (I0a)
- net DRA2: now also U540.6 (I2a); no longer U540.17 (I3b)
- net DRA3: now also U540.8 (I3a); no longer U540.15 (I2b)
- net DRA4: now also U540.11 (I0b); no longer U540.13 (I1b)
- net DRA5: now also U540.13 (I1b); no longer U540.11 (I0b)
- net DRA6: now also U540.15 (I2b); no longer U540.8 (I3a)
- net DRA7: now also U540.17 (I3b); no longer U540.6 (I2a)
- net DRA8: now also U541.2 (I0a); no longer U540.4 (I1a)
- net DRA9: now also U541.4 (I1a); no longer U540.2 (I0a)
- net DRAB0: now also R500-1.1, RN503.3 (R2), U502.2 (D0), U504.7 (D5); no longer R500-10.1, RN504.6 (R5), U502.11 (D9), U504.11 (D9)
- net DRAB1: now also R500-2.1, RN503.5 (R4), U502.3 (D1), U504.8 (D6); no longer R500-9.1, RN504.5 (R4), U502.10 (D8), U504.10 (D8)
- net DRAB2: now also R500-3.1, RN504.2 (R1), U502.4 (D2); no longer R500-8.1, RN504.4 (R3), U502.9 (D7)
- net DRAB3: now also R500-4.1, RN504.4 (R3), U502.5 (D3), U504.10 (D8); no longer R500-7.1, RN504.3 (R2), U502.8 (D6), U504.8 (D6)
- net DRAB4: now also R500-5.1, RN503.6 (R5), U502.6 (D4), U504.11 (D9); no longer R500-6.1, RN504.2 (R1), U502.7 (D5), U504.7 (D5)
- net DRAB5: now also R500-6.1, RN504.3 (R2), U502.7 (D5); no longer R500-5.1, RN503.6 (R5), U502.6 (D4)
- net DRAB6: now also R500-7.1, RN503.4 (R3), U502.8 (D6); no longer R500-4.1, RN503.5 (R4), U502.5 (D3)
- net DRAB7: now also R500-8.1, RN503.2 (R1), U502.9 (D7); no longer R500-3.1, RN503.4 (R3), U502.4 (D2)
- net DRAB8: now also R500-9.1, RN504.5 (R4), U502.10 (D8); no longer R500-2.1, RN503.3 (R2), U502.3 (D1)
- net DRAB9: now also R500-10.1, RN504.6 (R5); no longer R500-1.1, RN503.2 (R1)
- net DRAC0: now also U502.23 (Y0), U503.25 (A0), U505.5 (A0); no longer U502.14 (Y9), U503.6 (A10), U505.27 (A9)
- net DRAC1: now also U502.22 (Y1), U503.24 (A1), U505.4 (A1); no longer U502.15 (Y8), U503.5 (A11), U505.26 (A10)
- net DRAC2: now also U502.21 (Y2), U503.23 (A2), U505.3 (A2); no longer U502.16 (Y7), U503.4 (A12), U505.25 (A11)
- net DRAC3: now also U502.20 (Y3), U503.22 (A3), U505.2 (A3); no longer U502.17 (Y6), U503.3 (A13), U505.24 (A12)
- net DRAC4: now also U502.19 (Y4), U503.21 (A4), U505.1 (A4); no longer U502.18 (Y5), U503.2 (A14), U505.23 (A13)
- net DRAC5: now also U502.18 (Y5), U503.20 (A5), U505.44 (A5); no longer U502.19 (Y4), U503.1 (A15), U505.22 (A14)
- net DRAC6: now also U502.17 (Y6), U503.19 (A6), U505.43 (A6); no longer U502.20 (Y3), U503.48 (A16), U505.21 (A15)
- net DRAC7: now also U502.16 (Y7), U503.18 (A7), U505.42 (A7); no longer U502.21 (Y2), U503.17 (A17), U505.20 (A16)
- net DRAC8: now also U502.15 (Y8), U503.8 (A8), U505.28 (A8); no longer U502.22 (Y1), U503.16 (A18), U505.19 (A17)
- net DRAC9: now also U502.14 (Y9), U503.7 (A9); no longer U502.23 (Y0), U503.9 (A19)
- net DRAD0: now also U503.6 (A10), U504.18 (Y5), U505.27 (A9); no longer U503.25 (A0), U504.14 (Y9), U505.5 (A0)
- net DRAD1: now also U503.5 (A11), U504.17 (Y6), U505.26 (A10); no longer U503.24 (A1), U504.15 (Y8), U505.4 (A1)
- net DRAD2: now also U503.4 (A12), U505.25 (A11); no longer U503.23 (A2), U505.3 (A2)
- net DRAD3: now also U503.3 (A13), U504.15 (Y8), U505.24 (A12); no longer U503.22 (A3), U504.17 (Y6), U505.2 (A3)
- net DRAD4: now also U503.2 (A14), U504.14 (Y9), U505.23 (A13); no longer U503.21 (A4), U504.18 (Y5), U505.1 (A4)
- net DRAD5: now also U503.1 (A15), U505.22 (A14); no longer U503.20 (A5), U505.44 (A5)
- net DRAD6: now also U503.48 (A16), U505.21 (A15); no longer U503.19 (A6), U505.43 (A6)
- net DRAD7: now also U503.17 (A17), U505.20 (A16); no longer U503.18 (A7), U505.42 (A7)
- net DRAD8: now also U503.16 (A18), U505.19 (A17); no longer U503.8 (A8), U505.28 (A8)
- net DRAD9: now also U503.9 (A19); no longer U503.7 (A9)
- net GND: now also C540.1, C541.1, U541.15 (I2b); no longer U541.17 (I3b)
- net _MRAS1: now also R500-14.1, U501.1
- net _RAS0: now also U541.17 (I3b); no longer U541.13 (I1b)
- net _RAS1: now also U541.13 (I1b); no longer U541.15 (I2b)
- net at JA22.2 (C): now also U502.11 (D9); no longer U502.2 (D0)
- net at U541.3 (O3b): now also R500-15.2
- net at U541.5 (O2b): no longer R500-15.2
- net _MRAS0: now reaches R500-15.1, U501.2
Other:
- moved on the sheet: C540, C541

Commit message: Add files via upload
Parts:
- removed U505: CY62157, Package_SO:TSOP-II-44_10.16x18.41mm_P0.8mm, symbol Amiga-Library:CY62157
- added JA13: 8375/8372A, Jumper:SolderJumper-3_P1.3mm_Bridged12_RoundedPad1.0x1.5mm, symbol Jumper:SolderJumper_3_Bridged12
- renumbered JA22 to JA14
Connections:
- net DRA8: now also JA13.3 (B); no longer U541.2 (I0a)
- net DRA9: now also JA13.1 (A); no longer U541.4 (I1a)
- net DRAB0: now also JA14.1 (A); no longer U504.7 (D5)
- net DRAB9: now also U502.11 (D9); no longer JA14.1 (A)
- net DRABx: now reaches JA14.2 (C)
- net DRABx: now also U504.7 (D5); no longer U502.11 (D9)
- net DRA1 renamed DRA1-0
- net DRA2 renamed DRA2-1
- net DRA3 renamed DRA3-2
- net DRA4 renamed DRA4-3
- net DRA5 renamed DRA5-4
- net DRA6 renamed DRA6-5
- net DRA7 renamed DRA7-6
- net DRAD0 renamed DRADx
- new net DRA8-7: U541.2 (I0a)
- new net DRA9-8: JA13.2 (C), U541.4 (I1a)
Other:
- note removed: "2.0"
- moved on the sheet: JA14

Commit message: Add files via upload
Other:
- moved on the sheet: JA13
Changed lines of the file:
@@
 	7950 2800 6100 2800
 Wire Wire Line
-	7950 4200 6100 4200
+	7950 4200 7100 4200
 Wire Wire Line
 	7950 4300 6850 4300
@@
 	6100 2800 6000 2700
 Entry Wire Line
-	6100 4200 6000 4100
+	6100 3500 6000 3400
 Wire Bus Line
 	6000 1450 1550 1450
@@
 L Jumper:SolderJumper_3_Bridged12 JA?
 U 1 1 6183D00D
-P 6700 3700
+P 6700 4000
 AR Path="/61252A60/6183D00D" Ref="JA?"  Part="1"
 AR Path="/6089B263/6183D00D" Ref="JA13"  Part="1"
-F 0 "JA13" V 6654 3768 50  0000 L CNN
-F 1 "8375/8372A" V 6745 3768 50  0000 L CNN
-F 2 "Jumper:SolderJumper-3_P1.3mm_Bridged12_RoundedPad1.0x1.5mm" H 6700 3700 50  0001 C CNN
-F 3 "~" H 6700 3700 50  0001 C CNN
-	1    6700 3700
+F 0 "JA13" V 6654 4068 50  0000 L CNN
+F 1 "8375/8372A" V 6745 4068 50  0000 L CNN
+F 2 "Jumper:SolderJumper-3_P1.3mm_Bridged12_RoundedPad1.0x1.5mm" H 6700 4000 50  0001 C CNN
+F 3 "~" H 6700 4000 50  0001 C CNN
+	1    6700 4000
 	0    -1   -1   0
 $EndComp
 Wire Wire Line
-	6700 3500 6100 3500
-Wire Wire Line
-	6700 3900 6100 3900
-Entry Wire Line
-	6100 3500 6000 3400
-Entry Wire Line
-	6100 3900 6000 3800
-Wire Wire Line
-	6850 3700 6850 4300
-Text Label 6150 3900 0    51   ~ 0
+	6700 3800 6100 3800
+Wire Wire Line
+	6700 4200 6100 4200
+Entry Wire Line
+	6100 3800 6000 3700
+Entry Wire Line
+	6100 4200 6000 4100
+Text Label 6150 4200 0    51   ~ 0
 DRA9
-Text Label 6150 3500 0    51   ~ 0
+Text Label 6150 3800 0    51   ~ 0
 DRA8
 Entry Wire Line
@@
 Wire Wire Line
 	11250 4050 11700 4050
+Wire Wire Line
+	7100 4200 7100 3500
+Wire Wire Line
+	7100 3500 6100 3500
+Wire Wire Line
+	6850 4000 6850 4300
 Wire Bus Line
 	6000 1450 6000 4100

Commit message: Add files via upload
Other:
- note added: "J500 IS OMITTED\nPERMANENTLY SET \nTO MAX CHIP RAM"
- note added: "NOTE: The 8375 signal is the before the dash,\nthe 8372A signal is after the dash.\n\nJumpers default to 8375, all part numbers\ndefined with Agnus multiadapter."
- note removed: "J500 IS OMITTED\nPERMANENTLY SET \nTO 1M CHIP RAM"
Changed lines of the file:
@@
 	10700 6650 9100 6650
 Text Notes 9800 7600 0    50   ~ 0
-J500 IS OMITTED\nPERMANENTLY SET \nTO 1M CHIP RAM
+J500 IS OMITTED\nPERMANENTLY SET \nTO MAX CHIP RAM
 $Comp
 L Device:C C501
@@
 Wire Bus Line
 	15650 1350 15650 3300
+Text Notes 5100 1200 0    79   ~ 0
+NOTE: The 8375 signal is the before the dash,\nthe 8372A signal is after the dash.\n\nJumpers default to 8375, all part numbers\ndefined with Agnus multiadapter.
 $EndSCHEMATC

Commit message: Add files via upload
Connections:
- net DRA0 renamed DRA0-G
- net DRA9-8: no longer names the net of JA13.2 (C), U541.4 (I1a)
Other:
- note added: "DRA SIGNAL Description\n8372A Left - 8375 Right"
- note added: "Jumpers default to 8375, all part numbers\ndefined with Agnus multiadapter."
- note removed: "NOTE: The 8375 signal is the before the dash,\nthe 8372A signal is after the dash.\n\nJumpers default to 8375, all part numbers\ndefined with Agnus multiadapter."
- moved on the sheet: R500, U500A

Commit message: Add files via upload
Parts:
- U503: symbol Amiga-Library:CY62157 -> Amiga-Library:CY62167
Connections:
- net +5V: now also U503.37 (Vcc); no longer U503.11 (Vcc)
- net DRAB1: now also U504.6 (D4); no longer U504.8 (D6)
- net DRAB2: now also U504.7 (D5); no longer U504.9 (D7)
- net DRAB3: now also U504.8 (D6); no longer U504.10 (D8)
- net DRAB4: now also U504.9 (D7); no longer U504.11 (D9)
- net DRAB5: now also U504.10 (D8); no longer U504.6 (D4)
- net DRAB6: now also U504.11 (D9); no longer U504.5 (D3)
- net DRAB7: now also U504.2 (D0); no longer U504.4 (D2)
- net DRAB9: now also U504.4 (D2); no longer U504.2 (D0)
- net DRABx: now also U504.5 (D3); no longer U504.7 (D5)
- net DRAD1: now also U504.19 (Y4); no longer U504.17 (Y6)
- net DRAD2: now also U504.18 (Y5); no longer U504.16 (Y7)
- net DRAD3: now also U504.17 (Y6); no longer U504.15 (Y8)
- net DRAD4: now also U504.16 (Y7); no longer U504.14 (Y9)
- net DRAD5: now also U504.15 (Y8); no longer U504.19 (Y4)
- net DRAD6: now also U504.14 (Y9); no longer U504.20 (Y3)
- net DRAD7: now also U504.23 (Y0); no longer U504.21 (Y2)
- net DRAD9: now also U504.21 (Y2); no longer U504.23 (Y0)
- net DRADx: now also U504.20 (Y3); no longer U504.18 (Y5)
- net GND: now also U503.27 (Vss), U503.46 (Vss); no longer U503.12 (Vss), U503.34 (Vss)
Changed lines of the file:
@@
 	2100 7450 2750 7450
 $Comp
-L Amiga-Library:CY62157 U503
+L Amiga-Library:CY62167 U503
 U 2 1 60608AA1
 P 10050 9600
@@
 	12350 3650 11900 3650
 Wire Wire Line
-	12350 3750 11900 3750
+	12350 3750 12000 3750
 Wire Wire Line
 	12350 3850 11900 3850
 Wire Wire Line
-	12350 3950 12000 3950
+	12350 3950 11900 3950
 Wire Wire Line
 	12350 4050 11900 4050
@@
 Entry Wire Line
 	11900 3650 11800 3750
-Entry Wire Line
-	11900 3750 11800 3850
 Entry Wire Line
 	11900 3850 11800 3950
@@
 	11900 4350 11800 4450
 Text Label 12050 3450 0    51   ~ 0
-DRAB9
+DRAB7
 Text Label 12050 4350 0    51   ~ 0
-DRAB4
+DRAB6
 Text Label 12050 3550 0    51   ~ 0
 DRAB8
 Text Label 12050 3650 0    51   ~ 0
-DRAB7
+DRAB9
 Text Label 12050 3750 0    51   ~ 0
-DRAB6
+DRABx
 Text Label 12050 3850 0    51   ~ 0
+DRAB1
+Text Label 12050 3950 0    51   ~ 0
+DRAB2
+Text Label 12050 4050 0    51   ~ 0
+DRAB3
+Text Label 12050 4150 0    51   ~ 0
+DRAB4
+Text Label 12050 4250 0    51   ~ 0
 DRAB5
-Text Label 12050 3950 0    51   ~ 0
-DRABx
-Text Label 12050 4050 0    51   ~ 0
-DRAB1
-Text Label 12050 4150 0    51   ~ 0
-DRAB2
-Text Label 12050 4250 0    51   ~ 0
-DRAB3
 Text Label 13050 2850 0    51   ~ 0
 RAS
@@
 DRAC0
 Text Label 13050 3950 0    51   ~ 0
+DRAD2
+Text Label 13050 4050 0    51   ~ 0
+DRAD3
+Text Label 13050 4150 0    51   ~ 0
+DRAD4
+Text Label 13050 4250 0    51   ~ 0
+DRAD5
+Text Label 13050 4350 0    51   ~ 0
+DRAD6
+Text Label 13050 3750 0    51   ~ 0
 DRADx
-Text Label 13050 4050 0    51   ~ 0
-DRAD1
-Text Label 13050 4150 0    51   ~ 0
-DRAD2
-Text Label 13050 4250 0    51   ~ 0
-DRAD3
-Text Label 13050 4350 0    51   ~ 0
-DRAD4
-Text Label 13050 3750 0    51   ~ 0
-DRAD6
 Text Label 13050 3550 0    51   ~ 0
 DRAD8
 Text Label 13050 3650 0    51   ~ 0
-DRAD7
+DRAD9
 Text Label 14400 5950 0    51   ~ 0
 _SRAMCE
@@
 	11900 2700 12350 2700
 Text Label 13050 3450 0    51   ~ 0
-DRAD9
+DRAD7
 Text Label 13850 1800 2    51   ~ 0
 DRAD9
@@
 DRAC6
 Text Label 13050 3850 0    51   ~ 0
-DRAD5
+DRAD1
 Text Label 13850 3200 2    51   ~ 0
 DRAC5
@@
 Wire Wire Line
 	11550 4550 12000 4550
-Wire Wire Line
-	12000 4550 12000 3950
 Entry Wire Line
 	11700 4050 11800 4150
@@
 Wire Wire Line
 	1550 2800 7950 2800
+Entry Wire Line
+	11900 3950 11800 4050
+Wire Wire Line
+	12000 4550 12000 3750
 Wire Bus Line
 	11800 1750 11800 4450

Commit message: Add files via upload
Parts:
- JA13, JA14: footprint Jumper:SolderJumper-3_P1.3mm_Bridged12_RoundedPad1.0x1.5mm -> Jumper:SolderJumper-3_P1.3mm_Open_RoundedPad1.0x1.5mm; symbol Jumper:SolderJumper_3_Bridged12 -> Jumper:SolderJumper_3_Open
Other:
- note added: "DRA SIGNAL Description\n8375 Left - 8372A Right"
- note added: "JUMPERS MUST BE CONFIGURED BY AGNUS PART NUMBER"
- note removed: "DRA SIGNAL Description\n8372A Left - 8375 Right"
- note removed: "Jumpers default to 8375, all part numbers\ndefined with Agnus multiadapter."
Changed lines of the file:
@@
 Sheet 13 14
 Title "Amiga 2000 EATX"
-Date "2021-08-25"
+Date "2021-09-19"
 Rev "2.0"
 Comp ""
@@
 	4050 6500 4050 6100
 $Comp
-L Jumper:SolderJumper_3_Bridged12 JA?
+L Jumper:SolderJumper_3_Open JA?
 U 1 1 612556F6
 P 11250 4250
@@
 F 0 "JA14" V 11204 4318 50  0000 L CNN
 F 1 "8375/8372A" V 11295 4318 50  0000 L CNN
-F 2 "Jumper:SolderJumper-3_P1.3mm_Bridged12_RoundedPad1.0x1.5mm" H 11250 4250 50  0001 C CNN
+F 2 "Jumper:SolderJumper-3_P1.3mm_Open_RoundedPad1.0x1.5mm" H 11250 4250 50  0001 C CNN
 F 3 "~" H 11250 4250 50  0001 C CNN
 	1    11250 4250
@@
 DRAB9
 $Comp
-L Jumper:SolderJumper_3_Bridged12 JA?
+L Jumper:SolderJumper_3_Open JA?
 U 1 1 6183D00D
 P 6700 4000
@@
 F 0 "JA13" V 6654 4068 50  0000 L CNN
 F 1 "8375/8372A" V 6745 4068 50  0000 L CNN
-F 2 "Jumper:SolderJumper-3_P1.3mm_Bridged12_RoundedPad1.0x1.5mm" H 6700 4000 50  0001 C CNN
+F 2 "Jumper:SolderJumper-3_P1.3mm_Open_RoundedPad1.0x1.5mm" H 6700 4000 50  0001 C CNN
 F 3 "~" H 6700 4000 50  0001 C CNN
 	1    6700 4000
@@
 Wire Wire Line
 	6850 4000 6850 4300
-Text Notes 5100 1000 0    79   ~ 0
-Jumpers default to 8375, all part numbers\ndefined with Agnus multiadapter.
+Text Notes 3500 800  0    118  ~ 0
+JUMPERS MUST BE CONFIGURED BY AGNUS PART NUMBER
 Text Notes 1200 1100 0    79   ~ 0
-DRA SIGNAL Description\n8372A Left - 8375 Right
+DRA SIGNAL Description\n8375 Left - 8372A Right
 Text GLabel 1550 3050 0    51   Input ~ 0
 DRA8-7
