File: 2000EATX-KiCAD-INSANE-JUMPER-EDITION/Agnus-Multi.sch (KiCad schematic (older format))
At the start: 24 parts, among them J102 Short for NTSC

Commit message: Add files via upload
Parts:
- added C101: 0.1uF, Capacitor_SMD:C_1206_3216Metric, symbol Device:C
- added R109: 4.7k, Resistor_SMD:R_1206_3216Metric, symbol Device:R
- added unit 2 of U101
- gave numbers to parts that had none: 1
Connections:
- net +5V: now also C101.1, R109.1, U101.15 (VCC)
- net GND: now also C101.2, U101.58 (GND), U101.82 (GND)
- net XCLK: no longer names the net of JA1.3 (B)
- net _XCLKEN: no longer names the net of JA2.3 (B)
- net _XCLKEN: now also R109.2
- no-connect marks 1 -> 2
Changed lines of the file:
@@
 DRA0
 $Comp
-L Amiga-Library:Agnus_MULTI U?
+L Amiga-Library:Agnus_MULTI U101
 U 1 1 613F8639
 P 8950 4950
-F 0 "U?" H 8950 2127 50  0000 C CNN
+F 0 "U101" H 8950 2127 50  0000 C CNN
 F 1 "Agnus_MULTI" H 8950 2036 50  0000 C CNN
 F 2 "Package_LCC:PLCC-84_THT-Socket" H 8950 4830 50  0001 C CNN
@@
 	14700 7600 14700 7700
 $Comp
-L power:GND #PWR?
+L power:GND #PWR0356
 U 1 1 61475A2F
 P 14700 7700
-F 0 "#PWR?" H 14700 7450 50  0001 C CNN
+F 0 "#PWR0356" H 14700 7450 50  0001 C CNN
 F 1 "GND" H 14705 7527 50  0000 C CNN
 F 2 "" H 14700 7700 50  0001 C CNN
@@
 _CDAC
 Wire Wire Line
-	10700 6900 11600 6900
-Wire Wire Line
-	11600 6900 11600 8350
-Wire Wire Line
-	11600 8350 15250 8350
+	10700 6900 11400 6900
 Wire Wire Line
 	10700 7300 11550 7300
 Wire Wire Line
 	11550 7300 11550 8150
-Text GLabel 15250 8350 2    51   Input ~ 0
-_XCLKEN
 Wire Wire Line
 	9650 7100 10450 7100
@@
 Text GLabel 1550 2800 0    51   Output ~ 0
 DRD[0..15]
-$Comp
-L Jumper:SolderJumper_3_Bridged12 JA1
-U 1 1 61528D88
-P 6500 4200
-F 0 "JA1" V 6454 4268 50  0000 L CNN
-F 1 "8375/8372A" V 6545 4268 50  0000 L CNN
-F 2 "Jumper:SolderJumper-3_P1.3mm_Bridged12_RoundedPad1.0x1.5mm" H 6500 4200 50  0001 C CNN
-F 3 "~" H 6500 4200 50  0001 C CNN
-	1    6500 4200
-	0    -1   1    0
-$EndComp
 Wire Wire Line
 	6650 4200 6900 4200
@@
 Text GLabel 1550 4000 0    51   Input ~ 0
 A20
-Wire Wire Line
-	6500 4400 1550 4400
-Text GLabel 1550 4400 0    51   Input ~ 0
-XCLK
 Wire Wire Line
 	8250 6800 6800 6800
@@
 $EndComp
 $Comp
-L power:GND #PWR?
+L power:GND #PWR0358
 U 1 1 6172C6D7
 P 9250 9800
-F 0 "#PWR?" H 9250 9550 50  0001 C CNN
+F 0 "#PWR0358" H 9250 9550 50  0001 C CNN
 F 1 "GND" H 9255 9627 50  0000 C CNN
 F 2 "" H 9250 9800 50  0001 C CNN
@@
 	9000 9400 8550 9400
 $Comp
-L power:+5V #PWR?
+L power:+5V #PWR0359
 U 1 1 61780C14
 P 9000 9100
-F 0 "#PWR?" H 9000 8950 50  0001 C CNN
+F 0 "#PWR0359" H 9000 8950 50  0001 C CNN
 F 1 "+5V" H 9015 9273 50  0000 C CNN
 F 2 "" H 9000 9100 50  0001 C CNN
@@
 $EndComp
 $Comp
-L power:GND #PWR?
+L power:GND #PWR0360
 U 1 1 6178115A
 P 7750 9400
-F 0 "#PWR?" H 7750 9150 50  0001 C CNN
+F 0 "#PWR0360" H 7750 9150 50  0001 C CNN
 F 1 "GND" H 7755 9227 50  0000 C CNN
 F 2 "" H 7750 9400 50  0001 C CNN
@@
 Wire Wire Line
 	9400 9600 9900 9600
+Wire Wire Line
+	5350 10000 5350 10050
+Wire Wire Line
+	4350 9250 5350 9250
+Wire Wire Line
+	5350 9250 5350 9200
+$Comp
+L power:GND #PWR0362
+U 1 1 61ADE61F
+P 5350 10050
+F 0 "#PWR0362" H 5350 9800 50  0001 C CNN
+F 1 "GND" H 5355 9877 50  0000 C CNN
+F 2 "" H 5350 10050 50  0001 C CNN
+F 3 "" H 5350 10050 50  0001 C CNN
+	1    5350 10050
+	1    0    0    -1
+$EndComp
+$Comp
+L power:+5V #PWR0377
+U 1 1 61ADE92B
+P 5350 9200
+F 0 "#PWR0377" H 5350 9050 50  0001 C CNN
+F 1 "+5V" H 5365 9373 50  0000 C CNN
+F 2 "" H 5350 9200 50  0001 C CNN
+F 3 "" H 5350 9200 50  0001 C CNN
+	1    5350 9200
+	1    0    0    -1
+$EndComp
+$Comp
+L Device:C C101
+U 1 1 61AE14A0
+P 5350 9600
+F 0 "C101" H 5465 9646 50  0000 L CNN
+F 1 "0.1uF" H 5465 9555 50  0000 L CNN
+F 2 "Capacitor_SMD:C_1206_3216Metric" H 5388 9450 50  0001 C CNN
+F 3 "~" H 5350 9600 50  0001 C CNN
+	1    5350 9600
+	1    0    0    -1
+$EndComp
+Wire Wire Line
+	5350 9450 5350 9250
+Connection ~ 5350 9250
+Wire Wire Line
+	5350 9750 5350 10000
+Connection ~ 5350 10000
+$Comp
+L Amiga-Library:Agnus_MULTI U101
+U 2 1 61B0FA8D
+P 4350 9600
+F 0 "U101" H 4628 9621 50  0000 L CNN
+F 1 "Agnus_MULTI" H 4628 9530 50  0000 L CNN
+F 2 "Package_LCC:PLCC-84_THT-Socket" H 4350 9480 50  0001 C CNN
+F 3 "" H 4250 11150 50  0001 C CNN
+	2    4350 9600
+	1    0    0    -1
+$EndComp
+Wire Wire Line
+	4200 10000 4500 10000
+Connection ~ 4500 10000
+Wire Wire Line
+	4500 10000 5350 10000
+$Comp
+L Jumper:SolderJumper_3_Bridged12 JA1
+U 1 1 61528D88
+P 6500 4200
+F 0 "JA1" V 6454 4268 50  0000 L CNN
+F 1 "8375/8372A" V 6545 4268 50  0000 L CNN
+F 2 "Jumper:SolderJumper-3_P1.3mm_Bridged12_RoundedPad1.0x1.5mm" H 6500 4200 50  0001 C CNN
+F 3 "~" H 6500 4200 50  0001 C CNN
+	1    6500 4200
+	0    -1   1    0
+$EndComp
+NoConn ~ 6500 4400
+Wire Wire Line
+	11400 6900 11400 6150
+$Comp
+L Device:R R109
+U 1 1 612ECADF
+P 11400 6000
+F 0 "R109" H 11470 6046 50  0000 L CNN
+F 1 "4.7k" H 11470 5955 50  0000 L CNN
+F 2 "Resistor_SMD:R_1206_3216Metric" V 11330 6000 50  0001 C CNN
+F 3 "~" H 11400 6000 50  0001 C CNN
+	1    11400 6000
+	1    0    0    -1
+$EndComp
+$Comp
+L power:+5V #PWR0392
+U 1 1 612EECDA
+P 11400 5850
+F 0 "#PWR0392" H 11400 5700 50  0001 C CNN
+F 1 "+5V" H 11415 6023 50  0000 C CNN
+F 2 "" H 11400 5850 50  0001 C CNN
+F 3 "" H 11400 5850 50  0001 C CNN
+	1    11400 5850
+	1    0    0    -1
+$EndComp
 Wire Bus Line
 	10200 5650 10200 8750

Commit message: Add files via upload
Parts:
- removed JA10, JA11, JA12, JA13, JA14, JA15, JA16, JA7, JA8, JA9: 8375/8372A, Jumper:SolderJumper-3_P1.3mm_Bridged12_RoundedPad1.0x1.5mm, symbol Jumper:SolderJumper_3_Bridged12
- added JA7: 8372A, symbol Jumper:SolderJumper_2_Open
- J102: value Short for NTSC -> Short for NTSC or 8375
- renumbered JA21 to JA10, JA17 to JA11, JA18 to JA12, JA19 to JA8, JA20 to JA9
Connections:
- net DRA0: now also U101.42 (DRA0/GND), JA7.1 (A)
- net GND: now also JA1.3 (B), JA7.2 (B)
- net DRA8-7: now reaches U101.50 (DRA8/DRA7)
- net DRA6-5: now reaches U101.48 (DRA6/DRA5)
- net DRA4-3: now reaches U101.46 (DRA4/DRA3)
- net DRA7-6: now reaches U101.49 (DRA7/DRA6)
- net DRA5-4: now reaches U101.47 (DRA5/DRA4)
- net DRA2-1: now reaches U101.44 (DRA2/DRA1)
- net DRA3-2: now reaches U101.45 (DRA3/DRA2)
- net DRA1-0: now reaches U101.43 (DRA1/DRA0)
- net at U101.41 (GND/PAL-NTSC): now also J102.1 (Pin_1), R101.2
- net DRA8: no longer names the net of JA11.3 (B)
- no-connect marks 2 -> 1
Other:
- moved on the sheet: JA1, JA10

Commit message: Add files via upload
Parts:
- removed JA6: 8375/8372A, Jumper:SolderJumper-3_P1.3mm_Bridged12_RoundedPad1.0x1.5mm, symbol Jumper:SolderJumper_3_Bridged12
- removed unit 1 of U101
- added JA6: 8375/8372A, Jumper:SolderJumper-3_P1.3mm_Open_RoundedPad1.0x1.5mm, symbol Jumper:SolderJumper_3_Open
- added U?: Agnus_MULTI, Package_LCC:PLCC-84_THT-Socket, symbol Amiga-Library:Agnus_MULTI
- JA7: footprint (none) -> Jumper:SolderJumper-2_P1.3mm_Open_RoundedPad1.0x1.5mm
- U101: symbol Amiga-Library:Agnus_MULTI -> 2000ATX-rescue:Agnus_MULTI-Amiga-Library
Connections:
- net +5V: now also JA6.1 (A)
- net A1: now also U?.60 (A1)
- net A10: now also U?.69 (A10)
- net A11: now also U?.70 (A11)
- net A12: now also U?.71 (A12)
- net A13: now also U?.72 (A13)
- net A14: now also U?.73 (A14)
- net A15: now also U?.74 (A15)
- net A16: now also U?.75 (A16)
- net A17: now also U?.76 (A17)
- net A18: now also U?.77 (A18)
- net A19: now also U?.59 (A19)
- net A2: now also U?.61 (A2)
- net A3: now also U?.62 (A3)
- net A4: now also U?.63 (A4)
- net A5: now also U?.64 (A5)
- net A6: now also U?.65 (A6)
- net A7: now also U?.66 (A7)
- net A8: now also U?.67 (A8)
- net A9: now also U?.68 (A9)
- net AgnusCLK: now also U?.34 (28MHz)
- net CCK: now also JA6.3 (B)
- net DMAL: now also U?.18 (DMAL)
- net DRA0: now also U?.42 (DRA0/GND)
- net DRA1-0: now also U?.43 (DRA1/DRA0)
- net DRA2-1: now also U?.44 (DRA2/DRA1)
- net DRA3-2: now also U?.45 (DRA3/DRA2)
- net DRA4-3: now also U?.46 (DRA4/DRA3)
- net DRA5-4: now also U?.47 (DRA5/DRA4)
- net DRA6-5: now also U?.48 (DRA6/DRA5)
- net DRA7-6: now also U?.49 (DRA7/DRA6)
- net DRA8-7: now also U?.50 (DRA8/DRA7)
- net DRD0: now also U?.14 (DRD0)
- net DRD1: now also U?.13 (DRD1)
- net DRD10: now also U?.4 (DRD10)
- net DRD11: now also U?.3 (DRD11)
- net DRD12: now also U?.2 (DRD12)
- net DRD13: now also U?.1 (DRD13)
- net DRD14: now also U?.84 (DRD14)
- net DRD15: now also U?.83 (DRD15)
- net DRD2: now also U?.12 (DRD2)
- net DRD3: now also U?.11 (DRD3)
- net DRD4: now also U?.10 (DRD4)
- net DRD5: now also U?.9 (DRD5)
- net DRD6: now also U?.8 (DRD6)
- net DRD7: now also U?.7 (DRD7)
- net DRD8: now also U?.6 (DRD8)
- net DRD9: now also U?.5 (DRD9)
- net RGA1: now also U?.33 (RGA1)
- net RGA2: now also U?.32 (RGA2)
- net RGA3: now also U?.31 (RGA3)
- net RGA4: now also U?.30 (RGA4)
- net RGA5: now also U?.29 (RGA5)
- net RGA6: now also U?.28 (RGA6)
- net RGA7: now also U?.27 (RGA7)
- net RGA8: now also U?.26 (RGA8)
- net R_W: now also U?.22 (R/W)
- net _AS: now also U?.24 (_AS)
- net _BLS: now also U?.19 (_BLS)
- net _CSYNC: now also U?.80 (_CSYNC)
- net _DBR: now also U?.20 (_DBR)
- net _HSYNC: now also U?.81 (_HSYNC)
- net _INT3: now also U?.17 (_INTR)
- net _LPEN: now also U?.78 (_LPEN)
- net _RAMEN: now also U?.25 (_RAMEN)
- net _RAS0: now also U?.57 (_RAS0)
- net _RAS1: now also U?.56 (_RAS1)
- net _REGEN: now also U?.23 (_REGEN)
- net _RST: now also U?.16 (_RESET)
- net _VSYNC: now also U?.79 (_VSYNC)
- net _WE: now also U?.21 (_WE)
- net at JA10.2 (C): now also U?.55 (DRA9/_CASU)
- net at JA9.2 (C): now also U?.54 (_CASU/_CASL)
- net at JA8.2 (C): now also U?.53 (_CASL/_UDS)
- net at JA12.2 (C): now also U?.52 (_UDS/_LDS)
- net at JA11.2 (C): now also U?.51 (_LDS/DRA8)
- net DRA8: now reaches JA11.3 (B)
- net at JA1.2 (C): now also U?.35 (A20/XCLK)
- net at JA2.2 (C): now also U?.36 (_CDAC/_XCLKEN)
- net at JA3.2 (C): now also U?.37 (7MHz/_CDAC)
- net at JA4.2 (C): now also U?.38 (CCKQ/7MHz)
- net at JA5.2 (C): now also U?.39 (CCK/CCKQ)
- net at J102.1 (Pin_1), R101.2: now also U?.41 (GND/PAL-NTSC)
- new net: JA6.2 (C), U?.40 (14M_or_Vbb/CCK)
- no-connect marks 1 -> 0
Other:
- note added: "390554-01 is 14M...leave open\n318069-10 is Vbb...short to +5V"
- note added: "JUMPERS DEFAULT TO 390554-01"
- note added: "SUPPORTS 8372A (ALL PART NUMBERS)\nAND 8375 THE FOLLOWING PART NUMBERS:\n390554-01 AND COMPATIBLE (390554-02, 318069-12, 318069-13)\n318069-10 AND COMPATIBLE (318069-11, 390544-01, 390544-02)"
Changed lines of the file:
@@
 	9650 5350 12000 5350
-$Comp
-L Amiga-Library:Agnus_MULTI U101
-U 1 1 613F8639
-P 8950 4950
-F 0 "U101" H 8950 2127 50  0000 C CNN
-F 1 "Agnus_MULTI" H 8950 2036 50  0000 C CNN
-F 2 "Package_LCC:PLCC-84_THT-Socket" H 8950 4830 50  0001 C CNN
-F 3 "" H 8850 6500 50  0001 C CNN
-	1    8950 4950
-	1    0    0    -1
-$EndComp
 $Comp
 L power:GND #PWR0356
@@
 _RST
 $Comp
-L Jumper:SolderJumper_3_Bridged12 JA6
-U 1 1 615E718E
-P 10800 2550
-F 0 "JA6" V 10846 2618 50  0000 L CNN
-F 1 "8375/8372A" V 10755 2618 50  0000 L CNN
-F 2 "Jumper:SolderJumper-3_P1.3mm_Bridged12_RoundedPad1.0x1.5mm" H 10800 2550 50  0001 C CNN
-F 3 "~" H 10800 2550 50  0001 C CNN
-	1    10800 2550
-	0    1    -1   0
-$EndComp
-$Comp
 L Jumper:SolderJumper_3_Bridged12 JA5
 U 1 1 615E7A4E
@@
 Wire Wire Line
 	10250 2550 10650 2550
-Wire Wire Line
-	10800 2350 15100 2350
 Text GLabel 15250 2350 2    51   Output ~ 0
 CCK
-NoConn ~ 10800 2750
-Wire Wire Line
-	9650 3050 10200 3050
-Wire Wire Line
-	10200 3050 10200 2000
-Wire Wire Line
-	10200 2000 10650 2000
+Wire Wire Line
+	9650 3050 10150 3050
+Wire Wire Line
+	10150 3050 10150 2000
+Wire Wire Line
+	10150 2000 10650 2000
 Wire Wire Line
 	10800 2200 15100 2200
@@
 CCKQ
 Wire Wire Line
-	9650 2900 10150 2900
-Wire Wire Line
-	10150 2900 10150 1450
-Wire Wire Line
-	10150 1450 10650 1450
+	9650 2900 10000 2900
+Wire Wire Line
+	10000 2900 10000 1450
+Wire Wire Line
+	10000 1450 10650 1450
 Wire Wire Line
 	10800 1650 15100 1650
@@
 Connection ~ 5350 10000
 $Comp
-L Amiga-Library:Agnus_MULTI U101
+L 2000ATX-rescue:Agnus_MULTI-Amiga-Library U101
 U 2 1 61B0FA8D
 P 4350 9600
+AR Path="/61B0FA8D" Ref="U101"  Part="2"
+AR Path="/61252A60/61B0FA8D" Ref="U101"  Part="2"
 F 0 "U101" H 4628 9621 50  0000 L CNN
 F 1 "Agnus_MULTI" H 4628 9530 50  0000 L CNN
@@
 F 0 "JA7" V 13854 7868 50  0000 L CNN
 F 1 "8372A" V 13945 7868 50  0000 L CNN
-F 2 "" H 13900 7800 50  0001 C CNN
+F 2 "Jumper:SolderJumper-2_P1.3mm_Open_RoundedPad1.0x1.5mm" H 13900 7800 50  0001 C CNN
 F 3 "~" H 13900 7800 50  0001 C CNN
 	1    13900 7800
@@
 Wire Bus Line
 	1650 6300 1650 6350
+Text Label 1850 6200 0    51   ~ 0
+DRA8
+$Comp
+L Jumper:SolderJumper_3_Open JA6
+U 1 1 61426B23
+P 10800 2550
+F 0 "JA6" V 10846 2618 50  0000 L CNN
+F 1 "8375/8372A" V 10755 2618 50  0000 L CNN
+F 2 "Jumper:SolderJumper-3_P1.3mm_Open_RoundedPad1.0x1.5mm" H 10800 2550 50  0001 C CNN
+F 3 "~" H 10800 2550 50  0001 C CNN
+	1    10800 2550
+	0    1    -1   0
+$EndComp
+Wire Wire Line
+	10800 2350 15100 2350
+Wire Wire Line
+	10800 2750 15100 2750
+$Comp
+L power:+5V #PWR?
+U 1 1 6144A127
+P 15100 2650
+F 0 "#PWR?" H 15100 2500 50  0001 C CNN
+F 1 "+5V" H 15115 2823 50  0000 C CNN
+F 2 "" H 15100 2650 50  0001 C CNN
+F 3 "" H 15100 2650 50  0001 C CNN
+	1    15100 2650
+	1    0    0    -1
+$EndComp
+Wire Wire Line
+	15100 2750 15100 2650
+Text Notes 11400 2750 0    51   ~ 0
+390554-01 is 14M...leave open\n318069-10 is Vbb...short to +5V
+Text Notes 800  1600 0    157  ~ 0
+SUPPORTS 8372A (ALL PART NUMBERS)\nAND 8375 THE FOLLOWING PART NUMBERS:\n390554-01 AND COMPATIBLE (390554-02, 318069-12, 318069-13)\n318069-10 AND COMPATIBLE (318069-11, 390544-01, 390544-02)
+Text Notes 10500 1050 0    157  ~ 0
+JUMPERS DEFAULT TO 390554-01
 Wire Bus Line
 	10200 5650 10200 8750
@@
 Wire Bus Line
 	7700 4650 7700 6450
+$Comp
+L Amiga-Library:Agnus_MULTI U?
+U 1 1 614B5F28
+P 8950 4950
+F 0 "U?" H 8950 2127 50  0000 C CNN
+F 1 "Agnus_MULTI" H 8950 2036 50  0000 C CNN
+F 2 "Package_LCC:PLCC-84_THT-Socket" H 8950 4830 50  0001 C CNN
+F 3 "" H 8850 6500 50  0001 C CNN
+	1    8950 4950
+	1    0    0    -1
+$EndComp
 $EndSCHEMATC

Commit message: Add files via upload
Parts:
- removed J102: Short for NTSC or 8375, Connector_PinHeader_2.54mm:PinHeader_1x02_P2.54mm_Vertical, symbol Connector:Conn_01x02_Male
- added C112: 0.1uF, Capacitor_SMD:C_1206_3216Metric, symbol Device:C
- added J102: Short for 8327A NTSC or 8375, Jumper:SolderJumper-2_P1.3mm_Open_RoundedPad1.0x1.5mm, symbol Jumper:SolderJumper_2_Open
- gave numbers to parts that had none: 1
Connections:
- net +5V: now also C112.2
- net GND: now also C112.1, J102.1 (A)
- net at R101.2, U101.41 (GND/PAL-NTSC): now also J102.2 (B)
Changed lines of the file:
@@
 	10200 8750 1550 8750
 Text GLabel 1550 8750 0    51   Output ~ 0
-RGA[0..8]
+RGA[1..8]
 Wire Wire Line
 	8750 2500 8750 2400
@@
 Wire Wire Line
 	9900 9400 9000 9400
-$Comp
-L Connector:Conn_01x02_Male J102
-U 1 1 61740319
-P 8550 9200
-F 0 "J102" V 8500 9100 50  0000 L CNN
-F 1 "Short for NTSC or 8375" V 8400 8600 50  0000 L CNN
-F 2 "Connector_PinHeader_2.54mm:PinHeader_1x02_P2.54mm_Vertical" H 8550 9200 50  0001 C CNN
-F 3 "~" H 8550 9200 50  0001 C CNN
-	1    8550 9200
-	0    1    1    0
-$EndComp
-Wire Wire Line
-	8450 9400 7750 9400
+Wire Wire Line
+	8350 9400 7750 9400
 $Comp
 L Device:R R101
@@
 Connection ~ 9000 9400
 Wire Wire Line
-	9000 9400 8550 9400
+	9000 9400 8650 9400
 $Comp
 L power:+5V #PWR0359
@@
 	6500 4250 5300 4250
 $Comp
-L power:GND #PWR?
+L power:GND #PWR0211
 U 1 1 61486053
 P 5300 4250
-F 0 "#PWR?" H 5300 4000 50  0001 C CNN
+F 0 "#PWR0211" H 5300 4000 50  0001 C CNN
 F 1 "GND" H 5305 4077 50  0000 C CNN
 F 2 "" H 5300 4250 50  0001 C CNN
@@
 	10800 2350 15100 2350
 Wire Wire Line
-	10800 2750 15100 2750
-$Comp
-L power:+5V #PWR?
+	10800 2750 14050 2750
+$Comp
+L power:+5V #PWR0355
 U 1 1 6144A127
 P 15100 2650
-F 0 "#PWR?" H 15100 2500 50  0001 C CNN
+F 0 "#PWR0355" H 15100 2500 50  0001 C CNN
 F 1 "+5V" H 15115 2823 50  0000 C CNN
 F 2 "" H 15100 2650 50  0001 C CNN
@@
 Text Notes 10500 1050 0    157  ~ 0
 JUMPERS DEFAULT TO 390554-01
-Wire Bus Line
-	10200 5650 10200 8750
-Wire Bus Line
-	15150 4550 15150 7550
-Wire Bus Line
-	7700 2800 7700 4300
-Wire Bus Line
-	7700 4650 7700 6450
-$Comp
-L Amiga-Library:Agnus_MULTI U?
+$Comp
+L Amiga-Library:Agnus_MULTI U101
 U 1 1 614B5F28
 P 8950 4950
-F 0 "U?" H 8950 2127 50  0000 C CNN
+AR Path="/614B5F28" Ref="U101"  Part="1"
+AR Path="/61252A60/614B5F28" Ref="U101"  Part="1"
+F 0 "U101" H 8950 2127 50  0000 C CNN
 F 1 "Agnus_MULTI" H 8950 2036 50  0000 C CNN
 F 2 "Package_LCC:PLCC-84_THT-Socket" H 8950 4830 50  0001 C CNN
@@
 	1    0    0    -1
 $EndComp
+$Comp
+L Device:C C112
+U 1 1 6143A513
+P 14050 2600
+F 0 "C112" H 14165 2646 50  0000 L CNN
+F 1 "0.1uF" H 14165 2555 50  0000 L CNN
+F 2 "Capacitor_SMD:C_1206_3216Metric" H 14088 2450 50  0001 C CNN
+F 3 "~" H 14050 2600 50  0001 C CNN
+	1    14050 2600
+	1    0    0    -1
+$EndComp
+Connection ~ 14050 2750
+Wire Wire Line
+	14050 2750 15100 2750
+$Comp
+L power:GND #PWR0358
+U 1 1 6143E439
+P 13750 2450
+F 0 "#PWR0358" H 13750 2200 50  0001 C CNN
+F 1 "GND" H 13755 2277 50  0000 C CNN
+F 2 "" H 13750 2450 50  0001 C CNN
+F 3 "" H 13750 2450 50  0001 C CNN
+	1    13750 2450
+	1    0    0    -1
+$EndComp
+Wire Wire Line
+	13750 2450 14050 2450
+$Comp
+L Jumper:SolderJumper_2_Open J102
+U 1 1 61566589
+P 8500 9400
+F 0 "J102" H 8500 9500 50  0000 C CNN
+F 1 "Short for 8327A NTSC or 8375" H 8500 9250 50  0000 C CNN
+F 2 "Jumper:SolderJumper-2_P1.3mm_Open_RoundedPad1.0x1.5mm" H 8500 9400 50  0001 C CNN
+F 3 "~" H 8500 9400 50  0001 C CNN
+	1    8500 9400
+	1    0    0    -1
+$EndComp
+Wire Bus Line
+	10200 5650 10200 8750
+Wire Bus Line
+	15150 4550 15150 7550
+Wire Bus Line
+	7700 2800 7700 4300
+Wire Bus Line
+	7700 4650 7700 6450
 $EndSCHEMATC

Commit message: Add files via upload
Connections:
- net DRA0 renamed DRA0-G
Other:
- note added: "SIGNAL Description\n8375 Left - 8372A Right"
Changed lines of the file:
@@
 	2550 5800 1550 5800
 Wire Wire Line
-	6450 6200 1750 6200
-Wire Wire Line
-	13750 4650 15050 4650
+	6450 6200 1550 6200
+Wire Wire Line
+	13750 4650 15250 4650
 Text GLabel 15250 4150 2    51   Output ~ 0
 _WE
@@
 	10250 3950 15250 3950
 Wire Wire Line
-	15050 4950 13300 4950
+	15250 4950 13300 4950
 Wire Wire Line
 	13300 4950 13300 4550
@@
 	9650 4550 13300 4550
 Wire Wire Line
-	15050 5250 13150 5250
+	15250 5250 13150 5250
 Wire Wire Line
 	13150 5250 13150 4650
@@
 	12950 4750 12950 5650
 Wire Wire Line
-	12950 5650 15050 5650
-Wire Wire Line
-	15050 6000 12800 6000
+	12950 5650 15250 5650
+Wire Wire Line
+	15250 6000 12800 6000
 Wire Wire Line
 	12800 6000 12800 4850
@@
 	9650 4750 12950 4750
 Wire Wire Line
-	15050 6400 12600 6400
-Wire Wire Line
 	12600 6400 12600 4950
 Wire Wire Line
 	9650 4950 12600 4950
 Wire Wire Line
-	15050 6750 12450 6750
+	15250 6750 12450 6750
 Wire Wire Line
 	12450 6750 12450 5050
@@
 	12300 5150 12300 7100
 Wire Wire Line
-	12300 7100 15050 7100
-Wire Wire Line
-	15050 7450 12150 7450
+	12300 7100 15250 7100
+Wire Wire Line
+	15250 7450 12150 7450
 Wire Wire Line
 	12150 7450 12150 5250
@@
 	1    0    0    -1
 $EndComp
-Text Label 14700 4650 0    51   ~ 0
-DRA9
-Text Label 14700 4950 0    51   ~ 0
-DRA8-7
-Text Label 14700 5250 0    51   ~ 0
-DRA7-6
-Text Label 14700 5650 0    51   ~ 0
-DRA6-5
-Text Label 14700 6000 0    51   ~ 0
-DRA5-4
-Text Label 14700 6400 0    51   ~ 0
-DRA4-3
-Text Label 14700 6750 0    51   ~ 0
-DRA3-2
-Text Label 14700 7100 0    51   ~ 0
-DRA2-1
-Text Label 14700 7450 0    51   ~ 0
-DRA1-0
-Text Label 14700 7650 0    51   ~ 0
-DRA0
-Entry Wire Line
-	15050 4950 15150 4850
-Entry Wire Line
-	15050 4650 15150 4550
-Entry Wire Line
-	15050 5250 15150 5150
-Entry Wire Line
-	15050 5650 15150 5550
-Entry Wire Line
-	15050 6000 15150 5900
-Entry Wire Line
-	15050 6400 15150 6300
-Entry Wire Line
-	15050 6750 15150 6650
-Entry Wire Line
-	15050 7100 15150 7000
-Entry Wire Line
-	15050 7450 15150 7350
-Wire Bus Line
-	15150 4550 15250 4550
-Text GLabel 15250 4550 2    51   Output ~ 0
-DRA[0..9]
 Wire Wire Line
 	13900 7650 12000 7650
@@
 $EndComp
 Wire Wire Line
-	13900 7650 15050 7650
+	13900 7650 15250 7650
 Connection ~ 13900 7650
-Entry Wire Line
-	15050 7650 15150 7550
-Text GLabel 1550 6350 0    51   Output ~ 0
-DRA[0..9]
-Entry Wire Line
-	1750 6200 1650 6300
-Wire Bus Line
-	1650 6350 1550 6350
+Text GLabel 1550 6200 0    51   Output ~ 0
+DRA8
 Wire Wire Line
 	13900 7950 14500 7950
@@
 Wire Bus Line
 	1950 4650 1550 4650
-Wire Bus Line
-	1650 6300 1650 6350
-Text Label 1850 6200 0    51   ~ 0
-DRA8
 $Comp
 L Jumper:SolderJumper_3_Open JA6
@@
 	1    0    0    -1
 $EndComp
+Wire Wire Line
+	12600 6400 15250 6400
+Text Notes 16050 6300 2    79   ~ 0
+SIGNAL Description\n8375 Left - 8372A Right
+Text GLabel 15250 4950 2    51   Output ~ 0
+DRA8-7
+Text GLabel 15250 4650 2    51   Output ~ 0
+DRA9
+Text GLabel 15250 5250 2    51   Output ~ 0
+DRA7-6
+Text GLabel 15250 5650 2    51   Output ~ 0
+DRA6-5
+Text GLabel 15250 6000 2    51   Output ~ 0
+DRA5-4
+Text GLabel 15250 6400 2    51   Output ~ 0
+DRA4-3
+Text GLabel 15250 6750 2    51   Output ~ 0
+DRA3-2
+Text GLabel 15250 7100 2    51   Output ~ 0
+DRA2-1
+Text GLabel 15250 7450 2    51   Output ~ 0
+DRA1-0
+Text GLabel 15250 7650 2    51   Output ~ 0
+DRA0-G
 Wire Bus Line
 	10200 5650 10200 8750
 Wire Bus Line
-	15150 4550 15150 7550
-Wire Bus Line
 	7700 2800 7700 4300
