File: 2000EATX-KiCAD-INSANE-JUMPER-EDITION/Processor.sch (KiCad schematic (older format))
At the start: 19 parts, among them U100 MC68000, U103 74HCT245, U104 74HCT373, U105 74HCT245, U106 74HCT373, U303 74HCT08

Commit message: Add files via upload
Changed lines of the file:
@@
 Sheet 3 14
 Title "Amiga 2000 EATX"
-Date "2021-08-21"
+Date "2021-09-19"
 Rev "2.0"
 Comp ""
@@
 U 1 1 604AE2BE
 P 4750 4050
-F 0 "U100" H 4750 6631 50  0000 C CNN
+F 0 "U?" H 4750 6631 50  0000 C CNN
 F 1 "MC68000" H 4750 6540 50  0000 C CNN
 F 2 "Package_DIP:DIP-64_W22.86mm_Socket" H 4750 4050 50  0001 C CNN
@@
 U 1 1 604B0AF4
 P 7900 3100
-F 0 "U103" H 7900 4081 50  0000 C CNN
+F 0 "U?" H 7900 4081 50  0000 C CNN
 F 1 "74HCT245" H 7900 3990 50  0000 C CNN
 F 2 "Package_SO:SOIC-20W_7.5x12.8mm_P1.27mm" H 7900 3100 50  0001 C CNN
@@
 U 1 1 604B176E
 P 7900 5250
-F 0 "U105" H 7900 6231 50  0000 C CNN
+F 0 "U?" H 7900 6231 50  0000 C CNN
 F 1 "74HCT245" H 7900 6140 50  0000 C CNN
 F 2 "Package_SO:SOIC-20W_7.5x12.8mm_P1.27mm" H 7900 5250 50  0001 C CNN
@@
 U 1 1 604B299F
 P 9850 2550
-F 0 "U104" H 9850 3531 50  0000 C CNN
+F 0 "U?" H 9850 3531 50  0000 C CNN
 F 1 "74HCT373" H 9850 3440 50  0000 C CNN
 F 2 "Package_SO:SOIC-20W_7.5x12.8mm_P1.27mm" H 9850 2550 50  0001 C CNN
@@
 U 1 1 604B32EB
 P 9850 4700
-F 0 "U106" H 9850 5681 50  0000 C CNN
+F 0 "U?" H 9850 5681 50  0000 C CNN
 F 1 "74HCT373" H 9850 5590 50  0000 C CNN
 F 2 "Package_SO:SOIC-20W_7.5x12.8mm_P1.27mm" H 9850 4700 50  0001 C CNN
@@
 U 4 1 604B4590
 P 2600 2550
-F 0 "U303" H 2600 2875 50  0000 C CNN
+F 0 "U?" H 2600 2875 50  0000 C CNN
 F 1 "74HCT08" H 2600 2784 50  0000 C CNN
 F 2 "Package_SO:SOIC-14_3.9x8.7mm_P1.27mm" H 2600 2550 50  0001 C CNN
@@
 U 1 1 604BBC77
 P 5350 1450
-F 0 "C100" H 5442 1496 50  0000 L CNN
+F 0 "C?" H 5442 1496 50  0000 L CNN
 F 1 "0.1uF" H 5442 1405 50  0000 L CNN
 F 2 "Capacitor_SMD:C_1206_3216Metric" H 5350 1450 50  0001 C CNN
@@
 U 1 1 604BC934
 P 7300 4300
-F 0 "C105" H 7392 4346 50  0000 L CNN
+F 0 "C?" H 7392 4346 50  0000 L CNN
 F 1 "0.1uF" H 7392 4255 50  0000 L CNN
 F 2 "Capacitor_SMD:C_1206_3216Metric" H 7300 4300 50  0001 C CNN
@@
 U 1 1 604BD21B
 P 7350 2150
-F 0 "C103" H 7442 2196 50  0000 L CNN
+F 0 "C?" H 7442 2196 50  0000 L CNN
 F 1 "0.1uF" H 7442 2105 50  0000 L CNN
 F 2 "Capacitor_SMD:C_1206_3216Metric" H 7350 2150 50  0001 C CNN
@@
 U 1 1 604BDA4A
 P 10600 1700
-F 0 "C104" H 10692 1746 50  0000 L CNN
+F 0 "C?" H 10692 1746 50  0000 L CNN
 F 1 "0.1uF" H 10692 1655 50  0000 L CNN
 F 2 "Capacitor_SMD:C_1206_3216Metric" H 10600 1700 50  0001 C CNN
@@
 U 1 1 604BE218
 P 10650 3900
-F 0 "C106" H 10742 3946 50  0000 L CNN
+F 0 "C?" H 10742 3946 50  0000 L CNN
 F 1 "0.1uF" H 10742 3855 50  0000 L CNN
 F 2 "Capacitor_SMD:C_1206_3216Metric" H 10650 3900 50  0001 C CNN
@@
 U 1 1 604D36AF
 P 3700 4300
-F 0 "R917" H 3759 4346 50  0000 L CNN
+F 0 "R?" H 3759 4346 50  0000 L CNN
 F 1 "470" H 3759 4255 50  0000 L CNN
 F 2 "Resistor_SMD:R_1206_3216Metric" H 3700 4300 50  0001 C CNN
@@
 U 1 1 604D3E13
 P 3200 4450
-F 0 "R1000" H 3259 4496 50  0000 L CNN
+F 0 "R?" H 3259 4496 50  0000 L CNN
 F 1 "470" H 3259 4405 50  0000 L CNN
 F 2 "Resistor_SMD:R_1206_3216Metric" H 3200 4450 50  0001 C CNN
@@
 U 1 1 604D4948
 P 1950 4950
-F 0 "R111" H 2009 4996 50  0000 L CNN
+F 0 "R?" H 2009 4996 50  0000 L CNN
 F 1 "470" H 2009 4905 50  0000 L CNN
 F 2 "Resistor_SMD:R_1206_3216Metric" H 1950 4950 50  0001 C CNN
@@
 U 1 1 604D57CA
 P 2000 2350
-F 0 "R104" H 2059 2396 50  0000 L CNN
+F 0 "R?" H 2059 2396 50  0000 L CNN
 F 1 "4.7k" H 2059 2305 50  0000 L CNN
 F 2 "Resistor_SMD:R_1206_3216Metric" H 2000 2350 50  0001 C CNN
@@
 U 1 1 604D6FA2
 P 2800 3950
-F 0 "XR1" H 2859 3996 50  0000 L CNN
+F 0 "XR?" H 2859 3996 50  0000 L CNN
 F 1 "68" H 2859 3905 50  0000 L CNN
 F 2 "Resistor_SMD:R_1206_3216Metric" H 2800 3950 50  0001 C CNN
@@
 U 1 1 604D7BB8
 P 2800 4150
-F 0 "XC1" H 2892 4196 50  0000 L CNN
+F 0 "XC?" H 2892 4196 50  0000 L CNN
 F 1 "270pf" H 2892 4105 50  0000 L CNN
 F 2 "Capacitor_SMD:C_1206_3216Metric" H 2800 4150 50  0001 C CNN
@@
 U 1 1 6051F4AC
 P 5350 1550
-F 0 "#PWR0101" H 5350 1300 50  0001 C CNN
+F 0 "#PWR?" H 5350 1300 50  0001 C CNN
 F 1 "GND" H 5355 1377 50  0000 C CNN
 F 2 "" H 5350 1550 50  0001 C CNN
@@
 U 1 1 6051F9B4
 P 5350 1350
-F 0 "#PWR0102" H 5350 1200 50  0001 C CNN
+F 0 "#PWR?" H 5350 1200 50  0001 C CNN
 F 1 "+5V" H 5365 1523 50  0000 C CNN
 F 2 "" H 5350 1350 50  0001 C CNN
@@
 U 1 1 605323A6
 P 7350 2250
-F 0 "#PWR0103" H 7350 2000 50  0001 C CNN
+F 0 "#PWR?" H 7350 2000 50  0001 C CNN
 F 1 "GND" H 7355 2077 50  0000 C CNN
 F 2 "" H 7350 2250 50  0001 C CNN
@@
 U 1 1 60532D45
 P 7350 2050
-F 0 "#PWR0104" H 7350 1900 50  0001 C CNN
+F 0 "#PWR?" H 7350 1900 50  0001 C CNN
 F 1 "+5V" H 7365 2223 50  0000 C CNN
 F 2 "" H 7350 2050 50  0001 C CNN
@@
 U 1 1 6053C64D
 P 7900 3900
-F 0 "#PWR0105" H 7900 3650 50  0001 C CNN
+F 0 "#PWR?" H 7900 3650 50  0001 C CNN
 F 1 "GND" H 7905 3727 50  0000 C CNN
 F 2 "" H 7900 3900 50  0001 C CNN
@@
 U 1 1 6053CD93
 P 7300 4400
-F 0 "#PWR0106" H 7300 4150 50  0001 C CNN
+F 0 "#PWR?" H 7300 4150 50  0001 C CNN
 F 1 "GND" H 7305 4227 50  0000 C CNN
 F 2 "" H 7300 4400 50  0001 C CNN
@@
 U 1 1 6053D4DD
 P 7900 6050
-F 0 "#PWR0107" H 7900 5800 50  0001 C CNN
+F 0 "#PWR?" H 7900 5800 50  0001 C CNN
 F 1 "GND" H 7905 5877 50  0000 C CNN
 F 2 "" H 7900 6050 50  0001 C CNN
@@
 U 1 1 6053DCD8
 P 9850 5500
-F 0 "#PWR0108" H 9850 5250 50  0001 C CNN
+F 0 "#PWR?" H 9850 5250 50  0001 C CNN
 F 1 "GND" H 9855 5327 50  0000 C CNN
 F 2 "" H 9850 5500 50  0001 C CNN
@@
 U 1 1 6053E3AA
 P 7300 4200
-F 0 "#PWR0109" H 7300 4050 50  0001 C CNN
+F 0 "#PWR?" H 7300 4050 50  0001 C CNN
 F 1 "+5V" H 7315 4373 50  0000 C CNN
 F 2 "" H 7300 4200 50  0001 C CNN
@@
 U 1 1 605484D4
 P 10650 4000
-F 0 "#PWR0110" H 10650 3750 50  0001 C CNN
+F 0 "#PWR?" H 10650 3750 50  0001 C CNN
 F 1 "GND" H 10655 3827 50  0000 C CNN
 F 2 "" H 10650 4000 50  0001 C CNN
@@
 U 1 1 6054902B
 P 10600 1800
-F 0 "#PWR0111" H 10600 1550 50  0001 C CNN
+F 0 "#PWR?" H 10600 1550 50  0001 C CNN
 F 1 "GND" H 10605 1627 50  0000 C CNN
 F 2 "" H 10600 1800 50  0001 C CNN
@@
 U 1 1 60549A9D
 P 10600 1600
-F 0 "#PWR0112" H 10600 1450 50  0001 C CNN
+F 0 "#PWR?" H 10600 1450 50  0001 C CNN
 F 1 "+5V" H 10615 1773 50  0000 C CNN
 F 2 "" H 10600 1600 50  0001 C CNN
@@
 U 1 1 6054B765
 P 10650 3800
-F 0 "#PWR0113" H 10650 3650 50  0001 C CNN
+F 0 "#PWR?" H 10650 3650 50  0001 C CNN
 F 1 "+5V" H 10665 3973 50  0000 C CNN
 F 2 "" H 10650 3800 50  0001 C CNN
@@
 U 1 1 604CE9D6
 P 9850 3350
-F 0 "#PWR0114" H 9850 3100 50  0001 C CNN
+F 0 "#PWR?" H 9850 3100 50  0001 C CNN
 F 1 "GND" H 9855 3177 50  0000 C CNN
 F 2 "" H 9850 3350 50  0001 C CNN
@@
 U 1 1 604F5279
 P 2000 2250
-F 0 "#PWR0115" H 2000 2100 50  0001 C CNN
+F 0 "#PWR?" H 2000 2100 50  0001 C CNN
 F 1 "+5V" H 2015 2423 50  0000 C CNN
 F 2 "" H 2000 2250 50  0001 C CNN
@@
 U 1 1 604F5B47
 P 1050 800
-F 0 "#PWR0116" H 1050 650 50  0001 C CNN
+F 0 "#PWR?" H 1050 650 50  0001 C CNN
 F 1 "+5V" H 1065 973 50  0000 C CNN
 F 2 "" H 1050 800 50  0001 C CNN
@@
 U 1 1 60529232
 P 2800 4250
-F 0 "#PWR0117" H 2800 4000 50  0001 C CNN
+F 0 "#PWR?" H 2800 4000 50  0001 C CNN
 F 1 "GND" H 2805 4077 50  0000 C CNN
 F 2 "" H 2800 4250 50  0001 C CNN
@@
 U 1 1 60537B05
 P 1150 3550
-F 0 "#PWR0118" H 1150 3400 50  0001 C CNN
+F 0 "#PWR?" H 1150 3400 50  0001 C CNN
 F 1 "+5V" H 1165 3723 50  0000 C CNN
 F 2 "" H 1150 3550 50  0001 C CNN
@@
 U 1 1 605CF8B3
 P 1950 4850
-F 0 "#PWR0119" H 1950 4700 50  0001 C CNN
+F 0 "#PWR?" H 1950 4700 50  0001 C CNN
 F 1 "+5V" H 1965 5023 50  0000 C CNN
 F 2 "" H 1950 4850 50  0001 C CNN
@@
 U 1 1 60610E02
 P 4850 6450
-F 0 "#PWR0120" H 4850 6200 50  0001 C CNN
+F 0 "#PWR?" H 4850 6200 50  0001 C CNN
 F 1 "GND" H 4855 6277 50  0000 C CNN
 F 2 "" H 4850 6450 50  0001 C CNN
@@
 U 1 1 60653FAE
 P 3200 4350
-F 0 "#PWR0121" H 3200 4200 50  0001 C CNN
+F 0 "#PWR?" H 3200 4200 50  0001 C CNN
 F 1 "+5V" H 3215 4523 50  0000 C CNN
 F 2 "" H 3200 4350 50  0001 C CNN
@@
 U 1 1 6066D128
 P 3700 4200
-F 0 "#PWR0122" H 3700 4050 50  0001 C CNN
+F 0 "#PWR?" H 3700 4050 50  0001 C CNN
 F 1 "+5V" H 3715 4373 50  0000 C CNN
 F 2 "" H 3700 4200 50  0001 C CNN
@@
 U 1 1 6064DC50
 P 1450 1000
-F 0 "RN100" H 1938 1046 50  0000 L CNN
+F 0 "RN?" H 1938 1046 50  0000 L CNN
 F 1 "4.7k" H 1938 955 50  0000 L CNN
 F 2 "Resistor_THT:R_Array_SIP10" V 2025 1000 50  0001 C CNN
@@
 U 1 1 60685F24
 P 1550 3750
-F 0 "RN101" H 2038 3796 50  0000 L CNN
+F 0 "RN?" H 2038 3796 50  0000 L CNN
 F 1 "2.7k" H 2038 3705 50  0000 L CNN
 F 2 "Resistor_THT:R_Array_SIP10" V 2125 3750 50  0001 C CNN

Commit message: Add files via upload
Changed lines of the file:
@@
 encoding utf-8
 Sheet 3 14
-Title "Amiga 2000 EATX"
-Date "2021-09-19"
-Rev "2.0"
+Title ""
+Date ""
+Rev ""
 Comp ""
 Comment1 ""
@@
 U 1 1 604AE2BE
 P 4750 4050
-F 0 "U?" H 4750 6631 50  0000 C CNN
+F 0 "U100" H 4750 6631 50  0000 C CNN
 F 1 "MC68000" H 4750 6540 50  0000 C CNN
 F 2 "Package_DIP:DIP-64_W22.86mm_Socket" H 4750 4050 50  0001 C CNN
@@
 U 1 1 604B0AF4
 P 7900 3100
-F 0 "U?" H 7900 4081 50  0000 C CNN
+F 0 "U103" H 7900 4081 50  0000 C CNN
 F 1 "74HCT245" H 7900 3990 50  0000 C CNN
 F 2 "Package_SO:SOIC-20W_7.5x12.8mm_P1.27mm" H 7900 3100 50  0001 C CNN
@@
 U 1 1 604B176E
 P 7900 5250
-F 0 "U?" H 7900 6231 50  0000 C CNN
+F 0 "U105" H 7900 6231 50  0000 C CNN
 F 1 "74HCT245" H 7900 6140 50  0000 C CNN
 F 2 "Package_SO:SOIC-20W_7.5x12.8mm_P1.27mm" H 7900 5250 50  0001 C CNN
@@
 U 1 1 604B299F
 P 9850 2550
-F 0 "U?" H 9850 3531 50  0000 C CNN
+F 0 "U104" H 9850 3531 50  0000 C CNN
 F 1 "74HCT373" H 9850 3440 50  0000 C CNN
 F 2 "Package_SO:SOIC-20W_7.5x12.8mm_P1.27mm" H 9850 2550 50  0001 C CNN
@@
 U 1 1 604B32EB
 P 9850 4700
-F 0 "U?" H 9850 5681 50  0000 C CNN
+F 0 "U106" H 9850 5681 50  0000 C CNN
 F 1 "74HCT373" H 9850 5590 50  0000 C CNN
 F 2 "Package_SO:SOIC-20W_7.5x12.8mm_P1.27mm" H 9850 4700 50  0001 C CNN
@@
 U 4 1 604B4590
 P 2600 2550
-F 0 "U?" H 2600 2875 50  0000 C CNN
+F 0 "U303" H 2600 2875 50  0000 C CNN
 F 1 "74HCT08" H 2600 2784 50  0000 C CNN
 F 2 "Package_SO:SOIC-14_3.9x8.7mm_P1.27mm" H 2600 2550 50  0001 C CNN
@@
 U 1 1 604BBC77
 P 5350 1450
-F 0 "C?" H 5442 1496 50  0000 L CNN
+F 0 "C100" H 5442 1496 50  0000 L CNN
 F 1 "0.1uF" H 5442 1405 50  0000 L CNN
 F 2 "Capacitor_SMD:C_1206_3216Metric" H 5350 1450 50  0001 C CNN
@@
 U 1 1 604BC934
 P 7300 4300
-F 0 "C?" H 7392 4346 50  0000 L CNN
+F 0 "C105" H 7392 4346 50  0000 L CNN
 F 1 "0.1uF" H 7392 4255 50  0000 L CNN
 F 2 "Capacitor_SMD:C_1206_3216Metric" H 7300 4300 50  0001 C CNN
@@
 U 1 1 604BD21B
 P 7350 2150
-F 0 "C?" H 7442 2196 50  0000 L CNN
+F 0 "C103" H 7442 2196 50  0000 L CNN
 F 1 "0.1uF" H 7442 2105 50  0000 L CNN
 F 2 "Capacitor_SMD:C_1206_3216Metric" H 7350 2150 50  0001 C CNN
@@
 U 1 1 604BDA4A
 P 10600 1700
-F 0 "C?" H 10692 1746 50  0000 L CNN
+F 0 "C104" H 10692 1746 50  0000 L CNN
 F 1 "0.1uF" H 10692 1655 50  0000 L CNN
 F 2 "Capacitor_SMD:C_1206_3216Metric" H 10600 1700 50  0001 C CNN
@@
 U 1 1 604BE218
 P 10650 3900
-F 0 "C?" H 10742 3946 50  0000 L CNN
+F 0 "C106" H 10742 3946 50  0000 L CNN
 F 1 "0.1uF" H 10742 3855 50  0000 L CNN
 F 2 "Capacitor_SMD:C_1206_3216Metric" H 10650 3900 50  0001 C CNN
@@
 U 1 1 604D36AF
 P 3700 4300
-F 0 "R?" H 3759 4346 50  0000 L CNN
+F 0 "R917" H 3759 4346 50  0000 L CNN
 F 1 "470" H 3759 4255 50  0000 L CNN
 F 2 "Resistor_SMD:R_1206_3216Metric" H 3700 4300 50  0001 C CNN
@@
 U 1 1 604D3E13
 P 3200 4450
-F 0 "R?" H 3259 4496 50  0000 L CNN
+F 0 "R1000" H 3259 4496 50  0000 L CNN
 F 1 "470" H 3259 4405 50  0000 L CNN
 F 2 "Resistor_SMD:R_1206_3216Metric" H 3200 4450 50  0001 C CNN
@@
 U 1 1 604D4948
 P 1950 4950
-F 0 "R?" H 2009 4996 50  0000 L CNN
+F 0 "R111" H 2009 4996 50  0000 L CNN
 F 1 "470" H 2009 4905 50  0000 L CNN
 F 2 "Resistor_SMD:R_1206_3216Metric" H 1950 4950 50  0001 C CNN
@@
 U 1 1 604D57CA
 P 2000 2350
-F 0 "R?" H 2059 2396 50  0000 L CNN
+F 0 "R104" H 2059 2396 50  0000 L CNN
 F 1 "4.7k" H 2059 2305 50  0000 L CNN
 F 2 "Resistor_SMD:R_1206_3216Metric" H 2000 2350 50  0001 C CNN
@@
 U 1 1 604D6FA2
 P 2800 3950
-F 0 "XR?" H 2859 3996 50  0000 L CNN
+F 0 "XR1" H 2859 3996 50  0000 L CNN
 F 1 "68" H 2859 3905 50  0000 L CNN
 F 2 "Resistor_SMD:R_1206_3216Metric" H 2800 3950 50  0001 C CNN
@@
 U 1 1 604D7BB8
 P 2800 4150
-F 0 "XC?" H 2892 4196 50  0000 L CNN
+F 0 "XC1" H 2892 4196 50  0000 L CNN
 F 1 "270pf" H 2892 4105 50  0000 L CNN
 F 2 "Capacitor_SMD:C_1206_3216Metric" H 2800 4150 50  0001 C CNN
@@
 U 1 1 6051F4AC
 P 5350 1550
-F 0 "#PWR?" H 5350 1300 50  0001 C CNN
+F 0 "#PWR0101" H 5350 1300 50  0001 C CNN
 F 1 "GND" H 5355 1377 50  0000 C CNN
 F 2 "" H 5350 1550 50  0001 C CNN
@@
 U 1 1 6051F9B4
 P 5350 1350
-F 0 "#PWR?" H 5350 1200 50  0001 C CNN
+F 0 "#PWR0102" H 5350 1200 50  0001 C CNN
 F 1 "+5V" H 5365 1523 50  0000 C CNN
 F 2 "" H 5350 1350 50  0001 C CNN
@@
 U 1 1 605323A6
 P 7350 2250
-F 0 "#PWR?" H 7350 2000 50  0001 C CNN
+F 0 "#PWR0103" H 7350 2000 50  0001 C CNN
 F 1 "GND" H 7355 2077 50  0000 C CNN
 F 2 "" H 7350 2250 50  0001 C CNN
@@
 U 1 1 60532D45
 P 7350 2050
-F 0 "#PWR?" H 7350 1900 50  0001 C CNN
+F 0 "#PWR0104" H 7350 1900 50  0001 C CNN
 F 1 "+5V" H 7365 2223 50  0000 C CNN
 F 2 "" H 7350 2050 50  0001 C CNN
@@
 U 1 1 6053C64D
 P 7900 3900
-F 0 "#PWR?" H 7900 3650 50  0001 C CNN
+F 0 "#PWR0105" H 7900 3650 50  0001 C CNN
 F 1 "GND" H 7905 3727 50  0000 C CNN
 F 2 "" H 7900 3900 50  0001 C CNN
@@
 U 1 1 6053CD93
 P 7300 4400
-F 0 "#PWR?" H 7300 4150 50  0001 C CNN
+F 0 "#PWR0106" H 7300 4150 50  0001 C CNN
 F 1 "GND" H 7305 4227 50  0000 C CNN
 F 2 "" H 7300 4400 50  0001 C CNN
@@
 U 1 1 6053D4DD
 P 7900 6050
-F 0 "#PWR?" H 7900 5800 50  0001 C CNN
+F 0 "#PWR0107" H 7900 5800 50  0001 C CNN
 F 1 "GND" H 7905 5877 50  0000 C CNN
 F 2 "" H 7900 6050 50  0001 C CNN
@@
 U 1 1 6053DCD8
 P 9850 5500
-F 0 "#PWR?" H 9850 5250 50  0001 C CNN
+F 0 "#PWR0108" H 9850 5250 50  0001 C CNN
 F 1 "GND" H 9855 5327 50  0000 C CNN
 F 2 "" H 9850 5500 50  0001 C CNN
@@
 U 1 1 6053E3AA
 P 7300 4200
-F 0 "#PWR?" H 7300 4050 50  0001 C CNN
+F 0 "#PWR0109" H 7300 4050 50  0001 C CNN
 F 1 "+5V" H 7315 4373 50  0000 C CNN
 F 2 "" H 7300 4200 50  0001 C CNN
@@
 U 1 1 605484D4
 P 10650 4000
-F 0 "#PWR?" H 10650 3750 50  0001 C CNN
+F 0 "#PWR0110" H 10650 3750 50  0001 C CNN
 F 1 "GND" H 10655 3827 50  0000 C CNN
 F 2 "" H 10650 4000 50  0001 C CNN
@@
 U 1 1 6054902B
 P 10600 1800
-F 0 "#PWR?" H 10600 1550 50  0001 C CNN
+F 0 "#PWR0111" H 10600 1550 50  0001 C CNN
 F 1 "GND" H 10605 1627 50  0000 C CNN
 F 2 "" H 10600 1800 50  0001 C CNN
@@
 U 1 1 60549A9D
 P 10600 1600
-F 0 "#PWR?" H 10600 1450 50  0001 C CNN
+F 0 "#PWR0112" H 10600 1450 50  0001 C CNN
 F 1 "+5V" H 10615 1773 50  0000 C CNN
 F 2 "" H 10600 1600 50  0001 C CNN
@@
 U 1 1 6054B765
 P 10650 3800
-F 0 "#PWR?" H 10650 3650 50  0001 C CNN
+F 0 "#PWR0113" H 10650 3650 50  0001 C CNN
 F 1 "+5V" H 10665 3973 50  0000 C CNN
 F 2 "" H 10650 3800 50  0001 C CNN
@@
 U 1 1 604CE9D6
 P 9850 3350
-F 0 "#PWR?" H 9850 3100 50  0001 C CNN
+F 0 "#PWR0114" H 9850 3100 50  0001 C CNN
 F 1 "GND" H 9855 3177 50  0000 C CNN
 F 2 "" H 9850 3350 50  0001 C CNN
@@
 U 1 1 604F5279
 P 2000 2250
-F 0 "#PWR?" H 2000 2100 50  0001 C CNN
+F 0 "#PWR0115" H 2000 2100 50  0001 C CNN
 F 1 "+5V" H 2015 2423 50  0000 C CNN
 F 2 "" H 2000 2250 50  0001 C CNN
@@
 U 1 1 604F5B47
 P 1050 800
-F 0 "#PWR?" H 1050 650 50  0001 C CNN
+F 0 "#PWR0116" H 1050 650 50  0001 C CNN
 F 1 "+5V" H 1065 973 50  0000 C CNN
 F 2 "" H 1050 800 50  0001 C CNN
@@
 U 1 1 60529232
 P 2800 4250
-F 0 "#PWR?" H 2800 4000 50  0001 C CNN
+F 0 "#PWR0117" H 2800 4000 50  0001 C CNN
 F 1 "GND" H 2805 4077 50  0000 C CNN
 F 2 "" H 2800 4250 50  0001 C CNN
@@
 U 1 1 60537B05
 P 1150 3550
-F 0 "#PWR?" H 1150 3400 50  0001 C CNN
+F 0 "#PWR0118" H 1150 3400 50  0001 C CNN
 F 1 "+5V" H 1165 3723 50  0000 C CNN
 F 2 "" H 1150 3550 50  0001 C CNN
@@
 U 1 1 605CF8B3
 P 1950 4850
-F 0 "#PWR?" H 1950 4700 50  0001 C CNN
+F 0 "#PWR0119" H 1950 4700 50  0001 C CNN
 F 1 "+5V" H 1965 5023 50  0000 C CNN
 F 2 "" H 1950 4850 50  0001 C CNN
@@
 U 1 1 60610E02
 P 4850 6450
-F 0 "#PWR?" H 4850 6200 50  0001 C CNN
+F 0 "#PWR0120" H 4850 6200 50  0001 C CNN
 F 1 "GND" H 4855 6277 50  0000 C CNN
 F 2 "" H 4850 6450 50  0001 C CNN
@@
 U 1 1 60653FAE
 P 3200 4350
-F 0 "#PWR?" H 3200 4200 50  0001 C CNN
+F 0 "#PWR0121" H 3200 4200 50  0001 C CNN
 F 1 "+5V" H 3215 4523 50  0000 C CNN
 F 2 "" H 3200 4350 50  0001 C CNN
@@
 U 1 1 6066D128
 P 3700 4200
-F 0 "#PWR?" H 3700 4050 50  0001 C CNN
+F 0 "#PWR0122" H 3700 4050 50  0001 C CNN
 F 1 "+5V" H 3715 4373 50  0000 C CNN
 F 2 "" H 3700 4200 50  0001 C CNN
@@
 U 1 1 6064DC50
 P 1450 1000
-F 0 "RN?" H 1938 1046 50  0000 L CNN
+F 0 "RN100" H 1938 1046 50  0000 L CNN
 F 1 "4.7k" H 1938 955 50  0000 L CNN
 F 2 "Resistor_THT:R_Array_SIP10" V 2025 1000 50  0001 C CNN
@@
 U 1 1 60685F24
 P 1550 3750
-F 0 "RN?" H 2038 3796 50  0000 L CNN
+F 0 "RN101" H 2038 3796 50  0000 L CNN
 F 1 "2.7k" H 2038 3705 50  0000 L CNN
 F 2 "Resistor_THT:R_Array_SIP10" V 2125 3750 50  0001 C CNN

Commit message: Add files via upload
Other:
- moved on the sheet: C104, C106, U104, U106
