File: 2000EATX-KiCAD-INSANE-JUMPER-EDITION/clocks.sch (KiCad schematic (older format))
At the start: 32 parts, among them J900 Enable Chip RAM slowdown duri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, U102 GARY, U107 74HCT04, U109 74HC258, U302 74HCT32, U900 74HCT00, X1 28.63636MHz, X2 7C-28.63636MBB-T

Commit message: Add files via upload
Parts:
- added C109: 0.1uF, Capacitor_SMD:C_1206_3216Metric, symbol Device:C
- renumbered C666 to C111
Connections:
- net +5V: now also U109.16 (VCC), C109.2
- net GND: now also C109.1
Changed lines of the file:
@@
 $EndComp
 $Comp
-L power:GND #PWR?
+L power:GND #PWR0208
 U 1 1 62D48B9F
 P 5900 9450
-F 0 "#PWR?" H 5900 9200 50  0001 C CNN
+F 0 "#PWR0208" H 5900 9200 50  0001 C CNN
 F 1 "GND" H 5905 9277 50  0000 C CNN
 F 2 "" H 5900 9450 50  0001 C CNN
@@
 	6750 9250 7000 9250
 $Comp
-L Device:C C666
+L Device:C C111
 U 1 1 62F441F4
 P 7600 9400
-F 0 "C666" H 7715 9446 50  0000 L CNN
+F 0 "C111" H 7715 9446 50  0000 L CNN
 F 1 "22pF" H 7715 9355 50  0000 L CNN
 F 2 "Capacitor_SMD:C_1206_3216Metric" H 7638 9250 50  0001 C CNN
@@
 	7300 9250 7600 9250
 $Comp
-L power:GND #PWR?
+L power:GND #PWR0209
 U 1 1 62F7FE78
 P 7600 9550
-F 0 "#PWR?" H 7600 9300 50  0001 C CNN
+F 0 "#PWR0209" H 7600 9300 50  0001 C CNN
 F 1 "GND" H 7605 9377 50  0000 C CNN
 F 2 "" H 7600 9550 50  0001 C CNN
@@
 	5400 8150 5400 7950
 $Comp
-L power:GND #PWR?
+L power:GND #PWR0210
 U 1 1 62F9E115
 P 5000 7650
-F 0 "#PWR?" H 5000 7400 50  0001 C CNN
+F 0 "#PWR0210" H 5000 7400 50  0001 C CNN
 F 1 "GND" H 5005 7477 50  0000 C CNN
 F 2 "" H 5000 7650 50  0001 C CNN
@@
 	5400 8750 5400 8650
 $Comp
-L power:GND #PWR?
+L power:GND #PWR0211
 U 1 1 62FBCC02
 P 5000 8650
-F 0 "#PWR?" H 5000 8400 50  0001 C CNN
+F 0 "#PWR0211" H 5000 8400 50  0001 C CNN
 F 1 "GND" H 5005 8477 50  0000 C CNN
 F 2 "" H 5000 8650 50  0001 C CNN
@@
 Wire Wire Line
 	14550 2150 6250 2150
+$Comp
+L Device:C C109
+U 1 1 61996B04
+P 5250 7200
+F 0 "C109" H 5365 7246 50  0000 L CNN
+F 1 "0.1uF" H 5365 7155 50  0000 L CNN
+F 2 "Capacitor_SMD:C_1206_3216Metric" H 5288 7050 50  0001 C CNN
+F 3 "~" H 5250 7200 50  0001 C CNN
+	1    5250 7200
+	0    -1   -1   0
+$EndComp
+Wire Wire Line
+	5100 7200 5000 7200
+Wire Wire Line
+	5000 7200 5000 7650
+Connection ~ 5000 7650
+Wire Wire Line
+	5400 7200 5400 7550
+Wire Wire Line
+	5400 7550 5900 7550
+Wire Wire Line
+	5400 7200 5400 6800
+Connection ~ 5400 7200
+$Comp
+L power:+5V #PWR0361
+U 1 1 619C3755
+P 5400 6800
+F 0 "#PWR0361" H 5400 6650 50  0001 C CNN
+F 1 "+5V" H 5415 6973 50  0000 C CNN
+F 2 "" H 5400 6800 50  0001 C CNN
+F 3 "" H 5400 6800 50  0001 C CNN
+	1    5400 6800
+	1    0    0    -1
+$EndComp
 Wire Bus Line
 	4550 1950 4550 2550

Commit message: Add files via upload
Parts:
- removed R112: 150, Resistor_SMD:R_1206_3216Metric, symbol Device:R
- added FB103, FB104: Ferrite_Bead, Capacitor_SMD:C_1206_3216Metric, symbol Device:Ferrite_Bead
- J900: footprint Connector_PinHeader_2.54mm:PinHeader_1x02_P2.54mm_Vertical -> Jumper:SolderJumper-2_P1.3mm_Bridged_RoundedPad1.0x1.5mm; symbol Connector:Conn_01x02_Male -> Jumper:SolderJumper_2_Bridged
Connections:
- net 28M: now also FB104.2; no longer FB101.2, U109.13 (I1c)
- net AgnusCLK: now also FB103.1
- net GND: no longer U109.10 (I1d), U109.11 (I0d)
- net at U109.12 (Zc): now also FB103.2
- net at U109.9 (Zd): now also FB104.1
- new net: FB101.2, U109.10 (I1d), U109.11 (I0d), U109.13 (I1c)
- no-connect marks 4 -> 3
Other:
- moved on the sheet: C111
Changed lines of the file:
@@
 Wire Wire Line
 	3450 2650 4950 2650
-Wire Wire Line
-	2500 4600 1800 4600
 Text GLabel 1800 4600 0    50   Input ~ 0
 _BGACK
-Text GLabel 4950 3400 0    50   Output ~ 0
+Text GLabel 1800 3850 0    50   Output ~ 0
 _HLT
 Text GLabel 1750 5850 0    50   Input ~ 0
@@
 Connection ~ 3400 4600
 Wire Wire Line
-	3400 4600 2600 4600
+	3400 4600 2700 4600
 $Comp
 L power:+5V #PWR0246
@@
 $EndComp
 Wire Wire Line
-	3150 2650 1800 2650
-Text GLabel 1800 2650 0    50   Output ~ 0
+	3150 2650 2950 2650
+Text GLabel 1800 2800 0    50   Output ~ 0
 _VPA
 Wire Wire Line
@@
 Wire Wire Line
 	10300 6650 10300 6900
-Text GLabel 1750 9600 0    50   Output ~ 0
+Text GLabel 1700 10050 0    50   Output ~ 0
 28M
-Text GLabel 1750 9800 0    50   Input ~ 0
+Text GLabel 1700 9800 0    50   Input ~ 0
 _XCLKEN
 Text GLabel 1750 6450 0    50   Input ~ 0
 XCLK
 $Comp
-L Connector:Conn_01x02_Male J900
+L Jumper:SolderJumper_2_Bridged J900
 U 1 1 60632932
-P 2500 4800
-F 0 "J900" V 2654 4612 50  0000 R CNN
-F 1 "Enable Chip RAM slowdown during DMA" V 2563 4612 50  0000 R CNN
-F 2 "Connector_PinHeader_2.54mm:PinHeader_1x02_P2.54mm_Vertical" H 2500 4800 50  0001 C CNN
-F 3 "~" H 2500 4800 50  0001 C CNN
-	1    2500 4800
-	0    -1   -1   0
+P 2550 4600
+F 0 "J900" H 2600 4700 50  0000 R CNN
+F 1 "Enable Chip RAM slowdown during DMA" H 3300 4450 50  0000 R CNN
+F 2 "Jumper:SolderJumper-2_P1.3mm_Bridged_RoundedPad1.0x1.5mm" H 2550 4600 50  0001 C CNN
+F 3 "~" H 2550 4600 50  0001 C CNN
+	1    2550 4600
+	1    0    0    -1
 $EndComp
 $Comp
@@
 Wire Wire Line
 	9700 7650 10300 7650
-Wire Wire Line
-	1750 9600 3850 9600
 Text Notes 12300 9850 0    197  ~ 0
 CLOCKS AND GARY\nAmiga 2000 EATX
@@
 	4250 6450 1750 6450
 Wire Wire Line
-	5400 8550 4250 8550
-Wire Wire Line
-	4250 8550 4250 8700
-Wire Wire Line
-	4250 8700 3850 8700
-Wire Wire Line
-	3850 8700 3850 9600
-Wire Wire Line
 	5400 9050 3950 9050
 Wire Wire Line
 	3950 9050 3950 9800
 Wire Wire Line
-	3950 9800 1750 9800
+	3950 9800 1700 9800
 Wire Wire Line
 	5900 9450 5400 9450
@@
 	5400 9450 5400 9150
 Connection ~ 5900 9450
-Wire Wire Line
-	6400 8450 6750 8450
-Wire Wire Line
-	6750 8450 6750 9250
-Wire Wire Line
-	6750 9250 7000 9250
 $Comp
 L Device:C C111
 U 1 1 62F441F4
-P 7600 9400
-F 0 "C111" H 7715 9446 50  0000 L CNN
-F 1 "22pF" H 7715 9355 50  0000 L CNN
-F 2 "Capacitor_SMD:C_1206_3216Metric" H 7638 9250 50  0001 C CNN
-F 3 "~" H 7600 9400 50  0001 C CNN
-	1    7600 9400
-	1    0    0    -1
-$EndComp
-Wire Wire Line
-	7300 9250 7600 9250
+P 7600 8600
+F 0 "C111" H 7715 8646 50  0000 L CNN
+F 1 "22pF" H 7715 8555 50  0000 L CNN
+F 2 "Capacitor_SMD:C_1206_3216Metric" H 7638 8450 50  0001 C CNN
+F 3 "~" H 7600 8600 50  0001 C CNN
+	1    7600 8600
+	1    0    0    -1
+$EndComp
+Wire Wire Line
+	7300 8450 7600 8450
 $Comp
 L power:GND #PWR0209
 U 1 1 62F7FE78
-P 7600 9550
-F 0 "#PWR0209" H 7600 9300 50  0001 C CNN
-F 1 "GND" H 7605 9377 50  0000 C CNN
-F 2 "" H 7600 9550 50  0001 C CNN
-F 3 "" H 7600 9550 50  0001 C CNN
-	1    7600 9550
+P 7600 8750
+F 0 "#PWR0209" H 7600 8500 50  0001 C CNN
+F 1 "GND" H 7605 8577 50  0000 C CNN
+F 2 "" H 7600 8750 50  0001 C CNN
+F 3 "" H 7600 8750 50  0001 C CNN
+	1    7600 8750
 	1    0    0    -1
 $EndComp
@@
 L power:GND #PWR0210
 U 1 1 62F9E115
-P 5000 7650
-F 0 "#PWR0210" H 5000 7400 50  0001 C CNN
-F 1 "GND" H 5005 7477 50  0000 C CNN
-F 2 "" H 5000 7650 50  0001 C CNN
-F 3 "" H 5000 7650 50  0001 C CNN
-	1    5000 7650
-	1    0    0    -1
-$EndComp
-Wire Wire Line
-	5400 8850 5400 8750
-Wire Wire Line
-	5400 8650 5000 8650
-Connection ~ 5400 8750
-Wire Wire Line
-	5400 8750 5400 8650
-$Comp
-L power:GND #PWR0211
-U 1 1 62FBCC02
-P 5000 8650
-F 0 "#PWR0211" H 5000 8400 50  0001 C CNN
-F 1 "GND" H 5005 8477 50  0000 C CNN
-F 2 "" H 5000 8650 50  0001 C CNN
-F 3 "" H 5000 8650 50  0001 C CNN
-	1    5000 8650
-	1    0    0    -1
-$EndComp
-NoConn ~ 6400 8750
+P 5000 7800
+F 0 "#PWR0210" H 5000 7550 50  0001 C CNN
+F 1 "GND" H 5005 7627 50  0000 C CNN
+F 2 "" H 5000 7800 50  0001 C CNN
+F 3 "" H 5000 7800 50  0001 C CNN
+	1    5000 7800
+	1    0    0    -1
+$EndComp
 NoConn ~ 6400 8150
 NoConn ~ 6400 7850
-Connection ~ 3850 8700
-Wire Wire Line
-	3850 8600 3850 8700
 Connection ~ 3850 8300
 $Comp
@@
 	1    0    0    -1
 $EndComp
-$Comp
-L Device:R R112
-U 1 1 63028772
-P 7150 9250
-F 0 "R112" V 6943 9250 50  0000 C CNN
-F 1 "150" V 7034 9250 50  0000 C CNN
-F 2 "Resistor_SMD:R_1206_3216Metric" V 7080 9250 50  0001 C CNN
-F 3 "~" H 7150 9250 50  0001 C CNN
-	1    7150 9250
-	0    1    1    0
-$EndComp
 Text GLabel 14650 7750 2    51   Input ~ 0
 7MHz
 Wire Wire Line
-	7600 9250 8500 9250
-Connection ~ 7600 9250
-Text GLabel 1700 10050 0    51   Output ~ 0
+	7600 8450 8100 8450
+Connection ~ 7600 8450
+Text GLabel 1700 10250 0    51   Output ~ 0
 AgnusCLK
 Text GLabel 14550 2750 2    51   Input ~ 0
@@
 	1800 3500 4950 3500
 Wire Wire Line
-	1700 10050 8500 10050
-Wire Wire Line
-	8500 10050 8500 9250
+	1700 10250 8100 10250
 Wire Wire Line
 	4950 1550 3200 1550
@@
 	1    0    0    -1
 $EndComp
+Wire Wire Line
+	5400 8850 5250 8850
+Wire Wire Line
+	3850 8600 3850 8850
+Wire Wire Line
+	5250 8850 5250 8750
+Wire Wire Line
+	5250 8550 5400 8550
+Connection ~ 5250 8850
+Wire Wire Line
+	5250 8850 3850 8850
+Wire Wire Line
+	5400 8750 5250 8750
+Connection ~ 5250 8750
+Wire Wire Line
+	5250 8750 5250 8550
+Wire Wire Line
+	6400 8750 6600 8750
+Wire Wire Line
+	6600 8750 6600 10050
+Wire Wire Line
+	6600 10050 4600 10050
+$Comp
+L Device:Ferrite_Bead FB104
+U 1 1 614E0E5C
+P 4450 10050
+F 0 "FB104" V 4250 10050 50  0000 C CNN
+F 1 "Ferrite_Bead" V 4633 10050 50  0001 C CNN
+F 2 "Capacitor_SMD:C_1206_3216Metric" V 4380 10050 50  0001 C CNN
+F 3 "~" H 4450 10050 50  0001 C CNN
+	1    4450 10050
+	0    1    1    0
+$EndComp
+Wire Wire Line
+	4300 10050 1700 10050
+$Comp
+L Device:Ferrite_Bead FB103
+U 1 1 614F3561
+P 7150 8450
+F 0 "FB103" V 6950 8450 50  0000 C CNN
+F 1 "Ferrite_Bead" V 7333 8450 50  0001 C CNN
+F 2 "Capacitor_SMD:C_1206_3216Metric" V 7080 8450 50  0001 C CNN
+F 3 "~" H 7150 8450 50  0001 C CNN
+	1    7150 8450
+	0    1    1    0
+$EndComp
+Wire Wire Line
+	6400 8450 7000 8450
+Wire Wire Line
+	8100 10250 8100 8450
+Wire Wire Line
+	5000 7800 5000 7650
+Wire Wire Line
+	2400 4600 1800 4600
+Wire Wire Line
+	4950 3400 4450 3400
+Wire Wire Line
+	4450 3400 4450 3850
+Wire Wire Line
+	4450 3850 1750 3850
+Wire Wire Line
+	1800 2800 2950 2800
+Wire Wire Line
+	2950 2800 2950 2650
 Wire Bus Line
 	4550 1950 4550 2550

Commit message: Add files via upload
Other:
- note removed: "2.0"
Changed lines of the file:
@@
 Wire Wire Line
 	12050 6300 12900 6300
-Text Notes 15950 10350 0    51   ~ 0
-2.0
 Wire Wire Line
 	3850 7150 3850 8300

Commit message: Add files via upload
Connections:
- no-connect marks 3 -> 2
Changed lines of the file:
@@
 Sheet 9 14
 Title "Amiga 2000 EATX"
-Date "2021-08-21"
+Date "2021-09-19"
 Rev "2.0"
 Comp ""
@@
 Wire Wire Line
 	1750 5550 3750 5550
-NoConn ~ 9550 5300
 Wire Wire Line
 	14650 8250 12350 8250

Commit message: Add files via upload
Changed lines of the file:
@@
 	3300 1000 1850 1000
 Text GLabel 1800 2550 0    50   Input ~ 0
-A[17..23]
+A[1..23]
 Wire Wire Line
 	4950 1850 4650 1850
