File: 2000EATX-KiCAD-INSANE-JUMPER-EDITION/floppyparallel.sch (KiCad schematic (older format))
At the start: 50 parts, among them CN300 KEYBOARD, CN303 FLOPPY, CN305 DB25_Stack_FemaleAndMale, J301 SHORT FOR DF1, Q301 MMBT3904, U102 GARY, U108 74HCT74, U203 74LS38, U300 8520, U302 74HCT32, U607 74HCT08, U900 74HCT00

Commit message: Add files via upload
Parts:
- added C322, C323: 0.1uF, Capacitor_SMD:C_1206_3216Metric, symbol Device:C
- added CN304: EXTERNAL FLOPPY, Connector_PinHeader_2.54mm:PinHeader_2x10_P2.54mm_Vertical, symbol Connector_Generic:Conn_02x10_Odd_Even
- added EMI311, EMI312, EMI313, EMI314, EMI315, EMI316, EMI317, EMI318, EMI319, EMI320, EMI321, EMI322, EMI323, EMI324, EMI339, EMI340, EMI341: C_Feedthrough_Small, AmigaFootprints:C_1206_3216_Feedthrough, symbol Amiga-Library:C_Feedthrough_Small
- added F3, F4: Fuse, Fuse:Fuse_1206_3216Metric, symbol Device:Fuse
- added unit 1 of U203
- added unit 2 of U607
- CN303: value FLOPPY -> INTERNAL FLOPPY
Connections:
- net +5V: now also C323.2, F4.2, U203.1, U607.4
- net DIR: now also EMI317.1
- net GND: now also C322.1, C323.1, CN304.20 (Pin_20), CN304.5 (Pin_5), CN304.7 (Pin_7), EMI311.3, EMI312.3, EMI313.3, EMI314.3, EMI315.3, EMI316.3, EMI317.3, EMI318.3, EMI319.3, EMI320.3, EMI321.3, EMI322.3, EMI323.3, EMI324.3, EMI339.3, EMI340.3, EMI341.3
- net _BRST: now also U607.5
- net _CHNG: now also EMI341.1
- net _DKRD: now also EMI323.1
- net _DKWDB: now also EMI315.1
- net _DKWEB: now also EMI314.1
- net _INDEX: now also EMI340.1
- net _RDY: now also EMI322.1
- net _SIDE: now also EMI313.1
- net _STEP: now also EMI316.1
- net _TRK0: now also EMI339.1
- net _WPROT: now also EMI324.1
- net at U102.47 (MTRX): now also U203.2
- new net: CN304.1 (Pin_1), EMI322.2
- new net: CN304.10 (Pin_10), EMI316.2
- new net: CN304.11 (Pin_11), EMI317.2
- new net: CN304.12 (Pin_12), EMI311.2
- new net: CN304.13 (Pin_13), EMI318.2
- new net: CN304.14 (Pin_14), EMI319.2
- new net: CN304.15 (Pin_15), EMI312.2
- new net: CN304.16 (Pin_16), EMI340.2
- new net: CN304.17 (Pin_17), EMI341.2
- new net: CN304.18 (Pin_18), EMI320.2
- new net: CN304.19 (Pin_19), EMI321.2
- new net: CN304.2 (Pin_2), EMI313.2
- new net: CN304.3 (Pin_3), EMI323.2
- new net: CN304.4 (Pin_4), EMI324.2
- new net: CN304.6 (Pin_6), EMI339.2
- new net: CN304.8 (Pin_8), EMI314.2
- new net: CN304.9 (Pin_9), EMI315.2
- new net: EMI320.1, F3.1
- new net: EMI321.1, F4.1
- new net +12V: C322.2, F3.2
- new net _DKRST: EMI312.1, U607.6
- new net _MTRX: EMI311.1, U203.3
- new net _SEL2: EMI319.1
- new net _SEL3: EMI318.1
- no-connect marks 6 -> 5

Commit message: Add files via upload
Parts:
- EMI301, EMI302, EMI303, EMI304, EMI305, EMI306, EMI307, EMI308, EMI309, EMI335, EMI336, EMI337, EMI338: symbol Amiga-Library:C_Feedthrough -> Amiga-Library:C_Feedthrough_Small
Other:
- moved on the sheet: U302A
