File: 2000EATX-KiCAD-INSANE-JUMPER-EDITION/power.sch (KiCad schematic (older format))
At the start: 53 parts, among them CN400 ATX-24, J9003 Case Fan, J9100 POWER_SWITCH, Q9100 MMBT3904, U203 74LS38, U501 74HCT00, U607 74HCT08, U9000 MC7905, U9101 74HCT14, U9102 74HCT74

Commit message: Add files via upload
Parts:
- CN400: symbol Connector:ATX-24 -> Amiga-Library:ATX-24-Amiga
Connections:
- net +3V3: no longer CN400.1 (+3.3V), CN400.13 (+3.3V), CN400.2 (+3.3V)
Changed lines of the file:
@@
 $EndDescr
 $Comp
-L Connector:ATX-24 CN400
+L Amiga-Library:ATX-24-Amiga CN400
 U 1 1 60A50060
 P 1600 1600

Commit message: Add files via upload
Parts:
- removed U203: 74LS38, Package_SO:SOIC-14_3.9x8.7mm_P1.27mm, symbol 74xx:74LS38
- removed U607: 74HCT08, Package_SO:SOIC-14_3.9x8.7mm_P1.27mm, symbol 74xx:74LS08
Connections:
- no-connect marks 6 -> 4
Changed lines of the file:
@@
 	3200 6650 3200 6800
-$Comp
-L 74xx:74LS08 U607
-U 2 1 60FCEC3E
-P 10150 3650
-F 0 "U607" H 10150 3975 50  0000 C CNN
-F 1 "74HCT08" H 10150 3884 50  0000 C CNN
-F 2 "Package_SO:SOIC-14_3.9x8.7mm_P1.27mm" H 10150 3650 50  0001 C CNN
-F 3 "http://www.ti.com/lit/gpn/sn74LS08" H 10150 3650 50  0001 C CNN
-	2    10150 3650
-	1    0    0    -1
-$EndComp
 $Comp
 L power:GND #PWR0220
 U 1 1 6102ADE1
-P 9850 3900
-F 0 "#PWR0220" H 9850 3650 50  0001 C CNN
-F 1 "GND" H 9855 3727 50  0000 C CNN
-F 2 "" H 9850 3900 50  0001 C CNN
-F 3 "" H 9850 3900 50  0001 C CNN
-	1    9850 3900
+P 9850 2700
+F 0 "#PWR0220" H 9850 2450 50  0001 C CNN
+F 1 "GND" H 9855 2527 50  0000 C CNN
+F 2 "" H 9850 2700 50  0001 C CNN
+F 3 "" H 9850 2700 50  0001 C CNN
+	1    9850 2700
 	1    0    0    -1
 $EndComp
-Wire Wire Line
-	9850 3900 9850 3750
-Connection ~ 9850 3750
-Wire Wire Line
-	9850 3750 9850 3550
-NoConn ~ 10450 3650
 Text Notes 9700 850  0    118  ~ 0
 SPARES
-$Comp
-L 74xx:74LS38 U203
-U 1 1 61051305
-P 10150 3050
-F 0 "U203" H 10150 3375 50  0000 C CNN
-F 1 "74LS38" H 10150 3284 50  0000 C CNN
-F 2 "Package_SO:SOIC-14_3.9x8.7mm_P1.27mm" H 10150 3050 50  0001 C CNN
-F 3 "http://www.ti.com/lit/gpn/sn74LS38" H 10150 3050 50  0001 C CNN
-	1    10150 3050
-	1    0    0    -1
-$EndComp
-Wire Wire Line
-	9850 3550 9850 3150
-Connection ~ 9850 3550
-Connection ~ 9850 3150
-Wire Wire Line
-	9850 3150 9850 2950
-NoConn ~ 10450 3050
 $Comp
 L 74xx:74LS00 U501
@@
 	1    0    0    -1
 $EndComp
-Wire Wire Line
-	9850 2950 9850 2550
-Connection ~ 9850 2950
 Connection ~ 9850 2550
 Wire Wire Line
@@
 Wire Notes Line
 	10850 600  10850 4200
+Wire Wire Line
+	9850 2550 9850 2700
 $EndSCHEMATC
