File: 2000EATX-KiCAD-INSANE-JUMPER-EDITION/2000ATX.sch (KiCad schematic (older format))
At the start: 0 parts

Commit message: Add files via upload
Other:
- note added: "AGNUS CONFIG JUMPERS"
- note added: "Amiga 2000 EATX Details"
- note added: "OTHER JUMPERS"
- note removed: "PROCESSOR"
