File: 2000EATX-KiCAD-INSANE-JUMPER-EDITION/coprocessor.sch (KiCad schematic (older format))
At the start: 17 parts, among them CN600 Amiga-2000-CPU-Slot, U600 74HCT245, U601 74HCT245, U602 74HCT245, U603 74HCT245, U604 74HCT245, U605 74HCT245

Commit message: Add files via upload
Changed lines of the file:
@@
 Sheet 4 14
 Title "Amiga 2000 EATX"
-Date "2021-08-21"
+Date "2021-09-19"
 Rev "2.0"
 Comp ""
@@
 U 1 1 604CC309
 P 1800 3650
-F 0 "CN600" H 1700 5900 50  0000 L CNN
+F 0 "CN?" H 1700 5900 50  0000 L CNN
 F 1 "Amiga-2000-CPU-Slot" H 1350 1350 50  0000 L CNN
 F 2 "AmigaFootprints:Samtec_HLE-150-02-xx-DV-TE_2x43_P2.54mm_Horizontal" H 1800 5100 50  0001 C CNN
@@
 U 1 1 604D2A89
 P 1500 6250
-F 0 "#PWR0123" H 1500 6000 50  0001 C CNN
+F 0 "#PWR?" H 1500 6000 50  0001 C CNN
 F 1 "GND" H 1505 6077 50  0000 C CNN
 F 2 "" H 1500 6250 50  0001 C CNN
@@
 U 1 1 604D882A
 P 2100 1550
-F 0 "#PWR0124" H 2100 1400 50  0001 C CNN
+F 0 "#PWR?" H 2100 1400 50  0001 C CNN
 F 1 "+5V" H 2117 1773 50  0000 C CNN
 F 2 "" H 2100 1550 50  0001 C CNN
@@
 U 1 1 604D8A9E
 P 2250 1350
-F 0 "#PWR0125" H 2250 1200 50  0001 C CNN
+F 0 "#PWR?" H 2250 1200 50  0001 C CNN
 F 1 "-5V" H 2267 1573 50  0000 C CNN
 F 2 "" H 2250 1350 50  0001 C CNN
@@
 U 1 1 604DB1C1
 P 2400 1550
-F 0 "#PWR0126" H 2400 1400 50  0001 C CNN
+F 0 "#PWR?" H 2400 1400 50  0001 C CNN
 F 1 "+12V" H 2417 1773 50  0000 C CNN
 F 2 "" H 2400 1550 50  0001 C CNN
@@
 U 1 1 604DCE39
 P 5800 1600
-F 0 "U600" H 5800 2581 50  0000 C CNN
+F 0 "U?" H 5800 2581 50  0000 C CNN
 F 1 "74HCT245" H 5800 2490 50  0000 C CNN
 F 2 "Package_SO:SOIC-20W_7.5x12.8mm_P1.27mm" H 5800 1600 50  0001 C CNN
@@
 U 1 1 604DEF6B
 P 6850 3200
-F 0 "U601" H 6850 4181 50  0000 C CNN
+F 0 "U?" H 6850 4181 50  0000 C CNN
 F 1 "74HCT245" H 6850 4090 50  0000 C CNN
 F 2 "Package_SO:SOIC-20W_7.5x12.8mm_P1.27mm" H 6850 3200 50  0001 C CNN
@@
 U 1 1 604DFB80
 P 5850 4850
-F 0 "U602" H 5850 5831 50  0000 C CNN
+F 0 "U?" H 5850 5831 50  0000 C CNN
 F 1 "74HCT245" H 5850 5740 50  0000 C CNN
 F 2 "Package_SO:SOIC-20W_7.5x12.8mm_P1.27mm" H 5850 4850 50  0001 C CNN
@@
 U 1 1 604EA09A
 P 10250 2000
-F 0 "U603" H 10250 2981 50  0000 C CNN
+F 0 "U?" H 10250 2981 50  0000 C CNN
 F 1 "74HCT245" H 10250 2890 50  0000 C CNN
 F 2 "Package_SO:SOIC-20W_7.5x12.8mm_P1.27mm" H 10250 2000 50  0001 C CNN
@@
 U 1 1 604EACE6
 P 10250 4250
-F 0 "U604" H 10250 5231 50  0000 C CNN
+F 0 "U?" H 10250 5231 50  0000 C CNN
 F 1 "74HCT245" H 10250 5140 50  0000 C CNN
 F 2 "Package_SO:SOIC-20W_7.5x12.8mm_P1.27mm" H 10250 4250 50  0001 C CNN
@@
 U 1 1 604EBC1A
 P 3750 6700
-F 0 "U605" H 3750 7681 50  0000 C CNN
+F 0 "U?" H 3750 7681 50  0000 C CNN
 F 1 "74HCT245" H 3750 7590 50  0000 C CNN
 F 2 "Package_SO:SOIC-20W_7.5x12.8mm_P1.27mm" H 3750 6700 50  0001 C CNN
@@
 U 1 1 60551069
 P 5800 2400
-F 0 "#PWR0127" H 5800 2150 50  0001 C CNN
+F 0 "#PWR?" H 5800 2150 50  0001 C CNN
 F 1 "GND" H 5805 2227 50  0000 C CNN
 F 2 "" H 5800 2400 50  0001 C CNN
@@
 U 1 1 6056F1B9
 P 6850 4150
-F 0 "#PWR0128" H 6850 3900 50  0001 C CNN
+F 0 "#PWR?" H 6850 3900 50  0001 C CNN
 F 1 "GND" H 6855 3977 50  0000 C CNN
 F 2 "" H 6850 4150 50  0001 C CNN
@@
 U 1 1 6056F9E8
 P 5850 5650
-F 0 "#PWR0129" H 5850 5400 50  0001 C CNN
+F 0 "#PWR?" H 5850 5400 50  0001 C CNN
 F 1 "GND" H 5855 5477 50  0000 C CNN
 F 2 "" H 5850 5650 50  0001 C CNN
@@
 U 1 1 605B732B
 P 10250 2800
-F 0 "#PWR0130" H 10250 2550 50  0001 C CNN
+F 0 "#PWR?" H 10250 2550 50  0001 C CNN
 F 1 "GND" H 10255 2627 50  0000 C CNN
 F 2 "" H 10250 2800 50  0001 C CNN
@@
 U 1 1 605B78D1
 P 10250 5050
-F 0 "#PWR0131" H 10250 4800 50  0001 C CNN
+F 0 "#PWR?" H 10250 4800 50  0001 C CNN
 F 1 "GND" H 10255 4877 50  0000 C CNN
 F 2 "" H 10250 5050 50  0001 C CNN
@@
 U 1 1 607375B5
 P 7850 1800
-F 0 "#PWR0132" H 7850 1550 50  0001 C CNN
+F 0 "#PWR?" H 7850 1550 50  0001 C CNN
 F 1 "GND" H 7855 1627 50  0000 C CNN
 F 2 "" H 7850 1800 50  0001 C CNN
@@
 U 1 1 6073AFFD
 P 7850 4250
-F 0 "#PWR0133" H 7850 4000 50  0001 C CNN
+F 0 "#PWR?" H 7850 4000 50  0001 C CNN
 F 1 "GND" H 7855 4077 50  0000 C CNN
 F 2 "" H 7850 4250 50  0001 C CNN
@@
 U 1 1 60B411F4
 P 3750 7500
-F 0 "#PWR0134" H 3750 7250 50  0001 C CNN
+F 0 "#PWR?" H 3750 7250 50  0001 C CNN
 F 1 "GND" H 3755 7327 50  0000 C CNN
 F 2 "" H 3750 7500 50  0001 C CNN
@@
 U 1 1 60B454E3
 P 4400 5650
-F 0 "#PWR0135" H 4400 5500 50  0001 C CNN
+F 0 "#PWR?" H 4400 5500 50  0001 C CNN
 F 1 "+5V" H 4400 5800 50  0000 C CNN
 F 2 "" H 4400 5650 50  0001 C CNN
@@
 U 1 1 60B78755
 P 3250 7200
-F 0 "#PWR0136" H 3250 6950 50  0001 C CNN
+F 0 "#PWR?" H 3250 6950 50  0001 C CNN
 F 1 "GND" H 3255 7027 50  0000 C CNN
 F 2 "" H 3250 7200 50  0001 C CNN
@@
 U 1 1 60E11888
 P 3250 5800
-F 0 "C605" V 3479 5800 50  0000 C CNN
+F 0 "C?" V 3479 5800 50  0000 C CNN
 F 1 "0.1uF" V 3388 5800 50  0000 C CNN
 F 2 "Capacitor_SMD:C_1206_3216Metric" H 3250 5800 50  0001 C CNN
@@
 U 1 1 60E422B1
 P 3450 5800
-F 0 "#PWR0137" H 3450 5650 50  0001 C CNN
+F 0 "#PWR?" H 3450 5650 50  0001 C CNN
 F 1 "+5V" H 3467 6023 50  0000 C CNN
 F 2 "" H 3450 5800 50  0001 C CNN
@@
 U 1 1 60E42986
 P 3150 5800
-F 0 "#PWR0138" H 3150 5550 50  0001 C CNN
+F 0 "#PWR?" H 3150 5550 50  0001 C CNN
 F 1 "GND" H 3155 5627 50  0000 C CNN
 F 2 "" H 3150 5800 50  0001 C CNN
@@
 U 1 1 60E76DE4
 P 6600 4150
-F 0 "C602" V 6829 4150 50  0000 C CNN
+F 0 "C?" V 6829 4150 50  0000 C CNN
 F 1 "0.1uF" V 6738 4150 50  0000 C CNN
 F 2 "Capacitor_SMD:C_1206_3216Metric" H 6600 4150 50  0001 C CNN
@@
 U 1 1 60E79216
 P 7400 2400
-F 0 "C601" V 7629 2400 50  0000 C CNN
+F 0 "C?" V 7629 2400 50  0000 C CNN
 F 1 "0.1uF" V 7538 2400 50  0000 C CNN
 F 2 "Capacitor_SMD:C_1206_3216Metric" H 7400 2400 50  0001 C CNN
@@
 U 1 1 60E799DA
 P 6250 800
-F 0 "C600" V 6479 800 50  0000 C CNN
+F 0 "C?" V 6479 800 50  0000 C CNN
 F 1 "0.1uF" V 6388 800 50  0000 C CNN
 F 2 "Capacitor_SMD:C_1206_3216Metric" H 6250 800 50  0001 C CNN
@@
 U 1 1 60E7A171
 P 10700 1200
-F 0 "C603" V 10929 1200 50  0000 C CNN
+F 0 "C?" V 10929 1200 50  0000 C CNN
 F 1 "0.1uF" V 10838 1200 50  0000 C CNN
 F 2 "Capacitor_SMD:C_1206_3216Metric" H 10700 1200 50  0001 C CNN
@@
 U 1 1 60E7A9E7
 P 10800 3450
-F 0 "C604" V 11029 3450 50  0000 C CNN
+F 0 "C?" V 11029 3450 50  0000 C CNN
 F 1 "0.1uF" V 10938 3450 50  0000 C CNN
 F 2 "Capacitor_SMD:C_1206_3216Metric" H 10800 3450 50  0001 C CNN
@@
 U 1 1 60E7B497
 P 10900 3450
-F 0 "#PWR0139" H 10900 3200 50  0001 C CNN
+F 0 "#PWR?" H 10900 3200 50  0001 C CNN
 F 1 "GND" H 10905 3277 50  0000 C CNN
 F 2 "" H 10900 3450 50  0001 C CNN
@@
 U 1 1 60E7BCF4
 P 10800 1200
-F 0 "#PWR0140" H 10800 950 50  0001 C CNN
+F 0 "#PWR?" H 10800 950 50  0001 C CNN
 F 1 "GND" H 10805 1027 50  0000 C CNN
 F 2 "" H 10800 1200 50  0001 C CNN
@@
 U 1 1 60E7CCB0
 P 6350 800
-F 0 "#PWR0141" H 6350 550 50  0001 C CNN
+F 0 "#PWR?" H 6350 550 50  0001 C CNN
 F 1 "GND" H 6355 627 50  0000 C CNN
 F 2 "" H 6350 800 50  0001 C CNN
@@
 U 1 1 60E7E9FD
 P 7500 2400
-F 0 "#PWR0142" H 7500 2150 50  0001 C CNN
+F 0 "#PWR?" H 7500 2150 50  0001 C CNN
 F 1 "GND" H 7505 2227 50  0000 C CNN
 F 2 "" H 7500 2400 50  0001 C CNN
@@
 U 1 1 60E89AA3
 P 6200 4150
-F 0 "#PWR0143" H 6200 4000 50  0001 C CNN
+F 0 "#PWR?" H 6200 4000 50  0001 C CNN
 F 1 "+5V" H 6217 4373 50  0000 C CNN
 F 2 "" H 6200 4150 50  0001 C CNN
@@
 U 1 1 60FCDD63
 P 7150 2400
-F 0 "#PWR0144" H 7150 2250 50  0001 C CNN
+F 0 "#PWR?" H 7150 2250 50  0001 C CNN
 F 1 "+5V" H 7167 2623 50  0000 C CNN
 F 2 "" H 7150 2400 50  0001 C CNN
@@
 U 1 1 60FE91B2
 P 6050 800
-F 0 "#PWR0145" H 6050 650 50  0001 C CNN
+F 0 "#PWR?" H 6050 650 50  0001 C CNN
 F 1 "+5V" H 6067 1023 50  0000 C CNN
 F 2 "" H 6050 800 50  0001 C CNN
@@
 U 1 1 60FE967D
 P 10500 1200
-F 0 "#PWR0146" H 10500 1050 50  0001 C CNN
+F 0 "#PWR?" H 10500 1050 50  0001 C CNN
 F 1 "+5V" H 10517 1423 50  0000 C CNN
 F 2 "" H 10500 1200 50  0001 C CNN
@@
 U 1 1 60FE9CDB
 P 10500 3450
-F 0 "#PWR0147" H 10500 3300 50  0001 C CNN
+F 0 "#PWR?" H 10500 3300 50  0001 C CNN
 F 1 "+5V" H 10517 3673 50  0000 C CNN
 F 2 "" H 10500 3450 50  0001 C CNN
@@
 U 1 1 610452A3
 P 5300 2100
-F 0 "#PWR0148" H 5300 1850 50  0001 C CNN
+F 0 "#PWR?" H 5300 1850 50  0001 C CNN
 F 1 "GND" H 5305 1927 50  0000 C CNN
 F 2 "" H 5300 2100 50  0001 C CNN
@@
 U 1 1 61045A56
 P 5350 5350
-F 0 "#PWR0149" H 5350 5100 50  0001 C CNN
+F 0 "#PWR?" H 5350 5100 50  0001 C CNN
 F 1 "GND" H 5355 5177 50  0000 C CNN
 F 2 "" H 5350 5350 50  0001 C CNN
@@
 U 1 1 610463ED
 P 6350 3700
-F 0 "#PWR0150" H 6350 3450 50  0001 C CNN
+F 0 "#PWR?" H 6350 3450 50  0001 C CNN
 F 1 "GND" H 6355 3527 50  0000 C CNN
 F 2 "" H 6350 3700 50  0001 C CNN
@@
 U 1 1 606BE25A
 P 8050 1400
-F 0 "RNX1" V 8675 1400 50  0000 C CNN
+F 0 "RNX?" V 8675 1400 50  0000 C CNN
 F 1 "3.3k" V 8584 1400 50  0000 C CNN
 F 2 "Resistor_THT:R_Array_SIP10" V 8625 1400 50  0001 C CNN
@@
 U 1 1 60701175
 P 8100 3850
-F 0 "RNX2" V 8725 3850 50  0000 C CNN
+F 0 "RNX?" V 8725 3850 50  0000 C CNN
 F 1 "3.3k" V 8634 3850 50  0000 C CNN
 F 2 "Resistor_THT:R_Array_SIP10" V 8675 3850 50  0001 C CNN
@@
 U 1 1 61444A0D
 P 4600 5850
-F 0 "RN908" H 4888 5896 50  0000 L CNN
+F 0 "RN?" H 4888 5896 50  0000 L CNN
 F 1 "1k" H 4888 5805 50  0000 L CNN
 F 2 "Resistor_THT:R_Array_SIP6" V 4975 5850 50  0001 C CNN
@@
 U 1 1 61446021
 P 5400 6000
-F 0 "RN903" H 5688 6046 50  0000 L CNN
+F 0 "RN?" H 5688 6046 50  0000 L CNN
 F 1 "1k" H 5688 5955 50  0000 L CNN
 F 2 "Resistor_THT:R_Array_SIP6" V 5775 6000 50  0001 C CNN

Commit message: Add files via upload
Changed lines of the file:
@@
 encoding utf-8
 Sheet 4 14
-Title "Amiga 2000 EATX"
-Date "2021-09-19"
-Rev "2.0"
+Title ""
+Date ""
+Rev ""
 Comp ""
 Comment1 ""
@@
 U 1 1 604CC309
 P 1800 3650
-F 0 "CN?" H 1700 5900 50  0000 L CNN
+F 0 "CN600" H 1700 5900 50  0000 L CNN
 F 1 "Amiga-2000-CPU-Slot" H 1350 1350 50  0000 L CNN
 F 2 "AmigaFootprints:Samtec_HLE-150-02-xx-DV-TE_2x43_P2.54mm_Horizontal" H 1800 5100 50  0001 C CNN
@@
 U 1 1 604D2A89
 P 1500 6250
-F 0 "#PWR?" H 1500 6000 50  0001 C CNN
+F 0 "#PWR0123" H 1500 6000 50  0001 C CNN
 F 1 "GND" H 1505 6077 50  0000 C CNN
 F 2 "" H 1500 6250 50  0001 C CNN
@@
 U 1 1 604D882A
 P 2100 1550
-F 0 "#PWR?" H 2100 1400 50  0001 C CNN
+F 0 "#PWR0124" H 2100 1400 50  0001 C CNN
 F 1 "+5V" H 2117 1773 50  0000 C CNN
 F 2 "" H 2100 1550 50  0001 C CNN
@@
 U 1 1 604D8A9E
 P 2250 1350
-F 0 "#PWR?" H 2250 1200 50  0001 C CNN
+F 0 "#PWR0125" H 2250 1200 50  0001 C CNN
 F 1 "-5V" H 2267 1573 50  0000 C CNN
 F 2 "" H 2250 1350 50  0001 C CNN
@@
 U 1 1 604DB1C1
 P 2400 1550
-F 0 "#PWR?" H 2400 1400 50  0001 C CNN
+F 0 "#PWR0126" H 2400 1400 50  0001 C CNN
 F 1 "+12V" H 2417 1773 50  0000 C CNN
 F 2 "" H 2400 1550 50  0001 C CNN
@@
 U 1 1 604DCE39
 P 5800 1600
-F 0 "U?" H 5800 2581 50  0000 C CNN
+F 0 "U600" H 5800 2581 50  0000 C CNN
 F 1 "74HCT245" H 5800 2490 50  0000 C CNN
 F 2 "Package_SO:SOIC-20W_7.5x12.8mm_P1.27mm" H 5800 1600 50  0001 C CNN
@@
 U 1 1 604DEF6B
 P 6850 3200
-F 0 "U?" H 6850 4181 50  0000 C CNN
+F 0 "U601" H 6850 4181 50  0000 C CNN
 F 1 "74HCT245" H 6850 4090 50  0000 C CNN
 F 2 "Package_SO:SOIC-20W_7.5x12.8mm_P1.27mm" H 6850 3200 50  0001 C CNN
@@
 U 1 1 604DFB80
 P 5850 4850
-F 0 "U?" H 5850 5831 50  0000 C CNN
+F 0 "U602" H 5850 5831 50  0000 C CNN
 F 1 "74HCT245" H 5850 5740 50  0000 C CNN
 F 2 "Package_SO:SOIC-20W_7.5x12.8mm_P1.27mm" H 5850 4850 50  0001 C CNN
@@
 U 1 1 604EA09A
 P 10250 2000
-F 0 "U?" H 10250 2981 50  0000 C CNN
+F 0 "U603" H 10250 2981 50  0000 C CNN
 F 1 "74HCT245" H 10250 2890 50  0000 C CNN
 F 2 "Package_SO:SOIC-20W_7.5x12.8mm_P1.27mm" H 10250 2000 50  0001 C CNN
@@
 U 1 1 604EACE6
 P 10250 4250
-F 0 "U?" H 10250 5231 50  0000 C CNN
+F 0 "U604" H 10250 5231 50  0000 C CNN
 F 1 "74HCT245" H 10250 5140 50  0000 C CNN
 F 2 "Package_SO:SOIC-20W_7.5x12.8mm_P1.27mm" H 10250 4250 50  0001 C CNN
@@
 U 1 1 604EBC1A
 P 3750 6700
-F 0 "U?" H 3750 7681 50  0000 C CNN
+F 0 "U605" H 3750 7681 50  0000 C CNN
 F 1 "74HCT245" H 3750 7590 50  0000 C CNN
 F 2 "Package_SO:SOIC-20W_7.5x12.8mm_P1.27mm" H 3750 6700 50  0001 C CNN
@@
 U 1 1 60551069
 P 5800 2400
-F 0 "#PWR?" H 5800 2150 50  0001 C CNN
+F 0 "#PWR0127" H 5800 2150 50  0001 C CNN
 F 1 "GND" H 5805 2227 50  0000 C CNN
 F 2 "" H 5800 2400 50  0001 C CNN
@@
 U 1 1 6056F1B9
 P 6850 4150
-F 0 "#PWR?" H 6850 3900 50  0001 C CNN
+F 0 "#PWR0128" H 6850 3900 50  0001 C CNN
 F 1 "GND" H 6855 3977 50  0000 C CNN
 F 2 "" H 6850 4150 50  0001 C CNN
@@
 U 1 1 6056F9E8
 P 5850 5650
-F 0 "#PWR?" H 5850 5400 50  0001 C CNN
+F 0 "#PWR0129" H 5850 5400 50  0001 C CNN
 F 1 "GND" H 5855 5477 50  0000 C CNN
 F 2 "" H 5850 5650 50  0001 C CNN
@@
 U 1 1 605B732B
 P 10250 2800
-F 0 "#PWR?" H 10250 2550 50  0001 C CNN
+F 0 "#PWR0130" H 10250 2550 50  0001 C CNN
 F 1 "GND" H 10255 2627 50  0000 C CNN
 F 2 "" H 10250 2800 50  0001 C CNN
@@
 U 1 1 605B78D1
 P 10250 5050
-F 0 "#PWR?" H 10250 4800 50  0001 C CNN
+F 0 "#PWR0131" H 10250 4800 50  0001 C CNN
 F 1 "GND" H 10255 4877 50  0000 C CNN
 F 2 "" H 10250 5050 50  0001 C CNN
@@
 U 1 1 607375B5
 P 7850 1800
-F 0 "#PWR?" H 7850 1550 50  0001 C CNN
+F 0 "#PWR0132" H 7850 1550 50  0001 C CNN
 F 1 "GND" H 7855 1627 50  0000 C CNN
 F 2 "" H 7850 1800 50  0001 C CNN
@@
 U 1 1 6073AFFD
 P 7850 4250
-F 0 "#PWR?" H 7850 4000 50  0001 C CNN
+F 0 "#PWR0133" H 7850 4000 50  0001 C CNN
 F 1 "GND" H 7855 4077 50  0000 C CNN
 F 2 "" H 7850 4250 50  0001 C CNN
@@
 U 1 1 60B411F4
 P 3750 7500
-F 0 "#PWR?" H 3750 7250 50  0001 C CNN
+F 0 "#PWR0134" H 3750 7250 50  0001 C CNN
 F 1 "GND" H 3755 7327 50  0000 C CNN
 F 2 "" H 3750 7500 50  0001 C CNN
@@
 U 1 1 60B454E3
 P 4400 5650
-F 0 "#PWR?" H 4400 5500 50  0001 C CNN
+F 0 "#PWR0135" H 4400 5500 50  0001 C CNN
 F 1 "+5V" H 4400 5800 50  0000 C CNN
 F 2 "" H 4400 5650 50  0001 C CNN
@@
 U 1 1 60B78755
 P 3250 7200
-F 0 "#PWR?" H 3250 6950 50  0001 C CNN
+F 0 "#PWR0136" H 3250 6950 50  0001 C CNN
 F 1 "GND" H 3255 7027 50  0000 C CNN
 F 2 "" H 3250 7200 50  0001 C CNN
@@
 U 1 1 60E11888
 P 3250 5800
-F 0 "C?" V 3479 5800 50  0000 C CNN
+F 0 "C605" V 3479 5800 50  0000 C CNN
 F 1 "0.1uF" V 3388 5800 50  0000 C CNN
 F 2 "Capacitor_SMD:C_1206_3216Metric" H 3250 5800 50  0001 C CNN
@@
 U 1 1 60E422B1
 P 3450 5800
-F 0 "#PWR?" H 3450 5650 50  0001 C CNN
+F 0 "#PWR0137" H 3450 5650 50  0001 C CNN
 F 1 "+5V" H 3467 6023 50  0000 C CNN
 F 2 "" H 3450 5800 50  0001 C CNN
@@
 U 1 1 60E42986
 P 3150 5800
-F 0 "#PWR?" H 3150 5550 50  0001 C CNN
+F 0 "#PWR0138" H 3150 5550 50  0001 C CNN
 F 1 "GND" H 3155 5627 50  0000 C CNN
 F 2 "" H 3150 5800 50  0001 C CNN
@@
 U 1 1 60E76DE4
 P 6600 4150
-F 0 "C?" V 6829 4150 50  0000 C CNN
+F 0 "C602" V 6829 4150 50  0000 C CNN
 F 1 "0.1uF" V 6738 4150 50  0000 C CNN
 F 2 "Capacitor_SMD:C_1206_3216Metric" H 6600 4150 50  0001 C CNN
@@
 U 1 1 60E79216
 P 7400 2400
-F 0 "C?" V 7629 2400 50  0000 C CNN
+F 0 "C601" V 7629 2400 50  0000 C CNN
 F 1 "0.1uF" V 7538 2400 50  0000 C CNN
 F 2 "Capacitor_SMD:C_1206_3216Metric" H 7400 2400 50  0001 C CNN
@@
 U 1 1 60E799DA
 P 6250 800
-F 0 "C?" V 6479 800 50  0000 C CNN
+F 0 "C600" V 6479 800 50  0000 C CNN
 F 1 "0.1uF" V 6388 800 50  0000 C CNN
 F 2 "Capacitor_SMD:C_1206_3216Metric" H 6250 800 50  0001 C CNN
@@
 U 1 1 60E7A171
 P 10700 1200
-F 0 "C?" V 10929 1200 50  0000 C CNN
+F 0 "C603" V 10929 1200 50  0000 C CNN
 F 1 "0.1uF" V 10838 1200 50  0000 C CNN
 F 2 "Capacitor_SMD:C_1206_3216Metric" H 10700 1200 50  0001 C CNN
@@
 U 1 1 60E7A9E7
 P 10800 3450
-F 0 "C?" V 11029 3450 50  0000 C CNN
+F 0 "C604" V 11029 3450 50  0000 C CNN
 F 1 "0.1uF" V 10938 3450 50  0000 C CNN
 F 2 "Capacitor_SMD:C_1206_3216Metric" H 10800 3450 50  0001 C CNN
@@
 U 1 1 60E7B497
 P 10900 3450
-F 0 "#PWR?" H 10900 3200 50  0001 C CNN
+F 0 "#PWR0139" H 10900 3200 50  0001 C CNN
 F 1 "GND" H 10905 3277 50  0000 C CNN
 F 2 "" H 10900 3450 50  0001 C CNN
@@
 U 1 1 60E7BCF4
 P 10800 1200
-F 0 "#PWR?" H 10800 950 50  0001 C CNN
+F 0 "#PWR0140" H 10800 950 50  0001 C CNN
 F 1 "GND" H 10805 1027 50  0000 C CNN
 F 2 "" H 10800 1200 50  0001 C CNN
@@
 U 1 1 60E7CCB0
 P 6350 800
-F 0 "#PWR?" H 6350 550 50  0001 C CNN
+F 0 "#PWR0141" H 6350 550 50  0001 C CNN
 F 1 "GND" H 6355 627 50  0000 C CNN
 F 2 "" H 6350 800 50  0001 C CNN
@@
 U 1 1 60E7E9FD
 P 7500 2400
-F 0 "#PWR?" H 7500 2150 50  0001 C CNN
+F 0 "#PWR0142" H 7500 2150 50  0001 C CNN
 F 1 "GND" H 7505 2227 50  0000 C CNN
 F 2 "" H 7500 2400 50  0001 C CNN
@@
 U 1 1 60E89AA3
 P 6200 4150
-F 0 "#PWR?" H 6200 4000 50  0001 C CNN
+F 0 "#PWR0143" H 6200 4000 50  0001 C CNN
 F 1 "+5V" H 6217 4373 50  0000 C CNN
 F 2 "" H 6200 4150 50  0001 C CNN
@@
 U 1 1 60FCDD63
 P 7150 2400
-F 0 "#PWR?" H 7150 2250 50  0001 C CNN
+F 0 "#PWR0144" H 7150 2250 50  0001 C CNN
 F 1 "+5V" H 7167 2623 50  0000 C CNN
 F 2 "" H 7150 2400 50  0001 C CNN
@@
 U 1 1 60FE91B2
 P 6050 800
-F 0 "#PWR?" H 6050 650 50  0001 C CNN
+F 0 "#PWR0145" H 6050 650 50  0001 C CNN
 F 1 "+5V" H 6067 1023 50  0000 C CNN
 F 2 "" H 6050 800 50  0001 C CNN
@@
 U 1 1 60FE967D
 P 10500 1200
-F 0 "#PWR?" H 10500 1050 50  0001 C CNN
+F 0 "#PWR0146" H 10500 1050 50  0001 C CNN
 F 1 "+5V" H 10517 1423 50  0000 C CNN
 F 2 "" H 10500 1200 50  0001 C CNN
@@
 U 1 1 60FE9CDB
 P 10500 3450
-F 0 "#PWR?" H 10500 3300 50  0001 C CNN
+F 0 "#PWR0147" H 10500 3300 50  0001 C CNN
 F 1 "+5V" H 10517 3673 50  0000 C CNN
 F 2 "" H 10500 3450 50  0001 C CNN
@@
 U 1 1 610452A3
 P 5300 2100
-F 0 "#PWR?" H 5300 1850 50  0001 C CNN
+F 0 "#PWR0148" H 5300 1850 50  0001 C CNN
 F 1 "GND" H 5305 1927 50  0000 C CNN
 F 2 "" H 5300 2100 50  0001 C CNN
@@
 U 1 1 61045A56
 P 5350 5350
-F 0 "#PWR?" H 5350 5100 50  0001 C CNN
+F 0 "#PWR0149" H 5350 5100 50  0001 C CNN
 F 1 "GND" H 5355 5177 50  0000 C CNN
 F 2 "" H 5350 5350 50  0001 C CNN
@@
 U 1 1 610463ED
 P 6350 3700
-F 0 "#PWR?" H 6350 3450 50  0001 C CNN
+F 0 "#PWR0150" H 6350 3450 50  0001 C CNN
 F 1 "GND" H 6355 3527 50  0000 C CNN
 F 2 "" H 6350 3700 50  0001 C CNN
@@
 U 1 1 606BE25A
 P 8050 1400
-F 0 "RNX?" V 8675 1400 50  0000 C CNN
+F 0 "RNX1" V 8675 1400 50  0000 C CNN
 F 1 "3.3k" V 8584 1400 50  0000 C CNN
 F 2 "Resistor_THT:R_Array_SIP10" V 8625 1400 50  0001 C CNN
@@
 U 1 1 60701175
 P 8100 3850
-F 0 "RNX?" V 8725 3850 50  0000 C CNN
+F 0 "RNX2" V 8725 3850 50  0000 C CNN
 F 1 "3.3k" V 8634 3850 50  0000 C CNN
 F 2 "Resistor_THT:R_Array_SIP10" V 8675 3850 50  0001 C CNN
@@
 U 1 1 61444A0D
 P 4600 5850
-F 0 "RN?" H 4888 5896 50  0000 L CNN
+F 0 "RN908" H 4888 5896 50  0000 L CNN
 F 1 "1k" H 4888 5805 50  0000 L CNN
 F 2 "Resistor_THT:R_Array_SIP6" V 4975 5850 50  0001 C CNN
@@
 U 1 1 61446021
 P 5400 6000
-F 0 "RN?" H 5688 6046 50  0000 L CNN
+F 0 "RN903" H 5688 6046 50  0000 L CNN
 F 1 "1k" H 5688 5955 50  0000 L CNN
 F 2 "Resistor_THT:R_Array_SIP6" V 5775 6000 50  0001 C CNN

Commit message: Add files via upload
Other:
- moved on the sheet: C600, U600

Commit message: Add files via upload
Other:
- moved on the sheet: C601, C604
