File: 2000EATX-KiCAD-R121/memory.sch (KiCad schematic (older format))
At the start: 30 parts, among them U500 KICKSTART, U501 74HCT00, U502 CY74FCT821T, U503 CY62157, U504 CY74FCT821T, U540 74AHCT244, U541 74AHCT244

Commit message: Add files via upload
Parts:
- added unit 2 of U502
- added unit 2 of U504
Connections:
- net +5V: now also U500.22 (Vcc), U502.24 (Vcc), U504.24 (Vcc)
- net GND: now also U500.12 (Vss), U500.31 (Vss), U502.12 (GND), U504.12 (GND)
Other:
- moved on the sheet: C500, C501, C502, C503, C504, U500B, U501E, U503B
