File: 2000EATX-KiCAD-R21/video.sch (KiCad schematic (older format))
At the start: 37 parts, among them CN202 DB15_Female_HighDensity, CN203 Amiga-2000-Video-Slot, CN207 Amiga-2000-Video-Slot, J9004 HSYNC/COMPSYNC, U201 DENISE, U205 74AHCT244, U206 74AHCT244, U303 74HCT08

Commit message: Add files via upload
Parts:
- added C207: 0.1uF, Capacitor_SMD:C_1206_3216Metric, symbol Device:C
- added U207: 74HCT08, Package_SO:SOIC-14_3.9x8.7mm_P1.27mm, symbol 74xx:74LS08
Connections:
- net +VID: now also C207.1, U207.14 (VCC)
- net GND: now also C207.2, U207.7 (GND)
- net _VSYNC: now also U207.1, U207.2; no longer R203A1.2
- net at J9004.2 (C): now also U207.4, U207.5; no longer R203B1.2
- new net: R203A1.2, U207.3
- new net: R203B1.2, U207.6
Other:
- moved on the sheet: C201, EMI206, EMI207, EMI229, R203, R203A1, R203B1, U201B

Commit message: Add files via upload
Connections:
- net _HSYNC: now also U207.4, U207.5; no longer J9004.1 (A)
- net at U207.6: now also J9004.1 (A); no longer R203B1.2
- new net: J9004.2 (C), R203B1.2
Other:
- moved on the sheet: J9004, U207B
Changed lines of the file:
@@
 Sheet 6 14
 Title "Amiga 2000 EATX"
-Date "2021-10-08"
-Rev "2.0"
+Date "2021-10-28"
+Rev "2.1"
 Comp ""
 Comment1 ""
@@
 Connection ~ 8300 2700
 Wire Wire Line
-	8300 2700 8300 3550
+	8300 2700 8300 3450
 Wire Wire Line
 	5500 2850 5700 2850
@@
 L Jumper:Jumper_3_Bridged12 J9004
 U 1 1 60ED3751
-P 9950 3550
-F 0 "J9004" H 9950 3754 50  0000 C CNN
-F 1 "HSYNC/COMPSYNC" H 9950 3663 50  0000 C CNN
-F 2 "Connector_PinHeader_2.54mm:PinHeader_1x03_P2.54mm_Vertical" H 9950 3550 50  0001 C CNN
-F 3 "~" H 9950 3550 50  0001 C CNN
-	1    9950 3550
+P 10950 3550
+F 0 "J9004" H 10950 3754 50  0000 C CNN
+F 1 "HSYNC/COMPSYNC" H 10950 3663 50  0000 C CNN
+F 2 "Connector_PinHeader_2.54mm:PinHeader_1x03_P2.54mm_Vertical" H 10950 3550 50  0001 C CNN
+F 3 "~" H 10950 3550 50  0001 C CNN
+	1    10950 3550
 	1    0    0    -1
 $EndComp
@@
 $EndComp
 Wire Wire Line
-	10200 3550 11350 3550
+	11200 3550 11350 3550
 Wire Wire Line
 	11350 3550 11350 2850
 Connection ~ 11350 2850
-Wire Wire Line
-	8300 3550 9700 3550
 NoConn ~ 10300 5550
 NoConn ~ 10300 4950
@@
 L 74xx:74LS08 U207
 U 2 1 61824625
-P 10650 4000
-F 0 "U207" H 10650 4325 50  0000 C CNN
-F 1 "74HCT08" H 10650 4234 50  0000 C CNN
-F 2 "Package_SO:SOIC-14_3.9x8.7mm_P1.27mm" H 10650 4000 50  0001 C CNN
-F 3 "http://www.ti.com/lit/gpn/sn74LS08" H 10650 4000 50  0001 C CNN
-	2    10650 4000
+P 10000 3550
+F 0 "U207" H 10000 3875 50  0000 C CNN
+F 1 "74HCT08" H 10000 3784 50  0000 C CNN
+F 2 "Package_SO:SOIC-14_3.9x8.7mm_P1.27mm" H 10000 3550 50  0001 C CNN
+F 3 "http://www.ti.com/lit/gpn/sn74LS08" H 10000 3550 50  0001 C CNN
+	2    10000 3550
 	1    0    0    -1
 $EndComp
@@
 	8450 8000 8050 8000
 Wire Wire Line
-	10950 4300 10950 4000
-Wire Wire Line
-	10350 3900 10250 3900
-Wire Wire Line
-	9950 3900 9950 3700
-Wire Wire Line
-	10350 4100 10250 4100
-Wire Wire Line
-	10250 4100 10250 3900
-Connection ~ 10250 3900
-Wire Wire Line
-	10250 3900 9950 3900
-Wire Wire Line
 	1000 7800 6250 7800
 Wire Wire Line
@@
 Wire Wire Line
 	13050 7550 13050 7400
+Wire Wire Line
+	10950 3700 10950 4300
+Wire Wire Line
+	10300 3550 10700 3550
+Wire Wire Line
+	9700 3450 9600 3450
+Wire Wire Line
+	9700 3650 9600 3650
+Wire Wire Line
+	9600 3650 9600 3450
 Wire Bus Line
 	1150 4850 1150 5700
 Wire Bus Line
 	1150 3100 1150 4600
+Connection ~ 9600 3450
+Wire Wire Line
+	9600 3450 8300 3450
 $EndSCHEMATC
