File: 2000EATX-KiCAD-R22/Agnus-Multi.sch (KiCad schematic (older format))
At the start: 18 parts, among them J102 Short for 8327A NTSC or 8375, U101 Agnus_MULTI

Commit message: Add files via upload
Other:
- note added: "SUPPORTS 8372A (ALL PART NUMBERS)\nAND 8375 THE FOLLOWING PART NUMBERS:\n390544-01 AND COMPATIBLE (390544-02, 390554-01, 390554-02, \n318069-12, 318069-13) AND 318069-10, 318069-11"
- note removed: "SUPPORTS 8372A (ALL PART NUMBERS)\nAND 8375 THE FOLLOWING PART NUMBERS:\n390554-01 AND COMPATIBLE (390554-02, 318069-12, 318069-13)\n390544-01 AND COMPATIBLE (390544-02, 318069-10, 318069-11)"
Changed lines of the file:
@@
 390554-01 is 14M...leave open\n318069-10 is Vbb...short to GND
 Text Notes 800  1600 0    157  ~ 0
-SUPPORTS 8372A (ALL PART NUMBERS)\nAND 8375 THE FOLLOWING PART NUMBERS:\n390554-01 AND COMPATIBLE (390554-02, 318069-12, 318069-13)\n390544-01 AND COMPATIBLE (390544-02, 318069-10, 318069-11)
+SUPPORTS 8372A (ALL PART NUMBERS)\nAND 8375 THE FOLLOWING PART NUMBERS:\n390544-01 AND COMPATIBLE (390544-02, 390554-01, 390554-02, \n318069-12, 318069-13) AND 318069-10, 318069-11
 Text Notes 9000 850  0    157  ~ 0
 JUMPERS MUST BE CONFIGURED BY AGNUS PART NUMBER
