File: 2000EATX-KiCAD-R31/2000ATX.kicad_sch (KiCad schematic)
At the start: 0 parts

Commit message: Update Schematic 02-JUN-2024
Other:
- note added: "J503 = SRAM Vcc 1-2 3.3V 2-3 5V (Factory Default)"
- note removed: "J503 = SRAM Vcc 1-2 3.3V (Factory Default) 2-3 5V"
Changed lines of the file:
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@@
 		)
 	)
-	(text "J503 = SRAM Vcc\n  1-2 3.3V (Factory Default)\n  2-3 5V"
+	(text "J503 = SRAM Vcc\n  1-2 3.3V \n  2-3 5V (Factory Default)"
 		(exclude_from_sim no)
 		(at 114.046 125.222 0)
